File: connectors.sch (KiCad schematic (older format))
At the start: 23 parts, among them J4 Conn_01x03_Male

Commit message: fix all ERC errors
Changed lines of the file:
@@
 Text HLabel 4700 3500 2    50   Output ~ 0
 R_MTR_HALL_PHC
+$Comp
+L power:PWR_FLAG #FLG0104
+U 1 1 5F73A64F
+P 2850 4400
+F 0 "#FLG0104" H 2850 4475 50  0001 C CNN
+F 1 "PWR_FLAG" H 2850 4573 50  0000 C CNN
+F 2 "" H 2850 4400 50  0001 C CNN
+F 3 "~" H 2850 4400 50  0001 C CNN
+	1    2850 4400
+	-1   0    0    1
+$EndComp
+Wire Wire Line
+	2700 4400 2850 4400
+Connection ~ 2700 4400
 $EndSCHEMATC

Commit message: Add CAN transceiver
Parts:
- added C?: 4.7n, symbol Device:C
- added C?: 1u, symbol Device:C
- added D?: D_TVS_x2_AAC, symbol Device:D_TVS_x2_AAC
- added D?: D_Schottky, symbol Device:D_Schottky
- added D?: TVS, symbol Device:D_Zener
- added J?: Conn_01x05, symbol Connector_Generic:Conn_01x05
- added R?: 1M, symbol Device:R
Connections:
- net +VSW: now also D?.2 (A)
- net GND: now also C?.2, C?.2, D?.2 (A), D?.3 (common), J?.3 (Pin_3), R?.2
- new net: C?.1, D?.1 (K), D?.1 (K), J?.4 (Pin_4)
- new net: C?.1, J?.5 (Pin_5), R?.1
- new net CANH: D?.1 (A1), J?.1 (Pin_1)
- new net CANL: D?.2 (A2), J?.2 (Pin_2)
Other:
- note added: "CANH"
- note added: "CANL"
- note added: "CAN_GND"
- note added: "CAN_SHLD"
- note added: "VBUS"
Changed lines of the file:
@@
 $Descr A4 11693 8268
 encoding utf-8
-Sheet 5 13
+Sheet 5 14
 Title ""
 Date ""
@@
 	2700 4400 2850 4400
 Connection ~ 2700 4400
+$Comp
+L Connector_Generic:Conn_01x05 J?
+U 1 1 5F78B096
+P 2250 5850
+F 0 "J?" H 2168 6267 50  0000 C CNN
+F 1 "Conn_01x05" H 2168 6176 50  0000 C CNN
+F 2 "" H 2250 5850 50  0001 C CNN
+F 3 "~" H 2250 5850 50  0001 C CNN
+	1    2250 5850
+	-1   0    0    -1
+$EndComp
+Text HLabel 3800 5650 2    50   BiDi ~ 0
+CANH
+Wire Wire Line
+	2450 5650 2650 5650
+Text HLabel 3800 5750 2    50   BiDi ~ 0
+CANL
+Wire Wire Line
+	2450 5750 3450 5750
+$Comp
+L Device:D_TVS_x2_AAC D?
+U 1 1 5F79E74D
+P 3050 5200
+F 0 "D?" H 3050 5417 50  0000 C CNN
+F 1 "D_TVS_x2_AAC" H 3050 5326 50  0000 C CNN
+F 2 "" H 2900 5200 50  0001 C CNN
+F 3 "~" H 2900 5200 50  0001 C CNN
+	1    3050 5200
+	1    0    0    -1
+$EndComp
+Wire Wire Line
+	2700 5200 2650 5200
+Wire Wire Line
+	2650 5200 2650 5650
+Wire Wire Line
+	3400 5200 3450 5200
+Wire Wire Line
+	3450 5200 3450 5750
+$Comp
+L power:GND #PWR?
+U 1 1 5F7A3138
+P 3050 5400
+F 0 "#PWR?" H 3050 5150 50  0001 C CNN
+F 1 "GND" H 3055 5227 50  0000 C CNN
+F 2 "" H 3050 5400 50  0001 C CNN
+F 3 "" H 3050 5400 50  0001 C CNN
+	1    3050 5400
+	1    0    0    -1
+$EndComp
+Wire Wire Line
+	3050 5350 3050 5400
+Wire Wire Line
+	4350 5950 4350 5800
+$Comp
+L power:+VSW #PWR?
+U 1 1 5F7A9210
+P 4350 5450
+F 0 "#PWR?" H 4350 5300 50  0001 C CNN
+F 1 "+VSW" H 4365 5623 50  0000 C CNN
+F 2 "" H 4350 5450 50  0001 C CNN
+F 3 "" H 4350 5450 50  0001 C CNN
+	1    4350 5450
+	1    0    0    -1
+$EndComp
+Wire Wire Line
+	4350 5450 4350 5500
+$Comp
+L Device:D_Schottky D?
+U 1 1 5F7AAFC5
+P 4350 5650
+F 0 "D?" V 4396 5570 50  0000 R CNN
+F 1 "D_Schottky" V 4305 5570 50  0000 R CNN
+F 2 "" H 4350 5650 50  0001 C CNN
+F 3 "~" H 4350 5650 50  0001 C CNN
+	1    4350 5650
+	0    -1   -1   0
+$EndComp
+Text Notes 2150 5700 2    50   ~ 0
+CANH
+Text Notes 2150 5800 2    50   ~ 0
+CANL
+Text Notes 2150 5900 2    50   ~ 0
+CAN_GND
+Text Notes 2150 6000 2    50   ~ 0
+VBUS
+Text Notes 2150 6100 2    50   ~ 0
+CAN_SHLD
+$Comp
+L Device:D_Zener D?
+U 1 1 5F7DDDAC
+P 4350 6300
+F 0 "D?" V 4304 6380 50  0000 L CNN
+F 1 "TVS" V 4395 6380 50  0000 L CNN
+F 2 "" H 4350 6300 50  0001 C CNN
+F 3 "~" H 4350 6300 50  0001 C CNN
+	1    4350 6300
+	0    1    1    0
+$EndComp
+Wire Wire Line
+	4350 5950 4350 6150
+Connection ~ 4350 5950
+Wire Wire Line
+	4350 6450 4350 6700
+Wire Wire Line
+	2750 6700 2750 6750
+$Comp
+L power:GND #PWR?
+U 1 1 5F7A7150
+P 2750 6750
+F 0 "#PWR?" H 2750 6500 50  0001 C CNN
+F 1 "GND" H 2755 6577 50  0000 C CNN
+F 2 "" H 2750 6750 50  0001 C CNN
+F 3 "" H 2750 6750 50  0001 C CNN
+	1    2750 6750
+	1    0    0    -1
+$EndComp
+$Comp
+L Device:C C?
+U 1 1 5F7C92D2
+P 3950 6300
+F 0 "C?" H 4065 6346 50  0000 L CNN
+F 1 "1u" H 4065 6255 50  0000 L CNN
+F 2 "" H 3988 6150 50  0001 C CNN
+F 3 "~" H 3950 6300 50  0001 C CNN
+	1    3950 6300
+	1    0    0    -1
+$EndComp
+Wire Wire Line
+	3950 6450 3950 6700
+Wire Wire Line
+	3950 5950 3950 6150
+Wire Wire Line
+	2450 5950 3950 5950
+Connection ~ 3250 6700
+Wire Wire Line
+	3250 6700 3950 6700
+Wire Wire Line
+	2450 5850 2750 5850
+Wire Wire Line
+	2750 6700 3250 6700
+Connection ~ 3950 5950
+Wire Wire Line
+	3950 5950 4350 5950
+Connection ~ 3950 6700
+Wire Wire Line
+	3950 6700 4350 6700
+Connection ~ 2650 5650
+Connection ~ 3450 5750
+Wire Wire Line
+	2650 5650 3800 5650
+Wire Wire Line
+	3450 5750 3800 5750
+Wire Wire Line
+	3050 6500 3050 6550
+Wire Wire Line
+	3050 6150 3050 6200
+$Comp
+L Device:R R?
+U 1 1 5F7B4004
+P 3050 6350
+F 0 "R?" H 3120 6396 50  0000 L CNN
+F 1 "1M" H 3120 6305 50  0000 L CNN
+F 2 "" V 2980 6350 50  0001 C CNN
+F 3 "~" H 3050 6350 50  0001 C CNN
+	1    3050 6350
+	1    0    0    -1
+$EndComp
+Wire Wire Line
+	3250 6050 3250 6150
+Connection ~ 3250 6150
+$Comp
+L Device:C C?
+U 1 1 5F7B7D0B
+P 3450 6350
+F 0 "C?" H 3565 6396 50  0000 L CNN
+F 1 "4.7n" H 3565 6305 50  0000 L CNN
+F 2 "" H 3488 6200 50  0001 C CNN
+F 3 "~" H 3450 6350 50  0001 C CNN
+	1    3450 6350
+	1    0    0    -1
+$EndComp
+Wire Wire Line
+	3050 6150 3250 6150
+Wire Wire Line
+	3450 6150 3450 6200
+Wire Wire Line
+	3250 6150 3450 6150
+Wire Wire Line
+	3050 6550 3250 6550
+Wire Wire Line
+	3450 6550 3450 6500
+Wire Wire Line
+	3250 6550 3250 6700
+Connection ~ 3250 6550
+Wire Wire Line
+	3250 6550 3450 6550
+Wire Wire Line
+	2750 5850 2750 6700
+Wire Wire Line
+	2450 6050 3250 6050
+Connection ~ 2750 6700
 $EndSCHEMATC

Commit message: Do MCU bypassing according to datasheet; annotate
Parts:
- gave numbers to parts that had none: 7
Changed lines of the file:
@@
 Connection ~ 2700 4400
 $Comp
-L Connector_Generic:Conn_01x05 J?
+L Connector_Generic:Conn_01x05 J8
 U 1 1 5F78B096
 P 2250 5850
-F 0 "J?" H 2168 6267 50  0000 C CNN
+F 0 "J8" H 2168 6267 50  0000 C CNN
 F 1 "Conn_01x05" H 2168 6176 50  0000 C CNN
 F 2 "" H 2250 5850 50  0001 C CNN
@@
 	2450 5750 3450 5750
 $Comp
-L Device:D_TVS_x2_AAC D?
+L Device:D_TVS_x2_AAC D17
 U 1 1 5F79E74D
 P 3050 5200
-F 0 "D?" H 3050 5417 50  0000 C CNN
+F 0 "D17" H 3050 5417 50  0000 C CNN
 F 1 "D_TVS_x2_AAC" H 3050 5326 50  0000 C CNN
 F 2 "" H 2900 5200 50  0001 C CNN
@@
 	3450 5200 3450 5750
 $Comp
-L power:GND #PWR?
+L power:GND #PWR0224
 U 1 1 5F7A3138
 P 3050 5400
-F 0 "#PWR?" H 3050 5150 50  0001 C CNN
+F 0 "#PWR0224" H 3050 5150 50  0001 C CNN
 F 1 "GND" H 3055 5227 50  0000 C CNN
 F 2 "" H 3050 5400 50  0001 C CNN
@@
 	4350 5950 4350 5800
 $Comp
-L power:+VSW #PWR?
+L power:+VSW #PWR0225
 U 1 1 5F7A9210
 P 4350 5450
-F 0 "#PWR?" H 4350 5300 50  0001 C CNN
+F 0 "#PWR0225" H 4350 5300 50  0001 C CNN
 F 1 "+VSW" H 4365 5623 50  0000 C CNN
 F 2 "" H 4350 5450 50  0001 C CNN
@@
 	4350 5450 4350 5500
 $Comp
-L Device:D_Schottky D?
+L Device:D_Schottky D18
 U 1 1 5F7AAFC5
 P 4350 5650
-F 0 "D?" V 4396 5570 50  0000 R CNN
+F 0 "D18" V 4396 5570 50  0000 R CNN
 F 1 "D_Schottky" V 4305 5570 50  0000 R CNN
 F 2 "" H 4350 5650 50  0001 C CNN
@@
 CAN_SHLD
 $Comp
-L Device:D_Zener D?
+L Device:D_Zener D19
 U 1 1 5F7DDDAC
 P 4350 6300
-F 0 "D?" V 4304 6380 50  0000 L CNN
+F 0 "D19" V 4304 6380 50  0000 L CNN
 F 1 "TVS" V 4395 6380 50  0000 L CNN
 F 2 "" H 4350 6300 50  0001 C CNN
@@
 	2750 6700 2750 6750
 $Comp
-L power:GND #PWR?
+L power:GND #PWR0226
 U 1 1 5F7A7150
 P 2750 6750
-F 0 "#PWR?" H 2750 6500 50  0001 C CNN
+F 0 "#PWR0226" H 2750 6500 50  0001 C CNN
 F 1 "GND" H 2755 6577 50  0000 C CNN
 F 2 "" H 2750 6750 50  0001 C CNN
@@
 $EndComp
 $Comp
-L Device:C C?
+L Device:C C42
 U 1 1 5F7C92D2
 P 3950 6300
-F 0 "C?" H 4065 6346 50  0000 L CNN
+F 0 "C42" H 4065 6346 50  0000 L CNN
 F 1 "1u" H 4065 6255 50  0000 L CNN
 F 2 "" H 3988 6150 50  0001 C CNN
@@
 	3050 6150 3050 6200
 $Comp
-L Device:R R?
+L Device:R R45
 U 1 1 5F7B4004
 P 3050 6350
-F 0 "R?" H 3120 6396 50  0000 L CNN
+F 0 "R45" H 3120 6396 50  0000 L CNN
 F 1 "1M" H 3120 6305 50  0000 L CNN
 F 2 "" V 2980 6350 50  0001 C CNN
@@
 Connection ~ 3250 6150
 $Comp
-L Device:C C?
+L Device:C C41
 U 1 1 5F7B7D0B
 P 3450 6350
-F 0 "C?" H 3565 6396 50  0000 L CNN
+F 0 "C41" H 3565 6396 50  0000 L CNN
 F 1 "4.7n" H 3565 6305 50  0000 L CNN
 F 2 "" H 3488 6200 50  0001 C CNN

Commit message: Add +3.3V reverse current protection diode; add +3.3V on debug header
Parts:
- removed J4: Conn_01x03_Male, Connector_PinHeader_2.54mm:PinHeader_1x03_P2.54mm_Vertical, symbol Connector:Conn_01x03_Male
- added J4: Conn_01x04_Male, symbol Connector:Conn_01x04_Male
Connections:
- net +3V3: now also J4.4 (Pin_4)
- net GND: now also J4.2 (Pin_2)
- net MCU_SWCLK: now also J4.3 (Pin_3)
- net MCU_SWDIO: now also J4.1 (Pin_1)
Changed lines of the file:
@@
-$EndComp
-$Comp
-L Connector:Conn_01x03_Male J4
-U 1 1 5F75243E
-P 4500 900
-F 0 "J4" H 4608 1089 50  0000 C CNN
-F 1 "Conn_01x03_Male" H 4608 1090 50  0001 C CNN
-F 2 "Connector_PinHeader_2.54mm:PinHeader_1x03_P2.54mm_Vertical" H 4500 900 50  0001 C CNN
-F 3 "~" H 4500 900 50  0001 C CNN
-	1    4500 900
-	1    0    0    -1
 $EndComp
 $Comp
@@
 Wire Wire Line
 	3350 4300 3300 4300
-$Comp
-L power:GND #PWR0158
-U 1 1 5F7A90CE
-P 5300 900
-F 0 "#PWR0158" H 5300 650 50  0001 C CNN
-F 1 "GND" H 5305 727 50  0000 C CNN
-F 2 "" H 5300 900 50  0001 C CNN
-F 3 "" H 5300 900 50  0001 C CNN
-	1    5300 900
-	1    0    0    -1
-$EndComp
-Wire Wire Line
-	4700 900  5300 900
-Text HLabel 4700 800  2    50   BiDi ~ 0
+Wire Wire Line
+	4750 1150 5600 1150
+Text HLabel 4800 1050 2    50   BiDi ~ 0
 MCU_SWDIO
-Text HLabel 4700 1000 2    50   Output ~ 0
+Text HLabel 4800 1250 2    50   Output ~ 0
 MCU_SWCLK
 Text HLabel 3150 1150 2    50   Input ~ 0
@@
 	2450 6050 3250 6050
 Connection ~ 2750 6700
+$Comp
+L Connector:Conn_01x04_Male J4
+U 1 1 5F883EAC
+P 4550 1150
+F 0 "J4" H 4658 1431 50  0000 C CNN
+F 1 "Conn_01x04_Male" H 4658 1340 50  0000 C CNN
+F 2 "" H 4550 1150 50  0001 C CNN
+F 3 "~" H 4550 1150 50  0001 C CNN
+	1    4550 1150
+	1    0    0    -1
+$EndComp
+Wire Wire Line
+	4800 1050 4750 1050
+Wire Wire Line
+	4800 1250 4750 1250
+$Comp
+L power:+3.3V #PWR01
+U 1 1 5F88E1AC
+P 5400 900
+F 0 "#PWR01" H 5400 750 50  0001 C CNN
+F 1 "+3.3V" H 5415 1073 50  0000 C CNN
+F 2 "" H 5400 900 50  0001 C CNN
+F 3 "" H 5400 900 50  0001 C CNN
+	1    5400 900
+	1    0    0    -1
+$EndComp
+Wire Wire Line
+	5400 900  5400 1350
+Wire Wire Line
+	4750 1350 5400 1350
+Wire Wire Line
+	5600 1150 5600 1200
+$Comp
+L power:GND #PWR0158
+U 1 1 5F7A90CE
+P 5600 1200
+F 0 "#PWR0158" H 5600 950 50  0001 C CNN
+F 1 "GND" H 5605 1027 50  0000 C CNN
+F 2 "" H 5600 1200 50  0001 C CNN
+F 3 "" H 5600 1200 50  0001 C CNN
+	1    5600 1200
+	1    0    0    -1
+$EndComp
 $EndSCHEMATC

Commit message: Remove PWR_FLAG from UART header
Changed lines of the file:
@@
 R_MTR_HALL_PHC
-$Comp
-L power:PWR_FLAG #FLG0104
-U 1 1 5F73A64F
-P 2850 4400
-F 0 "#FLG0104" H 2850 4475 50  0001 C CNN
-F 1 "PWR_FLAG" H 2850 4573 50  0000 C CNN
-F 2 "" H 2850 4400 50  0001 C CNN
-F 3 "~" H 2850 4400 50  0001 C CNN
-	1    2850 4400
-	-1   0    0    1
-$EndComp
-Wire Wire Line
-	2700 4400 2850 4400
-Connection ~ 2700 4400
 $Comp
 L Connector_Generic:Conn_01x05 J8

Commit message: added footprints, continue layout
Parts:
- C41, C42: footprint (none) -> Capacitor_SMD:C_0805_2012Metric
- D17: footprint (none) -> Package_TO_SOT_SMD:SOT-23
- D18: value D_Schottky -> B5819W; footprint (none) -> Diode_SMD:D_SOD-123
- D19: value TVS -> 15V TVS C78409; footprint (none) -> Diode_SMD:D_SMB
- J10: renamed from UART_R1; value (none) -> UART_R1
- J4: footprint (none) -> Connector_PinHeader_2.54mm:PinHeader_1x04_P2.54mm_Vertical
- J8: footprint (none) -> Connector_PinHeader_2.54mm:PinHeader_1x05_P2.54mm_Vertical
- J9: renamed from UART_L1; value (none) -> UART_L1
- R45: footprint (none) -> Resistor_SMD:R_0603_1608Metric
Changed lines of the file:
@@
 $EndDescr
 $Comp
-L Connector:Conn_01x04_Male UART_L1
+L Connector:Conn_01x04_Male J9
 U 1 1 5F74D721
 P 2250 1850
-F 0 "UART_L1" H 2358 2039 50  0000 C CNN
-F 1 " " H 2358 2040 50  0001 C CNN
+F 0 "J9" H 2358 2039 50  0000 C CNN
+F 1 " UART_L1" H 2358 2040 50  0001 C CNN
 F 2 "Connector_PinHeader_2.54mm:PinHeader_1x04_P2.54mm_Vertical" H 2250 1850 50  0001 C CNN
 F 3 "~" H 2250 1850 50  0001 C CNN
@@
 $EndComp
 $Comp
-L Connector:Conn_01x04_Male UART_R1
+L Connector:Conn_01x04_Male J10
 U 1 1 5F750DE0
 P 2250 4200
-F 0 "UART_R1" H 2358 4389 50  0000 C CNN
-F 1 " " H 2358 4390 50  0001 C CNN
+F 0 "J10" H 2358 4389 50  0000 C CNN
+F 1 " UART_R1" H 2358 4390 50  0001 C CNN
 F 2 "Connector_PinHeader_2.54mm:PinHeader_1x04_P2.54mm_Vertical" H 2250 4200 50  0001 C CNN
 F 3 "~" H 2250 4200 50  0001 C CNN
@@
 F 0 "J8" H 2168 6267 50  0000 C CNN
 F 1 "Conn_01x05" H 2168 6176 50  0000 C CNN
-F 2 "" H 2250 5850 50  0001 C CNN
+F 2 "Connector_PinHeader_2.54mm:PinHeader_1x05_P2.54mm_Vertical" H 2250 5850 50  0001 C CNN
 F 3 "~" H 2250 5850 50  0001 C CNN
 	1    2250 5850
@@
 F 0 "D17" H 3050 5417 50  0000 C CNN
 F 1 "D_TVS_x2_AAC" H 3050 5326 50  0000 C CNN
-F 2 "" H 2900 5200 50  0001 C CNN
+F 2 "Package_TO_SOT_SMD:SOT-23" H 2900 5200 50  0001 C CNN
 F 3 "~" H 2900 5200 50  0001 C CNN
 	1    3050 5200
@@
 P 4350 5650
 F 0 "D18" V 4396 5570 50  0000 R CNN
-F 1 "D_Schottky" V 4305 5570 50  0000 R CNN
-F 2 "" H 4350 5650 50  0001 C CNN
+F 1 "B5819W" V 4305 5570 50  0000 R CNN
+F 2 "Diode_SMD:D_SOD-123" H 4350 5650 50  0001 C CNN
 F 3 "~" H 4350 5650 50  0001 C CNN
 	1    4350 5650
@@
 P 4350 6300
 F 0 "D19" V 4304 6380 50  0000 L CNN
-F 1 "TVS" V 4395 6380 50  0000 L CNN
-F 2 "" H 4350 6300 50  0001 C CNN
+F 1 "15V TVS C78409" V 4395 6380 50  0000 L CNN
+F 2 "Diode_SMD:D_SMB" H 4350 6300 50  0001 C CNN
 F 3 "~" H 4350 6300 50  0001 C CNN
 	1    4350 6300
@@
 F 0 "C42" H 4065 6346 50  0000 L CNN
 F 1 "1u" H 4065 6255 50  0000 L CNN
-F 2 "" H 3988 6150 50  0001 C CNN
+F 2 "Capacitor_SMD:C_0805_2012Metric" H 3988 6150 50  0001 C CNN
 F 3 "~" H 3950 6300 50  0001 C CNN
 	1    3950 6300
@@
 F 0 "R45" H 3120 6396 50  0000 L CNN
 F 1 "1M" H 3120 6305 50  0000 L CNN
-F 2 "" V 2980 6350 50  0001 C CNN
+F 2 "Resistor_SMD:R_0603_1608Metric" V 2980 6350 50  0001 C CNN
 F 3 "~" H 3050 6350 50  0001 C CNN
 	1    3050 6350
@@
 F 0 "C41" H 3565 6396 50  0000 L CNN
 F 1 "4.7n" H 3565 6305 50  0000 L CNN
-F 2 "" H 3488 6200 50  0001 C CNN
+F 2 "Capacitor_SMD:C_0805_2012Metric" H 3488 6200 50  0001 C CNN
 F 3 "~" H 3450 6350 50  0001 C CNN
 	1    3450 6350
@@
 F 0 "J4" H 4658 1431 50  0000 C CNN
 F 1 "Conn_01x04_Male" H 4658 1340 50  0000 C CNN
-F 2 "" H 4550 1150 50  0001 C CNN
+F 2 "Connector_PinHeader_2.54mm:PinHeader_1x04_P2.54mm_Vertical" H 4550 1150 50  0001 C CNN
 F 3 "~" H 4550 1150 50  0001 C CNN
 	1    4550 1150

Commit message: continue analog layout
Parts:
- added D29, D30, D31, D32, D33, D34: LED, LED_SMD:LED_0603_1608Metric, symbol Device:LED
Connections:
- net +3V3: now also D29.2 (A), D30.2 (A), D31.2 (A), D32.2 (A), D33.2 (A), D34.2 (A); no longer R16L1.1, R16L2.1, R17L1.1, R17L2.1, R18L1.1, R18L2.1
- new net: D29.1 (K), R16L1.1
- new net: D31.1 (K), R17L1.1
- new net: D33.1 (K), R18L1.1
- new net: D30.1 (K), R16L2.1
- new net: D32.1 (K), R17L2.1
- new net: D34.1 (K), R18L2.1
Other:
- moved on the sheet: C2, C41, C42, D0AL1, D17, D18, D19, HALL_R1, J10, J8, J9, R16L2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

Commit message: continue board layout, placed all components
Connections:
- net +VSW: now also J10.4 (Pin_4), J9.4 (Pin_4); no longer J10.1 (Pin_1), J9.1 (Pin_1)
- net GND: now also HALL_R1.1 (Pin_1), J10.1 (Pin_1), J9.1 (Pin_1); no longer HALL_R1.5 (Pin_5), J10.4 (Pin_4), J9.4 (Pin_4)
- net at J9.2 (Pin_2): now also R38.2; no longer R36.2
- net at J9.3 (Pin_3): now also R36.2; no longer R38.2
- net at C2.1, D0AL1.1 (K), HALL_L1.5 (Pin_5): now also HALL_R1.5 (Pin_5); no longer HALL_R1.1 (Pin_1)
- net at R16L2.2, R21L2.1: now also HALL_R1.4 (Pin_4); no longer HALL_R1.2 (Pin_2)
- net at R18L2.2, R19L2.1: now also HALL_R1.2 (Pin_2); no longer HALL_R1.4 (Pin_4)
- net at J10.2 (Pin_2): now also R37.2; no longer R35.2
- net at J10.3 (Pin_3): now also R35.2; no longer R37.2
Changed lines of the file:
@@
 L Connector:Conn_01x04_Male J9
 U 1 1 5F74D721
-P 2200 1350
-F 0 "J9" H 2308 1539 50  0000 C CNN
-F 1 " UART_L1" H 2308 1540 50  0001 C CNN
-F 2 "Connector_PinHeader_2.54mm:PinHeader_1x04_P2.54mm_Vertical" H 2200 1350 50  0001 C CNN
-F 3 "~" H 2200 1350 50  0001 C CNN
-	1    2200 1350
-	1    0    0    -1
+P 2200 1450
+F 0 "J9" H 2308 1639 50  0000 C CNN
+F 1 " UART_L1" H 2308 1640 50  0001 C CNN
+F 2 "Connector_PinHeader_2.54mm:PinHeader_1x04_P2.54mm_Vertical" H 2200 1450 50  0001 C CNN
+F 3 "~" H 2200 1450 50  0001 C CNN
+	1    2200 1450
+	1    0    0    1
 $EndComp
 $Comp
@@
 F 3 "~" H 2250 4500 50  0001 C CNN
 	1    2250 4500
-	1    0    0    -1
+	1    0    0    1
 $EndComp
 $Comp
 L Connector:Conn_01x04_Male J10
 U 1 1 5F750DE0
-P 2250 5300
-F 0 "J10" H 2358 5489 50  0000 C CNN
-F 1 " UART_R1" H 2358 5490 50  0001 C CNN
-F 2 "Connector_PinHeader_2.54mm:PinHeader_1x04_P2.54mm_Vertical" H 2250 5300 50  0001 C CNN
-F 3 "~" H 2250 5300 50  0001 C CNN
-	1    2250 5300
-	1    0    0    -1
+P 2250 5400
+F 0 "J10" H 2358 5589 50  0000 C CNN
+F 1 " UART_R1" H 2358 5590 50  0001 C CNN
+F 2 "Connector_PinHeader_2.54mm:PinHeader_1x04_P2.54mm_Vertical" H 2250 5400 50  0001 C CNN
+F 3 "~" H 2250 5400 50  0001 C CNN
+	1    2250 5400
+	1    0    0    1
 $EndComp
 $Comp
