File: connectors.sch (KiCad schematic (older format))
At the start: 36 parts, among them J10 UART_R1, J4 Conn_01x04_Male, J8 Conn_01x05, J9 UART_L1

Commit message: finish design
Parts:
- added R16L3, R16L4, R17L3, R17L4, R18L3, R18L4: 2K2, Resistor_SMD:R_0603_1608Metric, symbol Device:R
Connections:
- net +3V3: now also R16L3.1, R16L4.1, R17L3.1, R17L4.1, R18L3.1, R18L4.1
- net at HALL_L1.2 (Pin_2), R16L1.2, R21L1.1: now also R16L3.2
- net at HALL_L1.3 (Pin_3), R17L1.2, R20L1.1: now also R17L3.2
- net at HALL_L1.4 (Pin_4), R18L1.2, R19L1.1: now also R18L3.2
- net at HALL_R1.2 (Pin_2), R18L2.2, R19L2.1: now also R18L4.2
- net at HALL_R1.3 (Pin_3), R17L2.2, R20L2.1: now also R17L4.2
- net at HALL_R1.4 (Pin_4), R16L2.2, R21L2.1: now also R16L4.2
Changed lines of the file:
@@
 $EndComp
-Wire Wire Line
-	2450 2600 2900 2600
 Wire Wire Line
 	4050 2700 3250 2700
 Wire Wire Line
-	2450 2800 3600 2800
+	2450 2800 3500 2800
 Wire Wire Line
 	2900 2550 2900 2600
 Connection ~ 2900 2600
 Wire Wire Line
-	2900 2600 3800 2600
-Wire Wire Line
 	3250 2550 3250 2700
 Connection ~ 3250 2700
-Wire Wire Line
-	3250 2700 2450 2700
 Wire Wire Line
 	3600 2550 3600 2800
@@
 $EndComp
 Wire Wire Line
-	2450 4400 2900 4400
+	2450 4400 2800 4400
 Wire Wire Line
 	4050 4500 3250 4500
-Wire Wire Line
-	2450 4600 3600 4600
 Wire Wire Line
 	2900 4350 2900 4400
 Connection ~ 2900 4400
 Wire Wire Line
-	2900 4400 3800 4400
-Wire Wire Line
 	3250 4350 3250 4500
 Connection ~ 3250 4500
 Wire Wire Line
-	3250 4500 2450 4500
+	3250 4500 3150 4500
 Wire Wire Line
 	3600 4350 3600 4600
@@
 $EndComp
 Wire Wire Line
-	2900 1950 3250 1950
+	2900 1950 3150 1950
 Connection ~ 3250 1950
 Wire Wire Line
-	3250 1950 3600 1950
+	3250 1950 3500 1950
 Wire Wire Line
 	3250 1850 3250 1950
@@
 $EndComp
 Wire Wire Line
-	2900 3750 3250 3750
+	2900 3750 3150 3750
 Connection ~ 3250 3750
 Wire Wire Line
-	3250 3750 3600 3750
+	3250 3750 3500 3750
 Wire Wire Line
 	3250 3500 3250 3750
+$Comp
+L Device:R R16L3
+U 1 1 5F8901AA
+P 2800 2400
+F 0 "R16L3" H 2870 2446 50  0000 L CNN
+F 1 "2K2" H 2870 2355 50  0000 L CNN
+F 2 "Resistor_SMD:R_0603_1608Metric" V 2730 2400 50  0001 C CNN
+F 3 "~" H 2800 2400 50  0001 C CNN
+	1    2800 2400
+	1    0    0    -1
+$EndComp
+$Comp
+L Device:R R17L3
+U 1 1 5F890945
+P 3150 2400
+F 0 "R17L3" H 3220 2446 50  0000 L CNN
+F 1 "2K2" H 3220 2355 50  0000 L CNN
+F 2 "Resistor_SMD:R_0603_1608Metric" V 3080 2400 50  0001 C CNN
+F 3 "~" H 3150 2400 50  0001 C CNN
+	1    3150 2400
+	1    0    0    -1
+$EndComp
+$Comp
+L Device:R R18L3
+U 1 1 5F890B23
+P 3500 2400
+F 0 "R18L3" H 3570 2446 50  0000 L CNN
+F 1 "2K2" H 3570 2355 50  0000 L CNN
+F 2 "Resistor_SMD:R_0603_1608Metric" V 3430 2400 50  0001 C CNN
+F 3 "~" H 3500 2400 50  0001 C CNN
+	1    3500 2400
+	1    0    0    -1
+$EndComp
+Wire Wire Line
+	2450 2600 2800 2600
+Wire Wire Line
+	2800 2550 2800 2600
+Connection ~ 2800 2600
+Wire Wire Line
+	2800 2600 2900 2600
+Wire Wire Line
+	3500 2250 3500 1950
+Connection ~ 3500 1950
+Wire Wire Line
+	3500 1950 3600 1950
+Wire Wire Line
+	3150 2250 3150 1950
+Connection ~ 3150 1950
+Wire Wire Line
+	3150 1950 3250 1950
+Wire Wire Line
+	2800 2250 2800 1950
+Wire Wire Line
+	2800 1950 2900 1950
+Connection ~ 2900 1950
+$Comp
+L Device:R R16L4
+U 1 1 5F8A0AE7
+P 2800 4200
+F 0 "R16L4" H 2870 4246 50  0000 L CNN
+F 1 "2K2" H 2870 4155 50  0000 L CNN
+F 2 "Resistor_SMD:R_0603_1608Metric" V 2730 4200 50  0001 C CNN
+F 3 "~" H 2800 4200 50  0001 C CNN
+	1    2800 4200
+	1    0    0    -1
+$EndComp
+$Comp
+L Device:R R17L4
+U 1 1 5F8A0C56
+P 3150 4200
+F 0 "R17L4" H 3220 4246 50  0000 L CNN
+F 1 "2K2" H 3220 4155 50  0000 L CNN
+F 2 "Resistor_SMD:R_0603_1608Metric" V 3080 4200 50  0001 C CNN
+F 3 "~" H 3150 4200 50  0001 C CNN
+	1    3150 4200
+	1    0    0    -1
+$EndComp
+$Comp
+L Device:R R18L4
+U 1 1 5F8A0DC6
+P 3500 4200
+F 0 "R18L4" H 3570 4246 50  0000 L CNN
+F 1 "2K2" H 3570 4155 50  0000 L CNN
+F 2 "Resistor_SMD:R_0603_1608Metric" V 3430 4200 50  0001 C CNN
+F 3 "~" H 3500 4200 50  0001 C CNN
+	1    3500 4200
+	1    0    0    -1
+$EndComp
+Wire Wire Line
+	2800 4350 2800 4400
+Connection ~ 2800 4400
+Wire Wire Line
+	2800 4400 2900 4400
+Wire Wire Line
+	3500 4050 3500 3750
+Connection ~ 3500 3750
+Wire Wire Line
+	3500 3750 3600 3750
+Wire Wire Line
+	3150 4050 3150 3750
+Connection ~ 3150 3750
+Wire Wire Line
+	3150 3750 3250 3750
+Wire Wire Line
+	2800 4050 2800 3750
+Wire Wire Line
+	2800 3750 2900 3750
+Connection ~ 2900 3750
+Wire Wire Line
+	2900 4400 3800 4400
+Wire Wire Line
+	2450 4600 3500 4600
+Wire Wire Line
+	3150 4350 3150 4500
+Connection ~ 3150 4500
+Wire Wire Line
+	3150 4500 2450 4500
+Wire Wire Line
+	3500 4350 3500 4600
+Connection ~ 3500 4600
+Wire Wire Line
+	3500 4600 3600 4600
+Wire Wire Line
+	3250 2700 3150 2700
+Wire Wire Line
+	2900 2600 3800 2600
+Wire Wire Line
+	3150 2550 3150 2700
+Connection ~ 3150 2700
+Wire Wire Line
+	3150 2700 2450 2700
+Wire Wire Line
+	3500 2550 3500 2800
+Connection ~ 3500 2800
+Wire Wire Line
+	3500 2800 3600 2800
 $EndSCHEMATC

Commit message: added TVS diodes on HALL inputs
Parts:
- added U? (x2): SRV05-4, Package_TO_SOT_SMD:SOT-23-6, symbol Power_Protection:SRV05-4
Connections:
- net GND: now also U?.2 (VN), U?.2 (VN)
- net Hall_L_1: now reaches HALL_L1.2 (Pin_2), R16L1.2, R16L3.2, R21L1.1
- net Hall_L_1: now also U?.1 (IO1)
- net Hall_L_2: now reaches HALL_L1.3 (Pin_3), R17L1.2, R17L3.2, R20L1.1
- net Hall_L_2: now also U?.4 (IO3)
- net Hall_L_3: now reaches HALL_L1.4 (Pin_4), R18L1.2, R18L3.2, R19L1.1
- net Hall_L_3: now also U?.6 (IO4)
- net Hall_VCC: now reaches C2.1, D0AL1.1 (K), HALL_L1.5 (Pin_5), HALL_R1.5 (Pin_5)
- net Hall_VCC: now also U?.5 (VP), U?.5 (VP)
- net Hall_R_3: now reaches HALL_R1.2 (Pin_2), R18L2.2, R18L4.2, R19L2.1
- net Hall_R_3: now also U?.1 (IO1)
- net Hall_R_2: now reaches HALL_R1.3 (Pin_3), R17L2.2, R17L4.2, R20L2.1
- net Hall_R_2: now also U?.6 (IO4)
- net Hall_R_1: now reaches HALL_R1.4 (Pin_4), R16L2.2, R16L4.2, R21L2.1
- net Hall_R_1: now also U?.4 (IO3)
Changed lines of the file:
@@
-$EndComp
-$Comp
-L Connector:Conn_01x04_Male J10
-U 1 1 5F750DE0
-P 2250 5400
-F 0 "J10" H 2358 5589 50  0000 C CNN
-F 1 " UART_R1" H 2358 5590 50  0001 C CNN
-F 2 "Connector_PinHeader_2.54mm:PinHeader_1x04_P2.54mm_Vertical" H 2250 5400 50  0001 C CNN
-F 3 "~" H 2250 5400 50  0001 C CNN
-	1    2250 5400
-	1    0    0    1
 $EndComp
 $Comp
@@
 L power:GND #PWR0153
 U 1 1 5F7999C9
-P 1600 4500
-F 0 "#PWR0153" H 1600 4250 50  0001 C CNN
-F 1 "GND" H 1605 4327 50  0000 C CNN
-F 2 "" H 1600 4500 50  0001 C CNN
-F 3 "" H 1600 4500 50  0001 C CNN
-	1    1600 4500
+P 1600 4550
+F 0 "#PWR0153" H 1600 4300 50  0001 C CNN
+F 1 "GND" H 1605 4377 50  0000 C CNN
+F 2 "" H 1600 4550 50  0001 C CNN
+F 3 "" H 1600 4550 50  0001 C CNN
+	1    1600 4550
 	1    0    0    -1
 $EndComp
@@
 	1    0    0    -1
 $EndComp
-$Comp
-L power:+VSW #PWR0156
-U 1 1 5F79AEC1
-P 2700 5200
-F 0 "#PWR0156" H 2700 5050 50  0001 C CNN
-F 1 "+VSW" H 2715 5373 50  0000 C CNN
-F 2 "" H 2700 5200 50  0001 C CNN
-F 3 "" H 2700 5200 50  0001 C CNN
-	1    2700 5200
-	1    0    0    -1
-$EndComp
-Wire Wire Line
-	2700 5200 2450 5200
-$Comp
-L power:GND #PWR0157
-U 1 1 5F79BFBF
-P 2700 5500
-F 0 "#PWR0157" H 2700 5250 50  0001 C CNN
-F 1 "GND" H 2705 5327 50  0000 C CNN
-F 2 "" H 2700 5500 50  0001 C CNN
-F 3 "" H 2700 5500 50  0001 C CNN
-	1    2700 5500
-	1    0    0    -1
-$EndComp
-Wire Wire Line
-	2700 5500 2450 5500
-$Comp
-L Device:R R35
-U 1 1 5F79D104
-P 2850 5300
-F 0 "R35" V 2643 5300 50  0000 C CNN
-F 1 "100" V 2734 5300 50  0000 C CNN
-F 2 "Resistor_SMD:R_0603_1608Metric" V 2780 5300 50  0001 C CNN
-F 3 "~" H 2850 5300 50  0001 C CNN
-	1    2850 5300
-	0    1    1    0
-$EndComp
-$Comp
-L Device:R R37
-U 1 1 5F79D714
-P 3150 5400
-F 0 "R37" V 2943 5400 50  0000 C CNN
-F 1 "100" V 3034 5400 50  0000 C CNN
-F 2 "Resistor_SMD:R_0603_1608Metric" V 3080 5400 50  0001 C CNN
-F 3 "~" H 3150 5400 50  0001 C CNN
-	1    3150 5400
-	0    1    1    0
-$EndComp
-Wire Wire Line
-	2700 5300 2450 5300
-Wire Wire Line
-	3000 5400 2450 5400
-Wire Wire Line
-	3000 4850 3000 5300
-Wire Wire Line
-	3350 5000 3350 5400
-Wire Wire Line
-	3350 5400 3300 5400
 Wire Wire Line
 	4750 1150 5600 1150
@@
 Text HLabel 3350 900  2    50   Output ~ 0
 UART_L_RX
-Text HLabel 3000 4850 2    50   Input ~ 0
-UART_R_TX
-Text HLabel 3350 5000 2    50   Output ~ 0
-UART_R_RX
 Text HLabel 4700 2600 2    50   Output ~ 0
 L_MTR_HALL_PHC
@@
 Wire Wire Line
 	3500 2800 3600 2800
+Wire Wire Line
+	1600 4550 1600 4500
+Text HLabel 3000 4850 2    50   Input ~ 0
+UART_R_TX
+Text HLabel 3350 5000 2    50   Output ~ 0
+UART_R_RX
+Wire Wire Line
+	3350 5400 3300 5400
+Wire Wire Line
+	3350 5000 3350 5400
+Wire Wire Line
+	3000 4850 3000 5300
+Wire Wire Line
+	3000 5400 2450 5400
+Wire Wire Line
+	2700 5300 2450 5300
+$Comp
+L Device:R R37
+U 1 1 5F79D714
+P 3150 5400
+F 0 "R37" V 2943 5400 50  0000 C CNN
+F 1 "100" V 3034 5400 50  0000 C CNN
+F 2 "Resistor_SMD:R_0603_1608Metric" V 3080 5400 50  0001 C CNN
+F 3 "~" H 3150 5400 50  0001 C CNN
+	1    3150 5400
+	0    1    1    0
+$EndComp
+$Comp
+L Device:R R35
+U 1 1 5F79D104
+P 2850 5300
+F 0 "R35" V 2643 5300 50  0000 C CNN
+F 1 "100" V 2734 5300 50  0000 C CNN
+F 2 "Resistor_SMD:R_0603_1608Metric" V 2780 5300 50  0001 C CNN
+F 3 "~" H 2850 5300 50  0001 C CNN
+	1    2850 5300
+	0    1    1    0
+$EndComp
+Wire Wire Line
+	2700 5500 2450 5500
+$Comp
+L power:GND #PWR0157
+U 1 1 5F79BFBF
+P 2700 5500
+F 0 "#PWR0157" H 2700 5250 50  0001 C CNN
+F 1 "GND" H 2705 5327 50  0000 C CNN
+F 2 "" H 2700 5500 50  0001 C CNN
+F 3 "" H 2700 5500 50  0001 C CNN
+	1    2700 5500
+	1    0    0    -1
+$EndComp
+Wire Wire Line
+	2700 5200 2450 5200
+$Comp
+L power:+VSW #PWR0156
+U 1 1 5F79AEC1
+P 2700 5200
+F 0 "#PWR0156" H 2700 5050 50  0001 C CNN
+F 1 "+VSW" H 2715 5373 50  0000 C CNN
+F 2 "" H 2700 5200 50  0001 C CNN
+F 3 "" H 2700 5200 50  0001 C CNN
+	1    2700 5200
+	1    0    0    -1
+$EndComp
+$Comp
+L Connector:Conn_01x04_Male J10
+U 1 1 5F750DE0
+P 2250 5400
+F 0 "J10" H 2358 5589 50  0000 C CNN
+F 1 " UART_R1" H 2358 5590 50  0001 C CNN
+F 2 "Connector_PinHeader_2.54mm:PinHeader_1x04_P2.54mm_Vertical" H 2250 5400 50  0001 C CNN
+F 3 "~" H 2250 5400 50  0001 C CNN
+	1    2250 5400
+	1    0    0    1
+$EndComp
+$Comp
+L Power_Protection:SRV05-4 U?
+U 1 1 5F9B9AE8
+P 1300 2750
+F 0 "U?" H 1300 3431 50  0000 C CNN
+F 1 "SRV05-4" H 1300 3340 50  0000 C CNN
+F 2 "Package_TO_SOT_SMD:SOT-23-6" H 2000 2300 50  0001 C CNN
+F 3 "http://www.onsemi.com/pub/Collateral/SRV05-4-D.PDF" H 1300 2750 50  0001 C CNN
+	1    1300 2750
+	1    0    0    -1
+$EndComp
+Text Label 2450 2600 0    50   ~ 0
+Hall_L_1
+Text Label 2450 2700 0    50   ~ 0
+Hall_L_2
+Text Label 2450 2800 0    50   ~ 0
+Hall_L_3
+Text Label 1800 2850 0    50   ~ 0
+Hall_L_3
+Text Label 1800 2650 0    50   ~ 0
+Hall_L_2
+Text Label 800  2650 2    50   ~ 0
+Hall_L_1
+$Comp
+L power:GND #PWR?
+U 1 1 5F9C9519
+P 1300 3250
+F 0 "#PWR?" H 1300 3000 50  0001 C CNN
+F 1 "GND" H 1305 3077 50  0000 C CNN
+F 2 "" H 1300 3250 50  0001 C CNN
+F 3 "" H 1300 3250 50  0001 C CNN
+	1    1300 3250
+	1    0    0    -1
+$EndComp
+Text Label 2550 3150 0    50   ~ 0
+Hall_VCC
+Text Label 1300 2250 0    50   ~ 0
+Hall_VCC
+$Comp
+L Power_Protection:SRV05-4 U?
+U 1 1 5F9CA42C
+P 1350 5650
+F 0 "U?" H 1350 6331 50  0000 C CNN
+F 1 "SRV05-4" H 1350 6240 50  0000 C CNN
+F 2 "Package_TO_SOT_SMD:SOT-23-6" H 2050 5200 50  0001 C CNN
+F 3 "http://www.onsemi.com/pub/Collateral/SRV05-4-D.PDF" H 1350 5650 50  0001 C CNN
+	1    1350 5650
+	1    0    0    -1
+$EndComp
+$Comp
+L power:GND #PWR?
+U 1 1 5F9CA436
+P 1350 6150
+F 0 "#PWR?" H 1350 5900 50  0001 C CNN
+F 1 "GND" H 1355 5977 50  0000 C CNN
+F 2 "" H 1350 6150 50  0001 C CNN
+F 3 "" H 1350 6150 50  0001 C CNN
+	1    1350 6150
+	1    0    0    -1
+$EndComp
+Text Label 1350 5150 0    50   ~ 0
+Hall_VCC
+Text Label 2450 4400 0    50   ~ 0
+Hall_R_1
+Text Label 2450 4500 0    50   ~ 0
+Hall_R_2
+Text Label 2450 4600 0    50   ~ 0
+Hall_R_3
+Text Label 1850 5550 0    50   ~ 0
+Hall_R_1
+Text Label 1850 5750 0    50   ~ 0
+Hall_R_2
+Text Label 850  5550 2    50   ~ 0
+Hall_R_3
 $EndSCHEMATC

Commit message: add logos
Parts:
- gave numbers to parts that had none: 2
Changed lines of the file:
@@
 $EndComp
 $Comp
-L Power_Protection:SRV05-4 U?
+L Power_Protection:SRV05-4 U5
 U 1 1 5F9B9AE8
 P 1300 2750
-F 0 "U?" H 1300 3431 50  0000 C CNN
+F 0 "U5" H 1300 3431 50  0000 C CNN
 F 1 "SRV05-4" H 1300 3340 50  0000 C CNN
 F 2 "Package_TO_SOT_SMD:SOT-23-6" H 2000 2300 50  0001 C CNN
@@
 Hall_L_1
 $Comp
-L power:GND #PWR?
+L power:GND #PWR0241
 U 1 1 5F9C9519
 P 1300 3250
-F 0 "#PWR?" H 1300 3000 50  0001 C CNN
+F 0 "#PWR0241" H 1300 3000 50  0001 C CNN
 F 1 "GND" H 1305 3077 50  0000 C CNN
 F 2 "" H 1300 3250 50  0001 C CNN
@@
 Hall_VCC
 $Comp
-L Power_Protection:SRV05-4 U?
+L Power_Protection:SRV05-4 U15
 U 1 1 5F9CA42C
 P 1350 5650
-F 0 "U?" H 1350 6331 50  0000 C CNN
+F 0 "U15" H 1350 6331 50  0000 C CNN
 F 1 "SRV05-4" H 1350 6240 50  0000 C CNN
 F 2 "Package_TO_SOT_SMD:SOT-23-6" H 2050 5200 50  0001 C CNN
@@
 $EndComp
 $Comp
-L power:GND #PWR?
+L power:GND #PWR0242
 U 1 1 5F9CA436
 P 1350 6150
-F 0 "#PWR?" H 1350 5900 50  0001 C CNN
+F 0 "#PWR0242" H 1350 5900 50  0001 C CNN
 F 1 "GND" H 1355 5977 50  0000 C CNN
 F 2 "" H 1350 6150 50  0001 C CNN

Commit message: Minor changes to PCB; convert footprint library to .pretty format, add to project
Parts:
- D17: value D_TVS_x2_AAC -> PESD15VL2BT,215
Connections:
- no-connect marks 0 -> 2
Changed lines of the file:
@@
 P 4800 5800
 F 0 "D17" H 4800 6017 50  0000 C CNN
-F 1 "D_TVS_x2_AAC" H 4800 5926 50  0000 C CNN
+F 1 "PESD15VL2BT,215" H 4800 5926 50  0000 C CNN
 F 2 "Package_TO_SOT_SMD:SOT-23" H 4650 5800 50  0001 C CNN
 F 3 "~" H 4650 5800 50  0001 C CNN
@@
 Text Label 850  5550 2    50   ~ 0
 Hall_R_3
+NoConn ~ 850  5750
+NoConn ~ 800  2850
 $EndSCHEMATC

Commit message: modify hall sensor VCC so that overvoltage on one hall sensor will not affect the other motor
Parts:
- added C?: 100n, Capacitor_SMD:C_0603_1608Metric, symbol Device:C
- added D0AL?: 1N4148W, Diode_SMD:D_SOD-123, symbol Device:D
Connections:
- net +5V: now also D0AL?.2 (A)
- net GND: now also C?.2
- net Hall_VCC: no longer HALL_R1.5 (Pin_5), U15.5 (VP)
- new net Hall_VCC_2: C?.1, D0AL?.1 (K), HALL_R1.5 (Pin_5), U15.5 (VP)
Other:
- moved on the sheet: C2, D0AL1
Changed lines of the file:
@@
 	2450 4300 2550 4300
-Wire Wire Line
-	2550 4300 2550 4150
 Wire Wire Line
 	2550 2900 2450 2900
@@
 L Device:C C2
 U 1 1 5F79865D
-P 1600 4350
-F 0 "C2" H 1715 4350 50  0000 L CNN
-F 1 "100n" H 1715 4305 50  0001 L CNN
-F 2 "Capacitor_SMD:C_0603_1608Metric" H 1638 4200 50  0001 C CNN
-F 3 "~" H 1600 4350 50  0001 C CNN
-	1    1600 4350
-	1    0    0    -1
-$EndComp
-Wire Wire Line
-	2550 4150 1600 4150
-Wire Wire Line
-	1600 4150 1600 4200
-Connection ~ 2550 4150
+P 1950 3750
+F 0 "C2" H 2065 3750 50  0000 L CNN
+F 1 "100n" H 2065 3705 50  0001 L CNN
+F 2 "Capacitor_SMD:C_0603_1608Metric" H 1988 3600 50  0001 C CNN
+F 3 "~" H 1950 3750 50  0001 C CNN
+	1    1950 3750
+	1    0    0    -1
+$EndComp
+Wire Wire Line
+	1950 3550 1950 3600
 $Comp
 L power:GND #PWR0153
 U 1 1 5F7999C9
-P 1600 4550
-F 0 "#PWR0153" H 1600 4300 50  0001 C CNN
-F 1 "GND" H 1605 4377 50  0000 C CNN
-F 2 "" H 1600 4550 50  0001 C CNN
-F 3 "" H 1600 4550 50  0001 C CNN
-	1    1600 4550
+P 1950 3950
+F 0 "#PWR0153" H 1950 3700 50  0001 C CNN
+F 1 "GND" H 1955 3777 50  0000 C CNN
+F 2 "" H 1950 3950 50  0001 C CNN
+F 3 "" H 1950 3950 50  0001 C CNN
+	1    1950 3950
 	1    0    0    -1
 $EndComp
@@
 L Device:D D0AL1
 U 1 1 5F799DC8
-P 1600 4000
-F 0 "D0AL1" V 1646 3921 50  0000 R CNN
-F 1 "1N4148W" V 1555 3921 50  0000 R CNN
-F 2 "Diode_SMD:D_SOD-123" H 1600 4000 50  0001 C CNN
-F 3 "~" H 1600 4000 50  0001 C CNN
-	1    1600 4000
-	0    -1   -1   0
-$EndComp
-Connection ~ 1600 4150
+P 1950 3400
+F 0 "D0AL1" V 1996 3321 50  0000 R CNN
+F 1 "1N4148W" V 1905 3321 50  0000 R CNN
+F 2 "Diode_SMD:D_SOD-123" H 1950 3400 50  0001 C CNN
+F 3 "~" H 1950 3400 50  0001 C CNN
+	1    1950 3400
+	0    -1   -1   0
+$EndComp
 $Comp
 L power:+5V #PWR0154
 U 1 1 5F79A839
-P 1600 3850
-F 0 "#PWR0154" H 1600 3700 50  0001 C CNN
-F 1 "+5V" H 1615 4023 50  0000 C CNN
-F 2 "" H 1600 3850 50  0001 C CNN
-F 3 "" H 1600 3850 50  0001 C CNN
-	1    1600 3850
+P 1950 3250
+F 0 "#PWR0154" H 1950 3100 50  0001 C CNN
+F 1 "+5V" H 1965 3423 50  0000 C CNN
+F 2 "" H 1950 3250 50  0001 C CNN
+F 3 "" H 1950 3250 50  0001 C CNN
+	1    1950 3250
 	1    0    0    -1
 $EndComp
@@
 Wire Wire Line
 	3250 1850 3250 1950
-Wire Wire Line
-	2550 2900 2550 4150
 $Comp
 L Device:LED D?
@@
 	3500 2800 3600 2800
 Wire Wire Line
-	1600 4550 1600 4500
+	1950 3950 1950 3900
 Text HLabel 3000 4850 2    50   Input ~ 0
 UART_R_TX
@@
 $EndComp
 Text Label 1350 5150 0    50   ~ 0
-Hall_VCC
+Hall_VCC_2
 Text Label 2450 4400 0    50   ~ 0
 Hall_R_1
@@
 NoConn ~ 850  5750
 NoConn ~ 800  2850
+$Comp
+L Device:D D0AL?
+U 1 1 5F740132
+P 1400 4200
+F 0 "D0AL?" V 1446 4121 50  0000 R CNN
+F 1 "1N4148W" V 1355 4121 50  0000 R CNN
+F 2 "Diode_SMD:D_SOD-123" H 1400 4200 50  0001 C CNN
+F 3 "~" H 1400 4200 50  0001 C CNN
+	1    1400 4200
+	0    -1   -1   0
+$EndComp
+$Comp
+L Device:C C?
+U 1 1 5F7405CA
+P 1400 4550
+F 0 "C?" H 1515 4550 50  0000 L CNN
+F 1 "100n" H 1515 4505 50  0001 L CNN
+F 2 "Capacitor_SMD:C_0603_1608Metric" H 1438 4400 50  0001 C CNN
+F 3 "~" H 1400 4550 50  0001 C CNN
+	1    1400 4550
+	1    0    0    -1
+$EndComp
+Wire Wire Line
+	2550 2900 2550 3600
+Wire Wire Line
+	2550 3600 1950 3600
+Connection ~ 1950 3600
+$Comp
+L power:GND #PWR?
+U 1 1 5F7514FA
+P 1400 4700
+F 0 "#PWR?" H 1400 4450 50  0001 C CNN
+F 1 "GND" H 1405 4527 50  0000 C CNN
+F 2 "" H 1400 4700 50  0001 C CNN
+F 3 "" H 1400 4700 50  0001 C CNN
+	1    1400 4700
+	1    0    0    -1
+$EndComp
+$Comp
+L power:+5V #PWR?
+U 1 1 5F751715
+P 1400 4050
+F 0 "#PWR?" H 1400 3900 50  0001 C CNN
+F 1 "+5V" H 1415 4223 50  0000 C CNN
+F 2 "" H 1400 4050 50  0001 C CNN
+F 3 "" H 1400 4050 50  0001 C CNN
+	1    1400 4050
+	1    0    0    -1
+$EndComp
+Wire Wire Line
+	1400 4350 1400 4400
+Wire Wire Line
+	2550 4300 2550 4200
+Wire Wire Line
+	2550 4200 2100 4200
+Wire Wire Line
+	2100 4200 2100 4400
+Wire Wire Line
+	2100 4400 1400 4400
+Connection ~ 1400 4400
+Text Label 2100 4200 0    50   ~ 0
+Hall_VCC_2
 $EndSCHEMATC

Commit message: change Mosfet Driver to U3115S
Parts:
- gave numbers to parts that had none: 2
Changed lines of the file:
@@
 NoConn ~ 800  2850
 $Comp
-L Device:D D0AL?
+L Device:D D0AL2
 U 1 1 5F740132
 P 1400 4200
-F 0 "D0AL?" V 1446 4121 50  0000 R CNN
+F 0 "D0AL2" V 1446 4121 50  0000 R CNN
 F 1 "1N4148W" V 1355 4121 50  0000 R CNN
 F 2 "Diode_SMD:D_SOD-123" H 1400 4200 50  0001 C CNN
@@
 $EndComp
 $Comp
-L Device:C C?
+L Device:C C60
 U 1 1 5F7405CA
 P 1400 4550
-F 0 "C?" H 1515 4550 50  0000 L CNN
+F 0 "C60" H 1515 4550 50  0000 L CNN
 F 1 "100n" H 1515 4505 50  0001 L CNN
 F 2 "Capacitor_SMD:C_0603_1608Metric" H 1438 4400 50  0001 C CNN
@@
 Connection ~ 1950 3600
 $Comp
-L power:GND #PWR?
+L power:GND #PWR0243
 U 1 1 5F7514FA
 P 1400 4700
-F 0 "#PWR?" H 1400 4450 50  0001 C CNN
+F 0 "#PWR0243" H 1400 4450 50  0001 C CNN
 F 1 "GND" H 1405 4527 50  0000 C CNN
 F 2 "" H 1400 4700 50  0001 C CNN
@@
 $EndComp
 $Comp
-L power:+5V #PWR?
+L power:+5V #PWR0244
 U 1 1 5F751715
 P 1400 4050
-F 0 "#PWR?" H 1400 3900 50  0001 C CNN
+F 0 "#PWR0244" H 1400 3900 50  0001 C CNN
 F 1 "+5V" H 1415 4223 50  0000 C CNN
 F 2 "" H 1400 4050 50  0001 C CNN

Commit message: add silk screen, change diodes at DCDC converters, remove overcurrent detection, add 100nf
Parts:
- added D0AL3, D0AL4: 1N4148W, Diode_SMD:D_SOD-123, symbol Device:D
Connections:
- net +VSW: now also D0AL3.2 (A), D0AL4.2 (A); no longer J10.4 (Pin_4), J9.4 (Pin_4)
- new net: D0AL3.1 (K), J9.4 (Pin_4)
- new net: D0AL4.1 (K), J10.4 (Pin_4)
Changed lines of the file:
@@
 	1    0    0    -1
 $EndComp
-Wire Wire Line
-	2700 1250 2400 1250
 $Comp
 L Device:R R36
@@
 	1    0    0    -1
 $EndComp
-Wire Wire Line
-	2700 5200 2450 5200
 $Comp
 L power:+VSW #PWR0156
 U 1 1 5F79AEC1
-P 2700 5200
-F 0 "#PWR0156" H 2700 5050 50  0001 C CNN
-F 1 "+VSW" H 2715 5373 50  0000 C CNN
-F 2 "" H 2700 5200 50  0001 C CNN
-F 3 "" H 2700 5200 50  0001 C CNN
-	1    2700 5200
+P 2750 5200
+F 0 "#PWR0156" H 2750 5050 50  0001 C CNN
+F 1 "+VSW" H 2765 5373 50  0000 C CNN
+F 2 "" H 2750 5200 50  0001 C CNN
+F 3 "" H 2750 5200 50  0001 C CNN
+	1    2750 5200
 	1    0    0    -1
 $EndComp
@@
 Text Label 2100 4200 0    50   ~ 0
 Hall_VCC_2
+$Comp
+L Device:D D0AL4
+U 1 1 5F7CFD48
+P 2600 5200
+F 0 "D0AL4" V 2646 5121 50  0000 R CNN
+F 1 "1N4148W" V 2555 5121 50  0000 R CNN
+F 2 "Diode_SMD:D_SOD-123" H 2600 5200 50  0001 C CNN
+F 3 "~" H 2600 5200 50  0001 C CNN
+	1    2600 5200
+	1    0    0    -1
+$EndComp
+$Comp
+L Device:D D0AL3
+U 1 1 5F7D24AB
+P 2550 1250
+F 0 "D0AL3" V 2596 1171 50  0000 R CNN
+F 1 "1N4148W" V 2505 1171 50  0000 R CNN
+F 2 "Diode_SMD:D_SOD-123" H 2550 1250 50  0001 C CNN
+F 3 "~" H 2550 1250 50  0001 C CNN
+	1    2550 1250
+	1    0    0    -1
+$EndComp
 $EndSCHEMATC
