File: connectors.sch (KiCad schematic (older format))
At the start: 48 parts, among them J10 UART_R1, J4 Conn_01x04_Male, J8 Conn_01x05, J9 UART_L1, U15 SRV05-4, U5 SRV05-4

Commit message: add resistors on mosfet driver inputs, change board corners, fix labels
Parts:
- D19: value 15V TVS C78409 -> 15V C78409
- R16L1, R16L2, R16L3, R16L4, R17L1, R17L2, R17L3, R17L4, R18L1, R18L2, R18L3, R18L4: value 2K2 -> 2.2k
- R19L1, R19L2, R20L1, R20L2, R21L1, R21L2: value 3K3 -> 3.3k
Changed lines of the file:
@@
 P 2900 2400
 F 0 "R16L1" H 2970 2446 50  0000 L CNN
-F 1 "2K2" H 2970 2355 50  0000 L CNN
+F 1 "2.2k" H 2970 2355 50  0000 L CNN
 F 2 "Resistor_SMD:R_0603_1608Metric" V 2830 2400 50  0001 C CNN
 F 3 "~" H 2900 2400 50  0001 C CNN
@@
 P 3250 2400
 F 0 "R17L1" H 3320 2446 50  0000 L CNN
-F 1 "2K2" H 3320 2355 50  0000 L CNN
+F 1 "2.2k" H 3320 2355 50  0000 L CNN
 F 2 "Resistor_SMD:R_0603_1608Metric" V 3180 2400 50  0001 C CNN
 F 3 "~" H 3250 2400 50  0001 C CNN
@@
 P 3600 2400
 F 0 "R18L1" H 3670 2446 50  0000 L CNN
-F 1 "2K2" H 3670 2355 50  0000 L CNN
+F 1 "2.2k" H 3670 2355 50  0000 L CNN
 F 2 "Resistor_SMD:R_0603_1608Metric" V 3530 2400 50  0001 C CNN
 F 3 "~" H 3600 2400 50  0001 C CNN
@@
 P 3950 2600
 F 0 "R21L1" V 4157 2600 50  0000 C CNN
-F 1 "3K3" V 4066 2600 50  0000 C CNN
+F 1 "3.3k" V 4066 2600 50  0000 C CNN
 F 2 "Resistor_SMD:R_0603_1608Metric" V 3880 2600 50  0001 C CNN
 F 3 "~" H 3950 2600 50  0001 C CNN
@@
 P 4200 2700
 F 0 "R20L1" V 4407 2700 50  0000 C CNN
-F 1 "3K3" V 4316 2700 50  0000 C CNN
+F 1 "3.3k" V 4316 2700 50  0000 C CNN
 F 2 "Resistor_SMD:R_0603_1608Metric" V 4130 2700 50  0001 C CNN
 F 3 "~" H 4200 2700 50  0001 C CNN
@@
 P 4450 2800
 F 0 "R19L1" V 4657 2800 50  0000 C CNN
-F 1 "3K3" V 4566 2800 50  0000 C CNN
+F 1 "3.3k" V 4566 2800 50  0000 C CNN
 F 2 "Resistor_SMD:R_0603_1608Metric" V 4380 2800 50  0001 C CNN
 F 3 "~" H 4450 2800 50  0001 C CNN
@@
 P 2900 4200
 F 0 "R16L2" H 2970 4246 50  0000 L CNN
-F 1 "2K2" H 2970 4155 50  0000 L CNN
+F 1 "2.2k" H 2970 4155 50  0000 L CNN
 F 2 "Resistor_SMD:R_0603_1608Metric" V 2830 4200 50  0001 C CNN
 F 3 "~" H 2900 4200 50  0001 C CNN
@@
 P 3250 4200
 F 0 "R17L2" H 3320 4246 50  0000 L CNN
-F 1 "2K2" H 3320 4155 50  0000 L CNN
+F 1 "2.2k" H 3320 4155 50  0000 L CNN
 F 2 "Resistor_SMD:R_0603_1608Metric" V 3180 4200 50  0001 C CNN
 F 3 "~" H 3250 4200 50  0001 C CNN
@@
 P 3600 4200
 F 0 "R18L2" H 3670 4246 50  0000 L CNN
-F 1 "2K2" H 3670 4155 50  0000 L CNN
+F 1 "2.2k" H 3670 4155 50  0000 L CNN
 F 2 "Resistor_SMD:R_0603_1608Metric" V 3530 4200 50  0001 C CNN
 F 3 "~" H 3600 4200 50  0001 C CNN
@@
 P 3950 4400
 F 0 "R21L2" V 4157 4400 50  0000 C CNN
-F 1 "3K3" V 4066 4400 50  0000 C CNN
+F 1 "3.3k" V 4066 4400 50  0000 C CNN
 F 2 "Resistor_SMD:R_0603_1608Metric" V 3880 4400 50  0001 C CNN
 F 3 "~" H 3950 4400 50  0001 C CNN
@@
 P 4200 4500
 F 0 "R20L2" V 4407 4500 50  0000 C CNN
-F 1 "3K3" V 4316 4500 50  0000 C CNN
+F 1 "3.3k" V 4316 4500 50  0000 C CNN
 F 2 "Resistor_SMD:R_0603_1608Metric" V 4130 4500 50  0001 C CNN
 F 3 "~" H 4200 4500 50  0001 C CNN
@@
 P 4450 4600
 F 0 "R19L2" V 4657 4600 50  0000 C CNN
-F 1 "3K3" V 4566 4600 50  0000 C CNN
+F 1 "3.3k" V 4566 4600 50  0000 C CNN
 F 2 "Resistor_SMD:R_0603_1608Metric" V 4380 4600 50  0001 C CNN
 F 3 "~" H 4450 4600 50  0001 C CNN
@@
 Text Notes 3900 6700 2    50   ~ 0
 CAN_SHLD
-$Comp
-L Device:D_Zener D19
-U 1 1 5F7DDDAC
-P 6100 6900
-F 0 "D19" V 6054 6980 50  0000 L CNN
-F 1 "15V TVS C78409" V 6145 6980 50  0000 L CNN
-F 2 "Diode_SMD:D_SMB" H 6100 6900 50  0001 C CNN
-F 3 "~" H 6100 6900 50  0001 C CNN
-	1    6100 6900
-	0    1    1    0
-$EndComp
 Wire Wire Line
 	6100 6550 6100 6750
@@
 P 2800 2400
 F 0 "R16L3" H 2870 2446 50  0000 L CNN
-F 1 "2K2" H 2870 2355 50  0000 L CNN
+F 1 "2.2k" H 2870 2355 50  0000 L CNN
 F 2 "Resistor_SMD:R_0603_1608Metric" V 2730 2400 50  0001 C CNN
 F 3 "~" H 2800 2400 50  0001 C CNN
@@
 P 3150 2400
 F 0 "R17L3" H 3220 2446 50  0000 L CNN
-F 1 "2K2" H 3220 2355 50  0000 L CNN
+F 1 "2.2k" H 3220 2355 50  0000 L CNN
 F 2 "Resistor_SMD:R_0603_1608Metric" V 3080 2400 50  0001 C CNN
 F 3 "~" H 3150 2400 50  0001 C CNN
@@
 P 3500 2400
 F 0 "R18L3" H 3570 2446 50  0000 L CNN
-F 1 "2K2" H 3570 2355 50  0000 L CNN
+F 1 "2.2k" H 3570 2355 50  0000 L CNN
 F 2 "Resistor_SMD:R_0603_1608Metric" V 3430 2400 50  0001 C CNN
 F 3 "~" H 3500 2400 50  0001 C CNN
@@
 P 2800 4200
 F 0 "R16L4" H 2870 4246 50  0000 L CNN
-F 1 "2K2" H 2870 4155 50  0000 L CNN
+F 1 "2.2k" H 2870 4155 50  0000 L CNN
 F 2 "Resistor_SMD:R_0603_1608Metric" V 2730 4200 50  0001 C CNN
 F 3 "~" H 2800 4200 50  0001 C CNN
@@
 P 3150 4200
 F 0 "R17L4" H 3220 4246 50  0000 L CNN
-F 1 "2K2" H 3220 4155 50  0000 L CNN
+F 1 "2.2k" H 3220 4155 50  0000 L CNN
 F 2 "Resistor_SMD:R_0603_1608Metric" V 3080 4200 50  0001 C CNN
 F 3 "~" H 3150 4200 50  0001 C CNN
@@
 P 3500 4200
 F 0 "R18L4" H 3570 4246 50  0000 L CNN
-F 1 "2K2" H 3570 4155 50  0000 L CNN
+F 1 "2.2k" H 3570 4155 50  0000 L CNN
 F 2 "Resistor_SMD:R_0603_1608Metric" V 3430 4200 50  0001 C CNN
 F 3 "~" H 3500 4200 50  0001 C CNN
@@
 	1    0    0    -1
 $EndComp
+$Comp
+L Device:D_Zener D?
+U 1 1 5F7B04AF
+P 6100 6900
+AR Path="/5F7395DA/5F7B04AF" Ref="D?"  Part="1"
+AR Path="/5F74B195/5F7B04AF" Ref="D19"  Part="1"
+F 0 "D19" V 6054 6980 50  0000 L CNN
+F 1 "15V C78409" V 6250 6700 50  0000 L CNN
+F 2 "Diode_SMD:D_SMB" H 6100 6900 50  0001 C CNN
+F 3 "~" H 6100 6900 50  0001 C CNN
+	1    6100 6900
+	0    1    1    0
+$EndComp
 $EndSCHEMATC
