File: connectors.sch (KiCad schematic (older format))
At the start: 48 parts, among them J10 UART_R1, J4 Conn_01x04_Male, J8 Conn_01x05, J9 UART_L1, U15 SRV05-4, U5 SRV05-4

Commit message: added rs232, layout changes
Parts:
- added C77, C78, C79, C80, C81: 100nF, Capacitor_SMD:C_0603_1608Metric, symbol Device:C
- added U18: SP3232, Package_SO:TSSOP-16_4.4x5mm_P0.65mm, symbol Interface_UART:ICL3232
Connections:
- net +3V3: now also C78.2, U18.16 (VCC)
- net GND: now also C78.1, C80.2, C81.2, U18.11 (T1IN), U18.13 (R1IN), U18.15 (GND)
- net UART_L_RX: now also U18.7 (T2OUT); no longer R38.1
- net UART_L_TX: now also U18.8 (R2IN); no longer R36.1
- new net: C77.1, U18.1 (C1+)
- new net: C80.1, U18.2 (VS+)
- new net: C77.2, U18.3 (C1-)
- new net: C79.1, U18.4 (C2+)
- new net: C79.2, U18.5 (C2-)
- new net: C81.1, U18.6 (VS-)
- new net RS232_L_RX: R38.1, U18.10 (T2IN)
- new net RS232_L_TX: R36.1, U18.9 (R2OUT)
Other:
- moved on the sheet: C2, C41, C42, C60, D0AL1, D0AL2, D0AL3, D0AL4, D17, D18, D19, HALL_L1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

Commit message: Added LCSC Part # to most components
Parts:
- C2, C60: value 100n -> 100nF; LCSC Part # (none) -> C14663
- C41: value 4.7n -> 4.7nF; LCSC Part # (none) -> C53987
- C42: LCSC Part # (none) -> C28323
- D0AL1, D0AL2, D0AL3, D0AL4: LCSC Part # (none) -> C81598
- R16L1, R16L2, R16L3, R16L4, R17L1, R17L2, R17L3, R17L4, R18L1, R18L2, R18L3, R18L4: LCSC Part # (none) -> C4190
- R19L1, R19L2, R20L1, R20L2, R21L1, R21L2: LCSC Part # (none) -> C22978
- R35, R36, R37, R38: LCSC Part # (none) -> C22775
- R45: LCSC Part # (none) -> C22935
- U15, U5: LCSC Part # (none) -> C384887
Changed lines of the file:
@@
 F 2 "Resistor_SMD:R_0603_1608Metric" V 3030 1450 50  0001 C CNN
 F 3 "~" H 3100 1450 50  0001 C CNN
+F 4 "C22775" H 3100 1450 50  0001 C CNN "LCSC Part #"
 	1    3100 1450
 	0    1    1    0
@@
 F 2 "Resistor_SMD:R_0603_1608Metric" V 3280 1550 50  0001 C CNN
 F 3 "~" H 3350 1550 50  0001 C CNN
+F 4 "C22775" H 3350 1550 50  0001 C CNN "LCSC Part #"
 	1    3350 1550
 	0    1    1    0
@@
 F 2 "Resistor_SMD:R_0603_1608Metric" V 2980 2500 50  0001 C CNN
 F 3 "~" H 3050 2500 50  0001 C CNN
+F 4 "C4190" H 3050 2500 50  0001 C CNN "LCSC Part #"
 	1    3050 2500
 	1    0    0    -1
@@
 F 2 "Resistor_SMD:R_0603_1608Metric" V 3330 2500 50  0001 C CNN
 F 3 "~" H 3400 2500 50  0001 C CNN
+F 4 "C4190" H 3400 2500 50  0001 C CNN "LCSC Part #"
 	1    3400 2500
 	1    0    0    -1
@@
 F 2 "Resistor_SMD:R_0603_1608Metric" V 3680 2500 50  0001 C CNN
 F 3 "~" H 3750 2500 50  0001 C CNN
+F 4 "C4190" H 3750 2500 50  0001 C CNN "LCSC Part #"
 	1    3750 2500
 	1    0    0    -1
@@
 F 2 "Resistor_SMD:R_0603_1608Metric" V 4030 2700 50  0001 C CNN
 F 3 "~" H 4100 2700 50  0001 C CNN
+F 4 "C22978" H 4100 2700 50  0001 C CNN "LCSC Part #"
 	1    4100 2700
 	0    -1   -1   0
@@
 F 2 "Resistor_SMD:R_0603_1608Metric" V 4280 2800 50  0001 C CNN
 F 3 "~" H 4350 2800 50  0001 C CNN
+F 4 "C22978" H 4350 2800 50  0001 C CNN "LCSC Part #"
 	1    4350 2800
 	0    -1   -1   0
@@
 F 2 "Resistor_SMD:R_0603_1608Metric" V 4530 2900 50  0001 C CNN
 F 3 "~" H 4600 2900 50  0001 C CNN
+F 4 "C22978" H 4600 2900 50  0001 C CNN "LCSC Part #"
 	1    4600 2900
 	0    -1   -1   0
@@
 F 2 "Resistor_SMD:R_0603_1608Metric" V 2980 4300 50  0001 C CNN
 F 3 "~" H 3050 4300 50  0001 C CNN
+F 4 "C4190" H 3050 4300 50  0001 C CNN "LCSC Part #"
 	1    3050 4300
 	1    0    0    -1
@@
 F 2 "Resistor_SMD:R_0603_1608Metric" V 3330 4300 50  0001 C CNN
 F 3 "~" H 3400 4300 50  0001 C CNN
+F 4 "C4190" H 3400 4300 50  0001 C CNN "LCSC Part #"
 	1    3400 4300
 	1    0    0    -1
@@
 F 2 "Resistor_SMD:R_0603_1608Metric" V 3680 4300 50  0001 C CNN
 F 3 "~" H 3750 4300 50  0001 C CNN
+F 4 "C4190" H 3750 4300 50  0001 C CNN "LCSC Part #"
 	1    3750 4300
 	1    0    0    -1
@@
 F 2 "Resistor_SMD:R_0603_1608Metric" V 4030 4500 50  0001 C CNN
 F 3 "~" H 4100 4500 50  0001 C CNN
+F 4 "C22978" H 4100 4500 50  0001 C CNN "LCSC Part #"
 	1    4100 4500
 	0    -1   -1   0
@@
 F 2 "Resistor_SMD:R_0603_1608Metric" V 4280 4600 50  0001 C CNN
 F 3 "~" H 4350 4600 50  0001 C CNN
+F 4 "C22978" H 4350 4600 50  0001 C CNN "LCSC Part #"
 	1    4350 4600
 	0    -1   -1   0
@@
 F 2 "Resistor_SMD:R_0603_1608Metric" V 4530 4700 50  0001 C CNN
 F 3 "~" H 4600 4700 50  0001 C CNN
+F 4 "C22978" H 4600 4700 50  0001 C CNN "LCSC Part #"
 	1    4600 4700
 	0    -1   -1   0
@@
 P 2100 3850
 F 0 "C2" H 2215 3850 50  0000 L CNN
-F 1 "100n" H 2215 3805 50  0001 L CNN
+F 1 "100nF" H 2215 3805 50  0001 L CNN
 F 2 "Capacitor_SMD:C_0603_1608Metric" H 2138 3700 50  0001 C CNN
 F 3 "~" H 2100 3850 50  0001 C CNN
+F 4 "C14663" H 2100 3850 50  0001 C CNN "LCSC Part #"
 	1    2100 3850
 	1    0    0    -1
@@
 F 2 "Diode_SMD:D_SOD-123" H 2100 3500 50  0001 C CNN
 F 3 "~" H 2100 3500 50  0001 C CNN
+F 4 "C81598" H 2100 3500 50  0001 C CNN "LCSC Part #"
 	1    2100 3500
 	0    -1   -1   0
@@
 F 2 "Capacitor_SMD:C_0805_2012Metric" H 5888 6850 50  0001 C CNN
 F 3 "~" H 5850 7000 50  0001 C CNN
+F 4 "C28323" H 5850 7000 50  0001 C CNN "LCSC Part #"
 	1    5850 7000
 	1    0    0    -1
@@
 F 2 "Resistor_SMD:R_0603_1608Metric" V 4880 7050 50  0001 C CNN
 F 3 "~" H 4950 7050 50  0001 C CNN
+F 4 "C22935" H 4950 7050 50  0001 C CNN "LCSC Part #"
 	1    4950 7050
 	1    0    0    -1
@@
 P 5350 7050
 F 0 "C41" H 5465 7096 50  0000 L CNN
-F 1 "4.7n" H 5465 7005 50  0000 L CNN
+F 1 "4.7nF" H 5465 7005 50  0000 L CNN
 F 2 "Capacitor_SMD:C_0805_2012Metric" H 5388 6900 50  0001 C CNN
 F 3 "~" H 5350 7050 50  0001 C CNN
+F 4 "C53987" H 5350 7050 50  0001 C CNN "LCSC Part #"
 	1    5350 7050
 	1    0    0    -1
@@
 F 2 "Resistor_SMD:R_0603_1608Metric" V 2880 2500 50  0001 C CNN
 F 3 "~" H 2950 2500 50  0001 C CNN
+F 4 "C4190" H 2950 2500 50  0001 C CNN "LCSC Part #"
 	1    2950 2500
 	1    0    0    -1
@@
 F 2 "Resistor_SMD:R_0603_1608Metric" V 3230 2500 50  0001 C CNN
 F 3 "~" H 3300 2500 50  0001 C CNN
+F 4 "C4190" H 3300 2500 50  0001 C CNN "LCSC Part #"
 	1    3300 2500
 	1    0    0    -1
@@
 F 2 "Resistor_SMD:R_0603_1608Metric" V 3580 2500 50  0001 C CNN
 F 3 "~" H 3650 2500 50  0001 C CNN
+F 4 "C4190" H 3650 2500 50  0001 C CNN "LCSC Part #"
 	1    3650 2500
 	1    0    0    -1
@@
 F 2 "Resistor_SMD:R_0603_1608Metric" V 2880 4300 50  0001 C CNN
 F 3 "~" H 2950 4300 50  0001 C CNN
+F 4 "C4190" H 2950 4300 50  0001 C CNN "LCSC Part #"
 	1    2950 4300
 	1    0    0    -1
@@
 F 2 "Resistor_SMD:R_0603_1608Metric" V 3230 4300 50  0001 C CNN
 F 3 "~" H 3300 4300 50  0001 C CNN
+F 4 "C4190" H 3300 4300 50  0001 C CNN "LCSC Part #"
 	1    3300 4300
 	1    0    0    -1
@@
 F 2 "Resistor_SMD:R_0603_1608Metric" V 3580 4300 50  0001 C CNN
 F 3 "~" H 3650 4300 50  0001 C CNN
+F 4 "C4190" H 3650 4300 50  0001 C CNN "LCSC Part #"
 	1    3650 4300
 	1    0    0    -1
@@
 F 2 "Resistor_SMD:R_0603_1608Metric" V 3230 5500 50  0001 C CNN
 F 3 "~" H 3300 5500 50  0001 C CNN
+F 4 "C22775" H 3300 5500 50  0001 C CNN "LCSC Part #"
 	1    3300 5500
 	0    1    1    0
@@
 F 2 "Resistor_SMD:R_0603_1608Metric" V 2930 5400 50  0001 C CNN
 F 3 "~" H 3000 5400 50  0001 C CNN
+F 4 "C22775" H 3000 5400 50  0001 C CNN "LCSC Part #"
 	1    3000 5400
 	0    1    1    0
@@
 F 2 "Package_TO_SOT_SMD:SOT-23-6" H 2150 2400 50  0001 C CNN
 F 3 "http://www.onsemi.com/pub/Collateral/SRV05-4-D.PDF" H 1450 2850 50  0001 C CNN
+F 4 "C384887" H 1450 2850 50  0001 C CNN "LCSC Part #"
 	1    1450 2850
 	1    0    0    -1
@@
 F 2 "Package_TO_SOT_SMD:SOT-23-6" H 2200 5300 50  0001 C CNN
 F 3 "http://www.onsemi.com/pub/Collateral/SRV05-4-D.PDF" H 1500 5750 50  0001 C CNN
+F 4 "C384887" H 1500 5750 50  0001 C CNN "LCSC Part #"
 	1    1500 5750
 	1    0    0    -1
@@
 F 2 "Diode_SMD:D_SOD-123" H 1550 4300 50  0001 C CNN
 F 3 "~" H 1550 4300 50  0001 C CNN
+F 4 "C81598" H 1550 4300 50  0001 C CNN "LCSC Part #"
 	1    1550 4300
 	0    -1   -1   0
@@
 P 1550 4650
 F 0 "C60" H 1665 4650 50  0000 L CNN
-F 1 "100n" H 1665 4605 50  0001 L CNN
+F 1 "100nF" H 1665 4605 50  0001 L CNN
 F 2 "Capacitor_SMD:C_0603_1608Metric" H 1588 4500 50  0001 C CNN
 F 3 "~" H 1550 4650 50  0001 C CNN
+F 4 "C14663" H 1550 4650 50  0001 C CNN "LCSC Part #"
 	1    1550 4650
 	1    0    0    -1
@@
 F 2 "Diode_SMD:D_SOD-123" H 2750 5300 50  0001 C CNN
 F 3 "~" H 2750 5300 50  0001 C CNN
+F 4 "C81598" H 2750 5300 50  0001 C CNN "LCSC Part #"
 	1    2750 5300
 	1    0    0    -1
@@
 F 2 "Diode_SMD:D_SOD-123" H 2700 1350 50  0001 C CNN
 F 3 "~" H 2700 1350 50  0001 C CNN
+F 4 "C81598" H 2700 1350 50  0001 C CNN "LCSC Part #"
 	1    2700 1350
 	1    0    0    -1

Commit message: More adaptation to jlcpcb, parts checking
Parts:
- D17: LCSC Part # (none) -> C38838
- D18: LCSC Part # (none) -> C8598
- D19: LCSC Part # (none) -> C78409
- D29, D30, D31, D32, D33, D34: LCSC Part # (none) -> C2290
- HALL_L1, HALL_R1, J10, J4, J8, J9: place (none) -> dnp
Changed lines of the file:
@@
 F 2 "Connector_PinHeader_2.54mm:PinHeader_1x04_P2.54mm_Vertical" H 2350 1550 50  0001 C CNN
 F 3 "~" H 2350 1550 50  0001 C CNN
+F 4 "dnp" H 2350 1550 50  0001 C CNN "place"
 	1    2350 1550
 	1    0    0    1
@@
 F 2 "Connector_PinHeader_2.54mm:PinHeader_1x05_P2.54mm_Vertical" H 2400 2800 50  0001 C CNN
 F 3 "~" H 2400 2800 50  0001 C CNN
+F 4 "dnp" H 2400 2800 50  0001 C CNN "place"
 	1    2400 2800
 	1    0    0    -1
@@
 F 2 "Connector_PinHeader_2.54mm:PinHeader_1x05_P2.54mm_Vertical" H 2400 4600 50  0001 C CNN
 F 3 "~" H 2400 4600 50  0001 C CNN
+F 4 "dnp" H 2400 4600 50  0001 C CNN "place"
 	1    2400 4600
 	1    0    0    1
@@
 F 2 "Connector_PinHeader_2.54mm:PinHeader_1x05_P2.54mm_Vertical" H 4150 6550 50  0001 C CNN
 F 3 "~" H 4150 6550 50  0001 C CNN
+F 4 "dnp" H 4150 6550 50  0001 C CNN "place"
 	1    4150 6550
 	-1   0    0    -1
@@
 F 1 "PESD15VL2BT,215" H 4950 6026 50  0000 C CNN
 F 2 "Package_TO_SOT_SMD:SOT-23" H 4800 5900 50  0001 C CNN
-F 3 "~" H 4800 5900 50  0001 C CNN
+F 3 "" H 4800 5900 50  0001 C CNN
+F 4 "C38838" H 4950 5900 50  0001 C CNN "LCSC Part #"
 	1    4950 5900
 	1    0    0    -1
@@
 F 1 "B5819W" V 6205 6270 50  0000 R CNN
 F 2 "Diode_SMD:D_SOD-123" H 6250 6350 50  0001 C CNN
-F 3 "~" H 6250 6350 50  0001 C CNN
+F 3 "" H 6250 6350 50  0001 C CNN
+F 4 "C8598" H 6250 6350 50  0001 C CNN "LCSC Part #"
 	1    6250 6350
 	0    -1   -1   0
@@
 F 2 "Connector_PinHeader_2.54mm:PinHeader_1x04_P2.54mm_Vertical" H 4700 1250 50  0001 C CNN
 F 3 "~" H 4700 1250 50  0001 C CNN
+F 4 "dnp" H 4700 1250 50  0001 C CNN "place"
 	1    4700 1250
 	1    0    0    -1
@@
 F 1 "LED" H 3043 2036 50  0000 C CNN
 F 2 "LED_SMD:LED_0603_1608Metric" H 3050 2200 50  0001 C CNN
-F 3 "~" H 3050 2200 50  0001 C CNN
+F 3 "" H 3050 2200 50  0001 C CNN
+F 4 "C2290" H 3050 2200 50  0001 C CNN "LCSC Part #"
 	1    3050 2200
 	0    -1   -1   0
@@
 F 1 "LED" H 3393 2036 50  0000 C CNN
 F 2 "LED_SMD:LED_0603_1608Metric" H 3400 2200 50  0001 C CNN
-F 3 "~" H 3400 2200 50  0001 C CNN
+F 3 "" H 3400 2200 50  0001 C CNN
+F 4 "C2290" H 3400 2200 50  0001 C CNN "LCSC Part #"
 	1    3400 2200
 	0    -1   -1   0
@@
 F 1 "LED" H 3743 2036 50  0000 C CNN
 F 2 "LED_SMD:LED_0603_1608Metric" H 3750 2200 50  0001 C CNN
-F 3 "~" H 3750 2200 50  0001 C CNN
+F 3 "" H 3750 2200 50  0001 C CNN
+F 4 "C2290" H 3750 2200 50  0001 C CNN "LCSC Part #"
 	1    3750 2200
 	0    -1   -1   0
@@
 F 1 "LED" H 3043 3836 50  0000 C CNN
 F 2 "LED_SMD:LED_0603_1608Metric" H 3050 4000 50  0001 C CNN
-F 3 "~" H 3050 4000 50  0001 C CNN
+F 3 "" H 3050 4000 50  0001 C CNN
+F 4 "C2290" H 3050 4000 50  0001 C CNN "LCSC Part #"
 	1    3050 4000
 	0    -1   -1   0
@@
 F 1 "LED" H 3393 3836 50  0000 C CNN
 F 2 "LED_SMD:LED_0603_1608Metric" H 3400 4000 50  0001 C CNN
-F 3 "~" H 3400 4000 50  0001 C CNN
+F 3 "" H 3400 4000 50  0001 C CNN
+F 4 "C2290" H 3400 4000 50  0001 C CNN "LCSC Part #"
 	1    3400 4000
 	0    -1   -1   0
@@
 F 1 "LED" H 3743 3836 50  0000 C CNN
 F 2 "LED_SMD:LED_0603_1608Metric" H 3750 4000 50  0001 C CNN
-F 3 "~" H 3750 4000 50  0001 C CNN
+F 3 "" H 3750 4000 50  0001 C CNN
+F 4 "C2290" H 3750 4000 50  0001 C CNN "LCSC Part #"
 	1    3750 4000
 	0    -1   -1   0
@@
 F 2 "Connector_PinHeader_2.54mm:PinHeader_1x04_P2.54mm_Vertical" H 2400 5500 50  0001 C CNN
 F 3 "~" H 2400 5500 50  0001 C CNN
+F 4 "dnp" H 2400 5500 50  0001 C CNN "place"
 	1    2400 5500
 	1    0    0    1
@@
 F 2 "Diode_SMD:D_SMB" H 6250 7000 50  0001 C CNN
 F 3 "~" H 6250 7000 50  0001 C CNN
+F 4 "C78409" H 6250 7000 50  0001 C CNN "LCSC Part #"
 	1    6250 7000
 	0    1    1    0

Commit message: Changed emergency brake to uart2 connector
Parts:
- added C84: 100nF, Capacitor_SMD:C_0603_1608Metric, symbol Device:C
- added D12: CDSOD323, Diode_SMD:D_SOD-323, symbol input-board:CDSOD323-boardcomputer
- added R82: 1k, Resistor_SMD:R_0603_1608Metric, symbol Device:R
Connections:
- net +3V3: now also R82.1
- net GND: now also C84.2, D12.2 (A)
- net UART_R_RX: now also C84.1, D12.1 (K), R82.2
Changed lines of the file:
@@
 Text HLabel 3600 5400 2    50   Input ~ 0
 UART_R_TX
-Text HLabel 3600 5500 2    50   Output ~ 0
+Text HLabel 4350 5500 2    50   Output ~ 0
 UART_R_RX
 Wire Wire Line
@@
 	0    1    1    0
 $EndComp
+$Comp
+L Device:R R?
+U 1 1 604C8C5A
+P 4200 5350
+AR Path="/5F75358D/604C8C5A" Ref="R?"  Part="1"
+AR Path="/5F74B195/604C8C5A" Ref="R82"  Part="1"
+F 0 "R82" V 4300 5400 50  0000 C CNN
+F 1 "1k" V 4300 5250 50  0000 C CNN
+F 2 "Resistor_SMD:R_0603_1608Metric" V 4130 5350 50  0001 C CNN
+F 3 "~" H 4200 5350 50  0001 C CNN
+F 4 "C21190" H 4200 5350 50  0001 C CNN "LCSC Part #"
+	1    4200 5350
+	1    0    0    -1
+$EndComp
+$Comp
+L power:+3.3V #PWR?
+U 1 1 604C8C60
+P 4200 5200
+AR Path="/5F75358D/604C8C60" Ref="#PWR?"  Part="1"
+AR Path="/5F74B195/604C8C60" Ref="#PWR015"  Part="1"
+F 0 "#PWR015" H 4200 5050 50  0001 C CNN
+F 1 "+3.3V" V 4200 5450 50  0000 C CNN
+F 2 "" H 4200 5200 50  0001 C CNN
+F 3 "" H 4200 5200 50  0001 C CNN
+	1    4200 5200
+	1    0    0    -1
+$EndComp
+$Comp
+L input-board:CDSOD323-boardcomputer D?
+U 1 1 604C8C6F
+P 3850 5600
+AR Path="/5F75358D/604C8C6F" Ref="D?"  Part="1"
+AR Path="/5F74B195/604C8C6F" Ref="D12"  Part="1"
+F 0 "D12" V 4000 5700 50  0000 L CNN
+F 1 "CDSOD323" V 3900 5750 50  0000 L CNN
+F 2 "Diode_SMD:D_SOD-323" H 3850 5750 50  0001 C CNN
+F 3 "" H 3850 5750 50  0001 C CNN
+F 4 "C127526" V 3850 5600 50  0001 C CNN "LCSC Part #"
+	1    3850 5600
+	0    1    1    0
+$EndComp
+$Comp
+L Device:C C?
+U 1 1 604C8C7D
+P 3600 5650
+AR Path="/5F75358D/604C8C7D" Ref="C?"  Part="1"
+AR Path="/5F74B195/604C8C7D" Ref="C84"  Part="1"
+F 0 "C84" H 3250 5700 50  0000 L CNN
+F 1 "100nF" H 3250 5600 50  0000 L CNN
+F 2 "Capacitor_SMD:C_0603_1608Metric" H 3638 5500 50  0001 C CNN
+F 3 "~" H 3600 5650 50  0001 C CNN
+F 4 "C14663" H 3600 5650 50  0001 C CNN "LCSC Part #"
+	1    3600 5650
+	1    0    0    -1
+$EndComp
+Wire Wire Line
+	3600 5500 3850 5500
+Connection ~ 3600 5500
+Connection ~ 3850 5500
+Wire Wire Line
+	3850 5500 4200 5500
+Connection ~ 4200 5500
+Wire Wire Line
+	4200 5500 4350 5500
+$Comp
+L power:GND #PWR07
+U 1 1 604ED1CB
+P 3600 5800
+F 0 "#PWR07" H 3600 5550 50  0001 C CNN
+F 1 "GND" H 3605 5627 50  0000 C CNN
+F 2 "" H 3600 5800 50  0001 C CNN
+F 3 "" H 3600 5800 50  0001 C CNN
+	1    3600 5800
+	1    0    0    -1
+$EndComp
+$Comp
+L power:GND #PWR014
+U 1 1 604ED5D9
+P 3850 5800
+F 0 "#PWR014" H 3850 5550 50  0001 C CNN
+F 1 "GND" H 3855 5627 50  0000 C CNN
+F 2 "" H 3850 5800 50  0001 C CNN
+F 3 "" H 3850 5800 50  0001 C CNN
+	1    3850 5800
+	1    0    0    -1
+$EndComp
 $EndSCHEMATC
