File: hh_bridge.sch (KiCad schematic (older format))
At the start: 9 parts, among them U8 IRS2304

Commit message: Add CAN transceiver
Changed lines of the file:
@@
 $Descr A4 11693 8268
 encoding utf-8
-Sheet 13 13
+Sheet 8 14
 Title ""
 Date ""
@@
 AR Path="/5F7A3A2A/5F706578" Ref="C17"  Part="1"
 AR Path="/5F7A4E71/5F706578" Ref="C24"  Part="1"
-F 0 "C24" H 4618 3396 50  0000 L CNN
+F 0 "C1" H 4618 3396 50  0000 L CNN
 F 1 "47u LKMD0901K470MF" H 4618 3305 50  0000 L CNN
 F 2 "Capacitor_THT:CP_Radial_D8.0mm_P3.50mm" H 4538 3200 50  0001 C CNN
@@
 AR Path="/5F7A3A2A/5F707CCD" Ref="D10"  Part="1"
 AR Path="/5F7A4E71/5F707CCD" Ref="D11"  Part="1"
-F 0 "D11" H 4350 2284 50  0000 C CNN
+F 0 "D1" H 4350 2284 50  0000 C CNN
 F 1 "1N4148W" H 4350 2375 50  0000 C CNN
 F 2 "Diode_SMD:D_SOD-123" H 4350 2500 50  0001 C CNN
@@
 AR Path="/5F7A3A2A/5F77195C" Ref="#PWR0187"  Part="1"
 AR Path="/5F7A4E71/5F77195C" Ref="#PWR0191"  Part="1"
-F 0 "#PWR0191" H 3950 2250 50  0001 C CNN
+F 0 "#PWR0171" H 3950 2250 50  0001 C CNN
 F 1 "+VSW" H 3965 2573 50  0000 C CNN
 F 2 "" H 3950 2400 50  0001 C CNN
@@
 AR Path="/5F7A3A2A/5F771CDC" Ref="C16"  Part="1"
 AR Path="/5F7A4E71/5F771CDC" Ref="C18"  Part="1"
-F 0 "C18" H 3618 3996 50  0000 L CNN
+F 0 "C8" H 3618 3996 50  0000 L CNN
 F 1 "220u25V LKMD0901E221MF" H 3618 3905 50  0000 L CNN
 F 2 "Capacitor_THT:CP_Radial_D8.0mm_P3.50mm" H 3538 3800 50  0001 C CNN
@@
 AR Path="/5F7A3A2A/5F77283D" Ref="#PWR0188"  Part="1"
 AR Path="/5F7A4E71/5F77283D" Ref="#PWR0192"  Part="1"
-F 0 "#PWR0192" H 3500 3600 50  0001 C CNN
+F 0 "#PWR0172" H 3500 3600 50  0001 C CNN
 F 1 "+VSW" H 3515 3923 50  0000 C CNN
 F 2 "" H 3500 3750 50  0001 C CNN
@@
 AR Path="/5F7A3A2A/5F773E85" Ref="#PWR0189"  Part="1"
 AR Path="/5F7A4E71/5F773E85" Ref="#PWR0193"  Part="1"
-F 0 "#PWR0193" H 3750 3850 50  0001 C CNN
+F 0 "#PWR0173" H 3750 3850 50  0001 C CNN
 F 1 "GND" H 3755 3927 50  0000 C CNN
 F 2 "" H 3750 4100 50  0001 C CNN
@@
 AR Path="/5F7A3A2A/5F73738F" Ref="V9"  Part="1"
 AR Path="/5F7A4E71/5F73738F" Ref="V11"  Part="1"
-F 0 "V11" H 5755 3646 50  0000 L CNN
+F 0 "V1" H 5755 3646 50  0000 L CNN
 F 1 "CRSS042N10N" H 5755 3555 50  0000 L CNN
 F 2 "Package_TO_SOT_SMD:TO-263-2" H 5750 3525 50  0001 L CIN
@@
 AR Path="/5F7A3A2A/5F72B1D2" Ref="R32"  Part="1"
 AR Path="/5F7A4E71/5F72B1D2" Ref="R34"  Part="1"
-F 0 "R34" V 4993 3600 50  0000 C CNN
+F 0 "R10" V 4993 3600 50  0000 C CNN
 F 1 "68" V 5084 3600 50  0000 C CNN
 F 2 "Resistor_SMD:R_1206_3216Metric" V 5130 3600 50  0001 C CNN
@@
 AR Path="/5F7A3A2A/5F771122" Ref="U12"  Part="1"
 AR Path="/5F7A4E71/5F771122" Ref="U13"  Part="1"
-F 0 "U13" H 3950 3981 50  0000 C CNN
+F 0 "U8" H 3950 3981 50  0000 C CNN
 F 1 "IRS2304" H 3950 3890 50  0000 C CNN
 F 2 "Package_SO:SOIC-8_3.9x4.9mm_P1.27mm" H 3950 3300 50  0001 C CIN
@@
 AR Path="/5F7A3A2A/5F7824C8" Ref="R28"  Part="1"
 AR Path="/5F7A4E71/5F7824C8" Ref="R33"  Part="1"
-F 0 "R33" V 4993 3100 50  0000 C CNN
+F 0 "R13" V 4993 3100 50  0000 C CNN
 F 1 "68" V 5084 3100 50  0000 C CNN
 F 2 "Resistor_SMD:R_1206_3216Metric" V 5130 3100 50  0001 C CNN
@@
 AR Path="/5F7A3A2A/5F70E4C5" Ref="V8"  Part="1"
 AR Path="/5F7A4E71/5F70E4C5" Ref="V10"  Part="1"
-F 0 "V10" H 5755 3146 50  0000 L CNN
+F 0 "V0" H 5755 3146 50  0000 L CNN
 F 1 "CRSS042N10N" H 5755 3055 50  0000 L CNN
 F 2 "Package_TO_SOT_SMD:TO-263-2" H 5750 3025 50  0001 L CIN
@@
 AR Path="/5F7A3A2A/5F79127D" Ref="#PWR0190"  Part="1"
 AR Path="/5F7A4E71/5F79127D" Ref="#PWR0194"  Part="1"
-F 0 "#PWR0194" H 5650 2750 50  0001 C CNN
+F 0 "#PWR0174" H 5650 2750 50  0001 C CNN
 F 1 "+BATT" H 5665 3073 50  0000 C CNN
 F 2 "" H 5650 2900 50  0001 C CNN
@@
 AR Path="/5F7A3A2A/5F7BE8FF" Ref="C35"  Part="1"
 AR Path="/5F7A4E71/5F7BE8FF" Ref="C36"  Part="1"
-F 0 "C36" H 6818 2646 50  0000 L CNN
+F 0 "C31" H 6818 2646 50  0000 L CNN
 F 1 "47u LKMD0901K470MF" H 6818 2555 50  0000 L CNN
 F 2 "Capacitor_THT:CP_Radial_D8.0mm_P3.50mm" H 6738 2450 50  0001 C CNN
@@
 AR Path="/5F7A3A2A/5F7BF207" Ref="#PWR0201"  Part="1"
 AR Path="/5F7A4E71/5F7BF207" Ref="#PWR0202"  Part="1"
-F 0 "#PWR0202" H 6700 2300 50  0001 C CNN
+F 0 "#PWR0197" H 6700 2300 50  0001 C CNN
 F 1 "+BATT" H 6715 2623 50  0000 C CNN
 F 2 "" H 6700 2450 50  0001 C CNN

Commit message: Add missing FET driver connection
Connections:
- net MOTOR_PHASE: now also C1.2, U8.6 (VS)
Other:
- moved on the sheet: C1, C31, D1
Changed lines of the file:
@@
 L Device:CP C1
 U 1 1 5F706578
-P 4500 3350
+P 4500 3300
 AR Path="/5F7ECC6C/5F706578" Ref="C1"  Part="1"
 AR Path="/5F79FFE4/5F706578" Ref="C11"  Part="1"
@@
 AR Path="/5F7A3A2A/5F706578" Ref="C17"  Part="1"
 AR Path="/5F7A4E71/5F706578" Ref="C24"  Part="1"
-F 0 "C1" H 4618 3396 50  0000 L CNN
-F 1 "47u LKMD0901K470MF" H 4618 3305 50  0000 L CNN
-F 2 "Capacitor_THT:CP_Radial_D8.0mm_P3.50mm" H 4538 3200 50  0001 C CNN
-F 3 "~" H 4500 3350 50  0001 C CNN
-	1    4500 3350
+F 0 "C1" H 4618 3346 50  0000 L CNN
+F 1 "47u LKMD0901K470MF" H 4618 3255 50  0000 L CNN
+F 2 "Capacitor_THT:CP_Radial_D8.0mm_P3.50mm" H 4538 3150 50  0001 C CNN
+F 3 "~" H 4500 3300 50  0001 C CNN
+	1    4500 3300
 	1    0    0    -1
 $EndComp
@@
 L Device:D D1
 U 1 1 5F707CCD
-P 4350 2500
+P 4300 2500
 AR Path="/5F7ECC6C/5F707CCD" Ref="D1"  Part="1"
 AR Path="/5F79FFE4/5F707CCD" Ref="D7"  Part="1"
@@
 AR Path="/5F7A3A2A/5F707CCD" Ref="D10"  Part="1"
 AR Path="/5F7A4E71/5F707CCD" Ref="D11"  Part="1"
-F 0 "D1" H 4350 2284 50  0000 C CNN
-F 1 "1N4148W" H 4350 2375 50  0000 C CNN
-F 2 "Diode_SMD:D_SOD-123" H 4350 2500 50  0001 C CNN
-F 3 "~" H 4350 2500 50  0001 C CNN
-	1    4350 2500
+F 0 "D1" H 4300 2284 50  0000 C CNN
+F 1 "1N4148W" H 4300 2375 50  0000 C CNN
+F 2 "Diode_SMD:D_SOD-123" H 4300 2500 50  0001 C CNN
+F 3 "~" H 4300 2500 50  0001 C CNN
+	1    4300 2500
 	-1   0    0    1
 $EndComp
 Text HLabel 3650 3400 0    50   Input ~ 0
 H_BRIDGE_LO
-Text HLabel 6300 3800 2    50   UnSpc ~ 0
+Text HLabel 6300 3850 2    50   UnSpc ~ 0
 H_BRIDGE_GND
 Text HLabel 6300 3350 2    50   UnSpc ~ 0
@@
 	3500 3800 3500 3750
 Wire Wire Line
-	3500 4100 3750 4100
+	3500 4150 3750 4150
 $Comp
 L power:GND #PWR0173
 U 1 1 5F773E85
-P 3750 4100
+P 3750 4200
 AR Path="/5F7ECC6C/5F773E85" Ref="#PWR0173"  Part="1"
 AR Path="/5F79FFE4/5F773E85" Ref="#PWR0177"  Part="1"
@@
 AR Path="/5F7A3A2A/5F773E85" Ref="#PWR0189"  Part="1"
 AR Path="/5F7A4E71/5F773E85" Ref="#PWR0193"  Part="1"
-F 0 "#PWR0173" H 3750 3850 50  0001 C CNN
-F 1 "GND" H 3755 3927 50  0000 C CNN
-F 2 "" H 3750 4100 50  0001 C CNN
-F 3 "" H 3750 4100 50  0001 C CNN
-	1    3750 4100
-	1    0    0    -1
-$EndComp
-Connection ~ 3750 4100
-Wire Wire Line
-	3750 4100 3950 4100
+F 0 "#PWR0173" H 3750 3950 50  0001 C CNN
+F 1 "GND" H 3755 4027 50  0000 C CNN
+F 2 "" H 3750 4200 50  0001 C CNN
+F 3 "" H 3750 4200 50  0001 C CNN
+	1    3750 4200
+	1    0    0    -1
+$EndComp
+Connection ~ 3750 4150
+Wire Wire Line
+	3750 4150 3950 4150
 Wire Wire Line
 	3950 2400 3950 2500
-Wire Wire Line
-	4200 2500 3950 2500
 Connection ~ 3950 2500
 Wire Wire Line
 	4500 3000 4500 2500
-Wire Wire Line
-	4500 3200 4500 3000
-Connection ~ 4500 3000
 $Comp
 L Transistor_FET:BSP89 V1
@@
 Wire Wire Line
 	4250 3000 4500 3000
-Wire Wire Line
-	4250 3500 4500 3500
 $Comp
 L Device:R R10
@@
 $EndComp
 Wire Wire Line
-	3950 4100 3950 3800
-Wire Wire Line
 	3950 2500 3950 2800
 $Comp
@@
 L power:+BATT #PWR0174
 U 1 1 5F79127D
-P 5650 2900
+P 5650 2800
 AR Path="/5F7ECC6C/5F79127D" Ref="#PWR0174"  Part="1"
 AR Path="/5F79FFE4/5F79127D" Ref="#PWR0178"  Part="1"
@@
 AR Path="/5F7A3A2A/5F79127D" Ref="#PWR0190"  Part="1"
 AR Path="/5F7A4E71/5F79127D" Ref="#PWR0194"  Part="1"
-F 0 "#PWR0174" H 5650 2750 50  0001 C CNN
-F 1 "+BATT" H 5665 3073 50  0000 C CNN
-F 2 "" H 5650 2900 50  0001 C CNN
-F 3 "" H 5650 2900 50  0001 C CNN
-	1    5650 2900
+F 0 "#PWR0174" H 5650 2650 50  0001 C CNN
+F 1 "+BATT" H 5665 2973 50  0000 C CNN
+F 2 "" H 5650 2800 50  0001 C CNN
+F 3 "" H 5650 2800 50  0001 C CNN
+	1    5650 2800
 	1    0    0    -1
 $EndComp
@@
 	5650 3350 5650 3400
 Wire Wire Line
-	6300 3800 5650 3800
+	6300 3850 5650 3850
 $Comp
 L Device:CP C31
 U 1 1 5F7BE8FF
-P 6700 2600
+P 7100 3000
 AR Path="/5F7ECC6C/5F7BE8FF" Ref="C31"  Part="1"
 AR Path="/5F79FFE4/5F7BE8FF" Ref="C32"  Part="1"
@@
 AR Path="/5F7A3A2A/5F7BE8FF" Ref="C35"  Part="1"
 AR Path="/5F7A4E71/5F7BE8FF" Ref="C36"  Part="1"
-F 0 "C31" H 6818 2646 50  0000 L CNN
-F 1 "47u LKMD0901K470MF" H 6818 2555 50  0000 L CNN
-F 2 "Capacitor_THT:CP_Radial_D8.0mm_P3.50mm" H 6738 2450 50  0001 C CNN
-F 3 "~" H 6700 2600 50  0001 C CNN
-	1    6700 2600
+F 0 "C31" H 7218 3046 50  0000 L CNN
+F 1 "47u LKMD0901K470MF" H 7218 2955 50  0000 L CNN
+F 2 "Capacitor_THT:CP_Radial_D8.0mm_P3.50mm" H 7138 2850 50  0001 C CNN
+F 3 "~" H 7100 3000 50  0001 C CNN
+	1    7100 3000
 	1    0    0    -1
 $EndComp
@@
 L power:+BATT #PWR0197
 U 1 1 5F7BF207
-P 6700 2450
+P 7100 2800
 AR Path="/5F7ECC6C/5F7BF207" Ref="#PWR0197"  Part="1"
 AR Path="/5F79FFE4/5F7BF207" Ref="#PWR0198"  Part="1"
@@
 AR Path="/5F7A3A2A/5F7BF207" Ref="#PWR0201"  Part="1"
 AR Path="/5F7A4E71/5F7BF207" Ref="#PWR0202"  Part="1"
-F 0 "#PWR0197" H 6700 2300 50  0001 C CNN
-F 1 "+BATT" H 6715 2623 50  0000 C CNN
-F 2 "" H 6700 2450 50  0001 C CNN
-F 3 "" H 6700 2450 50  0001 C CNN
-	1    6700 2450
-	1    0    0    -1
-$EndComp
-Wire Wire Line
-	6700 2750 6700 3000
-Wire Wire Line
-	6700 3000 7100 3000
-Wire Wire Line
-	7100 3000 7100 4050
+F 0 "#PWR0197" H 7100 2650 50  0001 C CNN
+F 1 "+BATT" H 7115 2973 50  0000 C CNN
+F 2 "" H 7100 2800 50  0001 C CNN
+F 3 "" H 7100 2800 50  0001 C CNN
+	1    7100 2800
+	1    0    0    -1
+$EndComp
 Wire Wire Line
 	7100 4050 5650 4050
 Wire Wire Line
-	5650 4050 5650 3800
-Connection ~ 5650 3800
+	5650 4050 5650 3850
+Wire Wire Line
+	5500 3500 5500 3350
+Wire Wire Line
+	5500 3350 5650 3350
+Wire Wire Line
+	4500 3000 4500 3150
+Wire Wire Line
+	4250 3500 4500 3500
+Connection ~ 4500 3000
+Wire Wire Line
+	4500 3450 4500 3500
+Connection ~ 4500 3500
+Wire Wire Line
+	4500 3500 5500 3500
+Connection ~ 5650 3850
+Wire Wire Line
+	5650 3850 5650 3800
+Wire Wire Line
+	4150 2500 3950 2500
+Wire Wire Line
+	4450 2500 4500 2500
+Wire Wire Line
+	3750 4150 3750 4200
+Wire Wire Line
+	3500 4100 3500 4150
+Wire Wire Line
+	3950 3800 3950 4150
+Wire Wire Line
+	7100 3150 7100 4050
+Wire Wire Line
+	7100 2800 7100 2850
+Wire Wire Line
+	5650 2800 5650 2900
 $EndSCHEMATC

Commit message: added footprints, continue layout
Parts:
- added D23: 51V TVS C310059, Diode_SMD:D_SMC, symbol Device:D_Zener
Connections:
- net +BATT: now also D23.1 (K)
- net H_BRIDGE_GND: now also D23.2 (A)
Changed lines of the file:
@@
 $Descr A4 11693 8268
 encoding utf-8
-Sheet 8 14
+Sheet 11 14
 Title ""
 Date ""
@@
 AR Path="/5F7A3A2A/5F706578" Ref="C17"  Part="1"
 AR Path="/5F7A4E71/5F706578" Ref="C24"  Part="1"
-F 0 "C1" H 4618 3346 50  0000 L CNN
+F 0 "C15" H 4618 3346 50  0000 L CNN
 F 1 "47u LKMD0901K470MF" H 4618 3255 50  0000 L CNN
 F 2 "Capacitor_THT:CP_Radial_D8.0mm_P3.50mm" H 4538 3150 50  0001 C CNN
@@
 AR Path="/5F7A3A2A/5F707CCD" Ref="D10"  Part="1"
 AR Path="/5F7A4E71/5F707CCD" Ref="D11"  Part="1"
-F 0 "D1" H 4300 2284 50  0000 C CNN
+F 0 "D9" H 4300 2284 50  0000 C CNN
 F 1 "1N4148W" H 4300 2375 50  0000 C CNN
 F 2 "Diode_SMD:D_SOD-123" H 4300 2500 50  0001 C CNN
@@
 AR Path="/5F7A3A2A/5F77195C" Ref="#PWR0187"  Part="1"
 AR Path="/5F7A4E71/5F77195C" Ref="#PWR0191"  Part="1"
-F 0 "#PWR0171" H 3950 2250 50  0001 C CNN
+F 0 "#PWR0183" H 3950 2250 50  0001 C CNN
 F 1 "+VSW" H 3965 2573 50  0000 C CNN
 F 2 "" H 3950 2400 50  0001 C CNN
@@
 AR Path="/5F7A3A2A/5F771CDC" Ref="C16"  Part="1"
 AR Path="/5F7A4E71/5F771CDC" Ref="C18"  Part="1"
-F 0 "C8" H 3618 3996 50  0000 L CNN
+F 0 "C14" H 3618 3996 50  0000 L CNN
 F 1 "220u25V LKMD0901E221MF" H 3618 3905 50  0000 L CNN
 F 2 "Capacitor_THT:CP_Radial_D8.0mm_P3.50mm" H 3538 3800 50  0001 C CNN
@@
 AR Path="/5F7A3A2A/5F77283D" Ref="#PWR0188"  Part="1"
 AR Path="/5F7A4E71/5F77283D" Ref="#PWR0192"  Part="1"
-F 0 "#PWR0172" H 3500 3600 50  0001 C CNN
+F 0 "#PWR0184" H 3500 3600 50  0001 C CNN
 F 1 "+VSW" H 3515 3923 50  0000 C CNN
 F 2 "" H 3500 3750 50  0001 C CNN
@@
 AR Path="/5F7A3A2A/5F773E85" Ref="#PWR0189"  Part="1"
 AR Path="/5F7A4E71/5F773E85" Ref="#PWR0193"  Part="1"
-F 0 "#PWR0173" H 3750 3950 50  0001 C CNN
+F 0 "#PWR0185" H 3750 3950 50  0001 C CNN
 F 1 "GND" H 3755 4027 50  0000 C CNN
 F 2 "" H 3750 4200 50  0001 C CNN
@@
 AR Path="/5F7A3A2A/5F73738F" Ref="V9"  Part="1"
 AR Path="/5F7A4E71/5F73738F" Ref="V11"  Part="1"
-F 0 "V1" H 5755 3646 50  0000 L CNN
+F 0 "V7" H 5755 3646 50  0000 L CNN
 F 1 "CRSS042N10N" H 5755 3555 50  0000 L CNN
 F 2 "Package_TO_SOT_SMD:TO-263-2" H 5750 3525 50  0001 L CIN
@@
 AR Path="/5F7A3A2A/5F72B1D2" Ref="R32"  Part="1"
 AR Path="/5F7A4E71/5F72B1D2" Ref="R34"  Part="1"
-F 0 "R10" V 4993 3600 50  0000 C CNN
+F 0 "R21" V 4993 3600 50  0000 C CNN
 F 1 "68" V 5084 3600 50  0000 C CNN
 F 2 "Resistor_SMD:R_1206_3216Metric" V 5130 3600 50  0001 C CNN
@@
 AR Path="/5F7A3A2A/5F771122" Ref="U12"  Part="1"
 AR Path="/5F7A4E71/5F771122" Ref="U13"  Part="1"
-F 0 "U8" H 3950 3981 50  0000 C CNN
+F 0 "U11" H 3950 3981 50  0000 C CNN
 F 1 "IRS2304" H 3950 3890 50  0000 C CNN
 F 2 "Package_SO:SOIC-8_3.9x4.9mm_P1.27mm" H 3950 3300 50  0001 C CIN
@@
 AR Path="/5F7A3A2A/5F7824C8" Ref="R28"  Part="1"
 AR Path="/5F7A4E71/5F7824C8" Ref="R33"  Part="1"
-F 0 "R13" V 4993 3100 50  0000 C CNN
+F 0 "R18" V 4993 3100 50  0000 C CNN
 F 1 "68" V 5084 3100 50  0000 C CNN
 F 2 "Resistor_SMD:R_1206_3216Metric" V 5130 3100 50  0001 C CNN
@@
 AR Path="/5F7A3A2A/5F70E4C5" Ref="V8"  Part="1"
 AR Path="/5F7A4E71/5F70E4C5" Ref="V10"  Part="1"
-F 0 "V0" H 5755 3146 50  0000 L CNN
+F 0 "V6" H 5755 3146 50  0000 L CNN
 F 1 "CRSS042N10N" H 5755 3055 50  0000 L CNN
 F 2 "Package_TO_SOT_SMD:TO-263-2" H 5750 3025 50  0001 L CIN
@@
 AR Path="/5F7A3A2A/5F79127D" Ref="#PWR0190"  Part="1"
 AR Path="/5F7A4E71/5F79127D" Ref="#PWR0194"  Part="1"
-F 0 "#PWR0174" H 5650 2650 50  0001 C CNN
+F 0 "#PWR0186" H 5650 2650 50  0001 C CNN
 F 1 "+BATT" H 5665 2973 50  0000 C CNN
 F 2 "" H 5650 2800 50  0001 C CNN
@@
 AR Path="/5F7A3A2A/5F7BE8FF" Ref="C35"  Part="1"
 AR Path="/5F7A4E71/5F7BE8FF" Ref="C36"  Part="1"
-F 0 "C31" H 7218 3046 50  0000 L CNN
+F 0 "C34" H 7218 3046 50  0000 L CNN
 F 1 "47u LKMD0901K470MF" H 7218 2955 50  0000 L CNN
 F 2 "Capacitor_THT:CP_Radial_D8.0mm_P3.50mm" H 7138 2850 50  0001 C CNN
@@
 AR Path="/5F7A3A2A/5F7BF207" Ref="#PWR0201"  Part="1"
 AR Path="/5F7A4E71/5F7BF207" Ref="#PWR0202"  Part="1"
-F 0 "#PWR0197" H 7100 2650 50  0001 C CNN
+F 0 "#PWR0200" H 7100 2650 50  0001 C CNN
 F 1 "+BATT" H 7115 2973 50  0000 C CNN
 F 2 "" H 7100 2800 50  0001 C CNN
@@
 	3950 3800 3950 4150
 Wire Wire Line
-	7100 3150 7100 4050
+	7100 3150 7100 3350
 Wire Wire Line
 	7100 2800 7100 2850
 Wire Wire Line
 	5650 2800 5650 2900
+$Comp
+L Device:D_Zener D?
+U 1 1 5F72BDA4
+P 8200 3000
+AR Path="/5F7395DA/5F72BDA4" Ref="D?"  Part="1"
+AR Path="/5F7ECC6C/5F72BDA4" Ref="D23"  Part="1"
+AR Path="/5F79FFE4/5F72BDA4" Ref="D24"  Part="1"
+AR Path="/5F7A0EEE/5F72BDA4" Ref="D25"  Part="1"
+AR Path="/5F7A2640/5F72BDA4" Ref="D26"  Part="1"
+AR Path="/5F7A3A2A/5F72BDA4" Ref="D27"  Part="1"
+AR Path="/5F7A4E71/5F72BDA4" Ref="D28"  Part="1"
+F 0 "D26" V 8154 3080 50  0000 L CNN
+F 1 "51V TVS C310059" V 8245 3080 50  0000 L CNN
+F 2 "Diode_SMD:D_SMC" H 8200 3000 50  0001 C CNN
+F 3 "~" H 8200 3000 50  0001 C CNN
+	1    8200 3000
+	0    1    1    0
+$EndComp
+Wire Wire Line
+	8200 3150 8200 3350
+Wire Wire Line
+	7100 2800 8200 2800
+Connection ~ 7100 2800
+Wire Wire Line
+	8200 2800 8200 2850
+Wire Wire Line
+	8200 3350 7100 3350
+Connection ~ 7100 3350
+Wire Wire Line
+	7100 3350 7100 4050
 $EndSCHEMATC

Commit message: continue analog layout
Changed lines of the file:
@@
 $Descr A4 11693 8268
 encoding utf-8
-Sheet 11 14
+Sheet 12 14
 Title ""
 Date ""
@@
 AR Path="/5F7A3A2A/5F706578" Ref="C17"  Part="1"
 AR Path="/5F7A4E71/5F706578" Ref="C24"  Part="1"
-F 0 "C15" H 4618 3346 50  0000 L CNN
+F 0 "C24" H 4618 3346 50  0000 L CNN
 F 1 "47u LKMD0901K470MF" H 4618 3255 50  0000 L CNN
 F 2 "Capacitor_THT:CP_Radial_D8.0mm_P3.50mm" H 4538 3150 50  0001 C CNN
@@
 AR Path="/5F7A3A2A/5F707CCD" Ref="D10"  Part="1"
 AR Path="/5F7A4E71/5F707CCD" Ref="D11"  Part="1"
-F 0 "D9" H 4300 2284 50  0000 C CNN
+F 0 "D11" H 4300 2284 50  0000 C CNN
 F 1 "1N4148W" H 4300 2375 50  0000 C CNN
 F 2 "Diode_SMD:D_SOD-123" H 4300 2500 50  0001 C CNN
@@
 AR Path="/5F7A3A2A/5F77195C" Ref="#PWR0187"  Part="1"
 AR Path="/5F7A4E71/5F77195C" Ref="#PWR0191"  Part="1"
-F 0 "#PWR0183" H 3950 2250 50  0001 C CNN
+F 0 "#PWR0191" H 3950 2250 50  0001 C CNN
 F 1 "+VSW" H 3965 2573 50  0000 C CNN
 F 2 "" H 3950 2400 50  0001 C CNN
@@
 AR Path="/5F7A3A2A/5F771CDC" Ref="C16"  Part="1"
 AR Path="/5F7A4E71/5F771CDC" Ref="C18"  Part="1"
-F 0 "C14" H 3618 3996 50  0000 L CNN
+F 0 "C18" H 3618 3996 50  0000 L CNN
 F 1 "220u25V LKMD0901E221MF" H 3618 3905 50  0000 L CNN
 F 2 "Capacitor_THT:CP_Radial_D8.0mm_P3.50mm" H 3538 3800 50  0001 C CNN
@@
 AR Path="/5F7A3A2A/5F77283D" Ref="#PWR0188"  Part="1"
 AR Path="/5F7A4E71/5F77283D" Ref="#PWR0192"  Part="1"
-F 0 "#PWR0184" H 3500 3600 50  0001 C CNN
+F 0 "#PWR0192" H 3500 3600 50  0001 C CNN
 F 1 "+VSW" H 3515 3923 50  0000 C CNN
 F 2 "" H 3500 3750 50  0001 C CNN
@@
 AR Path="/5F7A3A2A/5F773E85" Ref="#PWR0189"  Part="1"
 AR Path="/5F7A4E71/5F773E85" Ref="#PWR0193"  Part="1"
-F 0 "#PWR0185" H 3750 3950 50  0001 C CNN
+F 0 "#PWR0193" H 3750 3950 50  0001 C CNN
 F 1 "GND" H 3755 4027 50  0000 C CNN
 F 2 "" H 3750 4200 50  0001 C CNN
@@
 AR Path="/5F7A3A2A/5F73738F" Ref="V9"  Part="1"
 AR Path="/5F7A4E71/5F73738F" Ref="V11"  Part="1"
-F 0 "V7" H 5755 3646 50  0000 L CNN
+F 0 "V11" H 5755 3646 50  0000 L CNN
 F 1 "CRSS042N10N" H 5755 3555 50  0000 L CNN
 F 2 "Package_TO_SOT_SMD:TO-263-2" H 5750 3525 50  0001 L CIN
@@
 AR Path="/5F7A3A2A/5F72B1D2" Ref="R32"  Part="1"
 AR Path="/5F7A4E71/5F72B1D2" Ref="R34"  Part="1"
-F 0 "R21" V 4993 3600 50  0000 C CNN
+F 0 "R34" V 4993 3600 50  0000 C CNN
 F 1 "68" V 5084 3600 50  0000 C CNN
 F 2 "Resistor_SMD:R_1206_3216Metric" V 5130 3600 50  0001 C CNN
@@
 AR Path="/5F7A3A2A/5F771122" Ref="U12"  Part="1"
 AR Path="/5F7A4E71/5F771122" Ref="U13"  Part="1"
-F 0 "U11" H 3950 3981 50  0000 C CNN
+F 0 "U13" H 3950 3981 50  0000 C CNN
 F 1 "IRS2304" H 3950 3890 50  0000 C CNN
 F 2 "Package_SO:SOIC-8_3.9x4.9mm_P1.27mm" H 3950 3300 50  0001 C CIN
@@
 AR Path="/5F7A3A2A/5F7824C8" Ref="R28"  Part="1"
 AR Path="/5F7A4E71/5F7824C8" Ref="R33"  Part="1"
-F 0 "R18" V 4993 3100 50  0000 C CNN
+F 0 "R33" V 4993 3100 50  0000 C CNN
 F 1 "68" V 5084 3100 50  0000 C CNN
 F 2 "Resistor_SMD:R_1206_3216Metric" V 5130 3100 50  0001 C CNN
@@
 AR Path="/5F7A3A2A/5F70E4C5" Ref="V8"  Part="1"
 AR Path="/5F7A4E71/5F70E4C5" Ref="V10"  Part="1"
-F 0 "V6" H 5755 3146 50  0000 L CNN
+F 0 "V10" H 5755 3146 50  0000 L CNN
 F 1 "CRSS042N10N" H 5755 3055 50  0000 L CNN
 F 2 "Package_TO_SOT_SMD:TO-263-2" H 5750 3025 50  0001 L CIN
@@
 AR Path="/5F7A3A2A/5F79127D" Ref="#PWR0190"  Part="1"
 AR Path="/5F7A4E71/5F79127D" Ref="#PWR0194"  Part="1"
-F 0 "#PWR0186" H 5650 2650 50  0001 C CNN
+F 0 "#PWR0194" H 5650 2650 50  0001 C CNN
 F 1 "+BATT" H 5665 2973 50  0000 C CNN
 F 2 "" H 5650 2800 50  0001 C CNN
@@
 AR Path="/5F7A3A2A/5F7BE8FF" Ref="C35"  Part="1"
 AR Path="/5F7A4E71/5F7BE8FF" Ref="C36"  Part="1"
-F 0 "C34" H 7218 3046 50  0000 L CNN
+F 0 "C36" H 7218 3046 50  0000 L CNN
 F 1 "47u LKMD0901K470MF" H 7218 2955 50  0000 L CNN
 F 2 "Capacitor_THT:CP_Radial_D8.0mm_P3.50mm" H 7138 2850 50  0001 C CNN
@@
 AR Path="/5F7A3A2A/5F7BF207" Ref="#PWR0201"  Part="1"
 AR Path="/5F7A4E71/5F7BF207" Ref="#PWR0202"  Part="1"
-F 0 "#PWR0200" H 7100 2650 50  0001 C CNN
+F 0 "#PWR0202" H 7100 2650 50  0001 C CNN
 F 1 "+BATT" H 7115 2973 50  0000 C CNN
 F 2 "" H 7100 2800 50  0001 C CNN
@@
 AR Path="/5F7A3A2A/5F72BDA4" Ref="D27"  Part="1"
 AR Path="/5F7A4E71/5F72BDA4" Ref="D28"  Part="1"
-F 0 "D26" V 8154 3080 50  0000 L CNN
+F 0 "D28" V 8154 3080 50  0000 L CNN
 F 1 "51V TVS C310059" V 8245 3080 50  0000 L CNN
 F 2 "Diode_SMD:D_SMC" H 8200 3000 50  0001 C CNN

Commit message: continue board layout, placed all components
Changed lines of the file:
@@
 AR Path="/5F7A3A2A/5F706578" Ref="C17"  Part="1"
 AR Path="/5F7A4E71/5F706578" Ref="C24"  Part="1"
-F 0 "C24" H 4618 3346 50  0000 L CNN
+F 0 "C17" H 4618 3346 50  0000 L CNN
 F 1 "47u LKMD0901K470MF" H 4618 3255 50  0000 L CNN
 F 2 "Capacitor_THT:CP_Radial_D8.0mm_P3.50mm" H 4538 3150 50  0001 C CNN
@@
 AR Path="/5F7A3A2A/5F707CCD" Ref="D10"  Part="1"
 AR Path="/5F7A4E71/5F707CCD" Ref="D11"  Part="1"
-F 0 "D11" H 4300 2284 50  0000 C CNN
+F 0 "D10" H 4300 2284 50  0000 C CNN
 F 1 "1N4148W" H 4300 2375 50  0000 C CNN
 F 2 "Diode_SMD:D_SOD-123" H 4300 2500 50  0001 C CNN
@@
 AR Path="/5F7A3A2A/5F771CDC" Ref="C16"  Part="1"
 AR Path="/5F7A4E71/5F771CDC" Ref="C18"  Part="1"
-F 0 "C18" H 3618 3996 50  0000 L CNN
+F 0 "C16" H 3618 3996 50  0000 L CNN
 F 1 "220u25V LKMD0901E221MF" H 3618 3905 50  0000 L CNN
 F 2 "Capacitor_THT:CP_Radial_D8.0mm_P3.50mm" H 3538 3800 50  0001 C CNN
@@
 AR Path="/5F7A3A2A/5F73738F" Ref="V9"  Part="1"
 AR Path="/5F7A4E71/5F73738F" Ref="V11"  Part="1"
-F 0 "V11" H 5755 3646 50  0000 L CNN
+F 0 "V9" H 5755 3646 50  0000 L CNN
 F 1 "CRSS042N10N" H 5755 3555 50  0000 L CNN
 F 2 "Package_TO_SOT_SMD:TO-263-2" H 5750 3525 50  0001 L CIN
@@
 AR Path="/5F7A3A2A/5F72B1D2" Ref="R32"  Part="1"
 AR Path="/5F7A4E71/5F72B1D2" Ref="R34"  Part="1"
-F 0 "R34" V 4993 3600 50  0000 C CNN
+F 0 "R32" V 4993 3600 50  0000 C CNN
 F 1 "68" V 5084 3600 50  0000 C CNN
 F 2 "Resistor_SMD:R_1206_3216Metric" V 5130 3600 50  0001 C CNN
@@
 AR Path="/5F7A3A2A/5F771122" Ref="U12"  Part="1"
 AR Path="/5F7A4E71/5F771122" Ref="U13"  Part="1"
-F 0 "U13" H 3950 3981 50  0000 C CNN
+F 0 "U12" H 3950 3981 50  0000 C CNN
 F 1 "IRS2304" H 3950 3890 50  0000 C CNN
 F 2 "Package_SO:SOIC-8_3.9x4.9mm_P1.27mm" H 3950 3300 50  0001 C CIN
@@
 AR Path="/5F7A3A2A/5F7824C8" Ref="R28"  Part="1"
 AR Path="/5F7A4E71/5F7824C8" Ref="R33"  Part="1"
-F 0 "R33" V 4993 3100 50  0000 C CNN
+F 0 "R28" V 4993 3100 50  0000 C CNN
 F 1 "68" V 5084 3100 50  0000 C CNN
 F 2 "Resistor_SMD:R_1206_3216Metric" V 5130 3100 50  0001 C CNN
@@
 AR Path="/5F7A3A2A/5F70E4C5" Ref="V8"  Part="1"
 AR Path="/5F7A4E71/5F70E4C5" Ref="V10"  Part="1"
-F 0 "V10" H 5755 3146 50  0000 L CNN
+F 0 "V8" H 5755 3146 50  0000 L CNN
 F 1 "CRSS042N10N" H 5755 3055 50  0000 L CNN
 F 2 "Package_TO_SOT_SMD:TO-263-2" H 5750 3025 50  0001 L CIN
@@
 AR Path="/5F7A3A2A/5F7BE8FF" Ref="C35"  Part="1"
 AR Path="/5F7A4E71/5F7BE8FF" Ref="C36"  Part="1"
-F 0 "C36" H 7218 3046 50  0000 L CNN
+F 0 "C35" H 7218 3046 50  0000 L CNN
 F 1 "47u LKMD0901K470MF" H 7218 2955 50  0000 L CNN
 F 2 "Capacitor_THT:CP_Radial_D8.0mm_P3.50mm" H 7138 2850 50  0001 C CNN
@@
 AR Path="/5F7A3A2A/5F72BDA4" Ref="D27"  Part="1"
 AR Path="/5F7A4E71/5F72BDA4" Ref="D28"  Part="1"
-F 0 "D28" V 8154 3080 50  0000 L CNN
+F 0 "D27" V 8154 3080 50  0000 L CNN
 F 1 "51V TVS C310059" V 8245 3080 50  0000 L CNN
 F 2 "Diode_SMD:D_SMC" H 8200 3000 50  0001 C CNN
