File: hh_bridge.sch (KiCad schematic (older format))
At the start: 10 parts, among them U8 IRS2304

Commit message: finish design
Changed lines of the file:
@@
 $Descr A4 11693 8268
 encoding utf-8
-Sheet 12 14
+Sheet 8 14
 Title ""
 Date ""
@@
 AR Path="/5F7A3A2A/5F706578" Ref="C17"  Part="1"
 AR Path="/5F7A4E71/5F706578" Ref="C24"  Part="1"
-F 0 "C17" H 4618 3346 50  0000 L CNN
+F 0 "C24" H 4618 3346 50  0000 L CNN
 F 1 "47u LKMD0901K470MF" H 4618 3255 50  0000 L CNN
 F 2 "Capacitor_THT:CP_Radial_D8.0mm_P3.50mm" H 4538 3150 50  0001 C CNN
@@
 AR Path="/5F7A3A2A/5F707CCD" Ref="D10"  Part="1"
 AR Path="/5F7A4E71/5F707CCD" Ref="D11"  Part="1"
-F 0 "D10" H 4300 2284 50  0000 C CNN
+F 0 "D11" H 4300 2284 50  0000 C CNN
 F 1 "1N4148W" H 4300 2375 50  0000 C CNN
 F 2 "Diode_SMD:D_SOD-123" H 4300 2500 50  0001 C CNN
@@
 AR Path="/5F7A3A2A/5F771CDC" Ref="C16"  Part="1"
 AR Path="/5F7A4E71/5F771CDC" Ref="C18"  Part="1"
-F 0 "C16" H 3618 3996 50  0000 L CNN
+F 0 "C18" H 3618 3996 50  0000 L CNN
 F 1 "220u25V LKMD0901E221MF" H 3618 3905 50  0000 L CNN
 F 2 "Capacitor_THT:CP_Radial_D8.0mm_P3.50mm" H 3538 3800 50  0001 C CNN
@@
 AR Path="/5F7A3A2A/5F73738F" Ref="V9"  Part="1"
 AR Path="/5F7A4E71/5F73738F" Ref="V11"  Part="1"
-F 0 "V9" H 5755 3646 50  0000 L CNN
+F 0 "V11" H 5755 3646 50  0000 L CNN
 F 1 "CRSS042N10N" H 5755 3555 50  0000 L CNN
 F 2 "Package_TO_SOT_SMD:TO-263-2" H 5750 3525 50  0001 L CIN
@@
 AR Path="/5F7A3A2A/5F72B1D2" Ref="R32"  Part="1"
 AR Path="/5F7A4E71/5F72B1D2" Ref="R34"  Part="1"
-F 0 "R32" V 4993 3600 50  0000 C CNN
+F 0 "R34" V 4993 3600 50  0000 C CNN
 F 1 "68" V 5084 3600 50  0000 C CNN
 F 2 "Resistor_SMD:R_1206_3216Metric" V 5130 3600 50  0001 C CNN
@@
 AR Path="/5F7A3A2A/5F771122" Ref="U12"  Part="1"
 AR Path="/5F7A4E71/5F771122" Ref="U13"  Part="1"
-F 0 "U12" H 3950 3981 50  0000 C CNN
+F 0 "U13" H 3950 3981 50  0000 C CNN
 F 1 "IRS2304" H 3950 3890 50  0000 C CNN
 F 2 "Package_SO:SOIC-8_3.9x4.9mm_P1.27mm" H 3950 3300 50  0001 C CIN
@@
 AR Path="/5F7A3A2A/5F7824C8" Ref="R28"  Part="1"
 AR Path="/5F7A4E71/5F7824C8" Ref="R33"  Part="1"
-F 0 "R28" V 4993 3100 50  0000 C CNN
+F 0 "R33" V 4993 3100 50  0000 C CNN
 F 1 "68" V 5084 3100 50  0000 C CNN
 F 2 "Resistor_SMD:R_1206_3216Metric" V 5130 3100 50  0001 C CNN
@@
 AR Path="/5F7A3A2A/5F70E4C5" Ref="V8"  Part="1"
 AR Path="/5F7A4E71/5F70E4C5" Ref="V10"  Part="1"
-F 0 "V8" H 5755 3146 50  0000 L CNN
+F 0 "V10" H 5755 3146 50  0000 L CNN
 F 1 "CRSS042N10N" H 5755 3055 50  0000 L CNN
 F 2 "Package_TO_SOT_SMD:TO-263-2" H 5750 3025 50  0001 L CIN
@@
 AR Path="/5F7A3A2A/5F7BE8FF" Ref="C35"  Part="1"
 AR Path="/5F7A4E71/5F7BE8FF" Ref="C36"  Part="1"
-F 0 "C35" H 7218 3046 50  0000 L CNN
+F 0 "C36" H 7218 3046 50  0000 L CNN
 F 1 "47u LKMD0901K470MF" H 7218 2955 50  0000 L CNN
 F 2 "Capacitor_THT:CP_Radial_D8.0mm_P3.50mm" H 7138 2850 50  0001 C CNN
@@
 AR Path="/5F7A3A2A/5F72BDA4" Ref="D27"  Part="1"
 AR Path="/5F7A4E71/5F72BDA4" Ref="D28"  Part="1"
-F 0 "D27" V 8154 3080 50  0000 L CNN
+F 0 "D28" V 8154 3080 50  0000 L CNN
 F 1 "51V TVS C310059" V 8245 3080 50  0000 L CNN
 F 2 "Diode_SMD:D_SMC" H 8200 3000 50  0001 C CNN

Commit message: finish layout
Changed lines of the file:
@@
 $Descr A4 11693 8268
 encoding utf-8
-Sheet 8 14
+Sheet 10 14
 Title ""
 Date ""
@@
 AR Path="/5F7A3A2A/5F706578" Ref="C17"  Part="1"
 AR Path="/5F7A4E71/5F706578" Ref="C24"  Part="1"
-F 0 "C24" H 4618 3346 50  0000 L CNN
+F 0 "C13" H 4618 3346 50  0000 L CNN
 F 1 "47u LKMD0901K470MF" H 4618 3255 50  0000 L CNN
 F 2 "Capacitor_THT:CP_Radial_D8.0mm_P3.50mm" H 4538 3150 50  0001 C CNN
@@
 AR Path="/5F7A3A2A/5F707CCD" Ref="D10"  Part="1"
 AR Path="/5F7A4E71/5F707CCD" Ref="D11"  Part="1"
-F 0 "D11" H 4300 2284 50  0000 C CNN
+F 0 "D8" H 4300 2284 50  0000 C CNN
 F 1 "1N4148W" H 4300 2375 50  0000 C CNN
 F 2 "Diode_SMD:D_SOD-123" H 4300 2500 50  0001 C CNN
@@
 AR Path="/5F7A3A2A/5F77195C" Ref="#PWR0187"  Part="1"
 AR Path="/5F7A4E71/5F77195C" Ref="#PWR0191"  Part="1"
-F 0 "#PWR0191" H 3950 2250 50  0001 C CNN
+F 0 "#PWR0179" H 3950 2250 50  0001 C CNN
 F 1 "+VSW" H 3965 2573 50  0000 C CNN
 F 2 "" H 3950 2400 50  0001 C CNN
@@
 AR Path="/5F7A3A2A/5F771CDC" Ref="C16"  Part="1"
 AR Path="/5F7A4E71/5F771CDC" Ref="C18"  Part="1"
-F 0 "C18" H 3618 3996 50  0000 L CNN
+F 0 "C12" H 3618 3996 50  0000 L CNN
 F 1 "220u25V LKMD0901E221MF" H 3618 3905 50  0000 L CNN
 F 2 "Capacitor_THT:CP_Radial_D8.0mm_P3.50mm" H 3538 3800 50  0001 C CNN
@@
 AR Path="/5F7A3A2A/5F77283D" Ref="#PWR0188"  Part="1"
 AR Path="/5F7A4E71/5F77283D" Ref="#PWR0192"  Part="1"
-F 0 "#PWR0192" H 3500 3600 50  0001 C CNN
+F 0 "#PWR0180" H 3500 3600 50  0001 C CNN
 F 1 "+VSW" H 3515 3923 50  0000 C CNN
 F 2 "" H 3500 3750 50  0001 C CNN
@@
 AR Path="/5F7A3A2A/5F773E85" Ref="#PWR0189"  Part="1"
 AR Path="/5F7A4E71/5F773E85" Ref="#PWR0193"  Part="1"
-F 0 "#PWR0193" H 3750 3950 50  0001 C CNN
+F 0 "#PWR0181" H 3750 3950 50  0001 C CNN
 F 1 "GND" H 3755 4027 50  0000 C CNN
 F 2 "" H 3750 4200 50  0001 C CNN
@@
 AR Path="/5F7A3A2A/5F73738F" Ref="V9"  Part="1"
 AR Path="/5F7A4E71/5F73738F" Ref="V11"  Part="1"
-F 0 "V11" H 5755 3646 50  0000 L CNN
+F 0 "V5" H 5755 3646 50  0000 L CNN
 F 1 "CRSS042N10N" H 5755 3555 50  0000 L CNN
 F 2 "Package_TO_SOT_SMD:TO-263-2" H 5750 3525 50  0001 L CIN
@@
 AR Path="/5F7A3A2A/5F72B1D2" Ref="R32"  Part="1"
 AR Path="/5F7A4E71/5F72B1D2" Ref="R34"  Part="1"
-F 0 "R34" V 4993 3600 50  0000 C CNN
+F 0 "R17" V 4993 3600 50  0000 C CNN
 F 1 "68" V 5084 3600 50  0000 C CNN
 F 2 "Resistor_SMD:R_1206_3216Metric" V 5130 3600 50  0001 C CNN
@@
 AR Path="/5F7A3A2A/5F771122" Ref="U12"  Part="1"
 AR Path="/5F7A4E71/5F771122" Ref="U13"  Part="1"
-F 0 "U13" H 3950 3981 50  0000 C CNN
+F 0 "U10" H 3950 3981 50  0000 C CNN
 F 1 "IRS2304" H 3950 3890 50  0000 C CNN
 F 2 "Package_SO:SOIC-8_3.9x4.9mm_P1.27mm" H 3950 3300 50  0001 C CIN
@@
 AR Path="/5F7A3A2A/5F7824C8" Ref="R28"  Part="1"
 AR Path="/5F7A4E71/5F7824C8" Ref="R33"  Part="1"
-F 0 "R33" V 4993 3100 50  0000 C CNN
+F 0 "R16" V 4993 3100 50  0000 C CNN
 F 1 "68" V 5084 3100 50  0000 C CNN
 F 2 "Resistor_SMD:R_1206_3216Metric" V 5130 3100 50  0001 C CNN
@@
 AR Path="/5F7A3A2A/5F70E4C5" Ref="V8"  Part="1"
 AR Path="/5F7A4E71/5F70E4C5" Ref="V10"  Part="1"
-F 0 "V10" H 5755 3146 50  0000 L CNN
+F 0 "V4" H 5755 3146 50  0000 L CNN
 F 1 "CRSS042N10N" H 5755 3055 50  0000 L CNN
 F 2 "Package_TO_SOT_SMD:TO-263-2" H 5750 3025 50  0001 L CIN
@@
 AR Path="/5F7A3A2A/5F79127D" Ref="#PWR0190"  Part="1"
 AR Path="/5F7A4E71/5F79127D" Ref="#PWR0194"  Part="1"
-F 0 "#PWR0194" H 5650 2650 50  0001 C CNN
+F 0 "#PWR0182" H 5650 2650 50  0001 C CNN
 F 1 "+BATT" H 5665 2973 50  0000 C CNN
 F 2 "" H 5650 2800 50  0001 C CNN
@@
 AR Path="/5F7A3A2A/5F7BE8FF" Ref="C35"  Part="1"
 AR Path="/5F7A4E71/5F7BE8FF" Ref="C36"  Part="1"
-F 0 "C36" H 7218 3046 50  0000 L CNN
+F 0 "C33" H 7218 3046 50  0000 L CNN
 F 1 "47u LKMD0901K470MF" H 7218 2955 50  0000 L CNN
 F 2 "Capacitor_THT:CP_Radial_D8.0mm_P3.50mm" H 7138 2850 50  0001 C CNN
@@
 AR Path="/5F7A3A2A/5F7BF207" Ref="#PWR0201"  Part="1"
 AR Path="/5F7A4E71/5F7BF207" Ref="#PWR0202"  Part="1"
-F 0 "#PWR0202" H 7100 2650 50  0001 C CNN
+F 0 "#PWR0199" H 7100 2650 50  0001 C CNN
 F 1 "+BATT" H 7115 2973 50  0000 C CNN
 F 2 "" H 7100 2800 50  0001 C CNN
@@
 AR Path="/5F7A3A2A/5F72BDA4" Ref="D27"  Part="1"
 AR Path="/5F7A4E71/5F72BDA4" Ref="D28"  Part="1"
-F 0 "D28" V 8154 3080 50  0000 L CNN
+F 0 "D25" V 8154 3080 50  0000 L CNN
 F 1 "51V TVS C310059" V 8245 3080 50  0000 L CNN
 F 2 "Diode_SMD:D_SMC" H 8200 3000 50  0001 C CNN

Commit message: added TVS diodes on HALL inputs
Changed lines of the file:
@@
 $Descr A4 11693 8268
 encoding utf-8
-Sheet 10 14
+Sheet 8 14
 Title ""
 Date ""
@@
 AR Path="/5F7A3A2A/5F706578" Ref="C17"  Part="1"
 AR Path="/5F7A4E71/5F706578" Ref="C24"  Part="1"
-F 0 "C13" H 4618 3346 50  0000 L CNN
+F 0 "C24" H 4618 3346 50  0000 L CNN
 F 1 "47u LKMD0901K470MF" H 4618 3255 50  0000 L CNN
 F 2 "Capacitor_THT:CP_Radial_D8.0mm_P3.50mm" H 4538 3150 50  0001 C CNN
@@
 AR Path="/5F7A3A2A/5F707CCD" Ref="D10"  Part="1"
 AR Path="/5F7A4E71/5F707CCD" Ref="D11"  Part="1"
-F 0 "D8" H 4300 2284 50  0000 C CNN
+F 0 "D11" H 4300 2284 50  0000 C CNN
 F 1 "1N4148W" H 4300 2375 50  0000 C CNN
 F 2 "Diode_SMD:D_SOD-123" H 4300 2500 50  0001 C CNN
@@
 AR Path="/5F7A3A2A/5F77195C" Ref="#PWR0187"  Part="1"
 AR Path="/5F7A4E71/5F77195C" Ref="#PWR0191"  Part="1"
-F 0 "#PWR0179" H 3950 2250 50  0001 C CNN
+F 0 "#PWR0191" H 3950 2250 50  0001 C CNN
 F 1 "+VSW" H 3965 2573 50  0000 C CNN
 F 2 "" H 3950 2400 50  0001 C CNN
@@
 AR Path="/5F7A3A2A/5F771CDC" Ref="C16"  Part="1"
 AR Path="/5F7A4E71/5F771CDC" Ref="C18"  Part="1"
-F 0 "C12" H 3618 3996 50  0000 L CNN
+F 0 "C18" H 3618 3996 50  0000 L CNN
 F 1 "220u25V LKMD0901E221MF" H 3618 3905 50  0000 L CNN
 F 2 "Capacitor_THT:CP_Radial_D8.0mm_P3.50mm" H 3538 3800 50  0001 C CNN
@@
 AR Path="/5F7A3A2A/5F77283D" Ref="#PWR0188"  Part="1"
 AR Path="/5F7A4E71/5F77283D" Ref="#PWR0192"  Part="1"
-F 0 "#PWR0180" H 3500 3600 50  0001 C CNN
+F 0 "#PWR0192" H 3500 3600 50  0001 C CNN
 F 1 "+VSW" H 3515 3923 50  0000 C CNN
 F 2 "" H 3500 3750 50  0001 C CNN
@@
 Wire Wire Line
 	3500 3800 3500 3750
-Wire Wire Line
-	3500 4150 3750 4150
 $Comp
 L power:GND #PWR0173
 U 1 1 5F773E85
-P 3750 4200
+P 3850 4150
 AR Path="/5F7ECC6C/5F773E85" Ref="#PWR0173"  Part="1"
 AR Path="/5F79FFE4/5F773E85" Ref="#PWR0177"  Part="1"
@@
 AR Path="/5F7A3A2A/5F773E85" Ref="#PWR0189"  Part="1"
 AR Path="/5F7A4E71/5F773E85" Ref="#PWR0193"  Part="1"
-F 0 "#PWR0181" H 3750 3950 50  0001 C CNN
-F 1 "GND" H 3755 4027 50  0000 C CNN
-F 2 "" H 3750 4200 50  0001 C CNN
-F 3 "" H 3750 4200 50  0001 C CNN
-	1    3750 4200
-	1    0    0    -1
-$EndComp
-Connection ~ 3750 4150
-Wire Wire Line
-	3750 4150 3950 4150
+F 0 "#PWR0193" H 3850 3900 50  0001 C CNN
+F 1 "GND" H 3855 3977 50  0000 C CNN
+F 2 "" H 3850 4150 50  0001 C CNN
+F 3 "" H 3850 4150 50  0001 C CNN
+	1    3850 4150
+	1    0    0    -1
+$EndComp
 Wire Wire Line
 	3950 2400 3950 2500
@@
 AR Path="/5F7A3A2A/5F73738F" Ref="V9"  Part="1"
 AR Path="/5F7A4E71/5F73738F" Ref="V11"  Part="1"
-F 0 "V5" H 5755 3646 50  0000 L CNN
+F 0 "V11" H 5755 3646 50  0000 L CNN
 F 1 "CRSS042N10N" H 5755 3555 50  0000 L CNN
 F 2 "Package_TO_SOT_SMD:TO-263-2" H 5750 3525 50  0001 L CIN
@@
 AR Path="/5F7A3A2A/5F72B1D2" Ref="R32"  Part="1"
 AR Path="/5F7A4E71/5F72B1D2" Ref="R34"  Part="1"
-F 0 "R17" V 4993 3600 50  0000 C CNN
+F 0 "R34" V 4993 3600 50  0000 C CNN
 F 1 "68" V 5084 3600 50  0000 C CNN
 F 2 "Resistor_SMD:R_1206_3216Metric" V 5130 3600 50  0001 C CNN
@@
 AR Path="/5F7A3A2A/5F771122" Ref="U12"  Part="1"
 AR Path="/5F7A4E71/5F771122" Ref="U13"  Part="1"
-F 0 "U10" H 3950 3981 50  0000 C CNN
+F 0 "U13" H 3950 3981 50  0000 C CNN
 F 1 "IRS2304" H 3950 3890 50  0000 C CNN
 F 2 "Package_SO:SOIC-8_3.9x4.9mm_P1.27mm" H 3950 3300 50  0001 C CIN
@@
 AR Path="/5F7A3A2A/5F7824C8" Ref="R28"  Part="1"
 AR Path="/5F7A4E71/5F7824C8" Ref="R33"  Part="1"
-F 0 "R16" V 4993 3100 50  0000 C CNN
+F 0 "R33" V 4993 3100 50  0000 C CNN
 F 1 "68" V 5084 3100 50  0000 C CNN
 F 2 "Resistor_SMD:R_1206_3216Metric" V 5130 3100 50  0001 C CNN
@@
 AR Path="/5F7A3A2A/5F70E4C5" Ref="V8"  Part="1"
 AR Path="/5F7A4E71/5F70E4C5" Ref="V10"  Part="1"
-F 0 "V4" H 5755 3146 50  0000 L CNN
+F 0 "V10" H 5755 3146 50  0000 L CNN
 F 1 "CRSS042N10N" H 5755 3055 50  0000 L CNN
 F 2 "Package_TO_SOT_SMD:TO-263-2" H 5750 3025 50  0001 L CIN
@@
 AR Path="/5F7A3A2A/5F79127D" Ref="#PWR0190"  Part="1"
 AR Path="/5F7A4E71/5F79127D" Ref="#PWR0194"  Part="1"
-F 0 "#PWR0182" H 5650 2650 50  0001 C CNN
+F 0 "#PWR0194" H 5650 2650 50  0001 C CNN
 F 1 "+BATT" H 5665 2973 50  0000 C CNN
 F 2 "" H 5650 2800 50  0001 C CNN
@@
 AR Path="/5F7A3A2A/5F7BE8FF" Ref="C35"  Part="1"
 AR Path="/5F7A4E71/5F7BE8FF" Ref="C36"  Part="1"
-F 0 "C33" H 7218 3046 50  0000 L CNN
+F 0 "C36" H 7218 3046 50  0000 L CNN
 F 1 "47u LKMD0901K470MF" H 7218 2955 50  0000 L CNN
 F 2 "Capacitor_THT:CP_Radial_D8.0mm_P3.50mm" H 7138 2850 50  0001 C CNN
@@
 AR Path="/5F7A3A2A/5F7BF207" Ref="#PWR0201"  Part="1"
 AR Path="/5F7A4E71/5F7BF207" Ref="#PWR0202"  Part="1"
-F 0 "#PWR0199" H 7100 2650 50  0001 C CNN
+F 0 "#PWR0202" H 7100 2650 50  0001 C CNN
 F 1 "+BATT" H 7115 2973 50  0000 C CNN
 F 2 "" H 7100 2800 50  0001 C CNN
@@
 Wire Wire Line
 	4450 2500 4500 2500
-Wire Wire Line
-	3750 4150 3750 4200
 Wire Wire Line
 	3500 4100 3500 4150
@@
 AR Path="/5F7A3A2A/5F72BDA4" Ref="D27"  Part="1"
 AR Path="/5F7A4E71/5F72BDA4" Ref="D28"  Part="1"
-F 0 "D25" V 8154 3080 50  0000 L CNN
+F 0 "D28" V 8154 3080 50  0000 L CNN
 F 1 "51V TVS C310059" V 8245 3080 50  0000 L CNN
 F 2 "Diode_SMD:D_SMC" H 8200 3000 50  0001 C CNN
@@
 Wire Wire Line
 	7100 3350 7100 4050
+Connection ~ 3850 4150
+Wire Wire Line
+	3850 4150 3950 4150
+Wire Wire Line
+	3500 4150 3850 4150
 $EndSCHEMATC
