File: hh_bridge.sch (KiCad schematic (older format))
At the start: 10 parts, among them U8 IRS2304

Commit message: change Mosfet Driver to U3115S
Parts:
- added R50: DNP 10k, Resistor_SMD:R_1206_3216Metric, symbol Device:R
- added R51: 10k IRF->DNP, Resistor_SMD:R_1206_3216Metric, symbol Device:R
- R10, R13: value 68 -> 20k
- U8: value IRS2304 -> IRS2304 || U3115S
Connections:
- net H_BRIDGE_GND: now also R51.1
- net MOTOR_PHASE: now also R50.1
- net at R10.2, U8.5 (LO): now also R51.2
- net at R13.2, U8.7 (HO): now also R50.2
Changed lines of the file:
@@
 $Descr A4 11693 8268
 encoding utf-8
-Sheet 9 14
+Sheet 10 14
 Title ""
 Date ""
@@
 AR Path="/5F7A3A2A/5F706578" Ref="C17"  Part="1"
 AR Path="/5F7A4E71/5F706578" Ref="C24"  Part="1"
-F 0 "C24" H 4618 3346 50  0000 L CNN
+F 0 "C13" H 4618 3346 50  0000 L CNN
 F 1 "47u LKMD0901K470MF" H 4618 3255 50  0000 L CNN
 F 2 "Capacitor_THT:CP_Radial_D8.0mm_P3.50mm" H 4538 3150 50  0001 C CNN
@@
 AR Path="/5F7A3A2A/5F707CCD" Ref="D10"  Part="1"
 AR Path="/5F7A4E71/5F707CCD" Ref="D11"  Part="1"
-F 0 "D11" H 4300 2284 50  0000 C CNN
+F 0 "D8" H 4300 2284 50  0000 C CNN
 F 1 "1N4148W" H 4300 2375 50  0000 C CNN
 F 2 "Diode_SMD:D_SOD-123" H 4300 2500 50  0001 C CNN
@@
 AR Path="/5F7A3A2A/5F771CDC" Ref="C16"  Part="1"
 AR Path="/5F7A4E71/5F771CDC" Ref="C18"  Part="1"
-F 0 "C18" H 3618 3996 50  0000 L CNN
+F 0 "C12" H 3618 3996 50  0000 L CNN
 F 1 "220u25V LKMD0901E221MF" H 3618 3905 50  0000 L CNN
 F 2 "Capacitor_THT:CP_Radial_D8.0mm_P3.50mm" H 3538 3800 50  0001 C CNN
@@
 AR Path="/5F7A3A2A/5F73738F" Ref="V9"  Part="1"
 AR Path="/5F7A4E71/5F73738F" Ref="V11"  Part="1"
-F 0 "V11" H 5755 3646 50  0000 L CNN
+F 0 "V5" H 5755 3646 50  0000 L CNN
 F 1 "CRSS042N10N" H 5755 3555 50  0000 L CNN
 F 2 "Package_TO_SOT_SMD:TO-263-2" H 5750 3525 50  0001 L CIN
@@
 AR Path="/5F7A3A2A/5F72B1D2" Ref="R32"  Part="1"
 AR Path="/5F7A4E71/5F72B1D2" Ref="R34"  Part="1"
-F 0 "R34" V 4993 3600 50  0000 C CNN
-F 1 "68" V 5084 3600 50  0000 C CNN
+F 0 "R17" V 4993 3600 50  0000 C CNN
+F 1 "20k" V 5084 3600 50  0000 C CNN
 F 2 "Resistor_SMD:R_1206_3216Metric" V 5130 3600 50  0001 C CNN
 F 3 "~" H 5200 3600 50  0001 C CNN
@@
 AR Path="/5F7A3A2A/5F771122" Ref="U12"  Part="1"
 AR Path="/5F7A4E71/5F771122" Ref="U13"  Part="1"
-F 0 "U13" H 3950 3981 50  0000 C CNN
-F 1 "IRS2304" H 3950 3890 50  0000 C CNN
+F 0 "U10" H 3950 3981 50  0000 C CNN
+F 1 "IRS2304 || U3115S" H 3950 3890 50  0000 C CNN
 F 2 "Package_SO:SOIC-8_3.9x4.9mm_P1.27mm" H 3950 3300 50  0001 C CIN
 F 3 "https://www.infineon.com/dgdl/irs2304spbf.pdf?fileId=5546d462533600a40153567a8fe72802" H 3950 3300 50  0001 C CNN
@@
 AR Path="/5F7A3A2A/5F7824C8" Ref="R28"  Part="1"
 AR Path="/5F7A4E71/5F7824C8" Ref="R33"  Part="1"
-F 0 "R33" V 4993 3100 50  0000 C CNN
-F 1 "68" V 5084 3100 50  0000 C CNN
+F 0 "R16" V 4993 3100 50  0000 C CNN
+F 1 "20k" V 5084 3100 50  0000 C CNN
 F 2 "Resistor_SMD:R_1206_3216Metric" V 5130 3100 50  0001 C CNN
 F 3 "~" H 5200 3100 50  0001 C CNN
@@
 AR Path="/5F7A3A2A/5F70E4C5" Ref="V8"  Part="1"
 AR Path="/5F7A4E71/5F70E4C5" Ref="V10"  Part="1"
-F 0 "V10" H 5755 3146 50  0000 L CNN
+F 0 "V4" H 5755 3146 50  0000 L CNN
 F 1 "CRSS042N10N" H 5755 3055 50  0000 L CNN
 F 2 "Package_TO_SOT_SMD:TO-263-2" H 5750 3025 50  0001 L CIN
@@
 $EndComp
 Wire Wire Line
-	4250 3600 5050 3600
-Wire Wire Line
-	5050 3100 4250 3100
+	4250 3600 4950 3600
 Wire Wire Line
 	5650 3300 5650 3350
@@
 	1    0    0    -1
 $EndComp
-Wire Wire Line
-	6300 3350 5650 3350
 Connection ~ 5650 3350
 Wire Wire Line
 	5650 3350 5650 3400
-Wire Wire Line
-	6300 3850 5650 3850
 $Comp
 L Device:CP C31
@@
 AR Path="/5F7A3A2A/5F7BE8FF" Ref="C35"  Part="1"
 AR Path="/5F7A4E71/5F7BE8FF" Ref="C36"  Part="1"
-F 0 "C36" H 7218 3046 50  0000 L CNN
+F 0 "C33" H 7218 3046 50  0000 L CNN
 F 1 "47u LKMD0901K470MF" H 7218 2955 50  0000 L CNN
 F 2 "Capacitor_THT:CP_Radial_D8.0mm_P3.50mm" H 7138 2850 50  0001 C CNN
@@
 	7100 4050 5650 4050
 Wire Wire Line
-	5650 4050 5650 3850
+	5650 4050 5650 3900
 Wire Wire Line
 	5500 3500 5500 3350
@@
 Connection ~ 4500 3500
 Wire Wire Line
-	4500 3500 5500 3500
+	4500 3500 4850 3500
 Connection ~ 5650 3850
 Wire Wire Line
@@
 AR Path="/5F7A3A2A/5F72BDA4" Ref="D27"  Part="1"
 AR Path="/5F7A4E71/5F72BDA4" Ref="D28"  Part="1"
-F 0 "D28" V 8154 3080 50  0000 L CNN
+F 0 "D25" V 8154 3080 50  0000 L CNN
 F 1 "51V TVS C310059" V 8245 3080 50  0000 L CNN
 F 2 "Diode_SMD:D_SMC" H 8200 3000 50  0001 C CNN
@@
 Wire Wire Line
 	3500 4150 3850 4150
+$Comp
+L Device:R R51
+U 1 1 5F76BFEE
+P 4950 3750
+AR Path="/5F7ECC6C/5F76BFEE" Ref="R51"  Part="1"
+AR Path="/5F79FFE4/5F76BFEE" Ref="R58"  Part="1"
+AR Path="/5F7A0EEE/5F76BFEE" Ref="R61"  Part="1"
+AR Path="/5F7A2640/5F76BFEE" Ref="R64"  Part="1"
+AR Path="/5F7A3A2A/5F76BFEE" Ref="R67"  Part="1"
+AR Path="/5F7A4E71/5F76BFEE" Ref="R70"  Part="1"
+F 0 "R61" V 4743 3750 50  0000 C CNN
+F 1 "10k IRF->DNP" V 4834 3750 50  0000 C CNN
+F 2 "Resistor_SMD:R_1206_3216Metric" V 4880 3750 50  0001 C CNN
+F 3 "~" H 4950 3750 50  0001 C CNN
+	1    4950 3750
+	-1   0    0    1
+$EndComp
+Connection ~ 4950 3600
+Wire Wire Line
+	4950 3600 5050 3600
+Wire Wire Line
+	5650 3900 4950 3900
+Connection ~ 5650 3900
+Wire Wire Line
+	5650 3900 5650 3850
+$Comp
+L Device:R R50
+U 1 1 5F76CC5E
+P 4850 3300
+AR Path="/5F7ECC6C/5F76CC5E" Ref="R50"  Part="1"
+AR Path="/5F79FFE4/5F76CC5E" Ref="R57"  Part="1"
+AR Path="/5F7A0EEE/5F76CC5E" Ref="R60"  Part="1"
+AR Path="/5F7A2640/5F76CC5E" Ref="R63"  Part="1"
+AR Path="/5F7A3A2A/5F76CC5E" Ref="R66"  Part="1"
+AR Path="/5F7A4E71/5F76CC5E" Ref="R69"  Part="1"
+F 0 "R60" V 4643 3300 50  0000 C CNN
+F 1 "DNP 10k" V 4734 3300 50  0000 C CNN
+F 2 "Resistor_SMD:R_1206_3216Metric" V 4780 3300 50  0001 C CNN
+F 3 "~" H 4850 3300 50  0001 C CNN
+	1    4850 3300
+	-1   0    0    1
+$EndComp
+Wire Wire Line
+	5650 3850 6300 3850
+Wire Wire Line
+	5650 3350 6300 3350
+Wire Wire Line
+	4250 3100 4850 3100
+Wire Wire Line
+	4850 3450 4850 3500
+Connection ~ 4850 3500
+Wire Wire Line
+	4850 3500 5500 3500
+Wire Wire Line
+	4850 3150 4850 3100
+Connection ~ 4850 3100
+Wire Wire Line
+	4850 3100 5050 3100
 $EndSCHEMATC

Commit message: add silk screen, change diodes at DCDC converters, remove overcurrent detection, add 100nf
Changed lines of the file:
@@
 AR Path="/5F7A3A2A/5F706578" Ref="C17"  Part="1"
 AR Path="/5F7A4E71/5F706578" Ref="C24"  Part="1"
-F 0 "C13" H 4618 3346 50  0000 L CNN
+F 0 "C24" H 4618 3346 50  0000 L CNN
 F 1 "47u LKMD0901K470MF" H 4618 3255 50  0000 L CNN
 F 2 "Capacitor_THT:CP_Radial_D8.0mm_P3.50mm" H 4538 3150 50  0001 C CNN
@@
 AR Path="/5F7A3A2A/5F707CCD" Ref="D10"  Part="1"
 AR Path="/5F7A4E71/5F707CCD" Ref="D11"  Part="1"
-F 0 "D8" H 4300 2284 50  0000 C CNN
+F 0 "D11" H 4300 2284 50  0000 C CNN
 F 1 "1N4148W" H 4300 2375 50  0000 C CNN
 F 2 "Diode_SMD:D_SOD-123" H 4300 2500 50  0001 C CNN
@@
 AR Path="/5F7A3A2A/5F771CDC" Ref="C16"  Part="1"
 AR Path="/5F7A4E71/5F771CDC" Ref="C18"  Part="1"
-F 0 "C12" H 3618 3996 50  0000 L CNN
+F 0 "C18" H 3618 3996 50  0000 L CNN
 F 1 "220u25V LKMD0901E221MF" H 3618 3905 50  0000 L CNN
 F 2 "Capacitor_THT:CP_Radial_D8.0mm_P3.50mm" H 3538 3800 50  0001 C CNN
@@
 AR Path="/5F7A3A2A/5F73738F" Ref="V9"  Part="1"
 AR Path="/5F7A4E71/5F73738F" Ref="V11"  Part="1"
-F 0 "V5" H 5755 3646 50  0000 L CNN
+F 0 "V11" H 5755 3646 50  0000 L CNN
 F 1 "CRSS042N10N" H 5755 3555 50  0000 L CNN
 F 2 "Package_TO_SOT_SMD:TO-263-2" H 5750 3525 50  0001 L CIN
@@
 AR Path="/5F7A3A2A/5F72B1D2" Ref="R32"  Part="1"
 AR Path="/5F7A4E71/5F72B1D2" Ref="R34"  Part="1"
-F 0 "R17" V 4993 3600 50  0000 C CNN
+F 0 "R34" V 4993 3600 50  0000 C CNN
 F 1 "20k" V 5084 3600 50  0000 C CNN
 F 2 "Resistor_SMD:R_1206_3216Metric" V 5130 3600 50  0001 C CNN
@@
 AR Path="/5F7A3A2A/5F771122" Ref="U12"  Part="1"
 AR Path="/5F7A4E71/5F771122" Ref="U13"  Part="1"
-F 0 "U10" H 3950 3981 50  0000 C CNN
+F 0 "U13" H 3950 3981 50  0000 C CNN
 F 1 "IRS2304 || U3115S" H 3950 3890 50  0000 C CNN
 F 2 "Package_SO:SOIC-8_3.9x4.9mm_P1.27mm" H 3950 3300 50  0001 C CIN
@@
 AR Path="/5F7A3A2A/5F7824C8" Ref="R28"  Part="1"
 AR Path="/5F7A4E71/5F7824C8" Ref="R33"  Part="1"
-F 0 "R16" V 4993 3100 50  0000 C CNN
+F 0 "R33" V 4993 3100 50  0000 C CNN
 F 1 "20k" V 5084 3100 50  0000 C CNN
 F 2 "Resistor_SMD:R_1206_3216Metric" V 5130 3100 50  0001 C CNN
@@
 AR Path="/5F7A3A2A/5F70E4C5" Ref="V8"  Part="1"
 AR Path="/5F7A4E71/5F70E4C5" Ref="V10"  Part="1"
-F 0 "V4" H 5755 3146 50  0000 L CNN
+F 0 "V10" H 5755 3146 50  0000 L CNN
 F 1 "CRSS042N10N" H 5755 3055 50  0000 L CNN
 F 2 "Package_TO_SOT_SMD:TO-263-2" H 5750 3025 50  0001 L CIN
@@
 AR Path="/5F7A3A2A/5F7BE8FF" Ref="C35"  Part="1"
 AR Path="/5F7A4E71/5F7BE8FF" Ref="C36"  Part="1"
-F 0 "C33" H 7218 3046 50  0000 L CNN
+F 0 "C36" H 7218 3046 50  0000 L CNN
 F 1 "47u LKMD0901K470MF" H 7218 2955 50  0000 L CNN
 F 2 "Capacitor_THT:CP_Radial_D8.0mm_P3.50mm" H 7138 2850 50  0001 C CNN
@@
 AR Path="/5F7A3A2A/5F72BDA4" Ref="D27"  Part="1"
 AR Path="/5F7A4E71/5F72BDA4" Ref="D28"  Part="1"
-F 0 "D25" V 8154 3080 50  0000 L CNN
+F 0 "D28" V 8154 3080 50  0000 L CNN
 F 1 "51V TVS C310059" V 8245 3080 50  0000 L CNN
 F 2 "Diode_SMD:D_SMC" H 8200 3000 50  0001 C CNN
@@
 AR Path="/5F7A3A2A/5F76BFEE" Ref="R67"  Part="1"
 AR Path="/5F7A4E71/5F76BFEE" Ref="R70"  Part="1"
-F 0 "R61" V 4743 3750 50  0000 C CNN
+F 0 "R70" V 4743 3750 50  0000 C CNN
 F 1 "10k IRF->DNP" V 4834 3750 50  0000 C CNN
 F 2 "Resistor_SMD:R_1206_3216Metric" V 4880 3750 50  0001 C CNN
@@
 AR Path="/5F7A3A2A/5F76CC5E" Ref="R66"  Part="1"
 AR Path="/5F7A4E71/5F76CC5E" Ref="R69"  Part="1"
-F 0 "R60" V 4643 3300 50  0000 C CNN
+F 0 "R69" V 4643 3300 50  0000 C CNN
 F 1 "DNP 10k" V 4734 3300 50  0000 C CNN
 F 2 "Resistor_SMD:R_1206_3216Metric" V 4780 3300 50  0001 C CNN

Commit message: fix labels
Changed lines of the file:
@@
 $Descr A4 11693 8268
 encoding utf-8
-Sheet 10 14
+Sheet 8 14
 Title ""
 Date ""
@@
 AR Path="/5F7A3A2A/5F706578" Ref="C17"  Part="1"
 AR Path="/5F7A4E71/5F706578" Ref="C24"  Part="1"
-F 0 "C24" H 4618 3346 50  0000 L CNN
+F 0 "C1" H 4618 3346 50  0000 L CNN
 F 1 "47u LKMD0901K470MF" H 4618 3255 50  0000 L CNN
 F 2 "Capacitor_THT:CP_Radial_D8.0mm_P3.50mm" H 4538 3150 50  0001 C CNN
@@
 AR Path="/5F7A3A2A/5F707CCD" Ref="D10"  Part="1"
 AR Path="/5F7A4E71/5F707CCD" Ref="D11"  Part="1"
-F 0 "D11" H 4300 2284 50  0000 C CNN
+F 0 "D1" H 4300 2284 50  0000 C CNN
 F 1 "1N4148W" H 4300 2375 50  0000 C CNN
 F 2 "Diode_SMD:D_SOD-123" H 4300 2500 50  0001 C CNN
@@
 AR Path="/5F7A3A2A/5F77195C" Ref="#PWR0187"  Part="1"
 AR Path="/5F7A4E71/5F77195C" Ref="#PWR0191"  Part="1"
-F 0 "#PWR0191" H 3950 2250 50  0001 C CNN
+F 0 "#PWR0171" H 3950 2250 50  0001 C CNN
 F 1 "+VSW" H 3965 2573 50  0000 C CNN
 F 2 "" H 3950 2400 50  0001 C CNN
@@
 AR Path="/5F7A3A2A/5F771CDC" Ref="C16"  Part="1"
 AR Path="/5F7A4E71/5F771CDC" Ref="C18"  Part="1"
-F 0 "C18" H 3618 3996 50  0000 L CNN
+F 0 "C8" H 3618 3996 50  0000 L CNN
 F 1 "220u25V LKMD0901E221MF" H 3618 3905 50  0000 L CNN
 F 2 "Capacitor_THT:CP_Radial_D8.0mm_P3.50mm" H 3538 3800 50  0001 C CNN
@@
 AR Path="/5F7A3A2A/5F77283D" Ref="#PWR0188"  Part="1"
 AR Path="/5F7A4E71/5F77283D" Ref="#PWR0192"  Part="1"
-F 0 "#PWR0192" H 3500 3600 50  0001 C CNN
+F 0 "#PWR0172" H 3500 3600 50  0001 C CNN
 F 1 "+VSW" H 3515 3923 50  0000 C CNN
 F 2 "" H 3500 3750 50  0001 C CNN
@@
 AR Path="/5F7A3A2A/5F773E85" Ref="#PWR0189"  Part="1"
 AR Path="/5F7A4E71/5F773E85" Ref="#PWR0193"  Part="1"
-F 0 "#PWR0193" H 3850 3900 50  0001 C CNN
+F 0 "#PWR0173" H 3850 3900 50  0001 C CNN
 F 1 "GND" H 3855 3977 50  0000 C CNN
 F 2 "" H 3850 4150 50  0001 C CNN
@@
 AR Path="/5F7A3A2A/5F73738F" Ref="V9"  Part="1"
 AR Path="/5F7A4E71/5F73738F" Ref="V11"  Part="1"
-F 0 "V11" H 5755 3646 50  0000 L CNN
+F 0 "V1" H 5755 3646 50  0000 L CNN
 F 1 "CRSS042N10N" H 5755 3555 50  0000 L CNN
 F 2 "Package_TO_SOT_SMD:TO-263-2" H 5750 3525 50  0001 L CIN
@@
 AR Path="/5F7A3A2A/5F72B1D2" Ref="R32"  Part="1"
 AR Path="/5F7A4E71/5F72B1D2" Ref="R34"  Part="1"
-F 0 "R34" V 4993 3600 50  0000 C CNN
+F 0 "R10" V 4993 3600 50  0000 C CNN
 F 1 "20k" V 5084 3600 50  0000 C CNN
 F 2 "Resistor_SMD:R_1206_3216Metric" V 5130 3600 50  0001 C CNN
@@
 AR Path="/5F7A3A2A/5F771122" Ref="U12"  Part="1"
 AR Path="/5F7A4E71/5F771122" Ref="U13"  Part="1"
-F 0 "U13" H 3950 3981 50  0000 C CNN
+F 0 "U8" H 3950 3981 50  0000 C CNN
 F 1 "IRS2304 || U3115S" H 3950 3890 50  0000 C CNN
 F 2 "Package_SO:SOIC-8_3.9x4.9mm_P1.27mm" H 3950 3300 50  0001 C CIN
@@
 AR Path="/5F7A3A2A/5F7824C8" Ref="R28"  Part="1"
 AR Path="/5F7A4E71/5F7824C8" Ref="R33"  Part="1"
-F 0 "R33" V 4993 3100 50  0000 C CNN
+F 0 "R13" V 4993 3100 50  0000 C CNN
 F 1 "20k" V 5084 3100 50  0000 C CNN
 F 2 "Resistor_SMD:R_1206_3216Metric" V 5130 3100 50  0001 C CNN
@@
 AR Path="/5F7A3A2A/5F70E4C5" Ref="V8"  Part="1"
 AR Path="/5F7A4E71/5F70E4C5" Ref="V10"  Part="1"
-F 0 "V10" H 5755 3146 50  0000 L CNN
+F 0 "V0" H 5755 3146 50  0000 L CNN
 F 1 "CRSS042N10N" H 5755 3055 50  0000 L CNN
 F 2 "Package_TO_SOT_SMD:TO-263-2" H 5750 3025 50  0001 L CIN
@@
 AR Path="/5F7A3A2A/5F79127D" Ref="#PWR0190"  Part="1"
 AR Path="/5F7A4E71/5F79127D" Ref="#PWR0194"  Part="1"
-F 0 "#PWR0194" H 5650 2650 50  0001 C CNN
+F 0 "#PWR0174" H 5650 2650 50  0001 C CNN
 F 1 "+BATT" H 5665 2973 50  0000 C CNN
 F 2 "" H 5650 2800 50  0001 C CNN
@@
 AR Path="/5F7A3A2A/5F7BE8FF" Ref="C35"  Part="1"
 AR Path="/5F7A4E71/5F7BE8FF" Ref="C36"  Part="1"
-F 0 "C36" H 7218 3046 50  0000 L CNN
+F 0 "C31" H 7218 3046 50  0000 L CNN
 F 1 "47u LKMD0901K470MF" H 7218 2955 50  0000 L CNN
 F 2 "Capacitor_THT:CP_Radial_D8.0mm_P3.50mm" H 7138 2850 50  0001 C CNN
@@
 AR Path="/5F7A3A2A/5F7BF207" Ref="#PWR0201"  Part="1"
 AR Path="/5F7A4E71/5F7BF207" Ref="#PWR0202"  Part="1"
-F 0 "#PWR0202" H 7100 2650 50  0001 C CNN
+F 0 "#PWR0197" H 7100 2650 50  0001 C CNN
 F 1 "+BATT" H 7115 2973 50  0000 C CNN
 F 2 "" H 7100 2800 50  0001 C CNN
@@
 AR Path="/5F7A3A2A/5F72BDA4" Ref="D27"  Part="1"
 AR Path="/5F7A4E71/5F72BDA4" Ref="D28"  Part="1"
-F 0 "D28" V 8154 3080 50  0000 L CNN
+F 0 "D23" V 8154 3080 50  0000 L CNN
 F 1 "51V TVS C310059" V 8245 3080 50  0000 L CNN
 F 2 "Diode_SMD:D_SMC" H 8200 3000 50  0001 C CNN
@@
 AR Path="/5F7A3A2A/5F76BFEE" Ref="R67"  Part="1"
 AR Path="/5F7A4E71/5F76BFEE" Ref="R70"  Part="1"
-F 0 "R70" V 4743 3750 50  0000 C CNN
+F 0 "R51" V 4743 3750 50  0000 C CNN
 F 1 "10k IRF->DNP" V 4834 3750 50  0000 C CNN
 F 2 "Resistor_SMD:R_1206_3216Metric" V 4880 3750 50  0001 C CNN
@@
 AR Path="/5F7A3A2A/5F76CC5E" Ref="R66"  Part="1"
 AR Path="/5F7A4E71/5F76CC5E" Ref="R69"  Part="1"
-F 0 "R69" V 4643 3300 50  0000 C CNN
+F 0 "R50" V 4643 3300 50  0000 C CNN
 F 1 "DNP 10k" V 4734 3300 50  0000 C CNN
 F 2 "Resistor_SMD:R_1206_3216Metric" V 4780 3300 50  0001 C CNN

Commit message: added capacitors
Parts:
- added C64: 2.2u 100V, Capacitor_SMD:C_1206_3216Metric, symbol Device:C
Connections:
- net +BATT: now also C64.1
- net H_BRIDGE_GND: now also C64.2
Changed lines of the file:
@@
 $Descr A4 11693 8268
 encoding utf-8
-Sheet 8 14
+Sheet 11 14
 Title ""
 Date ""
@@
 AR Path="/5F7A3A2A/5F706578" Ref="C17"  Part="1"
 AR Path="/5F7A4E71/5F706578" Ref="C24"  Part="1"
-F 0 "C1" H 4618 3346 50  0000 L CNN
+F 0 "C15" H 4618 3346 50  0000 L CNN
 F 1 "47u LKMD0901K470MF" H 4618 3255 50  0000 L CNN
 F 2 "Capacitor_THT:CP_Radial_D8.0mm_P3.50mm" H 4538 3150 50  0001 C CNN
@@
 AR Path="/5F7A3A2A/5F707CCD" Ref="D10"  Part="1"
 AR Path="/5F7A4E71/5F707CCD" Ref="D11"  Part="1"
-F 0 "D1" H 4300 2284 50  0000 C CNN
+F 0 "D9" H 4300 2284 50  0000 C CNN
 F 1 "1N4148W" H 4300 2375 50  0000 C CNN
 F 2 "Diode_SMD:D_SOD-123" H 4300 2500 50  0001 C CNN
@@
 AR Path="/5F7A3A2A/5F77195C" Ref="#PWR0187"  Part="1"
 AR Path="/5F7A4E71/5F77195C" Ref="#PWR0191"  Part="1"
-F 0 "#PWR0171" H 3950 2250 50  0001 C CNN
+F 0 "#PWR0183" H 3950 2250 50  0001 C CNN
 F 1 "+VSW" H 3965 2573 50  0000 C CNN
 F 2 "" H 3950 2400 50  0001 C CNN
@@
 AR Path="/5F7A3A2A/5F771CDC" Ref="C16"  Part="1"
 AR Path="/5F7A4E71/5F771CDC" Ref="C18"  Part="1"
-F 0 "C8" H 3618 3996 50  0000 L CNN
+F 0 "C14" H 3618 3996 50  0000 L CNN
 F 1 "220u25V LKMD0901E221MF" H 3618 3905 50  0000 L CNN
 F 2 "Capacitor_THT:CP_Radial_D8.0mm_P3.50mm" H 3538 3800 50  0001 C CNN
@@
 AR Path="/5F7A3A2A/5F77283D" Ref="#PWR0188"  Part="1"
 AR Path="/5F7A4E71/5F77283D" Ref="#PWR0192"  Part="1"
-F 0 "#PWR0172" H 3500 3600 50  0001 C CNN
+F 0 "#PWR0184" H 3500 3600 50  0001 C CNN
 F 1 "+VSW" H 3515 3923 50  0000 C CNN
 F 2 "" H 3500 3750 50  0001 C CNN
@@
 AR Path="/5F7A3A2A/5F773E85" Ref="#PWR0189"  Part="1"
 AR Path="/5F7A4E71/5F773E85" Ref="#PWR0193"  Part="1"
-F 0 "#PWR0173" H 3850 3900 50  0001 C CNN
+F 0 "#PWR0185" H 3850 3900 50  0001 C CNN
 F 1 "GND" H 3855 3977 50  0000 C CNN
 F 2 "" H 3850 4150 50  0001 C CNN
@@
 AR Path="/5F7A3A2A/5F73738F" Ref="V9"  Part="1"
 AR Path="/5F7A4E71/5F73738F" Ref="V11"  Part="1"
-F 0 "V1" H 5755 3646 50  0000 L CNN
+F 0 "V7" H 5755 3646 50  0000 L CNN
 F 1 "CRSS042N10N" H 5755 3555 50  0000 L CNN
 F 2 "Package_TO_SOT_SMD:TO-263-2" H 5750 3525 50  0001 L CIN
@@
 AR Path="/5F7A3A2A/5F72B1D2" Ref="R32"  Part="1"
 AR Path="/5F7A4E71/5F72B1D2" Ref="R34"  Part="1"
-F 0 "R10" V 4993 3600 50  0000 C CNN
+F 0 "R21" V 4993 3600 50  0000 C CNN
 F 1 "20k" V 5084 3600 50  0000 C CNN
 F 2 "Resistor_SMD:R_1206_3216Metric" V 5130 3600 50  0001 C CNN
@@
 AR Path="/5F7A3A2A/5F771122" Ref="U12"  Part="1"
 AR Path="/5F7A4E71/5F771122" Ref="U13"  Part="1"
-F 0 "U8" H 3950 3981 50  0000 C CNN
+F 0 "U11" H 3950 3981 50  0000 C CNN
 F 1 "IRS2304 || U3115S" H 3950 3890 50  0000 C CNN
 F 2 "Package_SO:SOIC-8_3.9x4.9mm_P1.27mm" H 3950 3300 50  0001 C CIN
@@
 AR Path="/5F7A3A2A/5F7824C8" Ref="R28"  Part="1"
 AR Path="/5F7A4E71/5F7824C8" Ref="R33"  Part="1"
-F 0 "R13" V 4993 3100 50  0000 C CNN
+F 0 "R18" V 4993 3100 50  0000 C CNN
 F 1 "20k" V 5084 3100 50  0000 C CNN
 F 2 "Resistor_SMD:R_1206_3216Metric" V 5130 3100 50  0001 C CNN
@@
 AR Path="/5F7A3A2A/5F70E4C5" Ref="V8"  Part="1"
 AR Path="/5F7A4E71/5F70E4C5" Ref="V10"  Part="1"
-F 0 "V0" H 5755 3146 50  0000 L CNN
+F 0 "V6" H 5755 3146 50  0000 L CNN
 F 1 "CRSS042N10N" H 5755 3055 50  0000 L CNN
 F 2 "Package_TO_SOT_SMD:TO-263-2" H 5750 3025 50  0001 L CIN
@@
 AR Path="/5F7A3A2A/5F79127D" Ref="#PWR0190"  Part="1"
 AR Path="/5F7A4E71/5F79127D" Ref="#PWR0194"  Part="1"
-F 0 "#PWR0174" H 5650 2650 50  0001 C CNN
+F 0 "#PWR0186" H 5650 2650 50  0001 C CNN
 F 1 "+BATT" H 5665 2973 50  0000 C CNN
 F 2 "" H 5650 2800 50  0001 C CNN
@@
 AR Path="/5F7A3A2A/5F7BE8FF" Ref="C35"  Part="1"
 AR Path="/5F7A4E71/5F7BE8FF" Ref="C36"  Part="1"
-F 0 "C31" H 7218 3046 50  0000 L CNN
+F 0 "C34" H 7218 3046 50  0000 L CNN
 F 1 "47u LKMD0901K470MF" H 7218 2955 50  0000 L CNN
 F 2 "Capacitor_THT:CP_Radial_D8.0mm_P3.50mm" H 7138 2850 50  0001 C CNN
@@
 AR Path="/5F7A3A2A/5F7BF207" Ref="#PWR0201"  Part="1"
 AR Path="/5F7A4E71/5F7BF207" Ref="#PWR0202"  Part="1"
-F 0 "#PWR0197" H 7100 2650 50  0001 C CNN
+F 0 "#PWR0200" H 7100 2650 50  0001 C CNN
 F 1 "+BATT" H 7115 2973 50  0000 C CNN
 F 2 "" H 7100 2800 50  0001 C CNN
@@
 AR Path="/5F7A3A2A/5F72BDA4" Ref="D27"  Part="1"
 AR Path="/5F7A4E71/5F72BDA4" Ref="D28"  Part="1"
-F 0 "D23" V 8154 3080 50  0000 L CNN
+F 0 "D26" V 8154 3080 50  0000 L CNN
 F 1 "51V TVS C310059" V 8245 3080 50  0000 L CNN
 F 2 "Diode_SMD:D_SMC" H 8200 3000 50  0001 C CNN
@@
 AR Path="/5F7A3A2A/5F76BFEE" Ref="R67"  Part="1"
 AR Path="/5F7A4E71/5F76BFEE" Ref="R70"  Part="1"
-F 0 "R51" V 4743 3750 50  0000 C CNN
+F 0 "R64" V 4743 3750 50  0000 C CNN
 F 1 "10k IRF->DNP" V 4834 3750 50  0000 C CNN
 F 2 "Resistor_SMD:R_1206_3216Metric" V 4880 3750 50  0001 C CNN
@@
 AR Path="/5F7A3A2A/5F76CC5E" Ref="R66"  Part="1"
 AR Path="/5F7A4E71/5F76CC5E" Ref="R69"  Part="1"
-F 0 "R50" V 4643 3300 50  0000 C CNN
+F 0 "R63" V 4643 3300 50  0000 C CNN
 F 1 "DNP 10k" V 4734 3300 50  0000 C CNN
 F 2 "Resistor_SMD:R_1206_3216Metric" V 4780 3300 50  0001 C CNN
@@
 Wire Wire Line
 	4850 3100 5050 3100
+$Comp
+L Device:C C?
+U 1 1 5F784928
+P 6750 3000
+AR Path="/5F784928" Ref="C?"  Part="1"
+AR Path="/5F7ECC6C/5F784928" Ref="C64"  Part="1"
+AR Path="/5F79FFE4/5F784928" Ref="C65"  Part="1"
+AR Path="/5F7A0EEE/5F784928" Ref="C66"  Part="1"
+AR Path="/5F7A2640/5F784928" Ref="C67"  Part="1"
+AR Path="/5F7A3A2A/5F784928" Ref="C68"  Part="1"
+AR Path="/5F7A4E71/5F784928" Ref="C69"  Part="1"
+F 0 "C67" H 6865 3046 50  0000 L CNN
+F 1 "2.2u 100V" H 6865 2955 50  0000 L CNN
+F 2 "Capacitor_SMD:C_1206_3216Metric" H 6788 2850 50  0001 C CNN
+F 3 "~" H 6750 3000 50  0001 C CNN
+	1    6750 3000
+	1    0    0    -1
+$EndComp
+Wire Wire Line
+	6750 2800 6750 2850
+Wire Wire Line
+	6750 2800 7100 2800
+Wire Wire Line
+	6750 3150 7100 3150
+Connection ~ 7100 3150
 $EndSCHEMATC
