File: hh_bridge.sch (KiCad schematic (older format))
At the start: 13 parts, among them U8 IRS2304 || U3115S

Commit message: add resistors on mosfet driver inputs, change board corners, fix labels
Parts:
- added R72, R73: 1k, Resistor_SMD:R_0603_1608Metric, symbol Device:R
- R10, R13: value 20k -> IRF->100 U51->20
- R50: value DNP 10k -> 10k IRF->DNP
Connections:
- net H_BRIDGE_HI: now also R72.2; no longer U8.2 (HIN)
- net H_BRIDGE_LO: now also R73.2; no longer U8.1 (LIN)
- new net: R73.1, U8.1 (LIN)
- new net: R72.1, U8.2 (HIN)
Changed lines of the file:
@@
 Comment4 ""
 $EndDescr
-Text HLabel 3650 3300 0    50   Input ~ 0
+Text HLabel 3350 3300 0    50   Input ~ 0
 H_BRIDGE_HI
 $Comp
@@
 AR Path="/5F7A4E71/5F706578" Ref="C24"  Part="1"
 F 0 "C15" H 4618 3346 50  0000 L CNN
-F 1 "47u LKMD0901K470MF" H 4618 3255 50  0000 L CNN
+F 1 "47u LKMD0901K470MF" H 3900 3450 50  0000 L CNN
 F 2 "Capacitor_THT:CP_Radial_D8.0mm_P3.50mm" H 4538 3150 50  0001 C CNN
 F 3 "~" H 4500 3300 50  0001 C CNN
@@
 AR Path="/5F7A3A2A/5F707CCD" Ref="D10"  Part="1"
 AR Path="/5F7A4E71/5F707CCD" Ref="D11"  Part="1"
-F 0 "D9" H 4300 2284 50  0000 C CNN
-F 1 "1N4148W" H 4300 2375 50  0000 C CNN
+F 0 "D9" H 4300 2283 50  0000 C CNN
+F 1 "1N4148W" H 4300 2374 50  0000 C CNN
 F 2 "Diode_SMD:D_SOD-123" H 4300 2500 50  0001 C CNN
 F 3 "~" H 4300 2500 50  0001 C CNN
@@
 	-1   0    0    1
 $EndComp
-Text HLabel 3650 3400 0    50   Input ~ 0
+Text HLabel 3350 3400 0    50   Input ~ 0
 H_BRIDGE_LO
 Text HLabel 6300 3850 2    50   UnSpc ~ 0
@@
 AR Path="/5F7A3A2A/5F771CDC" Ref="C16"  Part="1"
 AR Path="/5F7A4E71/5F771CDC" Ref="C18"  Part="1"
-F 0 "C14" H 3618 3996 50  0000 L CNN
-F 1 "220u25V LKMD0901E221MF" H 3618 3905 50  0000 L CNN
+F 0 "C14" H 3382 3996 50  0000 R CNN
+F 1 "220u25V LKMD0901E221MF" H 3382 3905 50  0000 R CNN
 F 2 "Capacitor_THT:CP_Radial_D8.0mm_P3.50mm" H 3538 3800 50  0001 C CNN
 F 3 "~" H 3500 3950 50  0001 C CNN
@@
 AR Path="/5F7A3A2A/5F73738F" Ref="V9"  Part="1"
 AR Path="/5F7A4E71/5F73738F" Ref="V11"  Part="1"
-F 0 "V7" H 5755 3646 50  0000 L CNN
-F 1 "CRSS042N10N" H 5755 3555 50  0000 L CNN
+F 0 "V7" H 5754 3646 50  0000 L CNN
+F 1 "CRSS042N10N" H 5754 3555 50  0000 L CNN
 F 2 "Package_TO_SOT_SMD:TO-263-2" H 5750 3525 50  0001 L CIN
 F 3 "https://www.infineon.com/dgdl/Infineon-BSP89-DS-v02_02-en.pdf?fileId=db3a30433b47825b013b4b8a07f90d55" H 5550 3600 50  0001 L CNN
@@
 AR Path="/5F7A3A2A/5F72B1D2" Ref="R32"  Part="1"
 AR Path="/5F7A4E71/5F72B1D2" Ref="R34"  Part="1"
-F 0 "R21" V 4993 3600 50  0000 C CNN
-F 1 "20k" V 5084 3600 50  0000 C CNN
+F 0 "R21" V 5200 3600 50  0000 C CNN
+F 1 "IRF->100 U51->20" V 5100 3550 50  0000 C CNN
 F 2 "Resistor_SMD:R_1206_3216Metric" V 5130 3600 50  0001 C CNN
 F 3 "~" H 5200 3600 50  0001 C CNN
@@
 AR Path="/5F7A3A2A/5F7824C8" Ref="R28"  Part="1"
 AR Path="/5F7A4E71/5F7824C8" Ref="R33"  Part="1"
-F 0 "R18" V 4993 3100 50  0000 C CNN
-F 1 "20k" V 5084 3100 50  0000 C CNN
+F 0 "R18" V 5200 3100 50  0000 C CNN
+F 1 "IRF->100 U51->20" V 5084 3100 50  0000 C CNN
 F 2 "Resistor_SMD:R_1206_3216Metric" V 5130 3100 50  0001 C CNN
 F 3 "~" H 5200 3100 50  0001 C CNN
@@
 AR Path="/5F7A3A2A/5F70E4C5" Ref="V8"  Part="1"
 AR Path="/5F7A4E71/5F70E4C5" Ref="V10"  Part="1"
-F 0 "V6" H 5755 3146 50  0000 L CNN
-F 1 "CRSS042N10N" H 5755 3055 50  0000 L CNN
+F 0 "V6" H 5754 3146 50  0000 L CNN
+F 1 "CRSS042N10N" H 5754 3055 50  0000 L CNN
 F 2 "Package_TO_SOT_SMD:TO-263-2" H 5750 3025 50  0001 L CIN
 F 3 "https://www.infineon.com/dgdl/Infineon-BSP89-DS-v02_02-en.pdf?fileId=db3a30433b47825b013b4b8a07f90d55" H 5550 3100 50  0001 L CNN
@@
 AR Path="/5F7A3A2A/5F76BFEE" Ref="R67"  Part="1"
 AR Path="/5F7A4E71/5F76BFEE" Ref="R70"  Part="1"
-F 0 "R64" V 4743 3750 50  0000 C CNN
-F 1 "10k IRF->DNP" V 4834 3750 50  0000 C CNN
+F 0 "R64" H 5019 3704 50  0000 L CNN
+F 1 "10k IRF->DNP" H 5019 3795 50  0000 L CNN
 F 2 "Resistor_SMD:R_1206_3216Metric" V 4880 3750 50  0001 C CNN
 F 3 "~" H 4950 3750 50  0001 C CNN
@@
 AR Path="/5F7A3A2A/5F76CC5E" Ref="R66"  Part="1"
 AR Path="/5F7A4E71/5F76CC5E" Ref="R69"  Part="1"
-F 0 "R63" V 4643 3300 50  0000 C CNN
-F 1 "DNP 10k" V 4734 3300 50  0000 C CNN
+F 0 "R63" H 4780 3254 50  0000 R CNN
+F 1 "10k IRF->DNP" H 4800 3350 50  0000 R CNN
 F 2 "Resistor_SMD:R_1206_3216Metric" V 4780 3300 50  0001 C CNN
 F 3 "~" H 4850 3300 50  0001 C CNN
@@
 AR Path="/5F7A3A2A/5F784928" Ref="C68"  Part="1"
 AR Path="/5F7A4E71/5F784928" Ref="C69"  Part="1"
-F 0 "C67" H 6865 3046 50  0000 L CNN
-F 1 "2.2u 100V" H 6865 2955 50  0000 L CNN
+F 0 "C67" H 6635 3046 50  0000 R CNN
+F 1 "2.2u 100V" H 6635 2955 50  0000 R CNN
 F 2 "Capacitor_SMD:C_1206_3216Metric" H 6788 2850 50  0001 C CNN
 F 3 "~" H 6750 3000 50  0001 C CNN
@@
 	6750 3150 7100 3150
 Connection ~ 7100 3150
+$Comp
+L Device:R R72
+U 1 1 5F7BAC08
+P 3500 3300
+AR Path="/5F7A2640/5F7BAC08" Ref="R72"  Part="1"
+AR Path="/5F7ECC6C/5F7BAC08" Ref="R52"  Part="1"
+AR Path="/5F79FFE4/5F7BAC08" Ref="R62"  Part="1"
+AR Path="/5F7A0EEE/5F7BAC08" Ref="R68"  Part="1"
+AR Path="/5F7A3A2A/5F7BAC08" Ref="R74"  Part="1"
+AR Path="/5F7A4E71/5F7BAC08" Ref="R76"  Part="1"
+F 0 "R72" V 3203 3300 50  0000 C CNN
+F 1 "1k" V 3294 3300 50  0000 C CNN
+F 2 "Resistor_SMD:R_0603_1608Metric" V 3250 2500 50  0001 C CNN
+F 3 "~" H 3500 3300 50  0001 C CNN
+	1    3500 3300
+	0    1    1    0
+$EndComp
+$Comp
+L Device:R R73
+U 1 1 5F7BB10C
+P 3500 3400
+AR Path="/5F7A2640/5F7BB10C" Ref="R73"  Part="1"
+AR Path="/5F7ECC6C/5F7BB10C" Ref="R59"  Part="1"
+AR Path="/5F79FFE4/5F7BB10C" Ref="R65"  Part="1"
+AR Path="/5F7A0EEE/5F7BB10C" Ref="R71"  Part="1"
+AR Path="/5F7A3A2A/5F7BB10C" Ref="R75"  Part="1"
+AR Path="/5F7A4E71/5F7BB10C" Ref="R77"  Part="1"
+F 0 "R73" V 3293 3400 50  0000 C CNN
+F 1 "1k" V 3384 3400 50  0000 C CNN
+F 2 "Resistor_SMD:R_0603_1608Metric" V 3430 3400 50  0001 C CNN
+F 3 "~" H 3500 3400 50  0001 C CNN
+	1    3500 3400
+	0    1    1    0
+$EndComp
 $EndSCHEMATC

Commit message: prepare production files
Parts:
- R10, R13: value IRF->100 U51->20 -> 100R
- R50, R51: value 10k IRF->DNP -> 10k
Changed lines of the file:
@@
 AR Path="/5F7A4E71/5F72B1D2" Ref="R34"  Part="1"
 F 0 "R21" V 5200 3600 50  0000 C CNN
-F 1 "IRF->100 U51->20" V 5100 3550 50  0000 C CNN
+F 1 "100R" V 5100 3550 50  0000 C CNN
 F 2 "Resistor_SMD:R_1206_3216Metric" V 5130 3600 50  0001 C CNN
 F 3 "~" H 5200 3600 50  0001 C CNN
@@
 AR Path="/5F7A4E71/5F7824C8" Ref="R33"  Part="1"
 F 0 "R18" V 5200 3100 50  0000 C CNN
-F 1 "IRF->100 U51->20" V 5084 3100 50  0000 C CNN
+F 1 "100R" V 5084 3100 50  0000 C CNN
 F 2 "Resistor_SMD:R_1206_3216Metric" V 5130 3100 50  0001 C CNN
 F 3 "~" H 5200 3100 50  0001 C CNN
@@
 AR Path="/5F7A4E71/5F76BFEE" Ref="R70"  Part="1"
 F 0 "R64" H 5019 3704 50  0000 L CNN
-F 1 "10k IRF->DNP" H 5019 3795 50  0000 L CNN
+F 1 "10k" H 5019 3795 50  0000 L CNN
 F 2 "Resistor_SMD:R_1206_3216Metric" V 4880 3750 50  0001 C CNN
 F 3 "~" H 4950 3750 50  0001 C CNN
@@
 AR Path="/5F7A4E71/5F76CC5E" Ref="R69"  Part="1"
 F 0 "R63" H 4780 3254 50  0000 R CNN
-F 1 "10k IRF->DNP" H 4800 3350 50  0000 R CNN
+F 1 "10k" H 4800 3350 50  0000 R CNN
 F 2 "Resistor_SMD:R_1206_3216Metric" V 4780 3300 50  0001 C CNN
 F 3 "~" H 4850 3300 50  0001 C CNN

Commit message: fix some bugs of the first revision
Parts:
- R10: value 100R -> 4.7
- R4.7: renamed from R13; value 100R -> 4.7
- U8: value IRS2304 || U3115S -> IRS2304; alternative (none) -> (alt U3115S different pinout)
Changed lines of the file:
@@
 $Descr A4 11693 8268
 encoding utf-8
-Sheet 11 14
+Sheet 12 14
 Title ""
 Date ""
@@
 AR Path="/5F7A3A2A/5F706578" Ref="C17"  Part="1"
 AR Path="/5F7A4E71/5F706578" Ref="C24"  Part="1"
-F 0 "C15" H 4618 3346 50  0000 L CNN
+F 0 "C24" H 4618 3346 50  0000 L CNN
 F 1 "47u LKMD0901K470MF" H 3900 3450 50  0000 L CNN
 F 2 "Capacitor_THT:CP_Radial_D8.0mm_P3.50mm" H 4538 3150 50  0001 C CNN
@@
 AR Path="/5F7A3A2A/5F707CCD" Ref="D10"  Part="1"
 AR Path="/5F7A4E71/5F707CCD" Ref="D11"  Part="1"
-F 0 "D9" H 4300 2283 50  0000 C CNN
+F 0 "D11" H 4300 2283 50  0000 C CNN
 F 1 "1N4148W" H 4300 2374 50  0000 C CNN
 F 2 "Diode_SMD:D_SOD-123" H 4300 2500 50  0001 C CNN
@@
 AR Path="/5F7A3A2A/5F77195C" Ref="#PWR0187"  Part="1"
 AR Path="/5F7A4E71/5F77195C" Ref="#PWR0191"  Part="1"
-F 0 "#PWR0183" H 3950 2250 50  0001 C CNN
+F 0 "#PWR0191" H 3950 2250 50  0001 C CNN
 F 1 "+VSW" H 3965 2573 50  0000 C CNN
 F 2 "" H 3950 2400 50  0001 C CNN
@@
 AR Path="/5F7A3A2A/5F771CDC" Ref="C16"  Part="1"
 AR Path="/5F7A4E71/5F771CDC" Ref="C18"  Part="1"
-F 0 "C14" H 3382 3996 50  0000 R CNN
+F 0 "C18" H 3382 3996 50  0000 R CNN
 F 1 "220u25V LKMD0901E221MF" H 3382 3905 50  0000 R CNN
 F 2 "Capacitor_THT:CP_Radial_D8.0mm_P3.50mm" H 3538 3800 50  0001 C CNN
@@
 AR Path="/5F7A3A2A/5F77283D" Ref="#PWR0188"  Part="1"
 AR Path="/5F7A4E71/5F77283D" Ref="#PWR0192"  Part="1"
-F 0 "#PWR0184" H 3500 3600 50  0001 C CNN
+F 0 "#PWR0192" H 3500 3600 50  0001 C CNN
 F 1 "+VSW" H 3515 3923 50  0000 C CNN
 F 2 "" H 3500 3750 50  0001 C CNN
@@
 AR Path="/5F7A3A2A/5F773E85" Ref="#PWR0189"  Part="1"
 AR Path="/5F7A4E71/5F773E85" Ref="#PWR0193"  Part="1"
-F 0 "#PWR0185" H 3850 3900 50  0001 C CNN
+F 0 "#PWR0193" H 3850 3900 50  0001 C CNN
 F 1 "GND" H 3855 3977 50  0000 C CNN
 F 2 "" H 3850 4150 50  0001 C CNN
@@
 AR Path="/5F7A3A2A/5F73738F" Ref="V9"  Part="1"
 AR Path="/5F7A4E71/5F73738F" Ref="V11"  Part="1"
-F 0 "V7" H 5754 3646 50  0000 L CNN
+F 0 "V11" H 5754 3646 50  0000 L CNN
 F 1 "CRSS042N10N" H 5754 3555 50  0000 L CNN
 F 2 "Package_TO_SOT_SMD:TO-263-2" H 5750 3525 50  0001 L CIN
@@
 AR Path="/5F7A3A2A/5F72B1D2" Ref="R32"  Part="1"
 AR Path="/5F7A4E71/5F72B1D2" Ref="R34"  Part="1"
-F 0 "R21" V 5200 3600 50  0000 C CNN
-F 1 "100R" V 5100 3550 50  0000 C CNN
+F 0 "R34" V 5200 3600 50  0000 C CNN
+F 1 "4.7" V 5100 3550 50  0000 C CNN
 F 2 "Resistor_SMD:R_1206_3216Metric" V 5130 3600 50  0001 C CNN
 F 3 "~" H 5200 3600 50  0001 C CNN
@@
 AR Path="/5F7A3A2A/5F771122" Ref="U12"  Part="1"
 AR Path="/5F7A4E71/5F771122" Ref="U13"  Part="1"
-F 0 "U11" H 3950 3981 50  0000 C CNN
-F 1 "IRS2304 || U3115S" H 3950 3890 50  0000 C CNN
+F 0 "U13" H 3950 3981 50  0000 C CNN
+F 1 "IRS2304" H 3950 3890 50  0000 C CNN
 F 2 "Package_SO:SOIC-8_3.9x4.9mm_P1.27mm" H 3950 3300 50  0001 C CIN
 F 3 "https://www.infineon.com/dgdl/irs2304spbf.pdf?fileId=5546d462533600a40153567a8fe72802" H 3950 3300 50  0001 C CNN
+F 4 "(alt U3115S different pinout)" H 3950 3300 50  0001 C CNN "alternative"
 	1    3950 3300
 	1    0    0    -1
 $EndComp
 $Comp
-L Device:R R13
+L Device:R R4.7
 U 1 1 5F7824C8
 P 5200 3100
-AR Path="/5F7ECC6C/5F7824C8" Ref="R13"  Part="1"
+AR Path="/5F7ECC6C/5F7824C8" Ref="R4.7"  Part="1"
 AR Path="/5F79FFE4/5F7824C8" Ref="R14"  Part="1"
 AR Path="/5F7A0EEE/5F7824C8" Ref="R16"  Part="1"
@@
 AR Path="/5F7A3A2A/5F7824C8" Ref="R28"  Part="1"
 AR Path="/5F7A4E71/5F7824C8" Ref="R33"  Part="1"
-F 0 "R18" V 5200 3100 50  0000 C CNN
-F 1 "100R" V 5084 3100 50  0000 C CNN
+F 0 "R4.7" V 5200 3100 50  0000 C CNN
+F 1 "4.7" V 5084 3100 50  0000 C CNN
 F 2 "Resistor_SMD:R_1206_3216Metric" V 5130 3100 50  0001 C CNN
 F 3 "~" H 5200 3100 50  0001 C CNN
@@
 AR Path="/5F7A3A2A/5F70E4C5" Ref="V8"  Part="1"
 AR Path="/5F7A4E71/5F70E4C5" Ref="V10"  Part="1"
-F 0 "V6" H 5754 3146 50  0000 L CNN
+F 0 "V10" H 5754 3146 50  0000 L CNN
 F 1 "CRSS042N10N" H 5754 3055 50  0000 L CNN
 F 2 "Package_TO_SOT_SMD:TO-263-2" H 5750 3025 50  0001 L CIN
@@
 AR Path="/5F7A3A2A/5F79127D" Ref="#PWR0190"  Part="1"
 AR Path="/5F7A4E71/5F79127D" Ref="#PWR0194"  Part="1"
-F 0 "#PWR0186" H 5650 2650 50  0001 C CNN
+F 0 "#PWR0194" H 5650 2650 50  0001 C CNN
 F 1 "+BATT" H 5665 2973 50  0000 C CNN
 F 2 "" H 5650 2800 50  0001 C CNN
@@
 AR Path="/5F7A3A2A/5F7BE8FF" Ref="C35"  Part="1"
 AR Path="/5F7A4E71/5F7BE8FF" Ref="C36"  Part="1"
-F 0 "C34" H 7218 3046 50  0000 L CNN
+F 0 "C36" H 7218 3046 50  0000 L CNN
 F 1 "47u LKMD0901K470MF" H 7218 2955 50  0000 L CNN
 F 2 "Capacitor_THT:CP_Radial_D8.0mm_P3.50mm" H 7138 2850 50  0001 C CNN
@@
 AR Path="/5F7A3A2A/5F7BF207" Ref="#PWR0201"  Part="1"
 AR Path="/5F7A4E71/5F7BF207" Ref="#PWR0202"  Part="1"
-F 0 "#PWR0200" H 7100 2650 50  0001 C CNN
+F 0 "#PWR0202" H 7100 2650 50  0001 C CNN
 F 1 "+BATT" H 7115 2973 50  0000 C CNN
 F 2 "" H 7100 2800 50  0001 C CNN
@@
 AR Path="/5F7A3A2A/5F72BDA4" Ref="D27"  Part="1"
 AR Path="/5F7A4E71/5F72BDA4" Ref="D28"  Part="1"
-F 0 "D26" V 8154 3080 50  0000 L CNN
+F 0 "D28" V 8154 3080 50  0000 L CNN
 F 1 "51V TVS C310059" V 8245 3080 50  0000 L CNN
 F 2 "Diode_SMD:D_SMC" H 8200 3000 50  0001 C CNN
@@
 AR Path="/5F7A3A2A/5F76BFEE" Ref="R67"  Part="1"
 AR Path="/5F7A4E71/5F76BFEE" Ref="R70"  Part="1"
-F 0 "R64" H 5019 3704 50  0000 L CNN
+F 0 "R70" H 5019 3704 50  0000 L CNN
 F 1 "10k" H 5019 3795 50  0000 L CNN
 F 2 "Resistor_SMD:R_1206_3216Metric" V 4880 3750 50  0001 C CNN
@@
 AR Path="/5F7A3A2A/5F76CC5E" Ref="R66"  Part="1"
 AR Path="/5F7A4E71/5F76CC5E" Ref="R69"  Part="1"
-F 0 "R63" H 4780 3254 50  0000 R CNN
+F 0 "R69" H 4780 3254 50  0000 R CNN
 F 1 "10k" H 4800 3350 50  0000 R CNN
 F 2 "Resistor_SMD:R_1206_3216Metric" V 4780 3300 50  0001 C CNN
@@
 AR Path="/5F7A3A2A/5F784928" Ref="C68"  Part="1"
 AR Path="/5F7A4E71/5F784928" Ref="C69"  Part="1"
-F 0 "C67" H 6635 3046 50  0000 R CNN
+F 0 "C69" H 6635 3046 50  0000 R CNN
 F 1 "2.2u 100V" H 6635 2955 50  0000 R CNN
 F 2 "Capacitor_SMD:C_1206_3216Metric" H 6788 2850 50  0001 C CNN
@@
 AR Path="/5F7A3A2A/5F7BAC08" Ref="R74"  Part="1"
 AR Path="/5F7A4E71/5F7BAC08" Ref="R76"  Part="1"
-F 0 "R72" V 3203 3300 50  0000 C CNN
+F 0 "R76" V 3203 3300 50  0000 C CNN
 F 1 "1k" V 3294 3300 50  0000 C CNN
 F 2 "Resistor_SMD:R_0603_1608Metric" V 3250 2500 50  0001 C CNN
@@
 AR Path="/5F7A3A2A/5F7BB10C" Ref="R75"  Part="1"
 AR Path="/5F7A4E71/5F7BB10C" Ref="R77"  Part="1"
-F 0 "R73" V 3293 3400 50  0000 C CNN
+F 0 "R77" V 3293 3400 50  0000 C CNN
 F 1 "1k" V 3384 3400 50  0000 C CNN
 F 2 "Resistor_SMD:R_0603_1608Metric" V 3430 3400 50  0001 C CNN
