File: hh_bridge.sch (KiCad schematic (older format))
At the start: 15 parts, among them U8 IRS2304

Commit message: MOVs placed
Parts:
- removed D23: 51V TVS C310059, Diode_SMD:D_SMC, symbol Device:D_Zener
- added RV1: Varistor, Bobbycar-FOC-hardware:MOV20, symbol Device:Varistor
Connections:
- net +BATT: now also RV1.1
- net H_BRIDGE_GND: now also RV1.2
Changed lines of the file:
@@
 $Descr A4 11693 8268
 encoding utf-8
-Sheet 11 14
+Sheet 10 14
 Title ""
 Date ""
@@
 AR Path="/5F7A3A2A/5F706578" Ref="C17"  Part="1"
 AR Path="/5F7A4E71/5F706578" Ref="C24"  Part="1"
-F 0 "C24" H 4618 3346 50  0000 L CNN
+F 0 "C13" H 4618 3346 50  0000 L CNN
 F 1 "47u LKMD0901K470MF" H 3900 3450 50  0000 L CNN
 F 2 "Capacitor_THT:CP_Radial_D8.0mm_P3.50mm" H 4538 3150 50  0001 C CNN
@@
 AR Path="/5F7A3A2A/5F707CCD" Ref="D10"  Part="1"
 AR Path="/5F7A4E71/5F707CCD" Ref="D11"  Part="1"
-F 0 "D11" H 4300 2283 50  0000 C CNN
+F 0 "D8" H 4300 2283 50  0000 C CNN
 F 1 "1N4148W" H 4300 2374 50  0000 C CNN
 F 2 "Diode_SMD:D_SOD-123" H 4300 2500 50  0001 C CNN
@@
 AR Path="/5F7A3A2A/5F77195C" Ref="#PWR0187"  Part="1"
 AR Path="/5F7A4E71/5F77195C" Ref="#PWR0191"  Part="1"
-F 0 "#PWR0191" H 3950 2250 50  0001 C CNN
+F 0 "#PWR0179" H 3950 2250 50  0001 C CNN
 F 1 "+VSW" H 3965 2573 50  0000 C CNN
 F 2 "" H 3950 2400 50  0001 C CNN
@@
 AR Path="/5F7A3A2A/5F771CDC" Ref="C16"  Part="1"
 AR Path="/5F7A4E71/5F771CDC" Ref="C18"  Part="1"
-F 0 "C18" H 3382 3996 50  0000 R CNN
+F 0 "C12" H 3382 3996 50  0000 R CNN
 F 1 "220u25V LKMD0901E221MF" H 3382 3905 50  0000 R CNN
 F 2 "Capacitor_THT:CP_Radial_D8.0mm_P3.50mm" H 3538 3800 50  0001 C CNN
@@
 AR Path="/5F7A3A2A/5F77283D" Ref="#PWR0188"  Part="1"
 AR Path="/5F7A4E71/5F77283D" Ref="#PWR0192"  Part="1"
-F 0 "#PWR0192" H 3500 3600 50  0001 C CNN
+F 0 "#PWR0180" H 3500 3600 50  0001 C CNN
 F 1 "+VSW" H 3515 3923 50  0000 C CNN
 F 2 "" H 3500 3750 50  0001 C CNN
@@
 AR Path="/5F7A3A2A/5F773E85" Ref="#PWR0189"  Part="1"
 AR Path="/5F7A4E71/5F773E85" Ref="#PWR0193"  Part="1"
-F 0 "#PWR0193" H 3850 3900 50  0001 C CNN
+F 0 "#PWR0181" H 3850 3900 50  0001 C CNN
 F 1 "GND" H 3855 3977 50  0000 C CNN
 F 2 "" H 3850 4150 50  0001 C CNN
@@
 AR Path="/5F7A3A2A/5F73738F" Ref="V9"  Part="1"
 AR Path="/5F7A4E71/5F73738F" Ref="V11"  Part="1"
-F 0 "V11" H 5754 3646 50  0000 L CNN
+F 0 "V5" H 5754 3646 50  0000 L CNN
 F 1 "CRSS042N10N" H 5754 3555 50  0000 L CNN
 F 2 "Package_TO_SOT_SMD:TO-263-2" H 5750 3525 50  0001 L CIN
@@
 AR Path="/5F7A3A2A/5F72B1D2" Ref="R32"  Part="1"
 AR Path="/5F7A4E71/5F72B1D2" Ref="R34"  Part="1"
-F 0 "R34" V 5200 3600 50  0000 C CNN
+F 0 "R17" V 5200 3600 50  0000 C CNN
 F 1 "4.7" V 5100 3550 50  0000 C CNN
 F 2 "Resistor_SMD:R_1206_3216Metric" V 5130 3600 50  0001 C CNN
@@
 AR Path="/5F7A3A2A/5F771122" Ref="U12"  Part="1"
 AR Path="/5F7A4E71/5F771122" Ref="U13"  Part="1"
-F 0 "U13" H 3950 3981 50  0000 C CNN
+F 0 "U10" H 3950 3981 50  0000 C CNN
 F 1 "IRS2304" H 3950 3890 50  0000 C CNN
 F 2 "Package_SO:SOIC-8_3.9x4.9mm_P1.27mm" H 3950 3300 50  0001 C CIN
@@
 AR Path="/5F7A3A2A/5F7824C8" Ref="R28"  Part="1"
 AR Path="/5F7A4E71/5F7824C8" Ref="R33"  Part="1"
-F 0 "R4.7" V 5200 3100 50  0000 C CNN
+F 0 "R16" V 5200 3100 50  0000 C CNN
 F 1 "4.7" V 5084 3100 50  0000 C CNN
 F 2 "Resistor_SMD:R_1206_3216Metric" V 5130 3100 50  0001 C CNN
@@
 AR Path="/5F7A3A2A/5F70E4C5" Ref="V8"  Part="1"
 AR Path="/5F7A4E71/5F70E4C5" Ref="V10"  Part="1"
-F 0 "V10" H 5754 3146 50  0000 L CNN
+F 0 "V4" H 5754 3146 50  0000 L CNN
 F 1 "CRSS042N10N" H 5754 3055 50  0000 L CNN
 F 2 "Package_TO_SOT_SMD:TO-263-2" H 5750 3025 50  0001 L CIN
@@
 AR Path="/5F7A3A2A/5F79127D" Ref="#PWR0190"  Part="1"
 AR Path="/5F7A4E71/5F79127D" Ref="#PWR0194"  Part="1"
-F 0 "#PWR0194" H 5650 2650 50  0001 C CNN
+F 0 "#PWR0182" H 5650 2650 50  0001 C CNN
 F 1 "+BATT" H 5665 2973 50  0000 C CNN
 F 2 "" H 5650 2800 50  0001 C CNN
@@
 AR Path="/5F7A3A2A/5F7BE8FF" Ref="C35"  Part="1"
 AR Path="/5F7A4E71/5F7BE8FF" Ref="C36"  Part="1"
-F 0 "C36" H 7218 3046 50  0000 L CNN
+F 0 "C33" H 7218 3046 50  0000 L CNN
 F 1 "47u LKMD0901K470MF" H 7218 2955 50  0000 L CNN
 F 2 "Capacitor_THT:CP_Radial_D8.0mm_P3.50mm" H 7138 2850 50  0001 C CNN
@@
 AR Path="/5F7A3A2A/5F7BF207" Ref="#PWR0201"  Part="1"
 AR Path="/5F7A4E71/5F7BF207" Ref="#PWR0202"  Part="1"
-F 0 "#PWR0202" H 7100 2650 50  0001 C CNN
+F 0 "#PWR0199" H 7100 2650 50  0001 C CNN
 F 1 "+BATT" H 7115 2973 50  0000 C CNN
 F 2 "" H 7100 2800 50  0001 C CNN
@@
 Wire Wire Line
 	5650 2800 5650 2900
-$Comp
-L Device:D_Zener D?
-U 1 1 5F72BDA4
-P 8200 3000
-AR Path="/5F7395DA/5F72BDA4" Ref="D?"  Part="1"
-AR Path="/5F7ECC6C/5F72BDA4" Ref="D23"  Part="1"
-AR Path="/5F79FFE4/5F72BDA4" Ref="D24"  Part="1"
-AR Path="/5F7A0EEE/5F72BDA4" Ref="D25"  Part="1"
-AR Path="/5F7A2640/5F72BDA4" Ref="D26"  Part="1"
-AR Path="/5F7A3A2A/5F72BDA4" Ref="D27"  Part="1"
-AR Path="/5F7A4E71/5F72BDA4" Ref="D28"  Part="1"
-F 0 "D28" V 8154 3080 50  0000 L CNN
-F 1 "51V TVS C310059" V 8245 3080 50  0000 L CNN
-F 2 "Diode_SMD:D_SMC" H 8200 3000 50  0001 C CNN
-F 3 "~" H 8200 3000 50  0001 C CNN
-	1    8200 3000
-	0    1    1    0
-$EndComp
 Wire Wire Line
 	8200 3150 8200 3350
@@
 AR Path="/5F7A3A2A/5F76BFEE" Ref="R67"  Part="1"
 AR Path="/5F7A4E71/5F76BFEE" Ref="R70"  Part="1"
-F 0 "R70" H 5019 3704 50  0000 L CNN
+F 0 "R61" H 5019 3704 50  0000 L CNN
 F 1 "10k" H 5019 3795 50  0000 L CNN
 F 2 "Resistor_SMD:R_1206_3216Metric" V 4880 3750 50  0001 C CNN
@@
 AR Path="/5F7A3A2A/5F76CC5E" Ref="R66"  Part="1"
 AR Path="/5F7A4E71/5F76CC5E" Ref="R69"  Part="1"
-F 0 "R69" H 4780 3254 50  0000 R CNN
+F 0 "R60" H 4780 3254 50  0000 R CNN
 F 1 "10k" H 4800 3350 50  0000 R CNN
 F 2 "Resistor_SMD:R_1206_3216Metric" V 4780 3300 50  0001 C CNN
@@
 AR Path="/5F7A3A2A/5F784928" Ref="C68"  Part="1"
 AR Path="/5F7A4E71/5F784928" Ref="C69"  Part="1"
-F 0 "C69" H 6635 3046 50  0000 R CNN
+F 0 "C66" H 6635 3046 50  0000 R CNN
 F 1 "2.2u 100V" H 6635 2955 50  0000 R CNN
 F 2 "Capacitor_SMD:C_1206_3216Metric" H 6788 2850 50  0001 C CNN
@@
 AR Path="/5F7A3A2A/5F7BAC08" Ref="R74"  Part="1"
 AR Path="/5F7A4E71/5F7BAC08" Ref="R76"  Part="1"
-F 0 "R76" V 3203 3300 50  0000 C CNN
+F 0 "R68" V 3203 3300 50  0000 C CNN
 F 1 "1k" V 3294 3300 50  0000 C CNN
 F 2 "Resistor_SMD:R_0603_1608Metric" V 3250 2500 50  0001 C CNN
@@
 AR Path="/5F7A3A2A/5F7BB10C" Ref="R75"  Part="1"
 AR Path="/5F7A4E71/5F7BB10C" Ref="R77"  Part="1"
-F 0 "R77" V 3293 3400 50  0000 C CNN
+F 0 "R71" V 3293 3400 50  0000 C CNN
 F 1 "1k" V 3384 3400 50  0000 C CNN
 F 2 "Resistor_SMD:R_0603_1608Metric" V 3430 3400 50  0001 C CNN
@@
 	0    1    1    0
 $EndComp
+$Comp
+L Device:Varistor RV1
+U 1 1 6020AE15
+P 8200 3000
+AR Path="/5F7ECC6C/6020AE15" Ref="RV1"  Part="1"
+AR Path="/5F79FFE4/6020AE15" Ref="RV2"  Part="1"
+AR Path="/5F7A0EEE/6020AE15" Ref="RV3"  Part="1"
+AR Path="/5F7A2640/6020AE15" Ref="RV4"  Part="1"
+AR Path="/5F7A3A2A/6020AE15" Ref="RV5"  Part="1"
+AR Path="/5F7A4E71/6020AE15" Ref="RV6"  Part="1"
+F 0 "RV3" H 8303 3046 50  0000 L CNN
+F 1 "Varistor" H 8303 2955 50  0000 L CNN
+F 2 "Bobbycar-FOC-hardware:MOV20" V 8130 3000 50  0001 C CNN
+F 3 "~" H 8200 3000 50  0001 C CNN
+	1    8200 3000
+	1    0    0    -1
+$EndComp
 $EndSCHEMATC

Commit message: Changed fet driver
Parts:
- U8: value IRS2304 -> UCC27712; LCSC Part # (none) -> C485818; alternative (alt U3115S different pinout) -> IRS2304 old
Changed lines of the file:
@@
 $Descr A4 11693 8268
 encoding utf-8
-Sheet 10 14
+Sheet 8 14
 Title ""
 Date ""
@@
 AR Path="/5F7A3A2A/5F706578" Ref="C17"  Part="1"
 AR Path="/5F7A4E71/5F706578" Ref="C24"  Part="1"
-F 0 "C13" H 4618 3346 50  0000 L CNN
+F 0 "C1" H 4618 3346 50  0000 L CNN
 F 1 "47u LKMD0901K470MF" H 3900 3450 50  0000 L CNN
 F 2 "Capacitor_THT:CP_Radial_D8.0mm_P3.50mm" H 4538 3150 50  0001 C CNN
@@
 AR Path="/5F7A3A2A/5F707CCD" Ref="D10"  Part="1"
 AR Path="/5F7A4E71/5F707CCD" Ref="D11"  Part="1"
-F 0 "D8" H 4300 2283 50  0000 C CNN
+F 0 "D1" H 4300 2283 50  0000 C CNN
 F 1 "1N4148W" H 4300 2374 50  0000 C CNN
 F 2 "Diode_SMD:D_SOD-123" H 4300 2500 50  0001 C CNN
@@
 AR Path="/5F7A3A2A/5F77195C" Ref="#PWR0187"  Part="1"
 AR Path="/5F7A4E71/5F77195C" Ref="#PWR0191"  Part="1"
-F 0 "#PWR0179" H 3950 2250 50  0001 C CNN
+F 0 "#PWR0171" H 3950 2250 50  0001 C CNN
 F 1 "+VSW" H 3965 2573 50  0000 C CNN
 F 2 "" H 3950 2400 50  0001 C CNN
@@
 AR Path="/5F7A3A2A/5F771CDC" Ref="C16"  Part="1"
 AR Path="/5F7A4E71/5F771CDC" Ref="C18"  Part="1"
-F 0 "C12" H 3382 3996 50  0000 R CNN
+F 0 "C8" H 3382 3996 50  0000 R CNN
 F 1 "220u25V LKMD0901E221MF" H 3382 3905 50  0000 R CNN
 F 2 "Capacitor_THT:CP_Radial_D8.0mm_P3.50mm" H 3538 3800 50  0001 C CNN
@@
 AR Path="/5F7A3A2A/5F77283D" Ref="#PWR0188"  Part="1"
 AR Path="/5F7A4E71/5F77283D" Ref="#PWR0192"  Part="1"
-F 0 "#PWR0180" H 3500 3600 50  0001 C CNN
+F 0 "#PWR0172" H 3500 3600 50  0001 C CNN
 F 1 "+VSW" H 3515 3923 50  0000 C CNN
 F 2 "" H 3500 3750 50  0001 C CNN
@@
 AR Path="/5F7A3A2A/5F773E85" Ref="#PWR0189"  Part="1"
 AR Path="/5F7A4E71/5F773E85" Ref="#PWR0193"  Part="1"
-F 0 "#PWR0181" H 3850 3900 50  0001 C CNN
+F 0 "#PWR0173" H 3850 3900 50  0001 C CNN
 F 1 "GND" H 3855 3977 50  0000 C CNN
 F 2 "" H 3850 4150 50  0001 C CNN
@@
 AR Path="/5F7A3A2A/5F73738F" Ref="V9"  Part="1"
 AR Path="/5F7A4E71/5F73738F" Ref="V11"  Part="1"
-F 0 "V5" H 5754 3646 50  0000 L CNN
+F 0 "V1" H 5754 3646 50  0000 L CNN
 F 1 "CRSS042N10N" H 5754 3555 50  0000 L CNN
 F 2 "Package_TO_SOT_SMD:TO-263-2" H 5750 3525 50  0001 L CIN
@@
 AR Path="/5F7A3A2A/5F72B1D2" Ref="R32"  Part="1"
 AR Path="/5F7A4E71/5F72B1D2" Ref="R34"  Part="1"
-F 0 "R17" V 5200 3600 50  0000 C CNN
+F 0 "R10" V 5200 3600 50  0000 C CNN
 F 1 "4.7" V 5100 3550 50  0000 C CNN
 F 2 "Resistor_SMD:R_1206_3216Metric" V 5130 3600 50  0001 C CNN
@@
 AR Path="/5F7A3A2A/5F771122" Ref="U12"  Part="1"
 AR Path="/5F7A4E71/5F771122" Ref="U13"  Part="1"
-F 0 "U10" H 3950 3981 50  0000 C CNN
-F 1 "IRS2304" H 3950 3890 50  0000 C CNN
+F 0 "U8" H 3950 3981 50  0000 C CNN
+F 1 "UCC27712" H 3950 3890 50  0000 C CNN
 F 2 "Package_SO:SOIC-8_3.9x4.9mm_P1.27mm" H 3950 3300 50  0001 C CIN
 F 3 "https://www.infineon.com/dgdl/irs2304spbf.pdf?fileId=5546d462533600a40153567a8fe72802" H 3950 3300 50  0001 C CNN
-F 4 "(alt U3115S different pinout)" H 3950 3300 50  0001 C CNN "alternative"
+F 4 "IRS2304 old" H 3950 3300 50  0001 C CNN "alternative"
+F 5 "C485818" H 3950 3300 50  0001 C CNN "LCSC Part #"
 	1    3950 3300
 	1    0    0    -1
@@
 AR Path="/5F7A3A2A/5F7824C8" Ref="R28"  Part="1"
 AR Path="/5F7A4E71/5F7824C8" Ref="R33"  Part="1"
-F 0 "R16" V 5200 3100 50  0000 C CNN
+F 0 "R4.7" V 5200 3100 50  0000 C CNN
 F 1 "4.7" V 5084 3100 50  0000 C CNN
 F 2 "Resistor_SMD:R_1206_3216Metric" V 5130 3100 50  0001 C CNN
@@
 AR Path="/5F7A3A2A/5F70E4C5" Ref="V8"  Part="1"
 AR Path="/5F7A4E71/5F70E4C5" Ref="V10"  Part="1"
-F 0 "V4" H 5754 3146 50  0000 L CNN
+F 0 "V0" H 5754 3146 50  0000 L CNN
 F 1 "CRSS042N10N" H 5754 3055 50  0000 L CNN
 F 2 "Package_TO_SOT_SMD:TO-263-2" H 5750 3025 50  0001 L CIN
@@
 AR Path="/5F7A3A2A/5F79127D" Ref="#PWR0190"  Part="1"
 AR Path="/5F7A4E71/5F79127D" Ref="#PWR0194"  Part="1"
-F 0 "#PWR0182" H 5650 2650 50  0001 C CNN
+F 0 "#PWR0174" H 5650 2650 50  0001 C CNN
 F 1 "+BATT" H 5665 2973 50  0000 C CNN
 F 2 "" H 5650 2800 50  0001 C CNN
@@
 AR Path="/5F7A3A2A/5F7BE8FF" Ref="C35"  Part="1"
 AR Path="/5F7A4E71/5F7BE8FF" Ref="C36"  Part="1"
-F 0 "C33" H 7218 3046 50  0000 L CNN
+F 0 "C31" H 7218 3046 50  0000 L CNN
 F 1 "47u LKMD0901K470MF" H 7218 2955 50  0000 L CNN
 F 2 "Capacitor_THT:CP_Radial_D8.0mm_P3.50mm" H 7138 2850 50  0001 C CNN
@@
 AR Path="/5F7A3A2A/5F7BF207" Ref="#PWR0201"  Part="1"
 AR Path="/5F7A4E71/5F7BF207" Ref="#PWR0202"  Part="1"
-F 0 "#PWR0199" H 7100 2650 50  0001 C CNN
+F 0 "#PWR0197" H 7100 2650 50  0001 C CNN
 F 1 "+BATT" H 7115 2973 50  0000 C CNN
 F 2 "" H 7100 2800 50  0001 C CNN
@@
 AR Path="/5F7A3A2A/5F76BFEE" Ref="R67"  Part="1"
 AR Path="/5F7A4E71/5F76BFEE" Ref="R70"  Part="1"
-F 0 "R61" H 5019 3704 50  0000 L CNN
+F 0 "R51" H 5019 3704 50  0000 L CNN
 F 1 "10k" H 5019 3795 50  0000 L CNN
 F 2 "Resistor_SMD:R_1206_3216Metric" V 4880 3750 50  0001 C CNN
@@
 AR Path="/5F7A3A2A/5F76CC5E" Ref="R66"  Part="1"
 AR Path="/5F7A4E71/5F76CC5E" Ref="R69"  Part="1"
-F 0 "R60" H 4780 3254 50  0000 R CNN
+F 0 "R50" H 4780 3254 50  0000 R CNN
 F 1 "10k" H 4800 3350 50  0000 R CNN
 F 2 "Resistor_SMD:R_1206_3216Metric" V 4780 3300 50  0001 C CNN
@@
 AR Path="/5F7A3A2A/5F784928" Ref="C68"  Part="1"
 AR Path="/5F7A4E71/5F784928" Ref="C69"  Part="1"
-F 0 "C66" H 6635 3046 50  0000 R CNN
+F 0 "C64" H 6635 3046 50  0000 R CNN
 F 1 "2.2u 100V" H 6635 2955 50  0000 R CNN
 F 2 "Capacitor_SMD:C_1206_3216Metric" H 6788 2850 50  0001 C CNN
@@
 AR Path="/5F7A3A2A/5F7BAC08" Ref="R74"  Part="1"
 AR Path="/5F7A4E71/5F7BAC08" Ref="R76"  Part="1"
-F 0 "R68" V 3203 3300 50  0000 C CNN
+F 0 "R52" V 3203 3300 50  0000 C CNN
 F 1 "1k" V 3294 3300 50  0000 C CNN
 F 2 "Resistor_SMD:R_0603_1608Metric" V 3250 2500 50  0001 C CNN
@@
 AR Path="/5F7A3A2A/5F7BB10C" Ref="R75"  Part="1"
 AR Path="/5F7A4E71/5F7BB10C" Ref="R77"  Part="1"
-F 0 "R71" V 3293 3400 50  0000 C CNN
+F 0 "R59" V 3293 3400 50  0000 C CNN
 F 1 "1k" V 3384 3400 50  0000 C CNN
 F 2 "Resistor_SMD:R_0603_1608Metric" V 3430 3400 50  0001 C CNN
@@
 AR Path="/5F7A3A2A/6020AE15" Ref="RV5"  Part="1"
 AR Path="/5F7A4E71/6020AE15" Ref="RV6"  Part="1"
-F 0 "RV3" H 8303 3046 50  0000 L CNN
+F 0 "RV1" H 8303 3046 50  0000 L CNN
 F 1 "Varistor" H 8303 2955 50  0000 L CNN
 F 2 "Bobbycar-FOC-hardware:MOV20" V 8130 3000 50  0001 C CNN

Commit message: Added FET for LED
Changed lines of the file:
@@
 AR Path="/5F7A3A2A/5F706578" Ref="C17"  Part="1"
 AR Path="/5F7A4E71/5F706578" Ref="C24"  Part="1"
-F 0 "C1" H 4618 3346 50  0000 L CNN
+F 0 "C24" H 4618 3346 50  0000 L CNN
 F 1 "47u LKMD0901K470MF" H 3900 3450 50  0000 L CNN
 F 2 "Capacitor_THT:CP_Radial_D8.0mm_P3.50mm" H 4538 3150 50  0001 C CNN
@@
 AR Path="/5F7A3A2A/5F707CCD" Ref="D10"  Part="1"
 AR Path="/5F7A4E71/5F707CCD" Ref="D11"  Part="1"
-F 0 "D1" H 4300 2283 50  0000 C CNN
+F 0 "D11" H 4300 2283 50  0000 C CNN
 F 1 "1N4148W" H 4300 2374 50  0000 C CNN
 F 2 "Diode_SMD:D_SOD-123" H 4300 2500 50  0001 C CNN
@@
 AR Path="/5F7A3A2A/5F77195C" Ref="#PWR0187"  Part="1"
 AR Path="/5F7A4E71/5F77195C" Ref="#PWR0191"  Part="1"
-F 0 "#PWR0171" H 3950 2250 50  0001 C CNN
+F 0 "#PWR0191" H 3950 2250 50  0001 C CNN
 F 1 "+VSW" H 3965 2573 50  0000 C CNN
 F 2 "" H 3950 2400 50  0001 C CNN
@@
 AR Path="/5F7A3A2A/5F771CDC" Ref="C16"  Part="1"
 AR Path="/5F7A4E71/5F771CDC" Ref="C18"  Part="1"
-F 0 "C8" H 3382 3996 50  0000 R CNN
+F 0 "C18" H 3382 3996 50  0000 R CNN
 F 1 "220u25V LKMD0901E221MF" H 3382 3905 50  0000 R CNN
 F 2 "Capacitor_THT:CP_Radial_D8.0mm_P3.50mm" H 3538 3800 50  0001 C CNN
@@
 AR Path="/5F7A3A2A/5F77283D" Ref="#PWR0188"  Part="1"
 AR Path="/5F7A4E71/5F77283D" Ref="#PWR0192"  Part="1"
-F 0 "#PWR0172" H 3500 3600 50  0001 C CNN
+F 0 "#PWR0192" H 3500 3600 50  0001 C CNN
 F 1 "+VSW" H 3515 3923 50  0000 C CNN
 F 2 "" H 3500 3750 50  0001 C CNN
@@
 AR Path="/5F7A3A2A/5F773E85" Ref="#PWR0189"  Part="1"
 AR Path="/5F7A4E71/5F773E85" Ref="#PWR0193"  Part="1"
-F 0 "#PWR0173" H 3850 3900 50  0001 C CNN
+F 0 "#PWR0193" H 3850 3900 50  0001 C CNN
 F 1 "GND" H 3855 3977 50  0000 C CNN
 F 2 "" H 3850 4150 50  0001 C CNN
@@
 AR Path="/5F7A3A2A/5F73738F" Ref="V9"  Part="1"
 AR Path="/5F7A4E71/5F73738F" Ref="V11"  Part="1"
-F 0 "V1" H 5754 3646 50  0000 L CNN
+F 0 "V11" H 5754 3646 50  0000 L CNN
 F 1 "CRSS042N10N" H 5754 3555 50  0000 L CNN
 F 2 "Package_TO_SOT_SMD:TO-263-2" H 5750 3525 50  0001 L CIN
@@
 AR Path="/5F7A3A2A/5F72B1D2" Ref="R32"  Part="1"
 AR Path="/5F7A4E71/5F72B1D2" Ref="R34"  Part="1"
-F 0 "R10" V 5200 3600 50  0000 C CNN
+F 0 "R34" V 5200 3600 50  0000 C CNN
 F 1 "4.7" V 5100 3550 50  0000 C CNN
 F 2 "Resistor_SMD:R_1206_3216Metric" V 5130 3600 50  0001 C CNN
@@
 AR Path="/5F7A3A2A/5F771122" Ref="U12"  Part="1"
 AR Path="/5F7A4E71/5F771122" Ref="U13"  Part="1"
-F 0 "U8" H 3950 3981 50  0000 C CNN
+F 0 "U13" H 3950 3981 50  0000 C CNN
 F 1 "UCC27712" H 3950 3890 50  0000 C CNN
 F 2 "Package_SO:SOIC-8_3.9x4.9mm_P1.27mm" H 3950 3300 50  0001 C CIN
@@
 AR Path="/5F7A3A2A/5F70E4C5" Ref="V8"  Part="1"
 AR Path="/5F7A4E71/5F70E4C5" Ref="V10"  Part="1"
-F 0 "V0" H 5754 3146 50  0000 L CNN
+F 0 "V10" H 5754 3146 50  0000 L CNN
 F 1 "CRSS042N10N" H 5754 3055 50  0000 L CNN
 F 2 "Package_TO_SOT_SMD:TO-263-2" H 5750 3025 50  0001 L CIN
@@
 AR Path="/5F7A3A2A/5F79127D" Ref="#PWR0190"  Part="1"
 AR Path="/5F7A4E71/5F79127D" Ref="#PWR0194"  Part="1"
-F 0 "#PWR0174" H 5650 2650 50  0001 C CNN
+F 0 "#PWR0194" H 5650 2650 50  0001 C CNN
 F 1 "+BATT" H 5665 2973 50  0000 C CNN
 F 2 "" H 5650 2800 50  0001 C CNN
@@
 AR Path="/5F7A3A2A/5F7BE8FF" Ref="C35"  Part="1"
 AR Path="/5F7A4E71/5F7BE8FF" Ref="C36"  Part="1"
-F 0 "C31" H 7218 3046 50  0000 L CNN
+F 0 "C36" H 7218 3046 50  0000 L CNN
 F 1 "47u LKMD0901K470MF" H 7218 2955 50  0000 L CNN
 F 2 "Capacitor_THT:CP_Radial_D8.0mm_P3.50mm" H 7138 2850 50  0001 C CNN
@@
 AR Path="/5F7A3A2A/5F7BF207" Ref="#PWR0201"  Part="1"
 AR Path="/5F7A4E71/5F7BF207" Ref="#PWR0202"  Part="1"
-F 0 "#PWR0197" H 7100 2650 50  0001 C CNN
+F 0 "#PWR0202" H 7100 2650 50  0001 C CNN
 F 1 "+BATT" H 7115 2973 50  0000 C CNN
 F 2 "" H 7100 2800 50  0001 C CNN
@@
 AR Path="/5F7A3A2A/5F76BFEE" Ref="R67"  Part="1"
 AR Path="/5F7A4E71/5F76BFEE" Ref="R70"  Part="1"
-F 0 "R51" H 5019 3704 50  0000 L CNN
+F 0 "R70" H 5019 3704 50  0000 L CNN
 F 1 "10k" H 5019 3795 50  0000 L CNN
 F 2 "Resistor_SMD:R_1206_3216Metric" V 4880 3750 50  0001 C CNN
@@
 AR Path="/5F7A3A2A/5F76CC5E" Ref="R66"  Part="1"
 AR Path="/5F7A4E71/5F76CC5E" Ref="R69"  Part="1"
-F 0 "R50" H 4780 3254 50  0000 R CNN
+F 0 "R69" H 4780 3254 50  0000 R CNN
 F 1 "10k" H 4800 3350 50  0000 R CNN
 F 2 "Resistor_SMD:R_1206_3216Metric" V 4780 3300 50  0001 C CNN
@@
 AR Path="/5F7A3A2A/5F784928" Ref="C68"  Part="1"
 AR Path="/5F7A4E71/5F784928" Ref="C69"  Part="1"
-F 0 "C64" H 6635 3046 50  0000 R CNN
+F 0 "C69" H 6635 3046 50  0000 R CNN
 F 1 "2.2u 100V" H 6635 2955 50  0000 R CNN
 F 2 "Capacitor_SMD:C_1206_3216Metric" H 6788 2850 50  0001 C CNN
@@
 AR Path="/5F7A3A2A/5F7BAC08" Ref="R74"  Part="1"
 AR Path="/5F7A4E71/5F7BAC08" Ref="R76"  Part="1"
-F 0 "R52" V 3203 3300 50  0000 C CNN
+F 0 "R76" V 3203 3300 50  0000 C CNN
 F 1 "1k" V 3294 3300 50  0000 C CNN
 F 2 "Resistor_SMD:R_0603_1608Metric" V 3250 2500 50  0001 C CNN
@@
 AR Path="/5F7A3A2A/5F7BB10C" Ref="R75"  Part="1"
 AR Path="/5F7A4E71/5F7BB10C" Ref="R77"  Part="1"
-F 0 "R59" V 3293 3400 50  0000 C CNN
+F 0 "R77" V 3293 3400 50  0000 C CNN
 F 1 "1k" V 3384 3400 50  0000 C CNN
 F 2 "Resistor_SMD:R_0603_1608Metric" V 3430 3400 50  0001 C CNN
@@
 AR Path="/5F7A3A2A/6020AE15" Ref="RV5"  Part="1"
 AR Path="/5F7A4E71/6020AE15" Ref="RV6"  Part="1"
-F 0 "RV1" H 8303 3046 50  0000 L CNN
+F 0 "RV6" H 8303 3046 50  0000 L CNN
 F 1 "Varistor" H 8303 2955 50  0000 L CNN
 F 2 "Bobbycar-FOC-hardware:MOV20" V 8130 3000 50  0001 C CNN
