File: Bobbycontroller.kicad_pcb (KiCad board)
At the start: 2 copper layers, 120 x 90 mm, 173 parts, among them J1 Conn_01x01_Male, J2 Conn_01x01_Male, J3 Conn_01x01_Male, J5 Conn_01x01_Male, J6 Conn_01x01_Male, J7 Conn_01x01_Male, Q2L1 MMBT5551, Q2R1 MMBT5551, Q6 MMBT5551, U1 L7805, U10 IRS2304, U11 IRS2304, U12 IRS2304, U13 IRS2304, U14 3PEAK TP09-SR, U2 AMS1117-3.3, U3 STM32F103RCTx, U4 3PEAK TP09-SR, U6 3PEAK TP09-SR, U7 MCP2542FDxMF, U8 IRS2304, U9 IRS2304

Commit message: added footprints, continue layout
Parts:
- added C19: 100n, Capacitor_SMD:C_0603_1608Metric, F.Cu at (214.4, 84.5)
- added C20: 100n, Capacitor_SMD:C_0603_1608Metric, F.Cu at (210.4, 87.0)
- added C21: 100n, Capacitor_SMD:C_0603_1608Metric, F.Cu at (214.4, 82.0)
- added C22: 4.7u, Capacitor_SMD:C_0805_2012Metric, F.Cu at (206.2, 85.2)
- added C23: 100n, Capacitor_SMD:C_0603_1608Metric, F.Cu at (210.4, 84.5)
- added C39: 10n, Capacitor_SMD:C_0603_1608Metric, F.Cu at (210.4, 82.0)
- added C40: 1u, Capacitor_SMD:C_0805_2012Metric, F.Cu at (206.2, 82.2)
- added C41: 4.7n, Capacitor_SMD:C_0805_2012Metric, F.Cu at (221.3, 63.6)
- added C42: 1u, Capacitor_SMD:C_0805_2012Metric, F.Cu at (210.9, 75.9)
- added C43: 0.1u, Capacitor_SMD:C_0603_1608Metric, F.Cu at (241.1, 68.5)
- added C44: 0.1u, Capacitor_SMD:C_0603_1608Metric, F.Cu at (245.1, 65.9)
- added C45: 0.1u, Capacitor_SMD:C_0603_1608Metric, F.Cu at (249.1, 63.4)
- added C6: 100n, Capacitor_SMD:C_0603_1608Metric, F.Cu at (242.5, 76.5)
- added D17: D_TVS_x2_AAC, Package_TO_SOT_SMD:SOT-23, F.Cu at (215.5, 67.8)
- added D18: B5819W, Diode_SMD:D_SOD-123, F.Cu at (216.2, 63.9)
- added D19: 15V TVS C78409, Diode_SMD:D_SMB, F.Cu at (276.4, 101.4)
- added D20: B5819W, Diode_SMD:D_SOD-123, F.Cu at (237.6, 76.9)
- added D21: 51V TVS C310059, Diode_SMD:D_SMC, F.Cu at (178.8, 152.8)
- added D22: 15V C78409, Diode_SMD:D_SMB, F.Cu at (264.0, 101.4)
- added D23: 51V TVS C310059, Diode_SMD:D_SMC, F.Cu at (147.7, 105.0)
- added D24: 51V TVS C310059, Diode_SMD:D_SMC, F.Cu at (147.7, 53.0)
- added D25: 51V TVS C310059, Diode_SMD:D_SMC, F.Cu at (147.7, 79.0)
- added D26: 51V TVS C310059, Diode_SMD:D_SMC, F.Cu at (52.3, 61.1)
- added D27: 51V TVS C310059, Diode_SMD:D_SMC, F.Cu at (52.3, 87.0)
- added D28: 51V TVS C310059, Diode_SMD:D_SMC, F.Cu at (52.3, 35.0)
- added F1: 2A C135342, Fuse:Fuse_1206_3216Metric, F.Cu at (185.0, 134.0)
- added J4: Conn_01x04_Male, Connector_PinHeader_2.54mm:PinHeader_1x04_P2.54mm_Vertical, F.Cu at (211.0, 64.5)
- added J8: Conn_01x05, Connector_PinHeader_2.54mm:PinHeader_1x05_P2.54mm_Vertical, F.Cu at (206.3, 64.5)
- added JP1: SolderJumper_2_Open, Jumper:SolderJumper-2_P1.3mm_Open_RoundedPad1.0x1.5mm, F.Cu at (236.9, 67.5)
- added JP2: SolderJumper_2_Open, Jumper:SolderJumper-2_P1.3mm_Open_RoundedPad1.0x1.5mm, F.Cu at (236.9, 64.0)
- added R45: 1M, Resistor_SMD:R_0603_1608Metric, F.Cu at (215.3, 71.3)
- added R46: 10k, Resistor_SMD:R_0603_1608Metric, F.Cu at (245.1, 63.4)
- added R47: 10k, Resistor_SMD:R_0603_1608Metric, F.Cu at (241.1, 65.9)
- added R48: 60.4, Resistor_SMD:R_0603_1608Metric, F.Cu at (236.8, 70.5)
- added R49: 60.4, Resistor_SMD:R_0603_1608Metric, F.Cu at (241.1, 63.4)
- J10: renamed from UART_R1; value (none) -> UART_R1
- J9: renamed from UART_L1; value (none) -> UART_L1
- moved U7 131.7 mm to (228.0, 73.0)
- moved D13 73.6 mm to (75.0, -10.0)
- moved D14 73.6 mm to (75.0, -8.50)
- moved D15 73.6 mm to (75.0, -7.00)
- moved D16 73.6 mm to (75.0, -5.50)
- moved R41 73.6 mm to (72.0, -10.0)
- moved R42 73.6 mm to (72.0, -8.50)
- moved R43 73.6 mm to (72.0, -7.00)
- moved R44 73.6 mm to (72.0, -5.50)
- moved R25 29.2 mm to (76.0, 55.0)
- moved D4 23.0 mm to (85.5, 62.0)
- moved D5 23.0 mm to (83.0, 62.0)
- moved R1 23.0 mm to (80.0, 65.5)
- moved R22 23.0 mm to (81.5, 52.0)
- moved R23 23.0 mm to (78.5, 52.0)
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Connections:
- Buck1 pad 1: +BATT -> Net-(Buck1-Pad1)
- R53 pad 1: +BATT -> Net-(R53-Pad1)
- R53 pad 2: Net-(R53-Pad2) -> +BATT
- R54 pad 1: Net-(R53-Pad2) -> /MCU/V_BATT_MEAS
- R54 pad 2: /MCU/V_BATT_MEAS -> Net-(R53-Pad1)
- U2 pad 3: (no net) -> Net-(D20-Pad1)
- U3 pad 46: (no net) -> /CONNECTORS/MCU_SWDIO
- U3 pad 49: (no net) -> /CONNECTORS/MCU_SWCLK
- U7 pad 6: (no net) -> /CAN/CANL
- U7 pad 7: (no net) -> /CAN/CANH
Routing:
- net +VSW: track 0.00 -> 140.4 mm
- net L_MTR_SHUNT: track 0.00 -> 39.2 mm
- net R_MTR_SHUNT: track 0.00 -> 38.8 mm
- net Net-(C24-Pad1): track 0.00 -> 25.5 mm
- net Net-(C17-Pad1): track 0.00 -> 25.3 mm
- net Net-(C15-Pad1): track 0.00 -> 24.8 mm
- net Net-(C1-Pad1): track 0.00 -> 24.3 mm
- net Net-(C13-Pad1): track 0.00 -> 24.3 mm
- net Net-(R21-Pad2): track 0.00 -> 23.6 mm
- net Net-(C11-Pad1): track 0.00 -> 23.6 mm
- net Net-(R32-Pad2): track 0.00 -> 22.5 mm
- net Net-(R34-Pad2): track 0.00 -> 22.4 mm
- net Net-(R15-Pad2): track 0.00 -> 22.1 mm
- net Net-(R10-Pad2): track 0.00 -> 21.9 mm
- net Net-(R17-Pad2): track 0.00 -> 21.7 mm
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- added copper zone on B.Cu, net /L_MTR_PHA
- added copper zone on F.Cu, net /L_MTR_PHA
- added copper zone on B.Cu, net /R_MTR_PHA
- added copper zone on F.Cu, net /R_MTR_PHA
- added copper zone on B.Cu, net GND
- added copper zone on B.Cu, net L_MTR_PHB
- added copper zone on F.Cu, net L_MTR_PHB
- added copper zone on B.Cu, net L_MTR_PHC
- added copper zone on F.Cu, net L_MTR_PHC
- added copper zone on B.Cu, net R_MTR_PHB
- added copper zone on F.Cu, net R_MTR_PHB
- added copper zone on B.Cu, net R_MTR_PHC
- added copper zone on F.Cu, net R_MTR_PHC

Commit message: continue analog layout
Parts:
- added D29: LED, LED_SMD:LED_0603_1608Metric, F.Cu at (110.3, 102.0)
- added D30: LED, LED_SMD:LED_0603_1608Metric, F.Cu at (87.7, 102.1)
- added D31: LED, LED_SMD:LED_0603_1608Metric, F.Cu at (107.2, 102.0)
- added D32: LED, LED_SMD:LED_0603_1608Metric, F.Cu at (90.8, 102.1)
- added D33: LED, LED_SMD:LED_0603_1608Metric, F.Cu at (104.2, 102.1)
- added D34: LED, LED_SMD:LED_0603_1608Metric, F.Cu at (93.8, 102.1)
- moved J4 97.0 mm to (116.5, 86.4), turned to 180 degrees
- moved J8 58.8 mm to (258.1, 36.6)
- moved D13 50.6 mm to (78.5, 40.5)
- moved D14 50.6 mm to (78.5, 42.0)
- moved D15 50.6 mm to (78.5, 43.5)
- moved D16 50.6 mm to (78.5, 45.0)
- moved R41 50.6 mm to (75.5, 40.5)
- moved R42 50.6 mm to (75.5, 42.0)
- moved R43 50.6 mm to (75.5, 43.5)
- moved R44 50.6 mm to (75.5, 45.0)
- moved C10 34.0 mm to (79.8, 63.4), turned to 90 degrees
- moved R50L1 20.9 mm to (110.8, 39.9), turned to 270 degrees
- moved R3 19.6 mm to (127.0, 39.3), turned to 180 degrees
- moved D3 19.0 mm to (123.7, 46.6), turned to 270 degrees
- moved R2 16.6 mm to (127.0, 41.0), turned to 180 degrees
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Connections:
- R16L1 pad 1: +3V3 -> Net-(D29-Pad1)
- R16L2 pad 1: +3V3 -> Net-(D30-Pad1)
- R17L1 pad 1: +3V3 -> Net-(D31-Pad1)
- R17L2 pad 1: +3V3 -> Net-(D32-Pad1)
- R18L1 pad 1: +3V3 -> Net-(D33-Pad1)
- R18L2 pad 1: +3V3 -> Net-(D34-Pad1)
Routing:
- net R_MTR_SHUNT: track 38.8 -> 103.3 mm, vias 0 -> 4
- net L_MTR_SHUNT: track 39.2 -> 94.7 mm, vias 0 -> 4
- net GND: track 0.00 -> 35.6 mm, vias 0 -> 1
- net +3V3: track 0.00 -> 33.2 mm
- net Net-(D3-Pad1): track 0.00 -> 24.1 mm
- net Net-(D3-Pad2): track 0.00 -> 22.7 mm
- net R_MTR_PHB: track 17.6 -> 32.4 mm, vias 41 -> 42
- net R_MTR_PHC: track 17.6 -> 32.2 mm, vias 41 -> 42
- net L_MTR_PHB: track 17.4 -> 31.1 mm, vias 55 -> 56
- net Net-(C18R1-Pad1): track 0.00 -> 13.2 mm
- net Net-(D6-Pad1): track 0.00 -> 12.9 mm
- net Net-(C18L1-Pad1): track 0.00 -> 12.4 mm
- net Net-(D4-Pad2): track 0.00 -> 12.2 mm
- net Net-(D6-Pad2): track 0.00 -> 11.9 mm
- net Net-(D5-Pad1): track 0.00 -> 9.34 mm
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- removed copper zone on B.Cu, net GND
Other:
- board text added: "3V3 CLK GND DIO"

Commit message: continue board layout, placed all components
Parts:
- added REF**: MountingHole_4.3mm_M4_Pad_Via, MountingHole:MountingHole_4.3mm_M4_Pad_Via, F.Cu at (44.0, 24.0)
- added REF**: MountingHole_4.3mm_M4_Pad_Via, MountingHole:MountingHole_4.3mm_M4_Pad_Via, F.Cu at (156.0, 24.0)
- added REF**: MountingHole_4.3mm_M4_Pad_Via, MountingHole:MountingHole_4.3mm_M4_Pad_Via, F.Cu at (156.0, 106.0)
- added REF**: MountingHole_4.3mm_M4_Pad_Via, MountingHole:MountingHole_4.3mm_M4_Pad_Via, F.Cu at (44.0, 106.0)
- moved D22 166.1 mm to (102.5, 62.6)
- moved R40 162.4 mm to (89.1, 62.0), turned to 90 degrees
- moved R39 159.2 mm to (90.8, 62.1), turned to 90 degrees
- moved D19 153.7 mm to (123.7, 84.8), turned to 90 degrees
- moved C37 153.6 mm to (92.6, 62.1), turned to 90 degrees
- moved C3 144.1 mm to (106.1, 67.2), turned to 90 degrees
- moved J8 138.0 mm to (127.8, 82.3)
- moved U1 137.0 mm to (112.8, 63.6)
- moved D21 136.7 mm to (82.9, 55.4), turned to 270 degrees
- moved Buck1 136.6 mm to (90.1, 54.7), turned to 90 degrees
- moved C45 135.7 mm to (116.3, 91.2), turned to 270 degrees
- moved C25 135.0 mm to (118.5, 43.1), turned to 90 degrees
- moved R46 134.4 mm to (113.1, 88.2), turned to 270 degrees
- moved C26 133.9 mm to (119.4, 75.0)
- moved F1 132.6 mm to (83.3, 48.9), turned to 180 degrees
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Connections:
- C43 pad 2: +3V3 -> GND
- C44 pad 2: +5V -> GND
- HALL_R1 pad 1: Net-(C2-Pad1) -> GND
- HALL_R1 pad 5: GND -> Net-(C2-Pad1)
- J10 pad 1: +VSW -> GND
- J10 pad 4: GND -> +VSW
- J9 pad 1: +VSW -> GND
- J9 pad 4: GND -> +VSW
- R16L2 pad 2: Net-(HALL_R1-Pad2) -> Net-(HALL_R1-Pad4)
- R18L2 pad 2: Net-(HALL_R1-Pad4) -> Net-(HALL_R1-Pad2)
- R19L2 pad 1: Net-(HALL_R1-Pad4) -> Net-(HALL_R1-Pad2)
- R21L2 pad 1: Net-(HALL_R1-Pad2) -> Net-(HALL_R1-Pad4)
- R35 pad 2: Net-(J10-Pad2) -> Net-(J10-Pad3)
- R36 pad 2: Net-(J9-Pad2) -> Net-(J9-Pad3)
- R37 pad 2: Net-(J10-Pad3) -> Net-(J10-Pad2)
- R38 pad 2: Net-(J9-Pad3) -> Net-(J9-Pad2)
Routing:
- net GND: track 35.6 -> 90.3 mm, vias 1 -> 11
- net /CAN/CANL: track 0.00 -> 28.6 mm
- net +VSW: track 140.8 -> 164.7 mm
- net +3V3: track 33.2 -> 56.5 mm
- net /CAN/CANH: track 0.00 -> 21.1 mm
- net Net-(C42-Pad1): track 0.00 -> 12.4 mm
- net /CONNECTORS/MCU_SWCLK: track 0.00 -> 11.1 mm, vias 0 -> 1
- net /CONNECTORS/MCU_SWDIO: track 0.00 -> 10.6 mm, vias 0 -> 1
- net Net-(C45-Pad1): track 0.00 -> 7.46 mm
- net Net-(C41-Pad1): track 0.00 -> 7.28 mm
- net +BATT: track 3.90 -> 10.7 mm, vias 72 -> 74
- net Net-(JP1-Pad2): track 0.00 -> 6.14 mm, vias 0 -> 2
- net +5V: track 0.00 -> 4.58 mm
- net Net-(JP2-Pad1): track 0.00 -> 3.99 mm
- net Net-(J10-Pad2): track 0.00 -> 3.50 mm
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- added copper zone on B.Cu, net GND
Other:
- board text added: "CANH CANL GND VBUS SHIELD"

Commit message: layout without hall sensor leds
Parts:
- moved D23 1.50 mm to (146.2, 104.9)
- moved C44 0.28 mm to (115.2, 80.8)
- moved D29 0.21 mm to (110.5, 102.0)
Routing:
- net +3V3: track 56.5 -> 232.6 mm, vias 0 -> 6
- net +5V: track 4.58 -> 137.3 mm, vias 0 -> 7
- net +VSW: track 164.7 -> 294.2 mm
- net /CURRENT_SENSE/L_MTR_OVERCUR: track 1.58 -> 84.6 mm, vias 0 -> 2
- net /CURRENT_SENSE/L_MTR_CURR: track 2.76 -> 78.1 mm, vias 0 -> 4
- net /R_MTR_PHC/H_BRIDGE_LO: track 0.00 -> 72.5 mm, vias 0 -> 2
- net GND: track 90.3 -> 161.8 mm, vias 11 -> 189
- net /R_MTR_PHC/H_BRIDGE_HI: track 0.00 -> 68.0 mm, vias 0 -> 2
- net /L_MTR_PHC/H_BRIDGE_LO: track 0.00 -> 64.9 mm, vias 0 -> 2
- net /CURRENT_SENSE/R_MTR_CURR: track 2.89 -> 66.6 mm, vias 0 -> 4
- net /MCU/L_MTR_PHC_SENSE: track 2.49 -> 66.0 mm, vias 0 -> 2
- net /MCU/V_BATT_MEAS: track 1.50 -> 62.9 mm, vias 0 -> 4
- net /MCU/L_MTR_PHB_SENSE: track 2.22 -> 63.6 mm, vias 0 -> 2
- net /CURRENT_SENSE/R_MTR_OVERCUR: track 0.00 -> 60.2 mm, vias 0 -> 4
- net /L_MTR_PHC/H_BRIDGE_HI: track 0.00 -> 58.6 mm, vias 0 -> 2
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- added copper zone on F.Cu, net GND

Commit message: finish design
Parts:
- removed REF** (x4): MountingHole_4.3mm_M4_Pad_Via, MountingHole:MountingHole_4.3mm_M4_Pad_Via
- added J11: Conn_01x01, MountingHole:MountingHole_4mm_Pad_Via, F.Cu at (44.0, 24.0)
- added J12: Conn_01x01, MountingHole:MountingHole_4mm_Pad_Via, F.Cu at (156.0, 24.0)
- added J13: Conn_01x01, MountingHole:MountingHole_4mm_Pad_Via, F.Cu at (156.0, 106.0)
- added J14: Conn_01x01, MountingHole:MountingHole_4mm_Pad_Via, F.Cu at (44.0, 106.0)
- added R16L3: 2K2, Resistor_SMD:R_0603_1608Metric, F.Cu at (109.9, 101.3)
- added R16L4: 2K2, Resistor_SMD:R_0603_1608Metric, F.Cu at (87.0, 101.3)
- added R17L3: 2K2, Resistor_SMD:R_0603_1608Metric, F.Cu at (106.7, 101.3)
- added R17L4: 2K2, Resistor_SMD:R_0603_1608Metric, F.Cu at (90.2, 101.3)
- added R18L3: 2K2, Resistor_SMD:R_0603_1608Metric, F.Cu at (103.5, 101.3)
- added R18L4: 2K2, Resistor_SMD:R_0603_1608Metric, F.Cu at (93.4, 101.3)
- moved D34 1.40 mm to (95.0, 101.3), turned to 90 degrees
- moved D31 1.29 mm to (108.3, 101.3), turned to 90 degrees
- moved D32 1.28 mm to (91.8, 101.3), turned to 90 degrees
- moved D29 1.22 mm to (111.5, 101.3), turned to 90 degrees
- moved D33 1.20 mm to (105.1, 101.3), turned to 90 degrees
- moved D30 1.19 mm to (88.6, 101.3), turned to 90 degrees
- moved R16L1 0.50 mm to (111.5, 104.5)
- moved R18L2 0.50 mm to (95.0, 104.5)
- moved R19L2 0.40 mm to (93.4, 104.5)
- moved R21L1 0.40 mm to (109.9, 104.5)
- moved R17L1 0.30 mm to (108.3, 104.5)
- moved R17L2 0.30 mm to (91.8, 104.5)
- moved R20L1 0.20 mm to (106.7, 104.5)
- moved R20L2 0.20 mm to (90.2, 104.5)
- moved R16L2 0.10 mm to (88.6, 104.5)
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Routing:
- net +3V3: track 232.6 -> 277.8 mm
- net Net-(HALL_R1-Pad3): track 0.00 -> 8.45 mm
- net Net-(HALL_L1-Pad4): track 0.00 -> 8.45 mm
- net Net-(HALL_L1-Pad2): track 0.00 -> 8.34 mm
- net Net-(HALL_R1-Pad4): track 0.00 -> 8.25 mm
- net Net-(HALL_L1-Pad3): track 0.00 -> 8.25 mm
- net Net-(HALL_R1-Pad2): track 0.00 -> 8.18 mm
- net /CONNECTORS/L_MTR_HALL_PHC: track 58.4 -> 60.3 mm
- net Net-(D34-Pad1): track 0.00 -> 1.62 mm
- net Net-(D33-Pad1): track 0.00 -> 1.62 mm
- net Net-(D32-Pad1): track 0.00 -> 1.62 mm
- net Net-(D31-Pad1): track 0.00 -> 1.62 mm
- net Net-(D29-Pad1): track 0.00 -> 1.62 mm
- net Net-(D30-Pad1): track 0.00 -> 1.62 mm
- net /CONNECTORS/L_MTR_HALL_PHB: track 56.9 -> 56.3 mm
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Other:
- board text added: "5V A B C GND"

Commit message: finish layout
Parts:
- added C46: 2.2u 100V, Capacitor_SMD:C_1206_3216Metric, B.Cu at (93.4, 16.5)
- added C47: 2.2u 100V, Capacitor_SMD:C_1206_3216Metric, B.Cu at (91.1, 16.5)
- added C48: 2.2u 100V, Capacitor_SMD:C_1206_3216Metric, B.Cu at (53.6, 16.5)
- added C49: 2.2u 100V, Capacitor_SMD:C_1206_3216Metric, B.Cu at (88.8, 16.5)
- added C50: 2.2u 100V, Capacitor_SMD:C_1206_3216Metric, B.Cu at (51.3, 16.5)
- added C51: 2.2u 100V, Capacitor_SMD:C_1206_3216Metric, B.Cu at (75.0, 16.5)
- added C52: 2.2u 100V, Capacitor_SMD:C_1206_3216Metric, B.Cu at (86.6, 16.5)
- added C53: 2.2u 100V, Capacitor_SMD:C_1206_3216Metric, B.Cu at (49.0, 16.5)
- added C54: 2.2u 100V, Capacitor_SMD:C_1206_3216Metric, B.Cu at (64.9, 16.6)
- added C55: 2.2u 100V, Capacitor_SMD:C_1206_3216Metric, B.Cu at (79.6, 16.5)
- added C56: 2.2u 100V, Capacitor_SMD:C_1206_3216Metric, B.Cu at (46.7, 16.5)
- added C57: 2.2u 100V, Capacitor_SMD:C_1206_3216Metric, B.Cu at (62.6, 16.6)
- added C58: 2.2u 100V, Capacitor_SMD:C_1206_3216Metric, B.Cu at (77.3, 16.5)
- added C59: 2.2u 100V, Capacitor_SMD:C_1206_3216Metric, B.Cu at (60.3, 16.6)
- added J15: -BATT, MountingHole:MountingHole_2.7mm_M2.5_Pad, F.Cu at (70.0, 13.4)
- added J16: +BATT, MountingHole:MountingHole_2.7mm_M2.5_Pad, F.Cu at (70.0, 22.0)
- added JP3: Jumper_2_Bridged, Jumper:SolderJumper-2_P1.3mm_Bridged2Bar_RoundedPad1.0x1.5mm, F.Cu at (62.2, 24.6)
- moved Buck1 31.6 mm to (60.1, 44.7)
- moved D13 31.6 mm to (48.5, 30.4)
- moved D14 31.6 mm to (48.5, 31.9)
- moved D15 31.6 mm to (48.5, 33.5)
- moved D16 31.6 mm to (48.5, 35.0)
- moved D30 31.6 mm to (58.6, 91.3)
- moved D4 31.6 mm to (46.4, 38.5)
- moved R18L4 31.6 mm to (63.4, 91.3)
- moved R19L2 31.6 mm to (63.4, 94.5)
- moved R23 31.6 mm to (44.4, 40.8)
- moved R24 31.6 mm to (43.6, 38.5)
- moved R26 31.6 mm to (43.6, 36.9)
- moved R29 31.6 mm to (43.9, 64.6)
- moved R30 31.6 mm to (45.9, 56.5)
- moved R31 31.6 mm to (43.9, 63.0)
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Routing:
- net GND: track 161.8 -> 164.8 mm
- net -BATT: track 0.00 -> 2.65 mm, vias 180 -> 172
Other:
- board text added: "GND +BATT"

Commit message: added TVS diodes on HALL inputs
Parts:
- added U15: SRV05-4, Package_TO_SOT_SMD:SOT-23-6, F.Cu at (54.3, 95.2)
- added U5: SRV05-4, Package_TO_SOT_SMD:SOT-23-6, F.Cu at (84.0, 94.6)
- turned LS1 to 90 degrees
Connections:
- net Net-(C2-Pad1) renamed /CONNECTORS/Hall_VCC
- net Net-(HALL_L1-Pad2) renamed /CONNECTORS/Hall_L_1
- net Net-(HALL_L1-Pad3) renamed /CONNECTORS/Hall_L_2
- net Net-(HALL_L1-Pad4) renamed /CONNECTORS/Hall_L_3
- net Net-(HALL_R1-Pad2) renamed /CONNECTORS/Hall_R_3
- net Net-(HALL_R1-Pad3) renamed /CONNECTORS/Hall_R_2
- net Net-(HALL_R1-Pad4) renamed /CONNECTORS/Hall_R_1
Routing:
- net /CONNECTORS/Hall_VCC: track 24.7 -> 48.8 mm
- net /CONNECTORS/Hall_R_3: track 8.18 -> 23.7 mm, vias 0 -> 1
- net /CONNECTORS/Hall_L_3: track 8.45 -> 23.5 mm, vias 0 -> 1
- net GND: track 164.8 -> 176.9 mm, vias 208 -> 210
- net /CONNECTORS/Hall_L_2: track 8.25 -> 19.3 mm, vias 0 -> 1
- net /CONNECTORS/Hall_R_2: track 8.45 -> 19.2 mm, vias 0 -> 1
- net Net-(D1AR1-Pad2): track 8.79 -> 16.1 mm, vias 0 -> 1
- net /CONNECTORS/Hall_R_1: track 8.25 -> 10.2 mm
- net /CONNECTORS/Hall_L_1: track 8.34 -> 10.1 mm
- net /MCU/L_MTR_PHB_SENSE: track 63.4 -> 64.2 mm
Other:
- board text added: "15V TX RX GND"

Commit message: add logos
Parts:
- added G***: LOGO, Local:lenas_bobbycar_logo, F.Cu at (50.9, 69.5)
- moved LS1 0.71 mm to (46.0, 88.5), turned to 0 degrees
Routing:
- net Net-(D1AR1-Pad2): track 16.1 -> 8.79 mm, vias 1 -> 0
- net GND: vias 210 -> 215
Other:
- board text added: "Bobbycar Graz FOC Motor Controller"
- board text added: "Version 1.0"
