File: Bobbycontroller.kicad_pcb (KiCad board)
At the start: 2 copper layers, 120 x 90 mm, 244 parts, among them J1 Conn_01x01_Male, J10 UART_R1, J11 Conn_01x01, J12 Conn_01x01, J13 Conn_01x01, J14 Conn_01x01, J15 -BATT, J16 +BATT, J2 Conn_01x01_Male, J3 Conn_01x01_Male, J4 Conn_01x04_Male, J5 Conn_01x01_Male, J6 Conn_01x01_Male, J7 Conn_01x01_Male, J8 Conn_01x05, J9 UART_L1, Q2L1 MMBT5551, Q2R1 MMBT5551, Q6 MMBT5551, U1 L7805, U10 IRS2304, U11 IRS2304, U12 IRS2304, U13 IRS2304, U14 3PEAK TP09-SR, U15 SRV05-4, U2 AMS1117-3.3, U3 STM32F103RCTx, U4 3PEAK TP09-SR, U5 SRV05-4, U6 3PEAK TP09-SR, U7 MCP2542FDxMF, U8 IRS2304, U9 IRS2304

Commit message: minor changes
Parts:
- moved C18 1.43 mm to (37.6, 92.8)
- moved J10 1.00 mm to (50.7, 98.0)
Routing:
- net +VSW: track 294.2 -> 295.5 mm
- net Net-(J10-Pad2): track 3.50 -> 2.90 mm

Commit message: Minor changes to PCB; convert footprint library to .pretty format, add to project
Parts:
- removed G***: LOGO, Local:lenas_bobbycar_logo
- removed JP3: Jumper_2_Bridged, Jumper:SolderJumper-2_P1.3mm_Bridged2Bar_RoundedPad1.0x1.5mm
- added LOGO1: Logo_Open_Hardware_Small, Bobbycar-FOC-hardware:lenas_bobbycar_logo, F.Cu at (51.2, 69.5)
- added NT1: Net-Tie_2, NetTie:NetTie-2_SMD_Pad2.0mm, F.Cu at (62.9, 24.0)
- added NT2: Net-Tie_2, NetTie:NetTie-2_SMD_Pad2.0mm, F.Cu at (77.1, 24.0)
- D17: value D_TVS_x2_AAC -> PESD15VL2BT,215
- moved C18L1 0.29 mm to (71.6, 33.8)
- moved R14 0.20 mm to (108.2, 67.0)
Connections:
- J11 pad 1: Net-(J11-Pad1) -> (no net)
- J12 pad 1: Net-(J12-Pad1) -> (no net)
- J13 pad 1: Net-(J13-Pad1) -> (no net)
- J14 pad 1: Net-(J14-Pad1) -> (no net)
Routing:
- net GND: track 176.9 -> 198.6 mm, vias 215 -> 252
- net -BATT: track 2.65 -> 10.8 mm
- net (no net): track 0.00 -> 1.32 mm
- net /CURRENT_SENSE/L_MTR_CURR: track 78.1 -> 79.1 mm
- net R_MTR_PHC: vias 42 -> 56
- net R_MTR_PHB: vias 42 -> 56
- net /R_MTR_PHA: vias 41 -> 55
Other:
- board text added: "blau"
- board text added: "gelb"
- board text added: "grün"

Commit message: modify hall sensor VCC so that overvoltage on one hall sensor will not affect the other motor
Parts:
- added C60: 100n, Capacitor_SMD:C_0603_1608Metric, F.Cu at (67.5, 94.5)
- added D0AL2: 1N4148W, Diode_SMD:D_SOD-123, F.Cu at (69.4, 92.5)
- moved D0AL1 1.85 mm to (69.4, 90.2)
- moved C2 1.26 mm to (70.5, 94.5)
Connections:
- HALL_R1 pad 5: /CONNECTORS/Hall_VCC -> /CONNECTORS/Hall_VCC_2
- U15 pad 5: /CONNECTORS/Hall_VCC -> /CONNECTORS/Hall_VCC_2
Routing:
- net /CONNECTORS/Hall_VCC_2: track 0.00 -> 24.0 mm
- net /CONNECTORS/Hall_VCC: track 48.8 -> 29.6 mm
- net +5V: track 137.3 -> 139.7 mm
- net GND: track 198.6 -> 198.8 mm, vias 252 -> 255

Commit message: change Mosfet Driver to U3115S
Parts:
- added R50: DNP 10k, Resistor_SMD:R_1206_3216Metric, F.Cu at (108.0, 96.6)
- added R51: DNP 10k, Resistor_SMD:R_1206_3216Metric, F.Cu at (114.0, 73.7)
- added R57: DNP 10k, Resistor_SMD:R_1206_3216Metric, F.Cu at (108.2, 70.5)
- added R58: DNP 10k, Resistor_SMD:R_1206_3216Metric, F.Cu at (114.0, 48.6)
- added R60: DNP 10k, Resistor_SMD:R_1206_3216Metric, F.Cu at (108.1, 44.1)
- added R61: DNP 10k, Resistor_SMD:R_1206_3216Metric, F.Cu at (114.0, 22.6)
- added R63: DNP 10k, Resistor_SMD:R_1206_3216Metric, F.Cu at (32.0, 76.0)
- added R64: DNP 10k, Resistor_SMD:R_1206_3216Metric, F.Cu at (25.5, 97.9)
- added R66: DNP 10k, Resistor_SMD:R_1206_3216Metric, F.Cu at (32.0, 50.0)
- added R67: DNP 10k, Resistor_SMD:R_1206_3216Metric, F.Cu at (26.0, 71.9)
- added R69: DNP 10k, Resistor_SMD:R_1206_3216Metric, F.Cu at (32.0, 24.6)
- added R70: DNP 10k, Resistor_SMD:R_1206_3216Metric, F.Cu at (25.5, 45.9)
- U10, U11, U12, U13, U8, U9: value IRS2304 -> IRS2304 || U3115S
Routing:
- net R_MTR_SHUNT: track 103.3 -> 112.3 mm
- net L_MTR_SHUNT: track 94.7 -> 103.2 mm
- net R_MTR_PHB: track 32.4 -> 40.5 mm
- net L_MTR_PHB: track 31.1 -> 38.9 mm, vias 56 -> 55
- net /L_MTR_PHA: track 18.5 -> 26.2 mm, vias 55 -> 54
- net /R_MTR_PHA: track 17.8 -> 25.3 mm
- net L_MTR_PHC: track 24.5 -> 31.8 mm, vias 56 -> 55
- net R_MTR_PHC: track 32.2 -> 37.5 mm
- net Net-(R13-Pad2): track 8.54 -> 12.2 mm
- net Net-(R14-Pad2): track 8.56 -> 12.1 mm
- net Net-(R16-Pad2): track 8.54 -> 11.6 mm
- net Net-(R28-Pad2): track 8.50 -> 11.6 mm
- net Net-(R18-Pad2): track 8.00 -> 11.0 mm
- net Net-(R32-Pad2): track 22.6 -> 25.0 mm
- net Net-(R21-Pad2): track 23.3 -> 25.7 mm
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
Commit message: add silk screen, change diodes at DCDC converters, remove overcurrent detection, add 100nf
Parts:
- removed C16L1, C16R1: 100n, Capacitor_SMD:C_0603_1608Metric
- removed Q2L1, Q2R1: MMBT5551, Package_TO_SOT_SMD:SOT-23
- removed R50L1, R50R1: 20k, Resistor_SMD:R_0603_1608Metric
- removed R51L1, R51R1: 510, Resistor_SMD:R_0603_1608Metric
- removed R52L1, R52R1: 1k, Resistor_SMD:R_0603_1608Metric
- added C61: 100nF 100V, Capacitor_SMD:C_0603_1608Metric, F.Cu at (56.1, 52.1)
- added C62: 100nF, Capacitor_SMD:C_0603_1608Metric, F.Cu at (64.2, 54.3)
- added D0AL3: 1N4148W, Diode_SMD:D_SOD-123, F.Cu at (95.0, 93.4)
- added D0AL4: 1N4148W, Diode_SMD:D_SOD-123, F.Cu at (45.2, 81.3)
- C37: value 100nF -> 33n
- R10, R13, R14, R15, R16, R17, R18, R21, R28, R32, R33, R34: value 68 -> 20k
- R51, R58, R61, R64, R67, R70: value DNP 10k -> 10k IRF->DNP
Connections:
- D22 pad 1: Net-(Buck1-Pad2) -> +VSW
- J10 pad 4: +VSW -> Net-(D0AL4-Pad1)
- J9 pad 4: +VSW -> Net-(D0AL3-Pad1)
- U3 pad 22: /CURRENT_SENSE/R_MTR_OVERCUR -> (no net)
- U3 pad 33: /CURRENT_SENSE/L_MTR_OVERCUR -> (no net)
Routing:
- net /CURRENT_SENSE/L_MTR_OVERCUR: track 85.0 -> 0.00 mm, vias 2 -> 0
- net /CURRENT_SENSE/R_MTR_OVERCUR: track 60.2 -> 0.00 mm, vias 4 -> 0
- net +3V3: track 277.8 -> 257.7 mm
- net Net-(D0AL4-Pad1): track 0.00 -> 18.3 mm, vias 0 -> 1
- net Net-(Q2L1-Pad2): track 6.36 -> 0.00 mm
- net Net-(D0AL3-Pad1): track 0.00 -> 3.29 mm
- net Net-(Buck1-Pad1): track 11.3 -> 14.5 mm
- net Net-(Q2R1-Pad2): track 3.07 -> 0.00 mm
- net Net-(Buck1-Pad2): track 21.2 -> 18.2 mm
- net /R_MTR_PH_SENSE/PH_AMP_A_OUT: track 45.2 -> 47.5 mm
- net +VSW: track 295.5 -> 293.5 mm, vias 0 -> 2
- net Net-(Q2R1-Pad1): track 1.70 -> 0.00 mm
- net Net-(Q2L1-Pad1): track 1.63 -> 0.00 mm
- net R_MTR_SHUNT: track 112.3 -> 110.7 mm
- net L_MTR_SHUNT: track 103.2 -> 101.7 mm
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Other:
- board text added: "Bobbycar Graz Dual FOC Motor Controller"
- board text added: "max. 12S (50.4V) max. 32A DC current (continuous)"
- board text added: "max. 12S (50.4V) max. 32A DC current max. 50A motor phase current"
- board text removed: "Bobbycar Graz FOC Motor Controller"

Commit message: fix silkscreen component references
Other:
- board text added: "blue"
- board text added: "green"
- board text added: "yellow"
- board text removed: "blau"
- board text removed: "gelb"
- board text removed: "grün"
Changed lines of the file:
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@@
   (general
     (thickness 1.6)
-    (drawings 63)
+    (drawings 66)
     (tracks 2840)
     (zones 0)
@@
   (page A4)
   (layers
-    (0 F.Cu signal)
-    (31 B.Cu signal)
+    (0 F.Cu signal hide)
+    (31 B.Cu signal hide)
     (32 B.Adhes user)
     (33 F.Adhes user)
     (34 B.Paste user)
     (35 F.Paste user)
-    (36 B.SilkS user)
+    (36 B.SilkS user hide)
     (37 F.SilkS user)
     (38 B.Mask user)
@@
     (tags capacitor)
     (attr smd)
-    (fp_text reference C61 (at 0 -1.43 90) (layer F.SilkS)
+    (fp_text reference C61 (at 3 -0.225 90) (layer F.SilkS)
       (effects (font (size 1 1) (thickness 0.15)))
     )
@@
     (tags SOD-123)
     (attr smd)
-    (fp_text reference D0AL4 (at -4.8 0.85) (layer F.SilkS)
+    (fp_text reference D0AL4 (at -4.775 -0.05) (layer F.SilkS)
       (effects (font (size 1 1) (thickness 0.15)))
     )
@@
     (tags SOD-123)
     (attr smd)
-    (fp_text reference D0AL3 (at 0 -2 90) (layer F.SilkS)
+    (fp_text reference D0AL3 (at -0.175 -1.875 90) (layer F.SilkS)
       (effects (font (size 1 1) (thickness 0.15)))
     )
@@
     (tags SOD-123)
     (attr smd)
-    (fp_text reference D0AL2 (at 0 -2) (layer F.SilkS)
+    (fp_text reference D0AL2 (at 1.35 -4.075) (layer F.SilkS)
       (effects (font (size 1 1) (thickness 0.15)))
     )
@@
     (tags "net tie")
     (attr virtual)
-    (fp_text reference NT2 (at 0 -2 90) (layer F.SilkS)
+    (fp_text reference NT2 (at 1.672 -2.24 90) (layer F.SilkS)
       (effects (font (size 1 1) (thickness 0.15)))
     )
@@
     (tags "net tie")
     (attr virtual)
-    (fp_text reference NT1 (at 0 -2 270) (layer F.SilkS)
+    (fp_text reference NT1 (at 0.872 2.64 270) (layer F.SilkS)
       (effects (font (size 1 1) (thickness 0.15)))
     )
@@
     (tags resistor)
     (attr smd)
-    (fp_text reference R18L4 (at -4.7 -3.2 90) (layer F.SilkS)
+    (fp_text reference R18L4 (at -4.675 -4.075 90) (layer F.SilkS)
       (effects (font (size 1 1) (thickness 0.15)))
     )
@@
     (descr "Through hole straight pin header, 1x04, 2.54mm pitch, single row")
     (tags "Through hole pin header THT 1x04 2.54mm single row")
-    (fp_text reference J9 (at 2 -0.6) (layer F.SilkS)
+    (fp_text reference J9 (at 2.775 -0.75) (layer F.SilkS)
       (effects (font (size 1 1) (thickness 0.15)))
     )
@@
     (tags diode)
     (attr smd)
-    (fp_text reference D34 (at 3.8 3.2 90) (layer F.SilkS)
+    (fp_text reference D34 (at 7.325 1.475 90) (layer F.SilkS)
       (effects (font (size 1 1) (thickness 0.15)))
     )
@@
     (tags resistor)
     (attr smd)
-    (fp_text reference R38R1 (at -1.55 3.725) (layer F.SilkS)
+    (fp_text reference R38R1 (at 0.825 -1.575) (layer F.SilkS)
       (effects (font (size 1 1) (thickness 0.15)))
     )
@@
     (tags resistor)
     (attr smd)
-    (fp_text reference R38L1 (at 0.75 -3.025) (layer F.SilkS)
+    (fp_text reference R38L1 (at 0.6 1.8) (layer F.SilkS)
       (effects (font (size 1 1) (thickness 0.15)))
     )
@@
     (tags resistor)
     (attr smd)
-    (fp_text reference R40 (at 0.245 -3.91 90) (layer F.SilkS)
+    (fp_text reference R40 (at -2.88 0.09 90) (layer F.SilkS)
       (effects (font (size 1 1) (thickness 0.15)))
     )
@@
     (tags resistor)
     (attr smd)
-    (fp_text reference R39 (at 0.22 -4.21 90) (layer F.SilkS)
+    (fp_text reference R39 (at -2.905 -0.06 90) (layer F.SilkS)
       (effects (font (size 1 1) (thickness 0.15)))
     )
@@
     (tags resistor)
     (attr smd)
-    (fp_text reference R37 (at 0.05 2.65 90) (layer F.SilkS)
+    (fp_text reference R37 (at -0.15 2.675 90) (layer F.SilkS)
       (effects (font (size 1 1) (thickness 0.15)))
     )
@@
     (tags resistor)
     (attr smd)
-    (fp_text reference R36 (at -3.1 0.1 90) (layer F.SilkS)
+    (fp_text reference R36 (at -2.9 0.1 90) (layer F.SilkS)
       (effects (font (size 1 1) (thickness 0.15)))
     )
@@
     (tags resistor)
     (attr smd)
-    (fp_text reference R35 (at 0 2.45 90) (layer F.SilkS)
+    (fp_text reference R35 (at -0.025 2.475 90) (layer F.SilkS)
       (effects (font (size 1 1) (thickness 0.15)))
     )
@@
     (tags resistor)
     (attr smd)
-    (fp_text reference R30 (at 1.2 -1.4) (layer F.SilkS)
+    (fp_text reference R30 (at 0.2 -1.425) (layer F.SilkS)
       (effects (font (size 1 1) (thickness 0.15)))
     )
@@
     (tags SOD-123)
     (attr smd)
-    (fp_text reference D0AL1 (at 1.25 -3.2 90) (layer F.SilkS)
+    (fp_text reference D0AL1 (at 1.225 -2.975 180) (layer F.SilkS)
       (effects (font (size 1 1) (thickness 0.15)))
     )
@@
     (tags SOD-123)
     (attr smd)
-    (fp_text reference D10 (at 3.7 0) (layer F.SilkS)
+    (fp_text reference D10 (at 3.7 -0.025) (layer F.SilkS)
       (effects (font (size 1 1) (thickness 0.15)))
     )
@@
     (tags SOD-123)
     (attr smd)
-    (fp_text reference D5 (at -0.6 -1.55) (layer F.SilkS)
+    (fp_text reference D5 (at -0.1 -1.825) (layer F.SilkS)
       (effects (font (size 1 1) (thickness 0.15)))
     )
@@
     (tags SOD-123)
     (attr smd)
-    (fp_text reference D1 (at 0 -0.2 180) (layer F.SilkS)
+    (fp_text reference D1 (at -3.125 -2.375 180) (layer F.SilkS)
       (effects (font (size 1 1) (thickness 0.15)))
     )
@@
     (tags capacitor)
     (attr smd)
-    (fp_text reference C37 (at 0.12 -4.66 90) (layer F.SilkS)
+    (fp_text reference C37 (at -2.905 -0.385 90) (layer F.SilkS)
       (effects (font (size 1 1) (thickness 0.15)))
     )
@@
     (descr "Generic Buzzer, D12mm height 9.5mm with RM7.6mm")
     (tags buzzer)
-    (fp_text reference LS1 (at -1.5 -4.9) (layer F.SilkS)
+    (fp_text reference LS1 (at -1.675 -5.1) (layer F.SilkS)
       (effects (font (size 1 1) (thickness 0.15)))
     )
@@
     )
   )
+  (gr_text yellow (at 34.675 32.75 90) (layer F.SilkS)
+    (effects (font (size 1 1) (thickness 0.15)))
+  )
+  (gr_text blue (at 34.75 84.825 90) (layer F.SilkS)
+    (effects (font (size 1 1) (thickness 0.15)))
+  )
+  (gr_text blue (at 34.65 59 90) (layer F.SilkS)
+    (effects (font (size 1 1) (thickness 0.15)))
+  )
   (gr_text "max. 12S (50.4V)\nmax. 32A DC current\nmax. 50A motor \nphase current" (at 225.5 46.55) (layer F.SilkS)
     (effects (font (size 0.8 0.8) (thickness 0.15)) (justify left))
@@
     (effects (font (size 0.8 0.8) (thickness 0.15)) (justify left))
   )
-  (gr_text gelb (at 105.25 35 90) (layer F.SilkS)
+  (gr_text yellow (at 105.25 35 90) (layer F.SilkS)
     (effects (font (size 1 1) (thickness 0.15)))
   )
-  (gr_text blau (at 105.25 61 90) (layer F.SilkS)
+  (gr_text blue (at 105.25 61 90) (layer F.SilkS)
     (effects (font (size 1 1) (thickness 0.15)))
   )
-  (gr_text grün (at 105.25 87 90) (layer F.SilkS)
+  (gr_text green (at 105.225 87.9 90) (layer F.SilkS)
     (effects (font (size 1 1) (thickness 0.15)))
   )

Commit message: fix labels
Other:
- board text removed: "max. 12S (50.4V) max. 32A DC current max. 50A motor phase current"

Commit message: round board corners
Other:
- outline, holes or cut-outs redrawn
- board text added: "Dual FOC Motor Controller @peterpoetzi @mickdermack"
- board text removed: "Bobbycar Graz Dual FOC Motor Controller"
Changed lines of the file:
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@@
   (general
     (thickness 1.6)
-    (drawings 65)
+    (drawings 69)
     (tracks 2840)
     (zones 0)
@@
   (page A4)
   (layers
-    (0 F.Cu signal hide)
-    (31 B.Cu signal hide)
+    (0 F.Cu signal)
+    (31 B.Cu signal)
     (32 B.Adhes user)
     (33 F.Adhes user)
@@
     (tags capacitor)
     (attr smd)
-    (fp_text reference C3 (at 0 -1.43 90) (layer F.SilkS)
+    (fp_text reference C3 (at 1.24 -1.43 90) (layer F.SilkS)
       (effects (font (size 1 1) (thickness 0.15)))
     )
@@
     )
   )
+  (gr_arc (start 128 12) (end 130 12) (angle -90) (layer Edge.Cuts) (width 0.05))
+  (gr_arc (start 128 98) (end 128 100) (angle -90) (layer Edge.Cuts) (width 0.05))
+  (gr_arc (start 12 98) (end 10 98) (angle -90) (layer Edge.Cuts) (width 0.05))
+  (gr_arc (start 12 12) (end 12 10) (angle -90) (layer Edge.Cuts) (width 0.05))
   (gr_text yellow (at 34.675 32.75 90) (layer F.SilkS)
     (effects (font (size 1 1) (thickness 0.15)))
@@
     (effects (font (size 1.5 1.5) (thickness 0.3)))
   )
-  (gr_text "Bobbycar Graz\nDual FOC Motor Controller" (at 64.4 59) (layer F.SilkS)
-    (effects (font (size 1.5 1.5) (thickness 0.3)))
+  (gr_text "Dual FOC Motor Controller\n@peterpoetzi @mickdermack" (at 63 59) (layer F.SilkS)
+    (effects (font (size 1.2 1.2) (thickness 0.2)))
   )
   (gr_text "15V TX RX GND" (at 92.4 99.5) (layer F.SilkS)
@@
     (arrow2b (pts (xy 122 57) (xy 123.126504 56.413579)))
   )
-  (gr_line (start 10 100) (end 10 10) (layer Edge.Cuts) (width 0.05))
-  (gr_line (start 130 100) (end 10 100) (layer Edge.Cuts) (width 0.05))
-  (gr_line (start 130 10) (end 130 100) (layer Edge.Cuts) (width 0.05))
-  (gr_line (start 10 10) (end 130 10) (layer Edge.Cuts) (width 0.05))
+  (gr_line (start 10 98) (end 10 12) (layer Edge.Cuts) (width 0.05))
+  (gr_line (start 128 100) (end 12 100) (layer Edge.Cuts) (width 0.05))
+  (gr_line (start 130 12) (end 130 98) (layer Edge.Cuts) (width 0.05))
+  (gr_line (start 12 10) (end 128 10) (layer Edge.Cuts) (width 0.05))
   (via (at 42 88) (size 0.8) (drill 0.4) (layers F.Cu B.Cu) (net 0))
   (segment (start 69.85 33.147) (end 69.85 34.462482) (width 0.5) (layer F.Cu) (net 0))
