File: Bobbycontroller.kicad_pcb (KiCad board)
At the start: 2 copper layers, 120 x 90 mm, 253 parts, among them J1 Conn_01x01_Male, J10 UART_R1, J11 Conn_01x01, J12 Conn_01x01, J13 Conn_01x01, J14 Conn_01x01, J15 -BATT, J16 +BATT, J2 Conn_01x01_Male, J3 Conn_01x01_Male, J4 Conn_01x04_Male, J5 Conn_01x01_Male, J6 Conn_01x01_Male, J7 Conn_01x01_Male, J8 Conn_01x05, J9 UART_L1, Q6 MMBT5551, U1 L7805, U10 IRS2304 || U3115S, U11 IRS2304 || U3115S, U12 IRS2304 || U3115S, U13 IRS2304 || U3115S, U14 3PEAK TP09-SR, U15 SRV05-4, U2 AMS1117-3.3, U3 STM32F103RCTx, U4 3PEAK TP09-SR, U5 SRV05-4, U6 3PEAK TP09-SR, U7 MCP2542FDxMF, U8 IRS2304 || U3115S, U9 IRS2304 || U3115S

Commit message: added capacitors
Parts:
- added C63: 100nF, Capacitor_SMD:C_0603_1608Metric, F.Cu at (76.8, 61.2)
- added C64: 2.2u 100V, Capacitor_SMD:C_1206_3216Metric, B.Cu at (123.3, 31.5)
- added C65: 2.2u 100V, Capacitor_SMD:C_1206_3216Metric, B.Cu at (123.3, 83.5)
- added C66: 2.2u 100V, Capacitor_SMD:C_1206_3216Metric, B.Cu at (123.3, 57.5)
- added C67: 2.2u 100V, Capacitor_SMD:C_1206_3216Metric, B.Cu at (17.2, 62.6)
- added C68: 2.2u 100V, Capacitor_SMD:C_1206_3216Metric, B.Cu at (17.1, 88.4)
- added C69: 2.2u 100V, Capacitor_SMD:C_1206_3216Metric, B.Cu at (17.2, 36.5)
- C25: value 470u 25V LKME0901E471MF -> 100u || 470u 25V LKME0901E471MF
Routing:
- net Net-(C63-Pad1): track 4.83 -> 10.1 mm
- net /L_MTR_PHB/H_BRIDGE_HI: track 45.3 -> 46.2 mm

Commit message: add resistors on mosfet driver inputs, change board corners, fix labels
Parts:
- added R52: 1k, Resistor_SMD:R_0603_1608Metric, F.Cu at (94.3, 86.5)
- added R59: 1k, Resistor_SMD:R_0603_1608Metric, F.Cu at (94.3, 84.9)
- added R62: 1k, Resistor_SMD:R_0603_1608Metric, F.Cu at (95.6, 59.5)
- added R65: 1k, Resistor_SMD:R_0603_1608Metric, F.Cu at (95.6, 57.8)
- added R68: 1k, Resistor_SMD:R_0603_1608Metric, F.Cu at (96.2, 37.7)
- added R71: 1k, Resistor_SMD:R_0603_1608Metric, F.Cu at (96.4, 33.7)
- added R72: 1k, Resistor_SMD:R_0603_1608Metric, F.Cu at (49.3, 81.1)
- added R73: 1k, Resistor_SMD:R_0603_1608Metric, F.Cu at (53.4, 82.0)
- added R74: 1k, Resistor_SMD:R_0603_1608Metric, F.Cu at (39.9, 55.0)
- added R75: 1k, Resistor_SMD:R_0603_1608Metric, F.Cu at (39.9, 53.3)
- added R76: 1k, Resistor_SMD:R_0603_1608Metric, F.Cu at (42.3, 27.9)
- added R77: 1k, Resistor_SMD:R_0603_1608Metric, F.Cu at (39.0, 27.9)
- C43, C44, C45: value 0.1u -> 100n
- D19: value 15V TVS C78409 -> 15V C78409
- R0N1L1, R0NL1: value 7m FMF25FPJR007-LHL -> 0.007 2512
- R0N1L2, R0NL2: value 7m -> 0.007 2512
- R10, R13, R14, R15, R16, R17, R18, R21, R28, R32, R33, R34: value 20k -> IRF->100 U51->20
- R16L1, R16L2, R16L3, R16L4, R17L1, R17L2, R17L3, R17L4, R18L1, R18L2, R18L3, R18L4: value 2K2 -> 2.2k
- R19L1, R19L2, R20L1, R20L2, R21L1, R21L2: value 3K3 -> 3.3k
- R48, R49: value 60.4 -> 56R
- R50, R57, R60, R63, R66, R69: value DNP 10k -> 10k IRF->DNP
- U3: value STM32F103RCTx -> STM32F103RCT
- moved D19 0.29 mm to (93.7, 74.5)
Connections:
- U10 pad 1: /L_MTR_PHC/H_BRIDGE_LO -> Net-(R71-Pad1)
- U10 pad 2: /L_MTR_PHC/H_BRIDGE_HI -> Net-(R68-Pad1)
- U11 pad 1: /R_MTR_PHA/H_BRIDGE_LO -> Net-(R73-Pad1)
- U11 pad 2: /R_MTR_PHA/H_BRIDGE_HI -> Net-(R72-Pad1)
- U12 pad 1: /R_MTR_PHB/H_BRIDGE_LO -> Net-(R75-Pad1)
- U12 pad 2: /R_MTR_PHB/H_BRIDGE_HI -> Net-(R74-Pad1)
- U13 pad 1: /R_MTR_PHC/H_BRIDGE_LO -> Net-(R77-Pad1)
- U13 pad 2: /R_MTR_PHC/H_BRIDGE_HI -> Net-(R76-Pad1)
- U8 pad 1: /L_MTR_PHA/H_BRIDGE_LO -> Net-(R59-Pad1)
- U8 pad 2: /L_MTR_PHA/H_BRIDGE_HI -> Net-(R52-Pad1)
- U9 pad 1: /L_MTR_PHB/H_BRIDGE_LO -> Net-(R65-Pad1)
- U9 pad 2: /L_MTR_PHB/H_BRIDGE_HI -> Net-(R62-Pad1)
Routing:
- net /R_MTR_PHA/H_BRIDGE_LO: track 29.1 -> 14.8 mm
- net Net-(R73-Pad1): track 0.00 -> 13.0 mm
- net /R_MTR_PHB/H_BRIDGE_HI: track 44.2 -> 56.8 mm
- net Net-(R75-Pad1): track 0.00 -> 11.0 mm
- net Net-(R77-Pad1): track 0.00 -> 10.5 mm, vias 0 -> 2
- net /L_MTR_PHC/H_BRIDGE_HI: track 58.6 -> 48.5 mm
- net /R_MTR_PHA/H_BRIDGE_HI: track 33.9 -> 24.0 mm
- net Net-(R72-Pad1): track 0.00 -> 9.64 mm
- net GND: track 198.9 -> 208.4 mm, vias 268 -> 276
- net Net-(R76-Pad1): track 0.00 -> 9.02 mm, vias 0 -> 2
- net /R_MTR_PHB/H_BRIDGE_LO: track 46.0 -> 54.1 mm
- net /R_MTR_PHC/H_BRIDGE_LO: track 73.4 -> 81.5 mm
- net /L_MTR_PHC/H_BRIDGE_LO: track 64.9 -> 57.9 mm
- net Net-(R74-Pad1): track 0.00 -> 6.87 mm
- net /R_MTR_PHC/H_BRIDGE_HI: track 68.3 -> 73.3 mm
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Other:
- outline, holes or cut-outs redrawn
- board text added: "capacitors: max 80V mosfets: max 100V DCDC: max 80V TVS diodes: max 51V"

Commit message: prepare production files
Routing:
- net GND: vias 276 -> 277
Changed lines of the file:
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@@
     (thickness 1.6)
     (drawings 52)
-    (tracks 2927)
+    (tracks 2928)
     (zones 0)
     (modules 272)
@@
   )
   (setup
-    (last_trace_width 0.25)
+    (last_trace_width 0.2)
     (user_trace_width 0.2)
     (user_trace_width 0.5)
@@
   (via (at 88.9 62.6) (size 0.8) (drill 0.4) (layers F.Cu B.Cu) (net 1))
   (via (at 86.1 64.6) (size 0.8) (drill 0.4) (layers F.Cu B.Cu) (net 1))
+  (via (at 66.3 96.1) (size 0.8) (drill 0.4) (layers F.Cu B.Cu) (net 1))
   (segment (start 60.86 52.9075) (end 60.81 52.8575) (width 0.5) (layer F.Cu) (net 2))
   (segment (start 62.56 52.9075) (end 60.86 52.9075) (width 0.5) (layer F.Cu) (net 2))

Commit message: production files
Parts:
- R10, R13, R14, R15, R16, R17, R18, R21, R28, R32, R33, R34: value IRF->100 U51->20 -> 100R
- R50, R51, R57, R58, R60, R61, R63, R64, R66, R67, R69, R70: value 10k IRF->DNP -> 10k

Commit message: fix some bugs of the first revision
Parts:
- added D35: 15V C78409, Diode_SMD:D_SMB, F.Cu at (106.0, 74.2)
- added D36: 15V C78409, Diode_SMD:D_SMB, F.Cu at (71.4, 57.2)
- added D37: 15V C78409, Diode_SMD:D_SMB, F.Cu at (38.9, 75.8)
- added D38: 15V C78409, Diode_SMD:D_SMB, F.Cu at (38.7, 49.5)
- added D39: 15V C78409, Diode_SMD:D_SMB, F.Cu at (79.1, 32.2)
- added R4.1: 4.7R, Resistor_SMD:R_1206_3216Metric, F.Cu at (53.0, 38.2)
- F1: value 2A C135342 -> 2A permanent fuse
- R10, R14, R15, R16, R17, R18, R21, R28, R32, R33, R34: value 100R -> 4.7
- R4.7: renamed from R13; value 100R -> 4.7
- R56: value 3k -> 200 - 500
- U10, U11, U12, U13, U8, U9: value IRS2304 || U3115S -> IRS2304
- moved F1 2.88 mm to (50.5, 38.2), turned to 90 degrees
- moved LOGO1 0.63 mm to (50.6, 69.7)
Connections:
- D21 pad 1: +BATT -> Net-(Buck1-Pad1)
- F1 pad 1: Net-(Buck1-Pad1) -> Net-(F1-Pad1)
Routing:
- net +VSW: track 293.8 -> 344.9 mm, vias 2 -> 4
- net GND: track 208.4 -> 219.3 mm, vias 277 -> 281
- net Net-(Buck1-Pad1): track 14.5 -> 22.4 mm
- net +BATT: track 28.1 -> 22.7 mm
- net Net-(F1-Pad1): track 0.00 -> 2.50 mm
- net +5V: track 141.6 -> 140.3 mm
Other:
- board text added: "50V 15V 5V 3.3V"
- board text added: "GND RX TX 15V"
- board text added: "Version 1.1"
- board text removed: "50V 12V 5V 3.3V"
- board text removed: "Version 1.0"

Commit message: Layout oscillator
Parts:
- added C70: 100n, Capacitor_SMD:C_0603_1608Metric, F.Cu at (55.4, 73.8)
- added X1: C252325, Bobbycar-FOC-hardware:Oscillator_C387448, F.Cu at (57.8, 73.0)
- moved C39 2.50 mm to (59.1, 78.9), turned to 270 degrees
- moved C4 1.15 mm to (58.6, 75.9)
- moved C40 0.97 mm to (57.3, 79.3), turned to 270 degrees
- moved R19 0.34 mm to (56.2, 76.0), turned to 0 degrees
Connections:
- U3 pad 5: (no net) -> Net-(U3-Pad5)
Routing:
- net +3V3: track 257.9 -> 253.5 mm
- net GND: track 219.3 -> 223.1 mm, vias 281 -> 285
- net Net-(U3-Pad5): track 0.00 -> 3.68 mm
- net /R_MTR_PH_SENSE/PH_AMP_B_OUT: track 37.6 -> 36.8 mm

Commit message: dcdc layout, MOV
Layout of new dcdc done, MOVs added but not routed
Parts:
- removed Buck1: XL7015, Package_TO_SOT_SMD:TO-252-5_TabPin3
- removed D12: 1N4148W, Diode_SMD:D_SOD-123
- removed D23, D24, D25, D26, D27, D28: 51V TVS C310059, Diode_SMD:D_SMC
- added C71: 2.2u 100V, Capacitor_SMD:C_1206_3216Metric, F.Cu at (60.5, 39.1)
- added C72: 2.2nF, Capacitor_SMD:C_0603_1608Metric, F.Cu at (62.0, 50.3)
- added C73: 2.2nF, Capacitor_SMD:C_0603_1608Metric, F.Cu at (67.3, 51.8)
- added C74: 2.2u 100V, Capacitor_SMD:C_1206_3216Metric, F.Cu at (71.9, 56.1)
- added R13: 124k, Resistor_SMD:R_0603_1608Metric, F.Cu at (57.1, 43.7)
- added R78: 562k, Resistor_SMD:R_0603_1608Metric, F.Cu at (65.0, 51.1)
- added RV1: Varistor, Bobbycar-FOC-hardware:MOV20, F.Cu at (4.06, 22.1)
- added RV2: Varistor, Bobbycar-FOC-hardware:MOV20, F.Cu at (136.0, 86.0)
- added RV3: Varistor, Bobbycar-FOC-hardware:MOV20, F.Cu at (4.32, 49.0)
- added RV4: Varistor, Bobbycar-FOC-hardware:MOV20, F.Cu at (136.0, 58.1)
- added RV5: Varistor, Bobbycar-FOC-hardware:MOV20, F.Cu at (6.10, 74.7)
- added RV6: Varistor, Bobbycar-FOC-hardware:MOV20, F.Cu at (136.0, 30.3)
- added U16: LM5164DDA, Package_SO:HSOP-8-1EP_3.9x4.9mm_P1.27mm_EP2.41x3.1mm_ThermalVias, F.Cu at (60.7, 45.7)
- C37: value 33n -> 47pF
- R39: value 30k -> 576k
- R40: value 2.7k -> 49.9k
- moved D36 35.8 mm to (106.2, 48.8)
- moved C61 12.1 mm to (61.2, 41.1), turned to 0 degrees
- moved C62 3.07 mm to (61.5, 52.8), turned to 90 degrees
- moved C37 2.51 mm to (65.0, 52.6), turned to 0 degrees
- moved R39 1.27 mm to (59.8, 52.8)
- moved R40 1.27 mm to (58.1, 52.8)
Connections:
- C37 pad 2: +VSW -> Net-(C37-Pad2)
Routing:
- net Net-(C72-Pad1): track 18.2 -> 10.9 mm
- net Net-(C37-Pad1): track 8.10 -> 13.2 mm, vias 0 -> 2
- net Net-(C37-Pad2): track 0.00 -> 3.01 mm
- net +VSW: track 344.9 -> 347.8 mm, vias 4 -> 3
- net Net-(C61-Pad1): track 22.4 -> 19.8 mm
- net Net-(C72-Pad2): track 0.00 -> 1.98 mm
- net Net-(R13-Pad1): track 0.00 -> 1.74 mm
- net GND: track 223.1 -> 222.9 mm, vias 285 -> 278

Commit message: MOVs placed
Parts:
- moved RV1 124.7 mm to (126.2, 47.0)
- moved RV6 123.1 mm to (14.0, 47.0)
- moved RV4 122.2 mm to (19.6, 20.8), turned to 225 degrees
- moved RV3 121.5 mm to (122.4, 20.3), turned to 125 degrees
- moved RV2 16.3 mm to (126.2, 72.9)
- moved RV5 8.32 mm to (14.2, 72.9)
