File: supplies.sch (KiCad schematic (older format))
At the start: 17 parts, among them U1 L7805, U2 AMS1117-3.3

Commit message: Add +3.3V reverse current protection diode; add +3.3V on debug header
Parts:
- added D20: D_Schottky, symbol Device:D_Schottky
- C6: value 100nF -> 100n; footprint Capacitor_SMD:C_0603_1608Metric -> (none)
Connections:
- net +3V3: now also C6.1; no longer C6.2
- net +5V: now also D20.2 (A); no longer U2.3 (VI)
- net GND: now also C6.2; no longer C6.1
- new net: D20.1 (K), U2.3 (VI)
Other:
- moved on the sheet: C26, U2
Changed lines of the file:
@@
 L Regulator_Linear:AMS1117-3.3 U2
 U 1 1 5F73F583
-P 8600 1450
-F 0 "U2" H 8600 1692 50  0000 C CNN
-F 1 "AMS1117-3.3" H 8600 1601 50  0000 C CNN
-F 2 "Package_TO_SOT_SMD:SOT-223-3_TabPin2" H 8600 1650 50  0001 C CNN
-F 3 "http://www.advanced-monolithic.com/pdf/ds1117.pdf" H 8700 1200 50  0001 C CNN
-	1    8600 1450
+P 9150 1450
+F 0 "U2" H 9150 1692 50  0000 C CNN
+F 1 "AMS1117-3.3" H 9150 1601 50  0000 C CNN
+F 2 "Package_TO_SOT_SMD:SOT-223-3_TabPin2" H 9150 1650 50  0001 C CNN
+F 3 "http://www.advanced-monolithic.com/pdf/ds1117.pdf" H 9250 1200 50  0001 C CNN
+	1    9150 1450
 	1    0    0    -1
 $EndComp
@@
 L Device:CP C26
 U 1 1 5F7432C1
-P 8950 1850
-F 0 "C26" H 9068 1896 50  0000 L CNN
-F 1 "470u 25V LKME0901E471MF" H 9068 1805 50  0000 L CNN
-F 2 "Capacitor_THT:CP_Radial_D10.0mm_P5.00mm" H 8988 1700 50  0001 C CNN
-F 3 "~" H 8950 1850 50  0001 C CNN
-	1    8950 1850
+P 9950 1750
+F 0 "C26" H 10068 1796 50  0000 L CNN
+F 1 "470u 25V LKME0901E471MF" H 10068 1705 50  0000 L CNN
+F 2 "Capacitor_THT:CP_Radial_D10.0mm_P5.00mm" H 9988 1600 50  0001 C CNN
+F 3 "~" H 9950 1750 50  0001 C CNN
+	1    9950 1750
 	1    0    0    -1
 $EndComp
@@
 	7650 1450 7650 1700
 Wire Wire Line
-	8900 1450 8950 1450
-Wire Wire Line
-	8950 1450 8950 1700
+	9950 1450 9950 1600
 $Comp
 L power:GND #PWR0123
 U 1 1 5F7440BE
-P 8950 2000
-F 0 "#PWR0123" H 8950 1750 50  0001 C CNN
-F 1 "GND" H 8955 1827 50  0000 C CNN
-F 2 "" H 8950 2000 50  0001 C CNN
-F 3 "" H 8950 2000 50  0001 C CNN
-	1    8950 2000
+P 9950 2100
+F 0 "#PWR0123" H 9950 1850 50  0001 C CNN
+F 1 "GND" H 9955 1927 50  0000 C CNN
+F 2 "" H 9950 2100 50  0001 C CNN
+F 3 "" H 9950 2100 50  0001 C CNN
+	1    9950 2100
 	1    0    0    -1
 $EndComp
@@
 L power:GND #PWR0124
 U 1 1 5F7441D8
-P 8600 1750
-F 0 "#PWR0124" H 8600 1500 50  0001 C CNN
-F 1 "GND" H 8605 1577 50  0000 C CNN
-F 2 "" H 8600 1750 50  0001 C CNN
-F 3 "" H 8600 1750 50  0001 C CNN
-	1    8600 1750
+P 9150 1750
+F 0 "#PWR0124" H 9150 1500 50  0001 C CNN
+F 1 "GND" H 9155 1577 50  0000 C CNN
+F 2 "" H 9150 1750 50  0001 C CNN
+F 3 "" H 9150 1750 50  0001 C CNN
+	1    9150 1750
 	1    0    0    -1
 $EndComp
@@
 L power:+3.3V #PWR0127
 U 1 1 5F744EDF
-P 8950 1150
-F 0 "#PWR0127" H 8950 1000 50  0001 C CNN
-F 1 "+3.3V" H 8965 1323 50  0000 C CNN
-F 2 "" H 8950 1150 50  0001 C CNN
-F 3 "" H 8950 1150 50  0001 C CNN
-	1    8950 1150
-	1    0    0    -1
-$EndComp
-Wire Wire Line
-	8950 1150 8950 1450
-Connection ~ 8950 1450
+P 9950 1150
+F 0 "#PWR0127" H 9950 1000 50  0001 C CNN
+F 1 "+3.3V" H 9965 1323 50  0000 C CNN
+F 2 "" H 9950 1150 50  0001 C CNN
+F 3 "" H 9950 1150 50  0001 C CNN
+	1    9950 1150
+	1    0    0    -1
+$EndComp
+Wire Wire Line
+	9950 1150 9950 1450
+Connection ~ 9950 1450
 Text HLabel 3650 1550 0    50   Input ~ 0
 V_BATT_MEAS
@@
 Wire Wire Line
 	7650 1450 8050 1450
-Wire Wire Line
-	8300 1450 8050 1450
 Connection ~ 8050 1450
-$Comp
-L Device:C C6
-U 1 1 5F7529AF
-P 9100 1450
-F 0 "C6" V 8848 1450 50  0000 C CNN
-F 1 "100nF" V 8939 1450 50  0000 C CNN
-F 2 "Capacitor_SMD:C_0603_1608Metric" H 9138 1300 50  0001 C CNN
-F 3 "~" H 9100 1450 50  0001 C CNN
-	1    9100 1450
-	0    1    1    0
-$EndComp
-$Comp
-L power:GND #PWR0130
-U 1 1 5F752FD7
-P 9250 1450
-F 0 "#PWR0130" H 9250 1200 50  0001 C CNN
-F 1 "GND" H 9255 1277 50  0000 C CNN
-F 2 "" H 9250 1450 50  0001 C CNN
-F 3 "" H 9250 1450 50  0001 C CNN
-	1    9250 1450
-	1    0    0    -1
-$EndComp
 $Comp
 L Connector_Generic:Conn_01x05 Buck1
@@
 	1    0    0    -1
 $EndComp
+$Comp
+L Device:D_Schottky D20
+U 1 1 5F877F67
+P 8550 1450
+F 0 "D20" H 8550 1233 50  0000 C CNN
+F 1 "D_Schottky" H 8550 1324 50  0000 C CNN
+F 2 "" H 8550 1450 50  0001 C CNN
+F 3 "~" H 8550 1450 50  0001 C CNN
+	1    8550 1450
+	-1   0    0    1
+$EndComp
+Wire Wire Line
+	8050 1450 8400 1450
+Wire Wire Line
+	8700 1450 8850 1450
+$Comp
+L Device:C C6
+U 1 1 5F87BC4D
+P 9550 1750
+F 0 "C6" H 9665 1796 50  0000 L CNN
+F 1 "100n" H 9665 1705 50  0000 L CNN
+F 2 "" H 9588 1600 50  0001 C CNN
+F 3 "~" H 9550 1750 50  0001 C CNN
+	1    9550 1750
+	1    0    0    -1
+$EndComp
+Wire Wire Line
+	9450 1450 9550 1450
+Wire Wire Line
+	9550 1450 9550 1600
+Wire Wire Line
+	9550 1450 9950 1450
+Connection ~ 9550 1450
+Wire Wire Line
+	9550 1900 9550 2050
+Wire Wire Line
+	9550 2050 9950 2050
+Wire Wire Line
+	9950 2050 9950 1900
+Wire Wire Line
+	9950 2050 9950 2100
+Connection ~ 9950 2050
 $EndSCHEMATC

Commit message: Add TVS diode, fuse to 15 V supply
Parts:
- added D21: D_Zener, symbol Device:D_Zener
- added D22: 15V, symbol Device:D_Zener
- added F1: 2A, symbol Device:Fuse
Connections:
- net +BATT: now also R53.2, D21.1 (K), F1.2; no longer Buck1.1 (Pin_1), R53.1
- net GND: now also D21.2 (A), D22.2 (A)
- net V_BATT_MEAS: now also R54.1; no longer R54.2
- net at Buck1.2 (Pin_2), D12.1 (K), L1.1: now also D22.1 (K)
- new net: Buck1.1 (Pin_1), F1.1
- new net: R53.1, R54.2
Other:
- note added: "beefy"
- moved on the sheet: C37, C38, D12, L1, R39, R53, R54, R55

Commit message: added footprints, continue layout
Parts:
- C6: footprint (none) -> Capacitor_SMD:C_0603_1608Metric
- D20: value D_Schottky -> B5819W; footprint (none) -> Diode_SMD:D_SOD-123
- D21: value D_Zener -> 51V TVS C310059; footprint (none) -> Diode_SMD:D_SMC
- D22: value 15V -> 15V C78409; footprint (none) -> Diode_SMD:D_SMB
- F1: value 2A -> 2A C135342; footprint (none) -> Fuse:Fuse_1206_3216Metric
Changed lines of the file:
@@
 P 8550 1450
 F 0 "D20" H 8550 1233 50  0000 C CNN
-F 1 "D_Schottky" H 8550 1324 50  0000 C CNN
-F 2 "" H 8550 1450 50  0001 C CNN
+F 1 "B5819W" H 8550 1324 50  0000 C CNN
+F 2 "Diode_SMD:D_SOD-123" H 8550 1450 50  0001 C CNN
 F 3 "~" H 8550 1450 50  0001 C CNN
 	1    8550 1450
@@
 F 0 "C6" H 9665 1796 50  0000 L CNN
 F 1 "100n" H 9665 1705 50  0000 L CNN
-F 2 "" H 9588 1600 50  0001 C CNN
+F 2 "Capacitor_SMD:C_0603_1608Metric" H 9588 1600 50  0001 C CNN
 F 3 "~" H 9550 1750 50  0001 C CNN
 	1    9550 1750
@@
 P 5200 3850
 F 0 "D21" V 5154 3930 50  0000 L CNN
-F 1 "D_Zener" V 5245 3930 50  0000 L CNN
-F 2 "" H 5200 3850 50  0001 C CNN
+F 1 "51V TVS C310059" V 5245 3930 50  0000 L CNN
+F 2 "Diode_SMD:D_SMC" H 5200 3850 50  0001 C CNN
 F 3 "~" H 5200 3850 50  0001 C CNN
 	1    5200 3850
@@
 P 5550 3500
 F 0 "F1" V 5353 3500 50  0000 C CNN
-F 1 "2A" V 5444 3500 50  0000 C CNN
-F 2 "" V 5480 3500 50  0001 C CNN
+F 1 "2A C135342" V 5444 3500 50  0000 C CNN
+F 2 "Fuse:Fuse_1206_3216Metric" V 5480 3500 50  0001 C CNN
 F 3 "~" H 5550 3500 50  0001 C CNN
 	1    5550 3500
@@
 P 6050 4000
 F 0 "D22" V 6004 4080 50  0000 L CNN
-F 1 "15V" V 6095 4080 50  0000 L CNN
-F 2 "" H 6050 4000 50  0001 C CNN
+F 1 "15V C78409" V 6095 4080 50  0000 L CNN
+F 2 "Diode_SMD:D_SMB" H 6050 4000 50  0001 C CNN
 F 3 "~" H 6050 4000 50  0001 C CNN
 	1    6050 4000

Commit message: added TVS diodes on HALL inputs
Changed lines of the file:
@@
 	8050 1450 8400 1450
 Wire Wire Line
-	8700 1450 8850 1450
+	8700 1450 8750 1200
 $Comp
 L Device:C C6
@@
 	0    1    1    0
 $EndComp
-Wire Wire Line
-	5200 4000 5200 4200
 $Comp
 L power:GND #PWR02
@@
 Wire Wire Line
 	6250 3400 6250 3700
+$Comp
+L power:PWR_FLAG #FLG0104
+U 1 1 5F987DA7
+P 8750 1200
+F 0 "#FLG0104" H 8750 1275 50  0001 C CNN
+F 1 "PWR_FLAG" H 8750 1373 50  0000 C CNN
+F 2 "" H 8750 1200 50  0001 C CNN
+F 3 "~" H 8750 1200 50  0001 C CNN
+	1    8750 1200
+	1    0    0    -1
+$EndComp
+Connection ~ 8750 1200
+Wire Wire Line
+	8750 1200 8850 1450
+Wire Wire Line
+	5200 4000 5200 4200
 $EndSCHEMATC

Commit message: add silk screen, change diodes at DCDC converters, remove overcurrent detection, add 100nf
Parts:
- added C61: 100nF 100V, Capacitor_SMD:C_0603_1608Metric, symbol Device:C
- added C62, C?: 100nF, Capacitor_SMD:C_0603_1608Metric, symbol Device:C
- C25: value 470u 25V LKME0901E471MF -> 100u || 470u 25V LKME0901E471MF
- C37: value 100nF -> 33n
Connections:
- net +VSW: now also D22.1 (K), C62.2
- net GND: now also C61.2, C62.1, C?.2
- net at D20.1 (K), U2.3 (VI): now also C?.1
- net at Buck1.1 (Pin_1), F1.1: now also C61.1
- net at Buck1.2 (Pin_2), D12.1 (K), L1.1: no longer D22.1 (K)
Other:
- moved on the sheet: D22
Changed lines of the file:
@@
 P 7650 1850
 F 0 "C25" H 7768 1896 50  0000 L CNN
-F 1 "470u 25V LKME0901E471MF" H 7768 1805 50  0000 L CNN
+F 1 "100u || 470u 25V LKME0901E471MF" H 7050 1400 50  0000 L CNN
 F 2 "Capacitor_THT:CP_Radial_D10.0mm_P5.00mm" H 7688 1700 50  0001 C CNN
 F 3 "~" H 7650 1850 50  0001 C CNN
@@
 P 7700 3500
 F 0 "C37" V 7448 3500 50  0000 C CNN
-F 1 "100nF" V 7539 3500 50  0000 C CNN
+F 1 "33n" V 7539 3500 50  0000 C CNN
 F 2 "Capacitor_SMD:C_0603_1608Metric" H 7738 3350 50  0001 C CNN
 F 3 "~" H 7700 3500 50  0001 C CNN
@@
 P 5200 3850
 F 0 "D21" V 5154 3930 50  0000 L CNN
-F 1 "51V TVS C310059" V 5245 3930 50  0000 L CNN
+F 1 "51V TVS C310059" V 5050 3900 50  0000 L CNN
 F 2 "Diode_SMD:D_SMC" H 5200 3850 50  0001 C CNN
 F 3 "~" H 5200 3850 50  0001 C CNN
@@
 $EndComp
 Wire Wire Line
-	5700 3500 5950 3500
-Wire Wire Line
 	5950 3500 5950 3400
 Wire Wire Line
@@
 L Device:D_Zener D22
 U 1 1 5F751B7B
-P 6050 4000
-F 0 "D22" V 6004 4080 50  0000 L CNN
-F 1 "15V C78409" V 6095 4080 50  0000 L CNN
-F 2 "Diode_SMD:D_SMB" H 6050 4000 50  0001 C CNN
-F 3 "~" H 6050 4000 50  0001 C CNN
-	1    6050 4000
+P 8450 4000
+F 0 "D22" V 8404 4080 50  0000 L CNN
+F 1 "15V C78409" V 8600 3800 50  0000 L CNN
+F 2 "Diode_SMD:D_SMB" H 8450 4000 50  0001 C CNN
+F 3 "~" H 8450 4000 50  0001 C CNN
+	1    8450 4000
 	0    1    1    0
 $EndComp
 Text Notes 5950 4100 1    50   ~ 0
 beefy
-$Comp
-L power:GND #PWR03
-U 1 1 5F7542DE
-P 6050 4200
-F 0 "#PWR03" H 6050 3950 50  0001 C CNN
-F 1 "GND" H 6055 4027 50  0000 C CNN
-F 2 "" H 6050 4200 50  0001 C CNN
-F 3 "" H 6050 4200 50  0001 C CNN
-	1    6050 4200
-	1    0    0    -1
-$EndComp
 Wire Wire Line
 	7650 1300 7650 1450
@@
 	1    0    0    -1
 $EndComp
-Wire Wire Line
-	6050 4150 6050 4200
-Wire Wire Line
-	6050 3800 6050 3850
-Connection ~ 6050 3800
 Wire Wire Line
 	7350 4100 7350 4200
@@
 Connection ~ 7700 3300
 Wire Wire Line
-	7700 3300 8700 3300
+	7700 3300 8150 3300
 Wire Wire Line
 	7700 3650 7700 3700
@@
 	5200 4000 5200 4200
 Connection ~ 8750 1200
+$Comp
+L Device:C C61
+U 1 1 5F7FE65A
+P 5650 4000
+F 0 "C61" H 5765 4046 50  0000 L CNN
+F 1 "100nF 100V" H 5765 3955 50  0000 L CNN
+F 2 "Capacitor_SMD:C_0603_1608Metric" H 5688 3850 50  0001 C CNN
+F 3 "~" H 5650 4000 50  0001 C CNN
+	1    5650 4000
+	1    0    0    -1
+$EndComp
+Wire Wire Line
+	5750 3850 5650 3850
+Wire Wire Line
+	5700 3500 5750 3500
+$Comp
+L power:GND #PWR0104
+U 1 1 5F80087C
+P 5650 4150
+F 0 "#PWR0104" H 5650 3900 50  0001 C CNN
+F 1 "GND" H 5655 3977 50  0000 C CNN
+F 2 "" H 5650 4150 50  0001 C CNN
+F 3 "" H 5650 4150 50  0001 C CNN
+	1    5650 4150
+	1    0    0    -1
+$EndComp
+Wire Wire Line
+	5750 3500 5750 3850
+Connection ~ 5750 3500
+Wire Wire Line
+	5750 3500 5950 3500
+$Comp
+L Device:C C62
+U 1 1 5F802D65
+P 8150 3700
+F 0 "C62" V 7898 3700 50  0000 C CNN
+F 1 "100nF" V 7989 3700 50  0000 C CNN
+F 2 "Capacitor_SMD:C_0603_1608Metric" H 8188 3550 50  0001 C CNN
+F 3 "~" H 8150 3700 50  0001 C CNN
+	1    8150 3700
+	-1   0    0    1
+$EndComp
+Wire Wire Line
+	8150 3550 8150 3300
+Connection ~ 8150 3300
+$Comp
+L power:GND #PWR0105
+U 1 1 5F804444
+P 8150 4200
+F 0 "#PWR0105" H 8150 3950 50  0001 C CNN
+F 1 "GND" H 8155 4027 50  0000 C CNN
+F 2 "" H 8150 4200 50  0001 C CNN
+F 3 "" H 8150 4200 50  0001 C CNN
+	1    8150 4200
+	1    0    0    -1
+$EndComp
+Wire Wire Line
+	8150 3850 8150 4200
+$Comp
+L power:GND #PWR0106
+U 1 1 5F81A9A1
+P 8450 4150
+F 0 "#PWR0106" H 8450 3900 50  0001 C CNN
+F 1 "GND" H 8455 3977 50  0000 C CNN
+F 2 "" H 8450 4150 50  0001 C CNN
+F 3 "" H 8450 4150 50  0001 C CNN
+	1    8450 4150
+	1    0    0    -1
+$EndComp
+Wire Wire Line
+	8450 3850 8450 3300
+Wire Wire Line
+	8150 3300 8450 3300
+Connection ~ 8450 3300
+Wire Wire Line
+	8450 3300 8700 3300
+$Comp
+L Device:C C?
+U 1 1 5F825126
+P 8700 1600
+F 0 "C?" H 8815 1646 50  0000 L CNN
+F 1 "100nF" H 8815 1555 50  0000 L CNN
+F 2 "Capacitor_SMD:C_0603_1608Metric" H 8738 1450 50  0001 C CNN
+F 3 "~" H 8700 1600 50  0001 C CNN
+	1    8700 1600
+	1    0    0    -1
+$EndComp
+Connection ~ 8700 1450
+$Comp
+L power:GND #PWR?
+U 1 1 5F82562F
+P 8700 1750
+F 0 "#PWR?" H 8700 1500 50  0001 C CNN
+F 1 "GND" H 8705 1577 50  0000 C CNN
+F 2 "" H 8700 1750 50  0001 C CNN
+F 3 "" H 8700 1750 50  0001 C CNN
+	1    8700 1750
+	1    0    0    -1
+$EndComp
 $EndSCHEMATC

Commit message: fix labels
Changed lines of the file:
@@
 	0    1    1    0
 $EndComp
-Text Notes 5950 4100 1    50   ~ 0
+Text Notes 8350 4100 1    50   ~ 0
 beefy
 Wire Wire Line
