File: supplies.sch (KiCad schematic (older format))
At the start: 24 parts, among them U1 L7805, U2 AMS1117-3.3

Commit message: added capacitors
Parts:
- gave numbers to parts that had none: 1
Changed lines of the file:
@@
 	8450 3300 8700 3300
 $Comp
-L Device:C C?
+L Device:C C63
 U 1 1 5F825126
 P 8700 1600
-F 0 "C?" H 8815 1646 50  0000 L CNN
+F 0 "C63" H 8815 1646 50  0000 L CNN
 F 1 "100nF" H 8815 1555 50  0000 L CNN
 F 2 "Capacitor_SMD:C_0603_1608Metric" H 8738 1450 50  0001 C CNN
@@
 Connection ~ 8700 1450
 $Comp
-L power:GND #PWR?
+L power:GND #PWR0112
 U 1 1 5F82562F
 P 8700 1750
-F 0 "#PWR?" H 8700 1500 50  0001 C CNN
+F 0 "#PWR0112" H 8700 1500 50  0001 C CNN
 F 1 "GND" H 8705 1577 50  0000 C CNN
 F 2 "" H 8700 1750 50  0001 C CNN

Commit message: fix some bugs of the first revision
Parts:
- added D35, D36, D37, D38, D39: 15V C78409, Diode_SMD:D_SMB, symbol Device:D_Zener
- added R4.1: 4.7R, Resistor_SMD:R_1206_3216Metric, symbol Device:R
- F1: value 2A C135342 -> 2A permanent fuse
Connections:
- net +BATT: no longer D21.1 (K)
- net +VSW: now also D35.1 (K), D36.1 (K), D37.1 (K), D38.1 (K), D39.1 (K)
- net GND: now also D35.2 (A), D36.2 (A), D37.2 (A), D38.2 (A), D39.2 (A)
- net at Buck1.1 (Pin_1), C61.1: now also D21.1 (K), R4.1.1; no longer F1.1
- new net: F1.1, R4.1.2
Other:
- moved on the sheet: F1
Changed lines of the file:
@@
 L power:+BATT #PWR0111
 U 1 1 5F82CD5F
-P 5200 3050
-F 0 "#PWR0111" H 5200 2900 50  0001 C CNN
-F 1 "+BATT" H 5215 3223 50  0000 C CNN
-F 2 "" H 5200 3050 50  0001 C CNN
-F 3 "" H 5200 3050 50  0001 C CNN
-	1    5200 3050
+P 4400 3200
+F 0 "#PWR0111" H 4400 3050 50  0001 C CNN
+F 1 "+BATT" H 4415 3373 50  0000 C CNN
+F 2 "" H 4400 3200 50  0001 C CNN
+F 3 "" H 4400 3200 50  0001 C CNN
+	1    4400 3200
 	1    0    0    -1
 $EndComp
@@
 	1    0    0    -1
 $EndComp
-Wire Wire Line
-	5200 3050 5200 3500
 $Comp
 L Device:Fuse F1
 U 1 1 5F74424C
-P 5550 3500
-F 0 "F1" V 5353 3500 50  0000 C CNN
-F 1 "2A C135342" V 5444 3500 50  0000 C CNN
-F 2 "Fuse:Fuse_1206_3216Metric" V 5480 3500 50  0001 C CNN
-F 3 "~" H 5550 3500 50  0001 C CNN
-	1    5550 3500
+P 4750 3500
+F 0 "F1" V 4553 3500 50  0000 C CNN
+F 1 "2A permanent fuse" V 4644 3500 50  0000 C CNN
+F 2 "Fuse:Fuse_1206_3216Metric" V 4680 3500 50  0001 C CNN
+F 3 "~" H 4750 3500 50  0001 C CNN
+	1    4750 3500
 	0    1    1    0
 $EndComp
 Wire Wire Line
 	5950 3500 5950 3400
-Wire Wire Line
-	5400 3500 5200 3500
 Connection ~ 5200 3500
 Wire Wire Line
@@
 Wire Wire Line
 	5750 3850 5650 3850
-Wire Wire Line
-	5700 3500 5750 3500
 $Comp
 L power:GND #PWR0104
@@
 	1    0    0    -1
 $EndComp
+$Comp
+L Device:D_Zener D39
+U 1 1 5F8C3D3D
+P 9750 3450
+F 0 "D39" V 9704 3530 50  0000 L CNN
+F 1 "15V C78409" V 9795 3530 50  0000 L CNN
+F 2 "Diode_SMD:D_SMB" H 9750 3450 50  0001 C CNN
+F 3 "~" H 9750 3450 50  0001 C CNN
+	1    9750 3450
+	0    1    1    0
+$EndComp
+$Comp
+L Device:D_Zener D38
+U 1 1 5F8C3BCF
+P 9550 3450
+F 0 "D38" V 9504 3530 50  0000 L CNN
+F 1 "15V C78409" V 9595 3530 50  0000 L CNN
+F 2 "Diode_SMD:D_SMB" H 9550 3450 50  0001 C CNN
+F 3 "~" H 9550 3450 50  0001 C CNN
+	1    9550 3450
+	0    1    1    0
+$EndComp
+$Comp
+L Device:D_Zener D37
+U 1 1 5F8C3A98
+P 9350 3450
+F 0 "D37" V 9304 3530 50  0000 L CNN
+F 1 "15V C78409" V 9395 3530 50  0000 L CNN
+F 2 "Diode_SMD:D_SMB" H 9350 3450 50  0001 C CNN
+F 3 "~" H 9350 3450 50  0001 C CNN
+	1    9350 3450
+	0    1    1    0
+$EndComp
+$Comp
+L Device:D_Zener D36
+U 1 1 5F8C3993
+P 9150 3450
+F 0 "D36" V 9104 3530 50  0000 L CNN
+F 1 "15V C78409" V 9300 3250 50  0000 L CNN
+F 2 "Diode_SMD:D_SMB" H 9150 3450 50  0001 C CNN
+F 3 "~" H 9150 3450 50  0001 C CNN
+	1    9150 3450
+	0    1    1    0
+$EndComp
+$Comp
+L Device:D_Zener D35
+U 1 1 5F8C33E4
+P 8950 3450
+F 0 "D35" V 8904 3530 50  0000 L CNN
+F 1 "15V C78409" V 8995 3530 50  0000 L CNN
+F 2 "Diode_SMD:D_SMB" H 8950 3450 50  0001 C CNN
+F 3 "~" H 8950 3450 50  0001 C CNN
+	1    8950 3450
+	0    1    1    0
+$EndComp
+Connection ~ 8950 3300
+Wire Wire Line
+	8950 3300 9150 3300
+Connection ~ 9150 3300
+Wire Wire Line
+	9150 3300 9350 3300
+Connection ~ 9350 3300
+Wire Wire Line
+	9350 3300 9550 3300
+Connection ~ 9550 3300
+Wire Wire Line
+	9550 3300 9750 3300
+Wire Wire Line
+	8700 3300 8950 3300
+Connection ~ 9150 3600
+Wire Wire Line
+	9150 3600 9350 3600
+Connection ~ 9350 3600
+Wire Wire Line
+	9350 3600 9550 3600
+Connection ~ 9550 3600
+Wire Wire Line
+	9550 3600 9750 3600
+Wire Wire Line
+	8950 3600 9150 3600
+$Comp
+L power:GND #PWR0113
+U 1 1 5F8CC748
+P 9750 3600
+F 0 "#PWR0113" H 9750 3350 50  0001 C CNN
+F 1 "GND" H 9755 3427 50  0000 C CNN
+F 2 "" H 9750 3600 50  0001 C CNN
+F 3 "" H 9750 3600 50  0001 C CNN
+	1    9750 3600
+	1    0    0    -1
+$EndComp
+Connection ~ 9750 3600
+$Comp
+L Device:R R4.?
+U 1 1 5F8F557C
+P 5050 3500
+AR Path="/5F7ECC6C/5F8F557C" Ref="R4.?"  Part="1"
+AR Path="/5F79FFE4/5F8F557C" Ref="R4.?"  Part="1"
+AR Path="/5F7A0EEE/5F8F557C" Ref="R4.?"  Part="1"
+AR Path="/5F7A2640/5F8F557C" Ref="R4.?"  Part="1"
+AR Path="/5F7A3A2A/5F8F557C" Ref="R4.?"  Part="1"
+AR Path="/5F7A4E71/5F8F557C" Ref="R4.?"  Part="1"
+AR Path="/5F7395DA/5F8F557C" Ref="R4.1"  Part="1"
+F 0 "R4.1" V 5050 3500 50  0000 C CNN
+F 1 "4.7R" V 4934 3500 50  0000 C CNN
+F 2 "Resistor_SMD:R_1206_3216Metric" V 4980 3500 50  0001 C CNN
+F 3 "~" H 5050 3500 50  0001 C CNN
+	1    5050 3500
+	0    1    1    0
+$EndComp
+Wire Wire Line
+	5200 3500 5750 3500
+Wire Wire Line
+	4600 3500 4400 3500
+Wire Wire Line
+	4400 3500 4400 3200
 $EndSCHEMATC

Commit message: Changed dcdc converter to lm5164
Parts:
- removed Buck1: XL7015, Package_TO_SOT_SMD:TO-252-5_TabPin3, symbol Connector_Generic:Conn_01x05
- removed D12: 1N4148W, Diode_SMD:D_SOD-123, symbol Device:D
- added C71, C74: 2.2u 100V, Capacitor_SMD:C_1206_3216Metric, symbol Device:C
- added C72, C73: 2.2nF, Capacitor_SMD:C_0603_1608Metric, symbol Device:C
- added R13: 124k, Resistor_SMD:R_0603_1608Metric, symbol Device:R
- added R78: 562k, Resistor_SMD:R_0603_1608Metric, symbol Device:R
- added U16: LM5164DDA, Package_SO:HSOP-8-1EP_3.9x4.9mm_P1.27mm_EP2.41x3.1mm_ThermalVias, symbol Regulator_Switching:LM5164DDA
- C37: value 33n -> 47pF
- R39: value 30k -> 576k
- R40: value 2.7k -> 49.9k
Connections:
- net +VSW: now also C73.1, C74.1; no longer C37.2
- net GND: now also C71.2, C74.2, R13.2, U16.1 (GND), U16.9 (EP)
- net at C61.1, D21.1 (K), R4.1.1: now also C71.1, U16.2 (VIN), U16.3 (EN/UVLO)
- net at L1.1: now also C72.1, R78.1, U16.8 (SW)
- net at C37.1, R39.1, R40.2: now also U16.5 (FB)
- new net: C37.2, C73.2, R78.2
- new net: R13.1, U16.4 (RON)
- new net: C72.2, U16.7 (BST)
Other:
- note added: "maybe we need a lower DCR inductor\nti suggestes 100mOhm"
- note removed: "VIN\nSW\nGND\nFB\nEN"
- moved on the sheet: C37, C38, C61, C62, D21, D22, D35, D36, D37, D38, D39, F1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

Commit message: Changed fet driver
Changed lines of the file:
@@
 U 1 1 5F74424C
 P 2650 3300
-F 0 "F1" V 2453 3300 50  0000 C CNN
-F 1 "2A permanent fuse" V 2544 3300 50  0000 C CNN
+F 0 "F1" V 2550 3300 50  0000 C CNN
+F 1 "2A permanent fuse" V 2750 3100 50  0000 C CNN
 F 2 "Fuse:Fuse_1206_3216Metric" V 2580 3300 50  0001 C CNN
 F 3 "~" H 2650 3300 50  0001 C CNN
@@
 AR Path="/5F7A4E71/5F8F557C" Ref="R4.?"  Part="1"
 AR Path="/5F7395DA/5F8F557C" Ref="R4.1"  Part="1"
-F 0 "R4.1" V 2950 3300 50  0000 C CNN
-F 1 "4.7R" V 2834 3300 50  0000 C CNN
+F 0 "R4.1" V 2850 3300 50  0000 C CNN
+F 1 "4.7R" V 3050 3300 50  0000 C CNN
 F 2 "Resistor_SMD:R_1206_3216Metric" V 2880 3300 50  0001 C CNN
 F 3 "~" H 2950 3300 50  0001 C CNN

Commit message: Added LCSC Part # to most components
Parts:
- C3, C5, C62, C63: LCSC Part # (none) -> C14663
- C37: LCSC Part # (none) -> C1671
- C6: value 100n -> 100nF; LCSC Part # (none) -> C14663
- C72, C73: LCSC Part # (none) -> C1604
- F1: LCSC Part # (none) -> C182310
- R13: LCSC Part # (none) -> C22788
- R39: LCSC Part # (none) -> C23207
- R40: LCSC Part # (none) -> C23184
- R53, R54: LCSC Part # (none) -> C22809
- R55: LCSC Part # (none) -> C21190
- R78: LCSC Part # (none) -> C23205
- R81: renamed from R4.1; value 4.7R -> 4.7; LCSC Part # (none) -> C17937
- U1: LCSC Part # (none) -> C310413
- U16: LCSC Part # (none) -> C477928
- U2: LCSC Part # (none) -> C426566
Changed lines of the file:
@@
 F 2 "Capacitor_SMD:C_0603_1608Metric" H 6588 1300 50  0001 C CNN
 F 3 "~" H 6550 1450 50  0001 C CNN
+F 4 "C14663" H 6550 1450 50  0001 C CNN "LCSC Part #"
 	1    6550 1450
 	0    1    1    0
@@
 F 2 "Package_TO_SOT_SMD:TO-263-2" H 7375 1300 50  0001 L CIN
 F 3 "http://www.st.com/content/ccc/resource/technical/document/datasheet/41/4f/b3/b0/12/d4/47/88/CD00000444.pdf/files/CD00000444.pdf/jcr:content/translations/en.CD00000444.pdf" H 7350 1400 50  0001 C CNN
+F 4 "C310413" H 7350 1450 50  0001 C CNN "LCSC Part #"
 	1    7350 1450
 	1    0    0    -1
@@
 F 2 "Package_TO_SOT_SMD:SOT-223-3_TabPin2" H 9150 1650 50  0001 C CNN
 F 3 "http://www.advanced-monolithic.com/pdf/ds1117.pdf" H 9250 1200 50  0001 C CNN
+F 4 "C426566" H 9150 1450 50  0001 C CNN "LCSC Part #"
 	1    9150 1450
 	1    0    0    -1
@@
 F 2 "Resistor_SMD:R_0603_1608Metric" V 3630 1700 50  0001 C CNN
 F 3 "~" H 3700 1700 50  0001 C CNN
+F 4 "C22809" H 3700 1700 50  0001 C CNN "LCSC Part #"
 	1    3700 1700
 	-1   0    0    1
@@
 F 2 "Resistor_SMD:R_0603_1608Metric" V 3630 2050 50  0001 C CNN
 F 3 "~" H 3700 2050 50  0001 C CNN
+F 4 "C22809" H 3700 2050 50  0001 C CNN "LCSC Part #"
 	1    3700 2050
 	-1   0    0    1
@@
 F 2 "Resistor_SMD:R_0603_1608Metric" V 3630 2450 50  0001 C CNN
 F 3 "~" H 3700 2450 50  0001 C CNN
+F 4 "C21190" H 3700 2450 50  0001 C CNN "LCSC Part #"
 	1    3700 2450
 	1    0    0    -1
@@
 F 2 "Capacitor_SMD:C_0603_1608Metric" H 8088 1450 50  0001 C CNN
 F 3 "~" H 8050 1600 50  0001 C CNN
+F 4 "C14663" H 8050 1600 50  0001 C CNN "LCSC Part #"
 	1    8050 1600
 	1    0    0    -1
@@
 F 2 "Resistor_SMD:R_0603_1608Metric" V 7680 3550 50  0001 C CNN
 F 3 "~" H 7750 3550 50  0001 C CNN
+F 4 "C23207" H 7750 3550 50  0001 C CNN "LCSC Part #"
 	1    7750 3550
 	-1   0    0    1
@@
 F 2 "Resistor_SMD:R_0603_1608Metric" V 7680 4300 50  0001 C CNN
 F 3 "~" H 7750 4300 50  0001 C CNN
+F 4 "C23184" H 7750 4300 50  0001 C CNN "LCSC Part #"
 	1    7750 4300
 	-1   0    0    1
@@
 F 2 "Capacitor_SMD:C_0603_1608Metric" H 7088 3700 50  0001 C CNN
 F 3 "~" H 7050 3850 50  0001 C CNN
+F 4 "C1671" H 7050 3850 50  0001 C CNN "LCSC Part #"
 	1    7050 3850
 	-1   0    0    1
@@
 P 9550 1750
 F 0 "C6" H 9665 1796 50  0000 L CNN
-F 1 "100n" H 9665 1705 50  0000 L CNN
+F 1 "100nF" H 9665 1705 50  0000 L CNN
 F 2 "Capacitor_SMD:C_0603_1608Metric" H 9588 1600 50  0001 C CNN
 F 3 "~" H 9550 1750 50  0001 C CNN
+F 4 "C14663" H 9550 1750 50  0001 C CNN "LCSC Part #"
 	1    9550 1750
 	1    0    0    -1
@@
 F 2 "Fuse:Fuse_1206_3216Metric" V 2580 3300 50  0001 C CNN
 F 3 "~" H 2650 3300 50  0001 C CNN
+F 4 "C182310" H 2650 3300 50  0001 C CNN "LCSC Part #"
 	1    2650 3300
 	0    1    1    0
@@
 F 2 "Capacitor_SMD:C_0603_1608Metric" H 8588 3550 50  0001 C CNN
 F 3 "~" H 8550 3700 50  0001 C CNN
+F 4 "C14663" H 8550 3700 50  0001 C CNN "LCSC Part #"
 	1    8550 3700
 	-1   0    0    1
@@
 F 2 "Capacitor_SMD:C_0603_1608Metric" H 8738 1450 50  0001 C CNN
 F 3 "~" H 8700 1600 50  0001 C CNN
+F 4 "C14663" H 8700 1600 50  0001 C CNN "LCSC Part #"
 	1    8700 1600
 	1    0    0    -1
@@
 AR Path="/5F7A3A2A/5F8F557C" Ref="R4.?"  Part="1"
 AR Path="/5F7A4E71/5F8F557C" Ref="R4.?"  Part="1"
-AR Path="/5F7395DA/5F8F557C" Ref="R4.1"  Part="1"
-F 0 "R4.1" V 2850 3300 50  0000 C CNN
-F 1 "4.7R" V 3050 3300 50  0000 C CNN
+AR Path="/5F7395DA/5F8F557C" Ref="R81"  Part="1"
+F 0 "R81" V 2850 3300 50  0000 C CNN
+F 1 "4.7" V 3050 3300 50  0000 C CNN
 F 2 "Resistor_SMD:R_1206_3216Metric" V 2880 3300 50  0001 C CNN
 F 3 "~" H 2950 3300 50  0001 C CNN
+F 4 "C17937" H 2950 3300 50  0001 C CNN "LCSC Part #"
 	1    2950 3300
 	0    1    1    0
@@
 F 2 "Package_SO:HSOP-8-1EP_3.9x4.9mm_P1.27mm_EP2.41x3.1mm_ThermalVias" H 5600 3150 50  0001 C CNN
 F 3 "https://www.ti.com/lit/ds/symlink/lm5164.pdf?ts=1598311864250&ref_url=https%253A%252F%252Fwww.ti.com%252Fproduct%252FLM5164%253FHQS%253DTI-null-null-octopart-df-pf-null-wwe" H 5250 3950 50  0001 C CNN
+F 4 "C477928" H 5550 3600 50  0001 C CNN "LCSC Part #"
 	1    5550 3600
 	1    0    0    -1
@@
 F 2 "Capacitor_SMD:C_0603_1608Metric" H 6438 3150 50  0001 C CNN
 F 3 "~" H 6400 3300 50  0001 C CNN
+F 4 "C1604" H 6400 3300 50  0001 C CNN "LCSC Part #"
 	1    6400 3300
 	0    1    1    0
@@
 F 2 "Resistor_SMD:R_0603_1608Metric" V 6780 3650 50  0001 C CNN
 F 3 "~" H 6850 3650 50  0001 C CNN
+F 4 "C23205" H 6850 3650 50  0001 C CNN "LCSC Part #"
 	1    6850 3650
 	0    -1   -1   0
@@
 F 2 "Capacitor_SMD:C_0603_1608Metric" H 7288 3500 50  0001 C CNN
 F 3 "~" H 7250 3650 50  0001 C CNN
+F 4 "C1604" H 7250 3650 50  0001 C CNN "LCSC Part #"
 	1    7250 3650
 	0    1    1    0
@@
 F 2 "Resistor_SMD:R_0603_1608Metric" V 4930 4050 50  0001 C CNN
 F 3 "~" H 5000 4050 50  0001 C CNN
+F 4 "C22788" H 5000 4050 50  0001 C CNN "LCSC Part #"
 	1    5000 4050
 	1    0    0    -1

Commit message: More adaptation to jlcpcb, parts checking
Parts:
- C25, C26, C38: place (none) -> hand
- C61: LCSC Part # (none) -> C113803
- C71, C74: footprint Capacitor_SMD:C_1206_3216Metric -> Capacitor_SMD:C_1210_3225Metric; LCSC Part # (none) -> C76685; place (none) -> hand
- D20: LCSC Part # (none) -> C8598
- D21: LCSC Part # (none) -> C10374
- D22, D35, D36, D37, D38, D39: LCSC Part # (none) -> C78409
- L1: LCSC Part # (none) -> C169378
- U1: LCSC Part # C310413 -> C15077
- U16: LCSC Part # C477928 -> (none); place (none) -> hand
Changed lines of the file:
@@
 F 2 "Package_TO_SOT_SMD:TO-263-2" H 7375 1300 50  0001 L CIN
 F 3 "http://www.st.com/content/ccc/resource/technical/document/datasheet/41/4f/b3/b0/12/d4/47/88/CD00000444.pdf/files/CD00000444.pdf/jcr:content/translations/en.CD00000444.pdf" H 7350 1400 50  0001 C CNN
-F 4 "C310413" H 7350 1450 50  0001 C CNN "LCSC Part #"
+F 4 "C15077" H 7350 1450 50  0001 C CNN "LCSC Part #"
 	1    7350 1450
 	1    0    0    -1
@@
 F 2 "Capacitor_THT:CP_Radial_D10.0mm_P5.00mm" H 7688 1700 50  0001 C CNN
 F 3 "~" H 7650 1850 50  0001 C CNN
+F 4 "hand" H 7650 1850 50  0001 C CNN "place"
 	1    7650 1850
 	1    0    0    -1
@@
 F 2 "Capacitor_THT:CP_Radial_D10.0mm_P5.00mm" H 9988 1600 50  0001 C CNN
 F 3 "~" H 9950 1750 50  0001 C CNN
+F 4 "hand" H 9950 1750 50  0001 C CNN "place"
 	1    9950 1750
 	1    0    0    -1
@@
 F 1 "SWRB1207S-101MT" V 7099 3300 50  0000 C CNN
 F 2 "Inductor_SMD:L_Wuerth_HCM-1240" H 7000 3300 50  0001 C CNN
-F 3 "~" H 7000 3300 50  0001 C CNN
+F 3 "https://datasheet.lcsc.com/szlcsc/Sunlord-SWRB1207S-101MT_C169378.pdf" H 7000 3300 50  0001 C CNN
+F 4 "C169378" H 7000 3300 50  0001 C CNN "LCSC Part #"
 	1    7000 3300
 	0    -1   -1   0
@@
 F 2 "Capacitor_THT:CP_Radial_D10.0mm_P5.00mm" H 9138 3600 50  0001 C CNN
 F 3 "~" H 9100 3750 50  0001 C CNN
+F 4 "hand" H 9100 3750 50  0001 C CNN "place"
 	1    9100 3750
 	1    0    0    -1
@@
 F 1 "B5819W" H 8550 1324 50  0000 C CNN
 F 2 "Diode_SMD:D_SOD-123" H 8550 1450 50  0001 C CNN
-F 3 "~" H 8550 1450 50  0001 C CNN
+F 3 "" H 8550 1450 50  0001 C CNN
+F 4 "C8598" H 8550 1450 50  0001 C CNN "LCSC Part #"
 	1    8550 1450
 	-1   0    0    1
@@
 F 2 "Diode_SMD:D_SMC" H 3100 3650 50  0001 C CNN
 F 3 "~" H 3100 3650 50  0001 C CNN
+F 4 "C10374" H 3100 3650 50  0001 C CNN "LCSC Part #"
 	1    3100 3650
 	0    1    1    0
@@
 F 2 "Diode_SMD:D_SMB" H 8850 3950 50  0001 C CNN
 F 3 "~" H 8850 3950 50  0001 C CNN
+F 4 "C78409" H 8850 3950 50  0001 C CNN "LCSC Part #"
 	1    8850 3950
 	0    1    1    0
@@
 F 2 "Capacitor_SMD:C_0603_1608Metric" H 4338 3700 50  0001 C CNN
 F 3 "~" H 4300 3850 50  0001 C CNN
+F 4 "C113803" H 4300 3850 50  0001 C CNN "LCSC Part #"
 	1    4300 3850
 	1    0    0    -1
@@
 F 2 "Diode_SMD:D_SMB" H 10150 3450 50  0001 C CNN
 F 3 "~" H 10150 3450 50  0001 C CNN
+F 4 "C78409" H 10150 3450 50  0001 C CNN "LCSC Part #"
 	1    10150 3450
 	0    1    1    0
@@
 F 2 "Diode_SMD:D_SMB" H 9950 3450 50  0001 C CNN
 F 3 "~" H 9950 3450 50  0001 C CNN
+F 4 "C78409" H 9950 3450 50  0001 C CNN "LCSC Part #"
 	1    9950 3450
 	0    1    1    0
@@
 F 2 "Diode_SMD:D_SMB" H 9750 3450 50  0001 C CNN
 F 3 "~" H 9750 3450 50  0001 C CNN
+F 4 "C78409" H 9750 3450 50  0001 C CNN "LCSC Part #"
 	1    9750 3450
 	0    1    1    0
@@
 F 2 "Diode_SMD:D_SMB" H 9550 3450 50  0001 C CNN
 F 3 "~" H 9550 3450 50  0001 C CNN
+F 4 "C78409" H 9550 3450 50  0001 C CNN "LCSC Part #"
 	1    9550 3450
 	0    1    1    0
@@
 F 2 "Diode_SMD:D_SMB" H 9350 3450 50  0001 C CNN
 F 3 "~" H 9350 3450 50  0001 C CNN
+F 4 "C78409" H 9350 3450 50  0001 C CNN "LCSC Part #"
 	1    9350 3450
 	0    1    1    0
@@
 F 2 "Package_SO:HSOP-8-1EP_3.9x4.9mm_P1.27mm_EP2.41x3.1mm_ThermalVias" H 5600 3150 50  0001 C CNN
 F 3 "https://www.ti.com/lit/ds/symlink/lm5164.pdf?ts=1598311864250&ref_url=https%253A%252F%252Fwww.ti.com%252Fproduct%252FLM5164%253FHQS%253DTI-null-null-octopart-df-pf-null-wwe" H 5250 3950 50  0001 C CNN
-F 4 "C477928" H 5550 3600 50  0001 C CNN "LCSC Part #"
+F 4 "" H 5550 3600 50  0001 C CNN "LCSC Part #"
+F 5 "hand" H 5550 3600 50  0001 C CNN "place"
 	1    5550 3600
 	1    0    0    -1
@@
 F 0 "C71" H 3885 3896 50  0000 R CNN
 F 1 "2.2u 100V" H 3885 3805 50  0000 R CNN
-F 2 "Capacitor_SMD:C_1206_3216Metric" H 4038 3700 50  0001 C CNN
+F 2 "Capacitor_SMD:C_1210_3225Metric" H 4038 3700 50  0001 C CNN
 F 3 "~" H 4000 3850 50  0001 C CNN
+F 4 "hand" H 4000 3850 50  0001 C CNN "place"
+F 5 "C76685" H 4000 3850 50  0001 C CNN "LCSC Part #"
 	1    4000 3850
 	1    0    0    -1
@@
 F 0 "C74" H 8135 3746 50  0000 R CNN
 F 1 "2.2u 100V" H 8135 3655 50  0000 R CNN
-F 2 "Capacitor_SMD:C_1206_3216Metric" H 8288 3550 50  0001 C CNN
+F 2 "Capacitor_SMD:C_1210_3225Metric" H 8288 3550 50  0001 C CNN
 F 3 "~" H 8250 3700 50  0001 C CNN
+F 4 "hand" H 8250 3700 50  0001 C CNN "place"
+F 5 "C76685" H 8250 3700 50  0001 C CNN "LCSC Part #"
 	1    8250 3700
 	1    0    0    -1

Commit message: Added pth caps to assembly
Parts:
- C25: value 100u || 470u 25V LKME0901E471MF -> 470u 25V LKME0901E471MF; footprint Capacitor_THT:CP_Radial_D10.0mm_P5.00mm -> Bobbycar-FOC-hardware:CP_Radial_D10.0mm_P5.00mm_mid; LCSC Part # (none) -> C105289; place hand -> (none)
- C26, C38: footprint Capacitor_THT:CP_Radial_D10.0mm_P5.00mm -> Bobbycar-FOC-hardware:CP_Radial_D10.0mm_P5.00mm_mid; LCSC Part # (none) -> C105289; place hand -> (none)
Changed lines of the file:
@@
 P 7650 1850
 F 0 "C25" H 7768 1896 50  0000 L CNN
-F 1 "100u || 470u 25V LKME0901E471MF" H 7050 1400 50  0000 L CNN
-F 2 "Capacitor_THT:CP_Radial_D10.0mm_P5.00mm" H 7688 1700 50  0001 C CNN
+F 1 "470u 25V LKME0901E471MF" H 7050 1400 50  0000 L CNN
+F 2 "Bobbycar-FOC-hardware:CP_Radial_D10.0mm_P5.00mm_mid" H 7688 1700 50  0001 C CNN
 F 3 "~" H 7650 1850 50  0001 C CNN
-F 4 "hand" H 7650 1850 50  0001 C CNN "place"
+F 4 "" H 7650 1850 50  0001 C CNN "place"
+F 5 "C105289" H 7650 1850 50  0001 C CNN "LCSC Part #"
 	1    7650 1850
 	1    0    0    -1
@@
 F 0 "C26" H 10068 1796 50  0000 L CNN
 F 1 "470u 25V LKME0901E471MF" H 10068 1705 50  0000 L CNN
-F 2 "Capacitor_THT:CP_Radial_D10.0mm_P5.00mm" H 9988 1600 50  0001 C CNN
+F 2 "Bobbycar-FOC-hardware:CP_Radial_D10.0mm_P5.00mm_mid" H 9988 1600 50  0001 C CNN
 F 3 "~" H 9950 1750 50  0001 C CNN
-F 4 "hand" H 9950 1750 50  0001 C CNN "place"
+F 4 "" H 9950 1750 50  0001 C CNN "place"
+F 5 "C105289" H 9950 1750 50  0001 C CNN "LCSC Part #"
 	1    9950 1750
 	1    0    0    -1
@@
 F 0 "C38" H 9218 3796 50  0000 L CNN
 F 1 "470u 25V LKME0901E471MF" H 9218 3705 50  0000 L CNN
-F 2 "Capacitor_THT:CP_Radial_D10.0mm_P5.00mm" H 9138 3600 50  0001 C CNN
+F 2 "Bobbycar-FOC-hardware:CP_Radial_D10.0mm_P5.00mm_mid" H 9138 3600 50  0001 C CNN
 F 3 "~" H 9100 3750 50  0001 C CNN
-F 4 "hand" H 9100 3750 50  0001 C CNN "place"
+F 4 "" H 9100 3750 50  0001 C CNN "place"
+F 5 "C105289" H 9100 3750 50  0001 C CNN "LCSC Part #"
 	1    9100 3750
 	1    0    0    -1
