File: Bobbycontroller.sch (KiCad schematic (older format))
At the start: 14 parts, among them J1 Conn_01x01_Male, J2 Conn_01x01_Male, J3 Conn_01x01_Male, J5 Conn_01x01_Male, J6 Conn_01x01_Male, J7 Conn_01x01_Male

Commit message: fix some errors
Connections:
- no-connect marks 0 -> 1
Changed lines of the file:
@@
 F10 "L_MTR_PHB_HI" I R 5900 1700 50
 F11 "L_MTR_PHC_HI" I R 5900 2200 50
-F12 "CHARGE_CONNECTED" I L 3150 4650 50
-F13 "SWDIO" I L 3150 4850 50
-F14 "SWCLK" I L 3150 4950 50
-F15 "R_MTR_PHB_LO" I R 5900 5650 50
-F16 "R_MTR_PHC_LO" I R 5900 6450 50
-F17 "L_MTR_HALL_PHA" I L 3150 3650 50
-F18 "L_MTR_HALL_PHB" I L 3150 3550 50
-F19 "L_MTR_HALL_PHC" I L 3150 3450 50
-F20 "UART_R_TX" I L 3150 4150 50
-F21 "UART_R_RX" I L 3150 4250 50
-F22 "L_MTR_OVERCUR" I L 3150 7000 50
-F23 "L_MTR_PHA_LO" I R 5900 1250 50
-F24 "L_MTR_PHB_LO" I R 5900 1800 50
-F25 "L_MTR_PHC_LO" I R 5900 2300 50
-F26 "R_MTR_CURR" I L 3150 6900 50
-F27 "L_MTR_CURR" I L 3150 7100 50
-F28 "V_BATT_MEAS" I L 3150 6350 50
-F29 "R_MTR_PHB_SENSE" I L 3150 2350 50
-F30 "L_MTR_PHB_SENSE" I L 3150 1600 50
-F31 "L_MTR_PHC_SENSE" I L 3150 1300 50
-F32 "R_MTR_PHA_HI" I R 5900 4700 50
-F33 "R_MTR_PHB_HI" I R 5900 5550 50
-F34 "R_MTR_PHC_HI" I R 5900 6350 50
-F35 "R_MTR_HALL_PHC" I L 3150 3250 50
-F36 "R_MTR_HALL_PHB" I L 3150 3150 50
-F37 "R_MTR_HALL_PHA" I L 3150 3050 50
+F12 "SWDIO" I L 3150 4850 50
+F13 "SWCLK" I L 3150 4950 50
+F14 "R_MTR_PHB_LO" I R 5900 5650 50
+F15 "R_MTR_PHC_LO" I R 5900 6450 50
+F16 "L_MTR_HALL_PHA" I L 3150 3650 50
+F17 "L_MTR_HALL_PHB" I L 3150 3550 50
+F18 "L_MTR_HALL_PHC" I L 3150 3450 50
+F19 "UART_R_TX" I L 3150 4150 50
+F20 "UART_R_RX" I L 3150 4250 50
+F21 "L_MTR_OVERCUR" I L 3150 7000 50
+F22 "L_MTR_PHA_LO" I R 5900 1250 50
+F23 "L_MTR_PHB_LO" I R 5900 1800 50
+F24 "L_MTR_PHC_LO" I R 5900 2300 50
+F25 "R_MTR_CURR" I L 3150 6900 50
+F26 "L_MTR_CURR" I L 3150 7100 50
+F27 "V_BATT_MEAS" I L 3150 6350 50
+F28 "R_MTR_PHB_SENSE" I L 3150 2350 50
+F29 "L_MTR_PHB_SENSE" I L 3150 1600 50
+F30 "L_MTR_PHC_SENSE" I L 3150 1300 50
+F31 "R_MTR_PHA_HI" I R 5900 4700 50
+F32 "R_MTR_PHB_HI" I R 5900 5550 50
+F33 "R_MTR_PHC_HI" I R 5900 6350 50
+F34 "R_MTR_HALL_PHC" I L 3150 3250 50
+F35 "R_MTR_HALL_PHB" I L 3150 3150 50
+F36 "R_MTR_HALL_PHA" I L 3150 3050 50
 $EndSheet
 $Sheet
@@
 $EndComp
 Wire Wire Line
-	3150 4650 3000 4650
-Wire Wire Line
 	3150 4550 3000 4550
 Wire Wire Line
 	3000 4550 3000 4650
-Connection ~ 3000 4650
 $Comp
 L power:+BATT #PWR0195
@@
 	-1   0    0    1
 $EndComp
+$Comp
+L power:+BATT #PWR0218
+U 1 1 5F71D61A
+P 10000 2850
+F 0 "#PWR0218" H 10000 2700 50  0001 C CNN
+F 1 "+BATT" H 10015 3023 50  0000 C CNN
+F 2 "" H 10000 2850 50  0001 C CNN
+F 3 "" H 10000 2850 50  0001 C CNN
+	1    10000 2850
+	1    0    0    -1
+$EndComp
+$Comp
+L power:-BATT #PWR0219
+U 1 1 5F71DB2B
+P 10250 2850
+F 0 "#PWR0219" H 10250 2700 50  0001 C CNN
+F 1 "-BATT" H 10265 3023 50  0000 C CNN
+F 2 "" H 10250 2850 50  0001 C CNN
+F 3 "" H 10250 2850 50  0001 C CNN
+	1    10250 2850
+	1    0    0    -1
+$EndComp
+$Comp
+L power:+VSW #PWR0220
+U 1 1 5F71E59F
+P 10500 2850
+F 0 "#PWR0220" H 10500 2700 50  0001 C CNN
+F 1 "+VSW" H 10515 3023 50  0000 C CNN
+F 2 "" H 10500 2850 50  0001 C CNN
+F 3 "" H 10500 2850 50  0001 C CNN
+	1    10500 2850
+	1    0    0    -1
+$EndComp
+$Comp
+L power:PWR_FLAG #FLG0101
+U 1 1 5F71E94D
+P 10000 2850
+F 0 "#FLG0101" H 10000 2925 50  0001 C CNN
+F 1 "PWR_FLAG" H 10000 3023 50  0000 C CNN
+F 2 "" H 10000 2850 50  0001 C CNN
+F 3 "~" H 10000 2850 50  0001 C CNN
+	1    10000 2850
+	-1   0    0    1
+$EndComp
+$Comp
+L power:PWR_FLAG #FLG0102
+U 1 1 5F71ED59
+P 10250 2850
+F 0 "#FLG0102" H 10250 2925 50  0001 C CNN
+F 1 "PWR_FLAG" H 10250 3023 50  0000 C CNN
+F 2 "" H 10250 2850 50  0001 C CNN
+F 3 "~" H 10250 2850 50  0001 C CNN
+	1    10250 2850
+	-1   0    0    1
+$EndComp
+$Comp
+L power:PWR_FLAG #FLG0103
+U 1 1 5F71EE95
+P 10500 2850
+F 0 "#FLG0103" H 10500 2925 50  0001 C CNN
+F 1 "PWR_FLAG" H 10500 3023 50  0000 C CNN
+F 2 "" H 10500 2850 50  0001 C CNN
+F 3 "~" H 10500 2850 50  0001 C CNN
+	1    10500 2850
+	-1   0    0    1
+$EndComp
+NoConn ~ 3150 4450
 $EndSCHEMATC

Commit message: fix all ERC errors
Connections:
- no-connect marks 1 -> 2
Changed lines of the file:
@@
 Wire Wire Line
 	1550 7050 1400 7050
-Text GLabel 8900 700  0    50   Input ~ 0
-L_MTR_PHA
 Text GLabel 8850 850  0    50   Input ~ 0
 L_MTR_PHB
@@
 	8100 1250 7700 1250
 Connection ~ 8100 1800
-Text GLabel 8900 4250 0    50   Input ~ 0
-R_MTR_PHA
 Text GLabel 8850 4400 0    50   Input ~ 0
 R_MTR_PHB
@@
 	8100 5850 8100 6050
 $Comp
-L power:GND #PWR0103
-U 1 1 5F70BA8E
-P 3000 4650
-F 0 "#PWR0103" H 3000 4400 50  0001 C CNN
-F 1 "GND" H 3005 4477 50  0000 C CNN
-F 2 "" H 3000 4650 50  0001 C CNN
-F 3 "" H 3000 4650 50  0001 C CNN
-	1    3000 4650
-	1    0    0    -1
-$EndComp
-Wire Wire Line
-	3150 4550 3000 4550
-Wire Wire Line
-	3000 4550 3000 4650
-$Comp
 L power:+BATT #PWR0195
 U 1 1 5F7AB0B8
@@
 $EndComp
 NoConn ~ 3150 4450
+NoConn ~ 3150 4550
+Text Label 8900 4250 2    50   ~ 0
+R_MTR_PHA
+Text Label 8900 700  2    50   ~ 0
+L_MTR_PHA
 $EndSCHEMATC

Commit message: Add CAN transceiver
Changed lines of the file:
@@
 $Descr A4 11693 8268
 encoding utf-8
-Sheet 1 13
+Sheet 1 14
 Title ""
 Date ""
@@
 F35 "R_MTR_HALL_PHB" I L 3150 3150 50
 F36 "R_MTR_HALL_PHA" I L 3150 3050 50
+F37 "CAN_RX" I L 3150 5650 50
+F38 "CAN_TX" O L 3150 5750 50
 $EndSheet
 $Sheet
@@
 F12 "R_MTR_HALL_PHB" I R 2800 3150 50
 F13 "R_MTR_HALL_PHC" I R 2800 3250 50
+F14 "CANH" B L 1550 4850 50
+F15 "CANL" B L 1550 4950 50
 $EndSheet
 $Sheet
@@
 Text Label 8900 700  2    50   ~ 0
 L_MTR_PHA
+$Sheet
+S 1550 5550 1250 300
+U 5F737F83
+F0 "CAN" 50
+F1 "CAN.sch" 50
+F2 "CAN_RX" O R 2800 5650 50
+F3 "CAN_TX" I R 2800 5750 50
+F4 "CANL" B L 1550 5750 50
+F5 "CANH" B L 1550 5650 50
+$EndSheet
+Wire Wire Line
+	3150 5650 2800 5650
+Wire Wire Line
+	3150 5750 2800 5750
+Wire Wire Line
+	1550 5650 1300 5650
+Wire Wire Line
+	1300 5650 1300 4850
+Wire Wire Line
+	1300 4850 1550 4850
+Wire Wire Line
+	1550 5750 1400 5750
+Wire Wire Line
+	1400 5750 1400 4950
+Wire Wire Line
+	1400 4950 1550 4950
 $EndSCHEMATC

Commit message: finish design
Parts:
- added J11, J? (x3): Conn_01x01, MountingHole:MountingHole_4mm_Pad_Via, symbol Connector_Generic:Conn_01x01
Changed lines of the file:
@@
 Wire Wire Line
 	1400 4950 1550 4950
+$Comp
+L Connector_Generic:Conn_01x01 J11
+U 1 1 5F8ED7E9
+P 10400 900
+F 0 "J11" H 10480 942 50  0000 L CNN
+F 1 "Conn_01x01" H 10480 851 50  0000 L CNN
+F 2 "MountingHole:MountingHole_4mm_Pad_Via" H 10400 900 50  0001 C CNN
+F 3 "~" H 10400 900 50  0001 C CNN
+	1    10400 900
+	1    0    0    -1
+$EndComp
+$Comp
+L Connector_Generic:Conn_01x01 J?
+U 1 1 5F8F0C04
+P 10400 1050
+F 0 "J?" H 10480 1092 50  0000 L CNN
+F 1 "Conn_01x01" H 10480 1001 50  0000 L CNN
+F 2 "MountingHole:MountingHole_4mm_Pad_Via" H 10400 1050 50  0001 C CNN
+F 3 "~" H 10400 1050 50  0001 C CNN
+	1    10400 1050
+	1    0    0    -1
+$EndComp
+$Comp
+L Connector_Generic:Conn_01x01 J?
+U 1 1 5F8F0EB7
+P 10400 1200
+F 0 "J?" H 10480 1242 50  0000 L CNN
+F 1 "Conn_01x01" H 10480 1151 50  0000 L CNN
+F 2 "MountingHole:MountingHole_4mm_Pad_Via" H 10400 1200 50  0001 C CNN
+F 3 "~" H 10400 1200 50  0001 C CNN
+	1    10400 1200
+	1    0    0    -1
+$EndComp
+$Comp
+L Connector_Generic:Conn_01x01 J?
+U 1 1 5F8F1012
+P 10400 1350
+F 0 "J?" H 10480 1392 50  0000 L CNN
+F 1 "Conn_01x01" H 10480 1301 50  0000 L CNN
+F 2 "MountingHole:MountingHole_4mm_Pad_Via" H 10400 1350 50  0001 C CNN
+F 3 "~" H 10400 1350 50  0001 C CNN
+	1    10400 1350
+	1    0    0    -1
+$EndComp
 $EndSCHEMATC

Commit message: finish layout
Parts:
- added C46, C47, C48, C49, C50, C51, C52, C53, C54, C55, C56, C57, C58, C59: 2.2u 100V, Capacitor_SMD:C_1206_3216Metric, symbol Device:C
- added J15: -BATT, MountingHole:MountingHole_2.7mm_M2.5_Pad, symbol Connector_Generic:Conn_01x01
- added J16: +BATT, MountingHole:MountingHole_2.7mm_M2.5_Pad, symbol Connector_Generic:Conn_01x01
- added JP3: Jumper_2_Bridged, Jumper:SolderJumper-2_P1.3mm_Bridged2Bar_RoundedPad1.0x1.5mm, symbol Jumper:Jumper_2_Bridged
- gave numbers to parts that had none: 3
Connections:
- net +BATT: now also C46.1, C47.1, C48.1, C49.1, C50.1, C51.1, C52.1, C53.1, C54.1, C55.1, C56.1, C57.1, C58.1, C59.1, J16.1 (Pin_1)
- net -BATT: now also C46.2, C47.2, C48.2, C49.2, C50.2, C51.2, C52.2, C53.2, C54.2, C55.2, C56.2, C57.2, C58.2, C59.2, J15.1 (Pin_1), JP3.1 (A)
- new net GND: JP3.2 (B)

Commit message: added TVS diodes on HALL inputs
Connections:
- no-connect marks 2 -> 6
Changed lines of the file:
@@
 $EndComp
 Connection ~ 9700 5950
+NoConn ~ 10200 900
+NoConn ~ 10200 1050
+NoConn ~ 10200 1200
+NoConn ~ 10200 1350
 $EndSCHEMATC

Commit message: Minor changes to PCB; convert footprint library to .pretty format, add to project
Parts:
- removed JP3: Jumper_2_Bridged, Jumper:SolderJumper-2_P1.3mm_Bridged2Bar_RoundedPad1.0x1.5mm, symbol Jumper:Jumper_2_Bridged
- added LOGO1: Logo_Open_Hardware_Small, Bobbycar-FOC-hardware:lenas_bobbycar_logo, symbol Graphic:Logo_Open_Hardware_Small
- added NT1, NT2: Net-Tie_2, NetTie:NetTie-2_SMD_Pad2.0mm, symbol Device:Net-Tie_2
- J11, J12, J13, J14: symbol Connector_Generic:Conn_01x01 -> Mechanical:MountingHole
Connections:
- net -BATT: now also NT1.1, NT2.1
- net GND: now also NT1.2, NT2.2
- no-connect marks 6 -> 2
Changed lines of the file:
@@
 	1400 4950 1550 4950
 $Comp
-L Connector_Generic:Conn_01x01 J11
+L Mechanical:MountingHole J11
 U 1 1 5F8ED7E9
-P 10400 900
-F 0 "J11" H 10480 942 50  0000 L CNN
-F 1 "Conn_01x01" H 10480 851 50  0000 L CNN
-F 2 "MountingHole:MountingHole_4mm_Pad_Via" H 10400 900 50  0001 C CNN
-F 3 "~" H 10400 900 50  0001 C CNN
-	1    10400 900
-	1    0    0    -1
-$EndComp
-$Comp
-L Connector_Generic:Conn_01x01 J12
+P 10400 700
+F 0 "J11" H 10480 742 50  0000 L CNN
+F 1 "Conn_01x01" H 10480 651 50  0000 L CNN
+F 2 "MountingHole:MountingHole_4mm_Pad_Via" H 10400 700 50  0001 C CNN
+F 3 "~" H 10400 700 50  0001 C CNN
+	1    10400 700
+	1    0    0    -1
+$EndComp
+$Comp
+L Mechanical:MountingHole J12
 U 1 1 5F8F0C04
-P 10400 1050
-F 0 "J12" H 10480 1092 50  0000 L CNN
-F 1 "Conn_01x01" H 10480 1001 50  0000 L CNN
-F 2 "MountingHole:MountingHole_4mm_Pad_Via" H 10400 1050 50  0001 C CNN
-F 3 "~" H 10400 1050 50  0001 C CNN
-	1    10400 1050
-	1    0    0    -1
-$EndComp
-$Comp
-L Connector_Generic:Conn_01x01 J13
+P 10400 850
+F 0 "J12" H 10480 892 50  0000 L CNN
+F 1 "Conn_01x01" H 10480 801 50  0000 L CNN
+F 2 "MountingHole:MountingHole_4mm_Pad_Via" H 10400 850 50  0001 C CNN
+F 3 "~" H 10400 850 50  0001 C CNN
+	1    10400 850
+	1    0    0    -1
+$EndComp
+$Comp
+L Mechanical:MountingHole J13
 U 1 1 5F8F0EB7
-P 10400 1200
-F 0 "J13" H 10480 1242 50  0000 L CNN
-F 1 "Conn_01x01" H 10480 1151 50  0000 L CNN
-F 2 "MountingHole:MountingHole_4mm_Pad_Via" H 10400 1200 50  0001 C CNN
-F 3 "~" H 10400 1200 50  0001 C CNN
-	1    10400 1200
-	1    0    0    -1
-$EndComp
-$Comp
-L Connector_Generic:Conn_01x01 J14
+P 10400 1000
+F 0 "J13" H 10480 1042 50  0000 L CNN
+F 1 "Conn_01x01" H 10480 951 50  0000 L CNN
+F 2 "MountingHole:MountingHole_4mm_Pad_Via" H 10400 1000 50  0001 C CNN
+F 3 "~" H 10400 1000 50  0001 C CNN
+	1    10400 1000
+	1    0    0    -1
+$EndComp
+$Comp
+L Mechanical:MountingHole J14
 U 1 1 5F8F1012
-P 10400 1350
-F 0 "J14" H 10480 1392 50  0000 L CNN
-F 1 "Conn_01x01" H 10480 1301 50  0000 L CNN
-F 2 "MountingHole:MountingHole_4mm_Pad_Via" H 10400 1350 50  0001 C CNN
-F 3 "~" H 10400 1350 50  0001 C CNN
-	1    10400 1350
+P 10400 1150
+F 0 "J14" H 10480 1192 50  0000 L CNN
+F 1 "Conn_01x01" H 10480 1101 50  0000 L CNN
+F 2 "MountingHole:MountingHole_4mm_Pad_Via" H 10400 1150 50  0001 C CNN
+F 3 "~" H 10400 1150 50  0001 C CNN
+	1    10400 1150
 	1    0    0    -1
 $EndComp
@@
 $EndComp
 $Comp
-L Jumper:Jumper_2_Bridged JP3
-U 1 1 5F8FED5A
-P 10350 2200
-F 0 "JP3" H 10350 2395 50  0000 C CNN
-F 1 "Jumper_2_Bridged" H 10350 2304 50  0000 C CNN
-F 2 "Jumper:SolderJumper-2_P1.3mm_Bridged2Bar_RoundedPad1.0x1.5mm" H 10350 2200 50  0001 C CNN
-F 3 "~" H 10350 2200 50  0001 C CNN
-	1    10350 2200
-	1    0    0    -1
-$EndComp
-$Comp
 L power:+BATT #PWR0235
 U 1 1 5F8FF3DE
@@
 $EndComp
 Connection ~ 9700 5950
-NoConn ~ 10200 900
-NoConn ~ 10200 1050
-NoConn ~ 10200 1200
-NoConn ~ 10200 1350
+$Comp
+L Device:Net-Tie_2 NT1
+U 1 1 5F73BECD
+P 10350 2100
+F 0 "NT1" H 10350 2281 50  0000 C CNN
+F 1 "Net-Tie_2" H 10350 2190 50  0000 C CNN
+F 2 "NetTie:NetTie-2_SMD_Pad2.0mm" H 10350 2100 50  0001 C CNN
+F 3 "~" H 10350 2100 50  0001 C CNN
+	1    10350 2100
+	1    0    0    -1
+$EndComp
+Wire Wire Line
+	10250 2100 10150 2100
+Wire Wire Line
+	10150 2100 10150 2200
+Wire Wire Line
+	10450 2100 10550 2100
+Wire Wire Line
+	10550 2100 10550 2200
+$Comp
+L power:PWR_FLAG #FLG0105
+U 1 1 5F75A34A
+P 10750 1950
+F 0 "#FLG0105" H 10750 2025 50  0001 C CNN
+F 1 "PWR_FLAG" H 10750 2123 50  0000 C CNN
+F 2 "" H 10750 1950 50  0001 C CNN
+F 3 "~" H 10750 1950 50  0001 C CNN
+	1    10750 1950
+	1    0    0    -1
+$EndComp
+Wire Wire Line
+	10750 1950 10750 2100
+Wire Wire Line
+	10750 2100 10550 2100
+Connection ~ 10550 2100
+$Comp
+L Graphic:Logo_Open_Hardware_Small LOGO1
+U 1 1 5F773897
+P 9800 1050
+F 0 "LOGO1" H 9800 1325 50  0001 C CNN
+F 1 "Logo_Open_Hardware_Small" H 9800 825 50  0001 C CNN
+F 2 "Bobbycar-FOC-hardware:lenas_bobbycar_logo" H 9800 1050 50  0001 C CNN
+F 3 "~" H 9800 1050 50  0001 C CNN
+	1    9800 1050
+	1    0    0    -1
+$EndComp
+$Comp
+L Device:Net-Tie_2 NT2
+U 1 1 5F7403BE
+P 10350 1800
+F 0 "NT2" H 10350 1981 50  0000 C CNN
+F 1 "Net-Tie_2" H 10350 1890 50  0000 C CNN
+F 2 "NetTie:NetTie-2_SMD_Pad2.0mm" H 10350 1800 50  0001 C CNN
+F 3 "~" H 10350 1800 50  0001 C CNN
+	1    10350 1800
+	1    0    0    -1
+$EndComp
+Wire Wire Line
+	10250 1800 10150 1800
+Wire Wire Line
+	10150 1800 10150 2100
+Connection ~ 10150 2100
+Wire Wire Line
+	10450 1800 10550 1800
+Wire Wire Line
+	10550 1800 10550 2100
 $EndSCHEMATC

Commit message: add resistors on mosfet driver inputs, change board corners, fix labels
Parts:
- R0N1L1, R0NL1: value 7m FMF25FPJR007-LHL -> 0.007 2512
- R0N1L2, R0NL2: value 7m -> 0.007 2512
Changed lines of the file:
@@
 P 8500 2650
 F 0 "R0N1L1" H 8570 2696 50  0000 L CNN
-F 1 "7m FMF25FPJR007-LHL" H 8570 2605 50  0000 L CNN
+F 1 "0.007 2512" H 8570 2605 50  0000 L CNN
 F 2 "Resistor_SMD:R_2512_6332Metric" V 8430 2650 50  0001 C CNN
 F 3 "~" H 8500 2650 50  0001 C CNN
@@
 P 8100 2650
 F 0 "R0NL1" H 8170 2696 50  0000 L CNN
-F 1 "7m FMF25FPJR007-LHL" H 8170 2605 50  0000 L CNN
+F 1 "0.007 2512" H 8170 2605 50  0000 L CNN
 F 2 "Resistor_SMD:R_2512_6332Metric" V 8030 2650 50  0001 C CNN
 F 3 "~" H 8100 2650 50  0001 C CNN
@@
 P 8500 6200
 F 0 "R0N1L2" H 8570 6246 50  0000 L CNN
-F 1 "7m" H 8570 6155 50  0000 L CNN
+F 1 "0.007 2512" H 8570 6155 50  0000 L CNN
 F 2 "Resistor_SMD:R_2512_6332Metric" V 8430 6200 50  0001 C CNN
 F 3 "~" H 8500 6200 50  0001 C CNN
@@
 P 8100 6200
 F 0 "R0NL2" H 8170 6246 50  0000 L CNN
-F 1 "7m" H 8170 6155 50  0000 L CNN
+F 1 "0.007 2512" H 8170 6155 50  0000 L CNN
 F 2 "Resistor_SMD:R_2512_6332Metric" V 8030 6200 50  0001 C CNN
 F 3 "~" H 8100 6200 50  0001 C CNN
