File: Bobbycontroller.sch (KiCad schematic (older format))
At the start: 37 parts, among them J1 Conn_01x01_Male, J11 Conn_01x01, J12 Conn_01x01, J13 Conn_01x01, J14 Conn_01x01, J15 -BATT, J16 +BATT, J2 Conn_01x01_Male, J3 Conn_01x01_Male, J5 Conn_01x01_Male, J6 Conn_01x01_Male, J7 Conn_01x01_Male

Commit message: added rs232, layout changes
Parts:
- LOGO1: footprint Bobbycar-FOC-hardware:lenas_bobbycar_logo -> (none)
Changed lines of the file:
@@
 F 0 "LOGO1" H 9800 1325 50  0001 C CNN
 F 1 "Logo_Open_Hardware_Small" H 9800 825 50  0001 C CNN
-F 2 "Bobbycar-FOC-hardware:lenas_bobbycar_logo" H 9800 1050 50  0001 C CNN
+F 2 "" H 9800 1050 50  0001 C CNN
 F 3 "~" H 9800 1050 50  0001 C CNN
 	1    9800 1050

Commit message: More adaptation to jlcpcb, parts checking
Parts:
- C27, C28, C29, C30, C46, C47, C48, C49, C50, C51, C52, C53, C54, C55, C56, C57, C58, C59: place (none) -> hand
- J1, J11, J12, J13, J14, J15, J16, J2, J3, J5, J6, J7, LOGO1, NT1, NT2: place (none) -> dnp
- R0N1L1, R0N1L2, R0NL1, R0NL2: LCSC Part # (none) -> C62405
Changed lines of the file:
@@
 F 2 "Resistor_SMD:R_2512_6332Metric" V 8430 2650 50  0001 C CNN
 F 3 "~" H 8500 2650 50  0001 C CNN
+F 4 "C62405" H 8500 2650 50  0001 C CNN "LCSC Part #"
 	1    8500 2650
 	1    0    0    -1
@@
 F 2 "Resistor_SMD:R_2512_6332Metric" V 8030 2650 50  0001 C CNN
 F 3 "~" H 8100 2650 50  0001 C CNN
+F 4 "C62405" H 8100 2650 50  0001 C CNN "LCSC Part #"
 	1    8100 2650
 	1    0    0    -1
@@
 F 2 "Resistor_SMD:R_2512_6332Metric" V 8430 6200 50  0001 C CNN
 F 3 "~" H 8500 6200 50  0001 C CNN
+F 4 "C62405" H 8500 6200 50  0001 C CNN "LCSC Part #"
 	1    8500 6200
 	1    0    0    -1
@@
 F 2 "Resistor_SMD:R_2512_6332Metric" V 8030 6200 50  0001 C CNN
 F 3 "~" H 8100 6200 50  0001 C CNN
+F 4 "C62405" H 8100 6200 50  0001 C CNN "LCSC Part #"
 	1    8100 6200
 	1    0    0    -1
@@
 F 1 "LKML1401K221MF" H 9918 5055 50  0000 L CNN
 F 2 "Capacitor_THT:CP_Radial_D12.5mm_P5.00mm" H 9838 4950 50  0001 C CNN
-F 3 "~" H 9800 5100 50  0001 C CNN
+F 3 "" H 9800 5100 50  0001 C CNN
+F 4 "hand" H 9800 5100 50  0001 C CNN "place"
 	1    9800 5100
 	1    0    0    -1
@@
 F 1 "LKML1401K221MF" H 10218 5055 50  0000 L CNN
 F 2 "Capacitor_THT:CP_Radial_D12.5mm_P5.00mm" H 10138 4950 50  0001 C CNN
-F 3 "~" H 10100 5100 50  0001 C CNN
+F 3 "" H 10100 5100 50  0001 C CNN
+F 4 "hand" H 10100 5100 50  0001 C CNN "place"
 	1    10100 5100
 	1    0    0    -1
@@
 F 1 "LKML1401K221MF" H 10468 5055 50  0000 L CNN
 F 2 "Capacitor_THT:CP_Radial_D12.5mm_P5.00mm" H 10388 4950 50  0001 C CNN
-F 3 "~" H 10350 5100 50  0001 C CNN
+F 3 "" H 10350 5100 50  0001 C CNN
+F 4 "hand" H 10350 5100 50  0001 C CNN "place"
 	1    10350 5100
 	1    0    0    -1
@@
 F 1 "LKML1401K221MF" H 10718 5055 50  0000 L CNN
 F 2 "Capacitor_THT:CP_Radial_D12.5mm_P5.00mm" H 10638 4950 50  0001 C CNN
-F 3 "~" H 10600 5100 50  0001 C CNN
+F 3 "" H 10600 5100 50  0001 C CNN
+F 4 "hand" H 10600 5100 50  0001 C CNN "place"
 	1    10600 5100
 	1    0    0    -1
@@
 F 2 "Connector_Pin:Pin_D1.4mm_L8.5mm_W2.8mm_FlatFork" H 9100 1400 50  0001 C CNN
 F 3 "~" H 9100 1400 50  0001 C CNN
+F 4 "dnp" H 9100 1400 50  0001 C CNN "place"
 	1    9100 1400
 	-1   0    0    1
@@
 F 2 "Connector_Pin:Pin_D1.4mm_L8.5mm_W2.8mm_FlatFork" H 9100 1500 50  0001 C CNN
 F 3 "~" H 9100 1500 50  0001 C CNN
+F 4 "dnp" H 9100 1500 50  0001 C CNN "place"
 	1    9100 1500
 	-1   0    0    1
@@
 F 2 "Connector_Pin:Pin_D1.4mm_L8.5mm_W2.8mm_FlatFork" H 9100 1600 50  0001 C CNN
 F 3 "~" H 9100 1600 50  0001 C CNN
+F 4 "dnp" H 9100 1600 50  0001 C CNN "place"
 	1    9100 1600
 	-1   0    0    1
@@
 F 2 "Connector_Pin:Pin_D1.4mm_L8.5mm_W2.8mm_FlatFork" H 9100 4950 50  0001 C CNN
 F 3 "~" H 9100 4950 50  0001 C CNN
+F 4 "dnp" H 9100 4950 50  0001 C CNN "place"
 	1    9100 4950
 	-1   0    0    1
@@
 F 2 "Connector_Pin:Pin_D1.4mm_L8.5mm_W2.8mm_FlatFork" H 9100 5050 50  0001 C CNN
 F 3 "~" H 9100 5050 50  0001 C CNN
+F 4 "dnp" H 9100 5050 50  0001 C CNN "place"
 	1    9100 5050
 	-1   0    0    1
@@
 F 2 "Connector_Pin:Pin_D1.4mm_L8.5mm_W2.8mm_FlatFork" H 9100 5150 50  0001 C CNN
 F 3 "~" H 9100 5150 50  0001 C CNN
+F 4 "dnp" H 9100 5150 50  0001 C CNN "place"
 	1    9100 5150
 	-1   0    0    1
@@
 F 1 "Conn_01x01" H 10480 651 50  0000 L CNN
 F 2 "MountingHole:MountingHole_4mm_Pad_Via" H 10400 700 50  0001 C CNN
-F 3 "~" H 10400 700 50  0001 C CNN
+F 3 "" H 10400 700 50  0001 C CNN
+F 4 "dnp" H 10400 700 50  0001 C CNN "place"
 	1    10400 700
 	1    0    0    -1
@@
 F 1 "Conn_01x01" H 10480 801 50  0000 L CNN
 F 2 "MountingHole:MountingHole_4mm_Pad_Via" H 10400 850 50  0001 C CNN
-F 3 "~" H 10400 850 50  0001 C CNN
+F 3 "" H 10400 850 50  0001 C CNN
+F 4 "dnp" H 10400 850 50  0001 C CNN "place"
 	1    10400 850
 	1    0    0    -1
@@
 F 1 "Conn_01x01" H 10480 951 50  0000 L CNN
 F 2 "MountingHole:MountingHole_4mm_Pad_Via" H 10400 1000 50  0001 C CNN
-F 3 "~" H 10400 1000 50  0001 C CNN
+F 3 "" H 10400 1000 50  0001 C CNN
+F 4 "dnp" H 10400 1000 50  0001 C CNN "place"
 	1    10400 1000
 	1    0    0    -1
@@
 F 1 "Conn_01x01" H 10480 1101 50  0000 L CNN
 F 2 "MountingHole:MountingHole_4mm_Pad_Via" H 10400 1150 50  0001 C CNN
-F 3 "~" H 10400 1150 50  0001 C CNN
+F 3 "" H 10400 1150 50  0001 C CNN
+F 4 "dnp" H 10400 1150 50  0001 C CNN "place"
 	1    10400 1150
 	1    0    0    -1
@@
 F 2 "MountingHole:MountingHole_2.7mm_M2.5_Pad" H 9450 2400 50  0001 C CNN
 F 3 "~" H 9450 2400 50  0001 C CNN
+F 4 "dnp" H 9450 2400 50  0001 C CNN "place"
 	1    9450 2400
 	0    1    1    0
@@
 F 2 "MountingHole:MountingHole_2.7mm_M2.5_Pad" H 9700 2400 50  0001 C CNN
 F 3 "~" H 9700 2400 50  0001 C CNN
+F 4 "dnp" H 9700 2400 50  0001 C CNN "place"
 	1    9700 2400
 	0    1    1    0
@@
 F 2 "Capacitor_SMD:C_1206_3216Metric" H 9738 5550 50  0001 C CNN
 F 3 "~" H 9700 5700 50  0001 C CNN
+F 4 "hand" H 9700 5700 50  0001 C CNN "place"
 	1    9700 5700
 	1    0    0    -1
@@
 F 2 "Capacitor_SMD:C_1206_3216Metric" H 9938 5550 50  0001 C CNN
 F 3 "~" H 9900 5700 50  0001 C CNN
+F 4 "hand" H 9900 5700 50  0001 C CNN "place"
 	1    9900 5700
 	1    0    0    -1
@@
 F 2 "Capacitor_SMD:C_1206_3216Metric" H 10138 5550 50  0001 C CNN
 F 3 "~" H 10100 5700 50  0001 C CNN
+F 4 "hand" H 10100 5700 50  0001 C CNN "place"
 	1    10100 5700
 	1    0    0    -1
@@
 F 2 "Capacitor_SMD:C_1206_3216Metric" H 10338 5550 50  0001 C CNN
 F 3 "~" H 10300 5700 50  0001 C CNN
+F 4 "hand" H 10300 5700 50  0001 C CNN "place"
 	1    10300 5700
 	1    0    0    -1
@@
 F 2 "Capacitor_SMD:C_1206_3216Metric" H 10538 5550 50  0001 C CNN
 F 3 "~" H 10500 5700 50  0001 C CNN
+F 4 "hand" H 10500 5700 50  0001 C CNN "place"
 	1    10500 5700
 	1    0    0    -1
@@
 F 2 "Capacitor_SMD:C_1206_3216Metric" H 10738 5550 50  0001 C CNN
 F 3 "~" H 10700 5700 50  0001 C CNN
+F 4 "hand" H 10700 5700 50  0001 C CNN "place"
 	1    10700 5700
 	1    0    0    -1
@@
 F 2 "Capacitor_SMD:C_1206_3216Metric" H 10938 5550 50  0001 C CNN
 F 3 "~" H 10900 5700 50  0001 C CNN
+F 4 "hand" H 10900 5700 50  0001 C CNN "place"
 	1    10900 5700
 	1    0    0    -1
@@
 F 2 "Capacitor_SMD:C_1206_3216Metric" H 9738 5950 50  0001 C CNN
 F 3 "~" H 9700 6100 50  0001 C CNN
+F 4 "hand" H 9700 6100 50  0001 C CNN "place"
 	1    9700 6100
 	1    0    0    -1
@@
 F 2 "Capacitor_SMD:C_1206_3216Metric" H 9938 5950 50  0001 C CNN
 F 3 "~" H 9900 6100 50  0001 C CNN
+F 4 "hand" H 9900 6100 50  0001 C CNN "place"
 	1    9900 6100
 	1    0    0    -1
@@
 F 2 "Capacitor_SMD:C_1206_3216Metric" H 10138 5950 50  0001 C CNN
 F 3 "~" H 10100 6100 50  0001 C CNN
+F 4 "hand" H 10100 6100 50  0001 C CNN "place"
 	1    10100 6100
 	1    0    0    -1
@@
 F 2 "Capacitor_SMD:C_1206_3216Metric" H 10338 5950 50  0001 C CNN
 F 3 "~" H 10300 6100 50  0001 C CNN
+F 4 "hand" H 10300 6100 50  0001 C CNN "place"
 	1    10300 6100
 	1    0    0    -1
@@
 F 2 "Capacitor_SMD:C_1206_3216Metric" H 10538 5950 50  0001 C CNN
 F 3 "~" H 10500 6100 50  0001 C CNN
+F 4 "hand" H 10500 6100 50  0001 C CNN "place"
 	1    10500 6100
 	1    0    0    -1
@@
 F 2 "Capacitor_SMD:C_1206_3216Metric" H 10738 5950 50  0001 C CNN
 F 3 "~" H 10700 6100 50  0001 C CNN
+F 4 "hand" H 10700 6100 50  0001 C CNN "place"
 	1    10700 6100
 	1    0    0    -1
@@
 F 2 "Capacitor_SMD:C_1206_3216Metric" H 10938 5950 50  0001 C CNN
 F 3 "~" H 10900 6100 50  0001 C CNN
+F 4 "hand" H 10900 6100 50  0001 C CNN "place"
 	1    10900 6100
 	1    0    0    -1
@@
 F 1 "Net-Tie_2" H 10350 2190 50  0000 C CNN
 F 2 "NetTie:NetTie-2_SMD_Pad2.0mm" H 10350 2100 50  0001 C CNN
-F 3 "~" H 10350 2100 50  0001 C CNN
+F 3 "" H 10350 2100 50  0001 C CNN
+F 4 "dnp" H 10350 2100 50  0001 C CNN "place"
 	1    10350 2100
 	1    0    0    -1
@@
 F 1 "Logo_Open_Hardware_Small" H 9800 825 50  0001 C CNN
 F 2 "" H 9800 1050 50  0001 C CNN
-F 3 "~" H 9800 1050 50  0001 C CNN
+F 3 "" H 9800 1050 50  0001 C CNN
+F 4 "dnp" H 9800 1050 50  0001 C CNN "place"
 	1    9800 1050
 	1    0    0    -1
@@
 F 1 "Net-Tie_2" H 10350 1890 50  0000 C CNN
 F 2 "NetTie:NetTie-2_SMD_Pad2.0mm" H 10350 1800 50  0001 C CNN
-F 3 "~" H 10350 1800 50  0001 C CNN
+F 3 "" H 10350 1800 50  0001 C CNN
+F 4 "dnp" H 10350 1800 50  0001 C CNN "place"
 	1    10350 1800
 	1    0    0    -1

Commit message: Added pth caps to assembly
Parts:
- R0N1L1, R0N1L2, R0NL1, R0NL2: value 0.007 2512 -> 0.004 2512; LCSC Part # C62405 -> C270946
Changed lines of the file:
@@
 P 8500 2650
 F 0 "R0N1L1" H 8570 2696 50  0000 L CNN
-F 1 "0.007 2512" H 8570 2605 50  0000 L CNN
+F 1 "0.004 2512" H 8570 2605 50  0000 L CNN
 F 2 "Resistor_SMD:R_2512_6332Metric" V 8430 2650 50  0001 C CNN
 F 3 "~" H 8500 2650 50  0001 C CNN
-F 4 "C62405" H 8500 2650 50  0001 C CNN "LCSC Part #"
+F 4 "C270946" H 8500 2650 50  0001 C CNN "LCSC Part #"
 	1    8500 2650
 	1    0    0    -1
@@
 P 8100 2650
 F 0 "R0NL1" H 8170 2696 50  0000 L CNN
-F 1 "0.007 2512" H 8170 2605 50  0000 L CNN
+F 1 "0.004 2512" H 8170 2605 50  0000 L CNN
 F 2 "Resistor_SMD:R_2512_6332Metric" V 8030 2650 50  0001 C CNN
 F 3 "~" H 8100 2650 50  0001 C CNN
-F 4 "C62405" H 8100 2650 50  0001 C CNN "LCSC Part #"
+F 4 "C270946" H 8100 2650 50  0001 C CNN "LCSC Part #"
 	1    8100 2650
 	1    0    0    -1
@@
 P 8500 6200
 F 0 "R0N1L2" H 8570 6246 50  0000 L CNN
-F 1 "0.007 2512" H 8570 6155 50  0000 L CNN
+F 1 "0.004 2512" H 8570 6155 50  0000 L CNN
 F 2 "Resistor_SMD:R_2512_6332Metric" V 8430 6200 50  0001 C CNN
 F 3 "~" H 8500 6200 50  0001 C CNN
-F 4 "C62405" H 8500 6200 50  0001 C CNN "LCSC Part #"
+F 4 "C270946" H 8500 6200 50  0001 C CNN "LCSC Part #"
 	1    8500 6200
 	1    0    0    -1
@@
 P 8100 6200
 F 0 "R0NL2" H 8170 6246 50  0000 L CNN
-F 1 "0.007 2512" H 8170 6155 50  0000 L CNN
+F 1 "0.004 2512" H 8170 6155 50  0000 L CNN
 F 2 "Resistor_SMD:R_2512_6332Metric" V 8030 6200 50  0001 C CNN
 F 3 "~" H 8100 6200 50  0001 C CNN
-F 4 "C62405" H 8100 6200 50  0001 C CNN "LCSC Part #"
+F 4 "C270946" H 8100 6200 50  0001 C CNN "LCSC Part #"
 	1    8100 6200
 	1    0    0    -1
