File: mcu.sch (KiCad schematic (older format))
At the start: 22 parts, among them Q6 MMBT5551, U3 STM32F103RCTx

Commit message: Fix MCU NRST connection
Connections:
- net at C4.1, R19.2: now also U3.7 (NRST)
Other:
- moved on the sheet: C4
Changed lines of the file:
@@
 L Device:C C4
 U 1 1 5F737CEC
-P 4400 1700
-F 0 "C4" H 4515 1700 50  0000 L CNN
-F 1 "100n" H 4515 1655 50  0001 L CNN
-F 2 "Capacitor_SMD:C_0603_1608Metric" H 4438 1550 50  0001 C CNN
-F 3 "~" H 4400 1700 50  0001 C CNN
-	1    4400 1700
+P 4400 1800
+F 0 "C4" H 4515 1800 50  0000 L CNN
+F 1 "100n" H 4515 1755 50  0001 L CNN
+F 2 "Capacitor_SMD:C_0603_1608Metric" H 4438 1650 50  0001 C CNN
+F 3 "~" H 4400 1800 50  0001 C CNN
+	1    4400 1800
 	1    0    0    -1
 $EndComp
@@
 L power:GND #PWR0148
 U 1 1 5F7384A8
-P 4400 1850
-F 0 "#PWR0148" H 4400 1600 50  0001 C CNN
-F 1 "GND" H 4405 1677 50  0000 C CNN
-F 2 "" H 4400 1850 50  0001 C CNN
-F 3 "" H 4400 1850 50  0001 C CNN
-	1    4400 1850
+P 4400 1950
+F 0 "#PWR0148" H 4400 1700 50  0001 C CNN
+F 1 "GND" H 4405 1777 50  0000 C CNN
+F 2 "" H 4400 1950 50  0001 C CNN
+F 3 "" H 4400 1950 50  0001 C CNN
+	1    4400 1950
 	1    0    0    -1
 $EndComp
@@
 Wire Wire Line
 	9300 4700 9450 4700
+Wire Wire Line
+	4400 1550 4400 1600
+Wire Wire Line
+	4400 1600 4400 1650
+Connection ~ 4400 1600
 $EndSCHEMATC

Commit message: fix some errors
Connections:
- net GND: now also U3.12 (VSSA), U3.18 (VSS), U3.31 (VSS), U3.47 (VSS), U3.63 (VSS)
- net CHARGE_CONNECTED: no longer names the net of U3.45 (PA12)
- no-connect marks 0 -> 15
Changed lines of the file:
@@
 	1    0    0    -1
 $EndComp
-Text HLabel 6350 2800 2    50   Output ~ 0
-SUPPLY_EN_MCU
 Text HLabel 6350 2900 2    50   Input ~ 0
 R_MTR_OVERCUR
@@
 Text HLabel 6350 3300 2    50   Input ~ 0
 L_MTR_PHC_HI
-Text HLabel 6350 3500 2    50   Input ~ 0
-CHARGE_CONNECTED
 Text HLabel 6350 3600 2    50   BiDi ~ 0
 SWDIO
@@
 	4400 1600 4400 1650
 Connection ~ 4400 1600
+NoConn ~ 4950 3600
+NoConn ~ 4950 3700
+NoConn ~ 4950 3800
+NoConn ~ 4950 4900
+NoConn ~ 4950 5300
+NoConn ~ 4950 5400
+NoConn ~ 4950 5500
+NoConn ~ 6350 4900
+NoConn ~ 6350 4800
+NoConn ~ 6350 4400
+NoConn ~ 6350 4300
+NoConn ~ 6350 3800
+NoConn ~ 6350 3400
+$Comp
+L power:GND #PWR0213
+U 1 1 5F71C540
+P 5450 5700
+F 0 "#PWR0213" H 5450 5450 50  0001 C CNN
+F 1 "GND" H 5455 5527 50  0000 C CNN
+F 2 "" H 5450 5700 50  0001 C CNN
+F 3 "" H 5450 5700 50  0001 C CNN
+	1    5450 5700
+	1    0    0    -1
+$EndComp
+$Comp
+L power:GND #PWR0214
+U 1 1 5F71CE6D
+P 5550 5700
+F 0 "#PWR0214" H 5550 5450 50  0001 C CNN
+F 1 "GND" H 5555 5527 50  0000 C CNN
+F 2 "" H 5550 5700 50  0001 C CNN
+F 3 "" H 5550 5700 50  0001 C CNN
+	1    5550 5700
+	1    0    0    -1
+$EndComp
+$Comp
+L power:GND #PWR0215
+U 1 1 5F71D00E
+P 5650 5700
+F 0 "#PWR0215" H 5650 5450 50  0001 C CNN
+F 1 "GND" H 5655 5527 50  0000 C CNN
+F 2 "" H 5650 5700 50  0001 C CNN
+F 3 "" H 5650 5700 50  0001 C CNN
+	1    5650 5700
+	1    0    0    -1
+$EndComp
+$Comp
+L power:GND #PWR0216
+U 1 1 5F71D1AF
+P 5750 5700
+F 0 "#PWR0216" H 5750 5450 50  0001 C CNN
+F 1 "GND" H 5755 5527 50  0000 C CNN
+F 2 "" H 5750 5700 50  0001 C CNN
+F 3 "" H 5750 5700 50  0001 C CNN
+	1    5750 5700
+	1    0    0    -1
+$EndComp
+$Comp
+L power:GND #PWR0217
+U 1 1 5F71D302
+P 5850 5700
+F 0 "#PWR0217" H 5850 5450 50  0001 C CNN
+F 1 "GND" H 5855 5527 50  0000 C CNN
+F 2 "" H 5850 5700 50  0001 C CNN
+F 3 "" H 5850 5700 50  0001 C CNN
+	1    5850 5700
+	1    0    0    -1
+$EndComp
+NoConn ~ 4950 2500
+NoConn ~ 6350 3500
+Text HLabel 6350 2800 2    50   Output ~ 0
+SUPPLY_EN_MCU
 $EndSCHEMATC

Commit message: Add CAN transceiver
Connections:
- net CAN_RX: now reaches U3.61 (PB8)
- net CAN_TX: now reaches U3.62 (PB9)
- no-connect marks 15 -> 13
Changed lines of the file:
@@
 $Descr A4 11693 8268
 encoding utf-8
-Sheet 4 13
+Sheet 4 14
 Title ""
 Date ""
@@
 NoConn ~ 4950 5400
 NoConn ~ 4950 5500
-NoConn ~ 6350 4900
-NoConn ~ 6350 4800
 NoConn ~ 6350 4400
 NoConn ~ 6350 4300
@@
 Text HLabel 6350 2800 2    50   Output ~ 0
 SUPPLY_EN_MCU
+Text HLabel 6350 4800 2    50   Input ~ 0
+CAN_RX
+Text HLabel 6350 4900 2    50   Output ~ 0
+CAN_TX
 $EndSCHEMATC

Commit message: Do MCU bypassing according to datasheet; annotate
Parts:
- added C39: 10n, symbol Device:C
- added C40: 1u, symbol Device:C
- C19, C20, C21, C23: footprint Capacitor_SMD:C_0603_1608Metric -> (none)
- C22: value 100n -> 4.7u; footprint Capacitor_SMD:C_0603_1608Metric -> (none)
Connections:
- net +3V3: now also C39.1, C40.1
- net GND: now also C39.2, C40.2

Commit message: added footprints, continue layout
Parts:
- C19, C20, C21, C23, C39: footprint (none) -> Capacitor_SMD:C_0603_1608Metric
- C22, C40: footprint (none) -> Capacitor_SMD:C_0805_2012Metric
Changed lines of the file:
@@
 F 0 "C23" H 5815 1396 50  0000 L CNN
 F 1 "100n" H 5815 1305 50  0000 L CNN
-F 2 "" H 5738 1200 50  0001 C CNN
+F 2 "Capacitor_SMD:C_0603_1608Metric" H 5738 1200 50  0001 C CNN
 F 3 "~" H 5700 1350 50  0001 C CNN
 	1    5700 1350
@@
 F 0 "C21" H 6315 1396 50  0000 L CNN
 F 1 "100n" H 6315 1305 50  0000 L CNN
-F 2 "" H 6238 1200 50  0001 C CNN
+F 2 "Capacitor_SMD:C_0603_1608Metric" H 6238 1200 50  0001 C CNN
 F 3 "~" H 6200 1350 50  0001 C CNN
 	1    6200 1350
@@
 F 0 "C19" H 6815 1396 50  0000 L CNN
 F 1 "100n" H 6815 1305 50  0000 L CNN
-F 2 "" H 6738 1200 50  0001 C CNN
+F 2 "Capacitor_SMD:C_0603_1608Metric" H 6738 1200 50  0001 C CNN
 F 3 "~" H 6700 1350 50  0001 C CNN
 	1    6700 1350
@@
 F 0 "C20" H 7315 1396 50  0000 L CNN
 F 1 "100n" H 7315 1305 50  0000 L CNN
-F 2 "" H 7238 1200 50  0001 C CNN
+F 2 "Capacitor_SMD:C_0603_1608Metric" H 7238 1200 50  0001 C CNN
 F 3 "~" H 7200 1350 50  0001 C CNN
 	1    7200 1350
@@
 F 0 "C22" H 7715 1396 50  0000 L CNN
 F 1 "4.7u" H 7715 1305 50  0000 L CNN
-F 2 "" H 7638 1200 50  0001 C CNN
+F 2 "Capacitor_SMD:C_0805_2012Metric" H 7638 1200 50  0001 C CNN
 F 3 "~" H 7600 1350 50  0001 C CNN
 	1    7600 1350
@@
 F 0 "C39" H 8215 1396 50  0000 L CNN
 F 1 "10n" H 8215 1305 50  0000 L CNN
-F 2 "" H 8138 1200 50  0001 C CNN
+F 2 "Capacitor_SMD:C_0603_1608Metric" H 8138 1200 50  0001 C CNN
 F 3 "~" H 8100 1350 50  0001 C CNN
 	1    8100 1350
@@
 F 0 "C40" H 8615 1396 50  0000 L CNN
 F 1 "1u" H 8615 1305 50  0000 L CNN
-F 2 "" H 8538 1200 50  0001 C CNN
+F 2 "Capacitor_SMD:C_0805_2012Metric" H 8538 1200 50  0001 C CNN
 F 3 "~" H 8500 1350 50  0001 C CNN
 	1    8500 1350

Commit message: add resistors on mosfet driver inputs, change board corners, fix labels
Parts:
- U3: value STM32F103RCTx -> STM32F103RCT
Changed lines of the file:
@@
 P 5650 3900
 F 0 "U3" H 5650 2011 50  0000 C CNN
-F 1 "STM32F103RCTx" H 5650 1920 50  0000 C CNN
+F 1 "STM32F103RCT" H 5650 1920 50  0000 C CNN
 F 2 "Package_QFP:LQFP-64_10x10mm_P0.5mm" H 5050 2200 50  0001 R CNN
 F 3 "http://www.st.com/st-web-ui/static/active/en/resource/technical/document/datasheet/CD00191185.pdf" H 5650 3900 50  0001 C CNN

Commit message: fix some bugs of the first revision
Parts:
- R56: value 3k -> 200 - 500
Changed lines of the file:
@@
 P 7300 2700
 F 0 "R56" V 7093 2700 50  0000 C CNN
-F 1 "3k" V 7184 2700 50  0000 C CNN
+F 1 "200 - 500" V 7184 2700 50  0000 C CNN
 F 2 "Resistor_SMD:R_0603_1608Metric" V 7230 2700 50  0001 C CNN
 F 3 "~" H 7300 2700 50  0001 C CNN

Commit message: Add oscillator for MCU
Parts:
- added C?: 100n, symbol Device:C
- added X?: C252325, Bobbycar-FOC-hardware:Oscillator_C387448, symbol Oscillator:ASDMB-xxxMHz
Connections:
- net +3V3: now also C?.1, X?.1 (Standby), X?.4 (VDD)
- net GND: now also C?.2, X?.2 (GND)
- net at U3.5 (PD0): now also X?.3 (Out)
- no-connect marks 13 -> 12
Changed lines of the file:
@@
 Wire Wire Line
 	6050 1150 6050 1800
-NoConn ~ 4950 3600
+$Comp
+L Oscillator:ASDMB-xxxMHz X?
+U 1 1 5F8CBBAB
+P 3500 3600
+F 0 "X?" H 3650 3350 50  0000 L CNN
+F 1 "C252325" H 3650 3250 50  0000 L CNN
+F 2 "Bobbycar-FOC-hardware:Oscillator_C387448" H 4200 3250 50  0001 C CNN
+F 3 "" H 3400 3600 50  0001 C CNN
+	1    3500 3600
+	1    0    0    -1
+$EndComp
+Wire Wire Line
+	3900 3600 4950 3600
+Wire Wire Line
+	3100 3600 3050 3600
+Wire Wire Line
+	3050 3600 3050 3250
+Wire Wire Line
+	3050 3250 3600 3250
+Wire Wire Line
+	3600 3250 3600 3300
+$Comp
+L power:+3.3V #PWR?
+U 1 1 5F8D1C3C
+P 3600 3200
+F 0 "#PWR?" H 3600 3050 50  0001 C CNN
+F 1 "+3.3V" H 3615 3373 50  0000 C CNN
+F 2 "" H 3600 3200 50  0001 C CNN
+F 3 "" H 3600 3200 50  0001 C CNN
+	1    3600 3200
+	1    0    0    -1
+$EndComp
+Wire Wire Line
+	3600 3200 3600 3250
+Connection ~ 3600 3250
+$Comp
+L power:GND #PWR?
+U 1 1 5F8D381D
+P 3600 4000
+F 0 "#PWR?" H 3600 3750 50  0001 C CNN
+F 1 "GND" H 3605 3827 50  0000 C CNN
+F 2 "" H 3600 4000 50  0001 C CNN
+F 3 "" H 3600 4000 50  0001 C CNN
+	1    3600 4000
+	1    0    0    -1
+$EndComp
+Wire Wire Line
+	3600 3900 3600 3950
+$Comp
+L Device:C C?
+U 1 1 5F8D5E88
+P 2700 3600
+F 0 "C?" H 2815 3646 50  0000 L CNN
+F 1 "100n" H 2815 3555 50  0000 L CNN
+F 2 "" H 2738 3450 50  0001 C CNN
+F 3 "~" H 2700 3600 50  0001 C CNN
+	1    2700 3600
+	1    0    0    -1
+$EndComp
+Wire Wire Line
+	3050 3250 2700 3250
+Wire Wire Line
+	2700 3250 2700 3450
+Connection ~ 3050 3250
+Wire Wire Line
+	2700 3750 2700 3950
+Wire Wire Line
+	2700 3950 3600 3950
+Connection ~ 3600 3950
+Wire Wire Line
+	3600 3950 3600 4000
 $EndSCHEMATC
