File: mcu.sch (KiCad schematic (older format))
At the start: 26 parts, among them Q6 MMBT5551, U3 STM32F103RCT

Commit message: Layout oscillator
Parts:
- C70: renamed from C?; footprint (none) -> Capacitor_SMD:C_0603_1608Metric
- gave numbers to parts that had none: 1
Changed lines of the file:
@@
 	6050 1150 6050 1800
 $Comp
-L Oscillator:ASDMB-xxxMHz X?
+L Oscillator:ASDMB-xxxMHz X1
 U 1 1 5F8CBBAB
 P 3500 3600
-F 0 "X?" H 3650 3350 50  0000 L CNN
+F 0 "X1" H 3650 3350 50  0000 L CNN
 F 1 "C252325" H 3650 3250 50  0000 L CNN
 F 2 "Bobbycar-FOC-hardware:Oscillator_C387448" H 4200 3250 50  0001 C CNN
@@
 	3600 3250 3600 3300
 $Comp
-L power:+3.3V #PWR?
+L power:+3.3V #PWR0114
 U 1 1 5F8D1C3C
 P 3600 3200
-F 0 "#PWR?" H 3600 3050 50  0001 C CNN
+F 0 "#PWR0114" H 3600 3050 50  0001 C CNN
 F 1 "+3.3V" H 3615 3373 50  0000 C CNN
 F 2 "" H 3600 3200 50  0001 C CNN
@@
 Connection ~ 3600 3250
 $Comp
-L power:GND #PWR?
+L power:GND #PWR0245
 U 1 1 5F8D381D
 P 3600 4000
-F 0 "#PWR?" H 3600 3750 50  0001 C CNN
+F 0 "#PWR0245" H 3600 3750 50  0001 C CNN
 F 1 "GND" H 3605 3827 50  0000 C CNN
 F 2 "" H 3600 4000 50  0001 C CNN
@@
 	3600 3900 3600 3950
 $Comp
-L Device:C C?
+L Device:C C70
 U 1 1 5F8D5E88
 P 2700 3600
-F 0 "C?" H 2815 3646 50  0000 L CNN
+F 0 "C70" H 2815 3646 50  0000 L CNN
 F 1 "100n" H 2815 3555 50  0000 L CNN
-F 2 "" H 2738 3450 50  0001 C CNN
+F 2 "Capacitor_SMD:C_0603_1608Metric" H 2738 3450 50  0001 C CNN
 F 3 "~" H 2700 3600 50  0001 C CNN
 	1    2700 3600

Commit message: Changed fet driver
Parts:
- R20, R44: value 1k -> 2k2
- R41: value 10k -> 100k
- R42: value 1k -> 47k
- R43: value 1k -> 10k
Other:
- note added: "UCC27517\nC99395\nFET Treiber\nhttps://www.ti.com/product/UCC27517"
Changed lines of the file:
@@
 P 7250 4200
 F 0 "R20" V 7457 4200 50  0000 C CNN
-F 1 "1k" V 7366 4200 50  0000 C CNN
+F 1 "2k2" V 7366 4200 50  0000 C CNN
 F 2 "Resistor_SMD:R_0603_1608Metric" V 7180 4200 50  0001 C CNN
 F 3 "~" H 7250 4200 50  0001 C CNN
@@
 P 9600 3850
 F 0 "R42" V 9807 3850 50  0000 C CNN
-F 1 "1k" V 9716 3850 50  0000 C CNN
+F 1 "47k" V 9716 3850 50  0000 C CNN
 F 2 "Resistor_SMD:R_0603_1608Metric" V 9530 3850 50  0001 C CNN
 F 3 "~" H 9600 3850 50  0001 C CNN
@@
 P 9600 4250
 F 0 "R43" V 9807 4250 50  0000 C CNN
-F 1 "1k" V 9716 4250 50  0000 C CNN
+F 1 "10k" V 9716 4250 50  0000 C CNN
 F 2 "Resistor_SMD:R_0603_1608Metric" V 9530 4250 50  0001 C CNN
 F 3 "~" H 9600 4250 50  0001 C CNN
@@
 P 9600 4700
 F 0 "R44" V 9807 4700 50  0000 C CNN
-F 1 "1k" V 9716 4700 50  0000 C CNN
+F 1 "2k2" V 9716 4700 50  0000 C CNN
 F 2 "Resistor_SMD:R_0603_1608Metric" V 9530 4700 50  0001 C CNN
 F 3 "~" H 9600 4700 50  0001 C CNN
@@
 P 9600 3400
 F 0 "R41" V 9807 3400 50  0000 C CNN
-F 1 "10k" V 9716 3400 50  0000 C CNN
+F 1 "100k" V 9716 3400 50  0000 C CNN
 F 2 "Resistor_SMD:R_0603_1608Metric" V 9530 3400 50  0001 C CNN
 F 3 "~" H 9600 3400 50  0001 C CNN
@@
 Wire Wire Line
 	3600 3950 3600 4000
+Text Notes 1600 5000 0    50   ~ 0
+UCC27517\nC99395\nFET Treiber\nhttps://www.ti.com/product/UCC27517
 $EndSCHEMATC

Commit message: Added FET for LED
Parts:
- added C75: 100n, Capacitor_SMD:C_0603_1608Metric, symbol Device:C
- added C76: 1u, Capacitor_SMD:C_0805_2012Metric, symbol Device:C
- added J17: Conn_01x01_Male, Connector_Pin:Pin_D1.4mm_L8.5mm_W2.8mm_FlatFork, symbol Connector:Conn_01x01_Male
- added R46, R47: 1k, Resistor_SMD:R_0603_1608Metric, symbol Device:R
- added R79: 4.7, Resistor_SMD:R_1206_3216Metric, symbol Device:R
- added U17: UCC27517, Package_TO_SOT_SMD:SOT-23-5, symbol Bobbycontroller:UCC27517
- added V12: CRSS042N10N, Package_TO_SOT_SMD:TO-263-2, symbol Transistor_FET:BSP89
Connections:
- net +3V3: now also R46.2
- net +VSW: now also C75.1, C76.1, U17.1 (VDD)
- net GND: now also C75.2, C76.2, R47.2, U17.2 (GND), U17.4 (IN-), V12.3 (S)
- net at U3.44 (PA11): now also R46.1, R47.1
- net at U3.55 (PB3): now also U17.3 (IN+)
- new net: R79.2, U17.5 (OUT)
- new net: R79.1, V12.1 (G)
- new net: J17.1 (Pin_1), V12.2 (D)
- no-connect marks 12 -> 10
Other:
- note added: "ID for CAN Address"
- note added: "LED-Light"
- note removed: "UCC27517\nC99395\nFET Treiber\nhttps://www.ti.com/product/UCC27517"
- moved on the sheet: R41, R42, R43, R44

Commit message: Routed FET and jumper
Parts:
- V12: value CRSS042N10N -> NCE0115K; footprint Package_TO_SOT_SMD:TO-263-2 -> Package_TO_SOT_SMD:TO-252-2
Connections:
- net L_MTR_OVERCUR: now also U3.44 (PA11); no longer U3.33 (PB12)
- net at R46.1, R47.1: now also U3.33 (PB12); no longer U3.44 (PA11)
Other:
- moved on the sheet: R46, R47
Changed lines of the file:
@@
 Text HLabel 6350 5100 2    50   Input ~ 0
 UART_R_RX
-Text HLabel 6350 5200 2    50   Input ~ 0
+Text HLabel 6350 3400 2    50   Input ~ 0
 L_MTR_OVERCUR
 Text HLabel 6350 5300 2    50   Output ~ 0
@@
 AR Path="/5F75358D/603858D6" Ref="V12"  Part="1"
 F 0 "V12" H 9304 4846 50  0000 L CNN
-F 1 "CRSS042N10N" H 9304 4755 50  0000 L CNN
-F 2 "Package_TO_SOT_SMD:TO-263-2" H 9300 4725 50  0001 L CIN
-F 3 "https://www.infineon.com/dgdl/Infineon-BSP89-DS-v02_02-en.pdf?fileId=db3a30433b47825b013b4b8a07f90d55" H 9100 4800 50  0001 L CNN
+F 1 "NCE0115K" H 9304 4755 50  0000 L CNN
+F 2 "Package_TO_SOT_SMD:TO-252-2" H 9300 4725 50  0001 L CIN
+F 3 "" H 9100 4800 50  0001 L CNN
 	1    9100 4800
 	1    0    0    -1
@@
 L Device:R R47
 U 1 1 603B7EB5
-P 7300 3500
-F 0 "R47" V 7200 3500 50  0000 C CNN
-F 1 "1k" V 7100 3500 50  0000 C CNN
-F 2 "Resistor_SMD:R_0603_1608Metric" V 7230 3500 50  0001 C CNN
-F 3 "~" H 7300 3500 50  0001 C CNN
-	1    7300 3500
+P 7300 5300
+F 0 "R47" V 7200 5300 50  0000 C CNN
+F 1 "1k" V 7100 5300 50  0000 C CNN
+F 2 "Resistor_SMD:R_0603_1608Metric" V 7230 5300 50  0001 C CNN
+F 3 "~" H 7300 5300 50  0001 C CNN
+	1    7300 5300
 	0    -1   -1   0
 $EndComp
@@
 L Device:R R46
 U 1 1 603B8184
-P 7300 3400
-F 0 "R46" V 7507 3400 50  0000 C CNN
-F 1 "1k" V 7416 3400 50  0000 C CNN
-F 2 "Resistor_SMD:R_0603_1608Metric" V 7230 3400 50  0001 C CNN
-F 3 "~" H 7300 3400 50  0001 C CNN
-	1    7300 3400
+P 7300 5200
+F 0 "R46" V 7507 5200 50  0000 C CNN
+F 1 "1k" V 7416 5200 50  0000 C CNN
+F 2 "Resistor_SMD:R_0603_1608Metric" V 7230 5200 50  0001 C CNN
+F 3 "~" H 7300 5200 50  0001 C CNN
+	1    7300 5200
 	0    -1   -1   0
 $EndComp
@@
 L power:+3.3V #PWR08
 U 1 1 603B83D0
-P 7450 3400
-F 0 "#PWR08" H 7450 3250 50  0001 C CNN
-F 1 "+3.3V" H 7465 3573 50  0000 C CNN
-F 2 "" H 7450 3400 50  0001 C CNN
-F 3 "" H 7450 3400 50  0001 C CNN
-	1    7450 3400
+P 7450 5200
+F 0 "#PWR08" H 7450 5050 50  0001 C CNN
+F 1 "+3.3V" H 7465 5373 50  0000 C CNN
+F 2 "" H 7450 5200 50  0001 C CNN
+F 3 "" H 7450 5200 50  0001 C CNN
+	1    7450 5200
 	1    0    0    -1
 $EndComp
@@
 L power:GND #PWR09
 U 1 1 603BA217
-P 7450 3500
-F 0 "#PWR09" H 7450 3250 50  0001 C CNN
-F 1 "GND" H 7455 3327 50  0000 C CNN
-F 2 "" H 7450 3500 50  0001 C CNN
-F 3 "" H 7450 3500 50  0001 C CNN
-	1    7450 3500
-	1    0    0    -1
-$EndComp
-Wire Wire Line
-	6350 3400 7150 3400
-Wire Wire Line
-	7150 3400 7150 3500
-Connection ~ 7150 3400
-Text Notes 7550 3450 0    50   ~ 0
+P 7450 5300
+F 0 "#PWR09" H 7450 5050 50  0001 C CNN
+F 1 "GND" H 7455 5127 50  0000 C CNN
+F 2 "" H 7450 5300 50  0001 C CNN
+F 3 "" H 7450 5300 50  0001 C CNN
+	1    7450 5300
+	1    0    0    -1
+$EndComp
+Wire Wire Line
+	6350 5200 7150 5200
+Wire Wire Line
+	7150 5200 7150 5300
+Connection ~ 7150 5200
+Text Notes 7550 5450 0    50   ~ 0
 ID for CAN Address
 $Comp

Commit message: Added LCSC Part # to most components
Parts:
- C19, C20, C21, C23, C4, C70, C75: value 100n -> 100nF; LCSC Part # (none) -> C14663
- C22: LCSC Part # (none) -> C1779
- C39: value 10n -> 10nF; LCSC Part # (none) -> C57112
- C40, C76: LCSC Part # (none) -> C28323
- D1AR1: LCSC Part # (none) -> C81598
- R19, R43: LCSC Part # (none) -> C25804
- R20, R44: value 2k2 -> 2.2k; LCSC Part # (none) -> C4190
- R41: LCSC Part # (none) -> C25803
- R42: LCSC Part # (none) -> C25819
- R46, R47: LCSC Part # (none) -> C21190
- R79: LCSC Part # (none) -> C17937
- U3: LCSC Part # (none) -> C8323
- V12: LCSC Part # (none) -> C108637
Changed lines of the file:
@@
 F 2 "Package_QFP:LQFP-64_10x10mm_P0.5mm" H 5050 2200 50  0001 R CNN
 F 3 "http://www.st.com/st-web-ui/static/active/en/resource/technical/document/datasheet/CD00191185.pdf" H 5650 3900 50  0001 C CNN
+F 4 "C8323" H 5650 3900 50  0001 C CNN "LCSC Part #"
 	1    5650 3900
 	1    0    0    -1
@@
 F 2 "Diode_SMD:D_SOD-123" H 7400 2350 50  0001 C CNN
 F 3 "~" H 7400 2350 50  0001 C CNN
+F 4 "C81598" H 7400 2350 50  0001 C CNN "LCSC Part #"
 	1    7400 2350
 	0    1    1    0
@@
 P 7250 4200
 F 0 "R20" V 7457 4200 50  0000 C CNN
-F 1 "2k2" V 7366 4200 50  0000 C CNN
+F 1 "2.2k" V 7366 4200 50  0000 C CNN
 F 2 "Resistor_SMD:R_0603_1608Metric" V 7180 4200 50  0001 C CNN
 F 3 "~" H 7250 4200 50  0001 C CNN
+F 4 "C4190" H 7250 4200 50  0001 C CNN "LCSC Part #"
 	1    7250 4200
 	0    -1   -1   0
@@
 F 2 "Resistor_SMD:R_0603_1608Metric" V 4330 1400 50  0001 C CNN
 F 3 "~" H 4400 1400 50  0001 C CNN
+F 4 "C25804" H 4400 1400 50  0001 C CNN "LCSC Part #"
 	1    4400 1400
 	1    0    0    -1
@@
 P 4400 1800
 F 0 "C4" H 4515 1800 50  0000 L CNN
-F 1 "100n" H 4515 1755 50  0001 L CNN
+F 1 "100nF" H 4515 1755 50  0001 L CNN
 F 2 "Capacitor_SMD:C_0603_1608Metric" H 4438 1650 50  0001 C CNN
 F 3 "~" H 4400 1800 50  0001 C CNN
+F 4 "C14663" H 4400 1800 50  0001 C CNN "LCSC Part #"
 	1    4400 1800
 	1    0    0    -1
@@
 F 2 "Resistor_SMD:R_0603_1608Metric" V 10080 2450 50  0001 C CNN
 F 3 "~" H 10150 2450 50  0001 C CNN
+F 4 "C25819" H 10150 2450 50  0001 C CNN "LCSC Part #"
 	1    10150 2450
 	0    -1   -1   0
@@
 F 2 "Resistor_SMD:R_0603_1608Metric" V 10080 2850 50  0001 C CNN
 F 3 "~" H 10150 2850 50  0001 C CNN
+F 4 "C25804" H 10150 2850 50  0001 C CNN "LCSC Part #"
 	1    10150 2850
 	0    -1   -1   0
@@
 P 10150 3300
 F 0 "R44" V 10357 3300 50  0000 C CNN
-F 1 "2k2" V 10266 3300 50  0000 C CNN
+F 1 "2.2k" V 10266 3300 50  0000 C CNN
 F 2 "Resistor_SMD:R_0603_1608Metric" V 10080 3300 50  0001 C CNN
 F 3 "~" H 10150 3300 50  0001 C CNN
+F 4 "C4190" H 10150 3300 50  0001 C CNN "LCSC Part #"
 	1    10150 3300
 	0    -1   -1   0
@@
 F 2 "Resistor_SMD:R_0603_1608Metric" V 10080 2000 50  0001 C CNN
 F 3 "~" H 10150 2000 50  0001 C CNN
+F 4 "C25803" H 10150 2000 50  0001 C CNN "LCSC Part #"
 	1    10150 2000
 	0    -1   -1   0
@@
 P 5700 1350
 F 0 "C23" H 5815 1396 50  0000 L CNN
-F 1 "100n" H 5815 1305 50  0000 L CNN
+F 1 "100nF" H 5815 1305 50  0000 L CNN
 F 2 "Capacitor_SMD:C_0603_1608Metric" H 5738 1200 50  0001 C CNN
 F 3 "~" H 5700 1350 50  0001 C CNN
+F 4 "C14663" H 5700 1350 50  0001 C CNN "LCSC Part #"
 	1    5700 1350
 	1    0    0    -1
@@
 P 6200 1350
 F 0 "C21" H 6315 1396 50  0000 L CNN
-F 1 "100n" H 6315 1305 50  0000 L CNN
+F 1 "100nF" H 6315 1305 50  0000 L CNN
 F 2 "Capacitor_SMD:C_0603_1608Metric" H 6238 1200 50  0001 C CNN
 F 3 "~" H 6200 1350 50  0001 C CNN
+F 4 "C14663" H 6200 1350 50  0001 C CNN "LCSC Part #"
 	1    6200 1350
 	1    0    0    -1
@@
 P 6700 1350
 F 0 "C19" H 6815 1396 50  0000 L CNN
-F 1 "100n" H 6815 1305 50  0000 L CNN
+F 1 "100nF" H 6815 1305 50  0000 L CNN
 F 2 "Capacitor_SMD:C_0603_1608Metric" H 6738 1200 50  0001 C CNN
 F 3 "~" H 6700 1350 50  0001 C CNN
+F 4 "C14663" H 6700 1350 50  0001 C CNN "LCSC Part #"
 	1    6700 1350
 	1    0    0    -1
@@
 P 7200 1350
 F 0 "C20" H 7315 1396 50  0000 L CNN
-F 1 "100n" H 7315 1305 50  0000 L CNN
+F 1 "100nF" H 7315 1305 50  0000 L CNN
 F 2 "Capacitor_SMD:C_0603_1608Metric" H 7238 1200 50  0001 C CNN
 F 3 "~" H 7200 1350 50  0001 C CNN
+F 4 "C14663" H 7200 1350 50  0001 C CNN "LCSC Part #"
 	1    7200 1350
 	1    0    0    -1
@@
 F 2 "Capacitor_SMD:C_0805_2012Metric" H 7638 1200 50  0001 C CNN
 F 3 "~" H 7600 1350 50  0001 C CNN
+F 4 "C1779" H 7600 1350 50  0001 C CNN "LCSC Part #"
 	1    7600 1350
 	1    0    0    -1
@@
 P 8100 1350
 F 0 "C39" H 8215 1396 50  0000 L CNN
-F 1 "10n" H 8215 1305 50  0000 L CNN
+F 1 "10nF" H 8215 1305 50  0000 L CNN
 F 2 "Capacitor_SMD:C_0603_1608Metric" H 8138 1200 50  0001 C CNN
 F 3 "~" H 8100 1350 50  0001 C CNN
+F 4 "C57112" H 8100 1350 50  0001 C CNN "LCSC Part #"
 	1    8100 1350
 	1    0    0    -1
@@
 F 2 "Capacitor_SMD:C_0805_2012Metric" H 8538 1200 50  0001 C CNN
 F 3 "~" H 8500 1350 50  0001 C CNN
+F 4 "C28323" H 8500 1350 50  0001 C CNN "LCSC Part #"
 	1    8500 1350
 	1    0    0    -1
@@
 P 2700 3600
 F 0 "C70" H 2815 3646 50  0000 L CNN
-F 1 "100n" H 2815 3555 50  0000 L CNN
+F 1 "100nF" H 2815 3555 50  0000 L CNN
 F 2 "Capacitor_SMD:C_0603_1608Metric" H 2738 3450 50  0001 C CNN
 F 3 "~" H 2700 3600 50  0001 C CNN
+F 4 "C14663" H 2700 3600 50  0001 C CNN "LCSC Part #"
 	1    2700 3600
 	1    0    0    -1
@@
 F 2 "Package_TO_SOT_SMD:TO-252-2" H 9300 4725 50  0001 L CIN
 F 3 "" H 9100 4800 50  0001 L CNN
+F 4 "C108637" H 9100 4800 50  0001 C CNN "LCSC Part #"
 	1    9100 4800
 	1    0    0    -1
@@
 F 2 "Resistor_SMD:R_1206_3216Metric" V 8630 4800 50  0001 C CNN
 F 3 "~" H 8700 4800 50  0001 C CNN
+F 4 "C17937" H 8700 4800 50  0001 C CNN "LCSC Part #"
 	1    8700 4800
 	0    1    1    0
@@
 P 8500 4100
 F 0 "C75" H 8615 4146 50  0000 L CNN
-F 1 "100n" H 8615 4055 50  0000 L CNN
+F 1 "100nF" H 8615 4055 50  0000 L CNN
 F 2 "Capacitor_SMD:C_0603_1608Metric" H 8538 3950 50  0001 C CNN
 F 3 "~" H 8500 4100 50  0001 C CNN
+F 4 "C14663" H 8500 4100 50  0001 C CNN "LCSC Part #"
 	1    8500 4100
 	1    0    0    -1
@@
 F 2 "Resistor_SMD:R_0603_1608Metric" V 7230 5300 50  0001 C CNN
 F 3 "~" H 7300 5300 50  0001 C CNN
+F 4 "C21190" H 7300 5300 50  0001 C CNN "LCSC Part #"
 	1    7300 5300
 	0    -1   -1   0
@@
 F 2 "Resistor_SMD:R_0603_1608Metric" V 7230 5200 50  0001 C CNN
 F 3 "~" H 7300 5200 50  0001 C CNN
+F 4 "C21190" H 7300 5200 50  0001 C CNN "LCSC Part #"
 	1    7300 5200
 	0    -1   -1   0
@@
 F 2 "Capacitor_SMD:C_0805_2012Metric" H 8938 3950 50  0001 C CNN
 F 3 "~" H 8900 4100 50  0001 C CNN
+F 4 "C28323" H 8900 4100 50  0001 C CNN "LCSC Part #"
 	1    8900 4100
 	1    0    0    -1

Commit message: More adaptation to jlcpcb, parts checking
Parts:
- D13, D14, D15, D16, D2: LCSC Part # (none) -> C2290
- J17: place (none) -> dnp
- LS1: place (none) -> hand
- Q6: LCSC Part # (none) -> C2145
- R56: value 200 - 500 -> 220; LCSC Part # (none) -> C22962
- U3: LCSC Part # C8323 -> (none); place (none) -> hand
- X1: value C252325 -> 8MHz 2520; LCSC Part # (none) -> C390520
Changed lines of the file:
@@
 F 2 "Package_QFP:LQFP-64_10x10mm_P0.5mm" H 5050 2200 50  0001 R CNN
 F 3 "http://www.st.com/st-web-ui/static/active/en/resource/technical/document/datasheet/CD00191185.pdf" H 5650 3900 50  0001 C CNN
-F 4 "C8323" H 5650 3900 50  0001 C CNN "LCSC Part #"
+F 4 "" H 5650 3900 50  0001 C CNN "LCSC Part #"
+F 5 "hand" H 5650 3900 50  0001 C CNN "place"
 	1    5650 3900
 	1    0    0    -1
@@
 P 7300 2700
 F 0 "R56" V 7093 2700 50  0000 C CNN
-F 1 "200 - 500" V 7184 2700 50  0000 C CNN
+F 1 "220" V 7184 2700 50  0000 C CNN
 F 2 "Resistor_SMD:R_0603_1608Metric" V 7230 2700 50  0001 C CNN
 F 3 "~" H 7300 2700 50  0001 C CNN
+F 4 "C22962" H 7300 2700 50  0001 C CNN "LCSC Part #"
 	1    7300 2700
 	0    1    1    0
@@
 F 1 "MMBT5551" H 7841 2655 50  0000 L CNN
 F 2 "Package_TO_SOT_SMD:SOT-23" H 7850 2800 50  0001 C CNN
-F 3 "~" H 7650 2700 50  0001 C CNN
+F 3 "" H 7650 2700 50  0001 C CNN
+F 4 "C2145" H 7650 2700 50  0001 C CNN "LCSC Part #"
 	1    7650 2700
 	1    0    0    -1
@@
 F 1 "FS1212 #Rastermaß 6.5" H 8120 2150 50  0000 L CNN
 F 2 "Buzzer_Beeper:Buzzer_12x9.5RM7.6" H 7950 2000 50  0001 C CNN
-F 3 "~" H 7940 2150 50  0001 C CNN
+F 3 "" H 7940 2150 50  0001 C CNN
+F 4 "hand" H 7950 2200 50  0001 C CNN "place"
 	1    7950 2200
 	1    0    0    -1
@@
 F 1 "LED" H 7543 4036 50  0000 C CNN
 F 2 "LED_SMD:LED_0603_1608Metric" H 7550 4200 50  0001 C CNN
-F 3 "~" H 7550 4200 50  0001 C CNN
+F 3 "" H 7550 4200 50  0001 C CNN
+F 4 "C2290" H 7550 4200 50  0001 C CNN "LCSC Part #"
 	1    7550 4200
 	-1   0    0    1
@@
 F 1 "LED" H 10443 1836 50  0000 C CNN
 F 2 "LED_SMD:LED_0603_1608Metric" H 10450 2000 50  0001 C CNN
-F 3 "~" H 10450 2000 50  0001 C CNN
+F 3 "" H 10450 2000 50  0001 C CNN
+F 4 "C2290" H 10450 2000 50  0001 C CNN "LCSC Part #"
 	1    10450 2000
 	-1   0    0    1
@@
 F 1 "LED" H 10443 2286 50  0000 C CNN
 F 2 "LED_SMD:LED_0603_1608Metric" H 10450 2450 50  0001 C CNN
-F 3 "~" H 10450 2450 50  0001 C CNN
+F 3 "" H 10450 2450 50  0001 C CNN
+F 4 "C2290" H 10450 2450 50  0001 C CNN "LCSC Part #"
 	1    10450 2450
 	-1   0    0    1
@@
 F 1 "LED" H 10443 2686 50  0000 C CNN
 F 2 "LED_SMD:LED_0603_1608Metric" H 10450 2850 50  0001 C CNN
-F 3 "~" H 10450 2850 50  0001 C CNN
+F 3 "" H 10450 2850 50  0001 C CNN
+F 4 "C2290" H 10450 2850 50  0001 C CNN "LCSC Part #"
 	1    10450 2850
 	-1   0    0    1
@@
 F 1 "LED" H 10443 3136 50  0000 C CNN
 F 2 "LED_SMD:LED_0603_1608Metric" H 10450 3300 50  0001 C CNN
-F 3 "~" H 10450 3300 50  0001 C CNN
+F 3 "" H 10450 3300 50  0001 C CNN
+F 4 "C2290" H 10450 3300 50  0001 C CNN "LCSC Part #"
 	1    10450 3300
 	-1   0    0    1
@@
 P 3500 3600
 F 0 "X1" H 3650 3350 50  0000 L CNN
-F 1 "C252325" H 3650 3250 50  0000 L CNN
+F 1 "8MHz 2520" H 3650 3250 50  0000 L CNN
 F 2 "Bobbycar-FOC-hardware:Oscillator_C387448" H 4200 3250 50  0001 C CNN
 F 3 "" H 3400 3600 50  0001 C CNN
+F 4 "C390520" H 3500 3600 50  0001 C CNN "LCSC Part #"
 	1    3500 3600
 	1    0    0    -1
@@
 F 2 "Connector_Pin:Pin_D1.4mm_L8.5mm_W2.8mm_FlatFork" H 9400 4500 50  0001 C CNN
 F 3 "~" H 9400 4500 50  0001 C CNN
+F 4 "dnp" H 9400 4500 50  0001 C CNN "place"
 	1    9400 4500
 	-1   0    0    1

Commit message: Added emergency-break connector
Parts:
- added C84: 100nF, Capacitor_SMD:C_0603_1608Metric, symbol Device:C
- added D12: CDSOD323, Diode_SMD:D_SOD-323, symbol input-board:CDSOD323-boardcomputer
- added J18: Conn_01x02, Connector_Molex:Molex_PicoBlade_53047-0210_1x02_P1.25mm_Vertical, symbol Connector_Generic:Conn_01x02
- added R82: 1k, Resistor_SMD:R_0603_1608Metric, symbol Device:R
- added R83: 100, Resistor_SMD:R_0603_1608Metric, symbol Device:R
Connections:
- net +3V3: now also R82.2
- net GND: now also C84.2, D12.2 (A), J18.2 (Pin_2)
- net at U3.45 (PA12): now also C84.1, D12.1 (K), R82.1, R83.2
- new net: J18.1 (Pin_1), R83.1
- no-connect marks 10 -> 9
Other:
- moved on the sheet: C75, C76, J17, R79, U17, V12

Commit message: Changed emergency brake to uart2 connector
Parts:
- removed C84: 100nF, Capacitor_SMD:C_0603_1608Metric, symbol Device:C
- removed D12: CDSOD323, Diode_SMD:D_SOD-323, symbol input-board:CDSOD323-boardcomputer
- removed J18: Conn_01x02, Connector_Molex:Molex_PicoBlade_53047-0210_1x02_P1.25mm_Vertical, symbol Connector_Generic:Conn_01x02
- removed R82: 1k, Resistor_SMD:R_0603_1608Metric, symbol Device:R
- removed R83: 100, Resistor_SMD:R_0603_1608Metric, symbol Device:R
Changed lines of the file:
@@
 Text Notes 9700 4350 0    50   ~ 0
 LED-Light
-$Comp
-L Connector_Generic:Conn_01x02 J18
-U 1 1 604B57CC
-P 8750 3500
-F 0 "J18" H 8830 3492 50  0000 L CNN
-F 1 "Conn_01x02" H 8830 3401 50  0000 L CNN
-F 2 "Connector_Molex:Molex_PicoBlade_53047-0210_1x02_P1.25mm_Vertical" H 8750 3500 50  0001 C CNN
-F 3 "~" H 8750 3500 50  0001 C CNN
-	1    8750 3500
-	1    0    0    -1
-$EndComp
-$Comp
-L Device:R R82
-U 1 1 604B8BE5
-P 8300 3350
-F 0 "R82" V 8400 3400 50  0000 C CNN
-F 1 "1k" V 8400 3250 50  0000 C CNN
-F 2 "Resistor_SMD:R_0603_1608Metric" V 8230 3350 50  0001 C CNN
-F 3 "~" H 8300 3350 50  0001 C CNN
-F 4 "C21190" H 8300 3350 50  0001 C CNN "LCSC Part #"
-	1    8300 3350
-	0    -1   -1   0
-$EndComp
-$Comp
-L power:+3.3V #PWR014
-U 1 1 604B9333
-P 8450 3350
-F 0 "#PWR014" H 8450 3200 50  0001 C CNN
-F 1 "+3.3V" V 8450 3600 50  0000 C CNN
-F 2 "" H 8450 3350 50  0001 C CNN
-F 3 "" H 8450 3350 50  0001 C CNN
-	1    8450 3350
-	0    1    1    0
-$EndComp
-$Comp
-L power:GND #PWR07
-U 1 1 604C25D2
-P 7850 3800
-F 0 "#PWR07" H 7850 3550 50  0001 C CNN
-F 1 "GND" H 7855 3627 50  0000 C CNN
-F 2 "" H 7850 3800 50  0001 C CNN
-F 3 "" H 7850 3800 50  0001 C CNN
-	1    7850 3800
-	1    0    0    -1
-$EndComp
-Wire Wire Line
-	8150 3500 8150 3350
-Connection ~ 8150 3500
-$Comp
-L input-board:CDSOD323-boardcomputer D12
-U 1 1 604E029D
-P 8150 3600
-F 0 "D12" V 8300 3700 50  0000 L CNN
-F 1 "CDSOD323" V 8400 3400 50  0000 L CNN
-F 2 "Diode_SMD:D_SOD-323" H 8150 3750 50  0001 C CNN
-F 3 "" H 8150 3750 50  0001 C CNN
-F 4 "C127526" V 8150 3600 50  0001 C CNN "LCSC Part #"
-	1    8150 3600
-	0    1    1    0
-$EndComp
-$Comp
-L Device:R R?
-U 1 1 605069DF
-P 8300 3500
-AR Path="/5F74B195/605069DF" Ref="R?"  Part="1"
-AR Path="/5F75358D/605069DF" Ref="R83"  Part="1"
-F 0 "R83" V 8400 3500 50  0000 C CNN
-F 1 "100" V 8450 3650 50  0000 C CNN
-F 2 "Resistor_SMD:R_0603_1608Metric" V 8230 3500 50  0001 C CNN
-F 3 "~" H 8300 3500 50  0001 C CNN
-F 4 "C22775" H 8300 3500 50  0001 C CNN "LCSC Part #"
-	1    8300 3500
-	0    1    1    0
-$EndComp
-$Comp
-L Device:C C84
-U 1 1 6050851D
-P 7850 3650
-F 0 "C84" H 7500 3700 50  0000 L CNN
-F 1 "100nF" H 7500 3600 50  0000 L CNN
-F 2 "Capacitor_SMD:C_0603_1608Metric" H 7888 3500 50  0001 C CNN
-F 3 "~" H 7850 3650 50  0001 C CNN
-F 4 "C14663" H 7850 3650 50  0001 C CNN "LCSC Part #"
-	1    7850 3650
-	1    0    0    -1
-$EndComp
-Wire Wire Line
-	6350 3500 7850 3500
-Connection ~ 7850 3500
-Wire Wire Line
-	7850 3500 8150 3500
-Wire Wire Line
-	7850 3800 8150 3800
-Wire Wire Line
-	8550 3800 8550 3600
-Connection ~ 7850 3800
-Connection ~ 8150 3800
-Wire Wire Line
-	8150 3800 8550 3800
-Wire Wire Line
-	8450 3500 8550 3500
 $EndSCHEMATC
