File: mcu.sch (KiCad schematic (older format))
At the start: 34 parts, among them J17 Conn_01x01_Male, Q6 MMBT5551, U17 UCC27517, U3 STM32F103RCT, X1 8MHz 2520

Commit message: Added pth caps to assembly
Parts:
- R42: value 47k -> 20k; LCSC Part # C25819 -> C4184
- R43: value 10k -> 3.3k; LCSC Part # C25804 -> C22978
- R44: value 2.2k -> 1k; LCSC Part # C4190 -> C21190
Changed lines of the file:
@@
 P 10150 2450
 F 0 "R42" V 10357 2450 50  0000 C CNN
-F 1 "47k" V 10266 2450 50  0000 C CNN
+F 1 "20k" V 10266 2450 50  0000 C CNN
 F 2 "Resistor_SMD:R_0603_1608Metric" V 10080 2450 50  0001 C CNN
 F 3 "~" H 10150 2450 50  0001 C CNN
-F 4 "C25819" H 10150 2450 50  0001 C CNN "LCSC Part #"
+F 4 "C4184" H 10150 2450 50  0001 C CNN "LCSC Part #"
 	1    10150 2450
 	0    -1   -1   0
@@
 P 10150 2850
 F 0 "R43" V 10357 2850 50  0000 C CNN
-F 1 "10k" V 10266 2850 50  0000 C CNN
+F 1 "3.3k" V 10266 2850 50  0000 C CNN
 F 2 "Resistor_SMD:R_0603_1608Metric" V 10080 2850 50  0001 C CNN
 F 3 "~" H 10150 2850 50  0001 C CNN
-F 4 "C25804" H 10150 2850 50  0001 C CNN "LCSC Part #"
+F 4 "C22978" H 10150 2850 50  0001 C CNN "LCSC Part #"
 	1    10150 2850
 	0    -1   -1   0
@@
 P 10150 3300
 F 0 "R44" V 10357 3300 50  0000 C CNN
-F 1 "2.2k" V 10266 3300 50  0000 C CNN
+F 1 "1k" V 10266 3300 50  0000 C CNN
 F 2 "Resistor_SMD:R_0603_1608Metric" V 10080 3300 50  0001 C CNN
 F 3 "~" H 10150 3300 50  0001 C CNN
-F 4 "C4190" H 10150 3300 50  0001 C CNN "LCSC Part #"
+F 4 "C21190" H 10150 3300 50  0001 C CNN "LCSC Part #"
 	1    10150 3300
 	0    -1   -1   0
