File: CAN.sch (KiCad schematic (older format))
At the start: 10 parts

Commit message: Do MCU bypassing according to datasheet; annotate
Parts:
- gave numbers to parts that had none: 10
Changed lines of the file:
@@
 $EndDescr
 $Comp
-L Interface_CAN_LIN:MCP2542FDxMF U?
+L Interface_CAN_LIN:MCP2542FDxMF U7
 U 1 1 5F738629
 P 4750 3600
-F 0 "U?" H 5100 3200 50  0000 C CNN
+F 0 "U7" H 5100 3200 50  0000 C CNN
 F 1 "MCP2542FDxMF" H 5100 3100 50  0000 C CNN
 F 2 "Package_DFN_QFN:DFN-8-1EP_3x3mm_P0.65mm_EP1.55x2.4mm" H 4750 3100 50  0001 C CIN
@@
 	5850 2850 5850 3500
 $Comp
-L power:GND #PWR?
+L power:GND #PWR0227
 U 1 1 5F747B70
 P 4750 4150
-F 0 "#PWR?" H 4750 3900 50  0001 C CNN
+F 0 "#PWR0227" H 4750 3900 50  0001 C CNN
 F 1 "GND" H 4755 3977 50  0000 C CNN
 F 2 "" H 4750 4150 50  0001 C CNN
@@
 	4750 4000 4750 4100
 $Comp
-L power:+3.3V #PWR?
+L power:+3.3V #PWR0228
 U 1 1 5F74847C
 P 4550 2700
-F 0 "#PWR?" H 4550 2550 50  0001 C CNN
+F 0 "#PWR0228" H 4550 2550 50  0001 C CNN
 F 1 "+3.3V" H 4565 2873 50  0000 C CNN
 F 2 "" H 4550 2700 50  0001 C CNN
@@
 	4650 3000 4650 3150
 $Comp
-L power:+5V #PWR?
+L power:+5V #PWR0229
 U 1 1 5F74B31E
 P 4900 2450
-F 0 "#PWR?" H 4900 2300 50  0001 C CNN
+F 0 "#PWR0229" H 4900 2300 50  0001 C CNN
 F 1 "+5V" H 4915 2623 50  0000 C CNN
 F 2 "" H 4900 2450 50  0001 C CNN
@@
 	4750 3000 4750 3150
 $Comp
-L Device:C C?
+L Device:C C43
 U 1 1 5F74BE20
 P 4200 2950
-F 0 "C?" H 4315 2996 50  0000 L CNN
+F 0 "C43" H 4315 2996 50  0000 L CNN
 F 1 "0.1u" H 4315 2905 50  0000 L CNN
 F 2 "" H 4238 2800 50  0001 C CNN
@@
 	4200 3150 4650 3150
 $Comp
-L Device:C C?
+L Device:C C44
 U 1 1 5F751476
 P 5150 2950
-F 0 "C?" H 5265 2996 50  0000 L CNN
+F 0 "C44" H 5265 2996 50  0000 L CNN
 F 1 "0.1u" H 5265 2905 50  0000 L CNN
 F 2 "" H 5188 2800 50  0001 C CNN
@@
 	4750 4100 4750 4150
 $Comp
-L Device:R R?
+L Device:R R46
 U 1 1 5F739A95
 P 6250 3400
-F 0 "R?" H 6320 3446 50  0000 L CNN
+F 0 "R46" H 6320 3446 50  0000 L CNN
 F 1 "10k" H 6320 3355 50  0000 L CNN
 F 2 "" V 6180 3400 50  0001 C CNN
@@
 $EndComp
 $Comp
-L Device:R R?
+L Device:R R47
 U 1 1 5F739F21
 P 6250 3800
-F 0 "R?" H 6320 3846 50  0000 L CNN
+F 0 "R47" H 6320 3846 50  0000 L CNN
 F 1 "10k" H 6320 3755 50  0000 L CNN
 F 2 "" V 6180 3800 50  0001 C CNN
@@
 $EndComp
 $Comp
-L Device:R R?
+L Device:R R48
 U 1 1 5F73A83D
 P 6650 3400
-F 0 "R?" H 6720 3446 50  0000 L CNN
+F 0 "R48" H 6720 3446 50  0000 L CNN
 F 1 "60.4" H 6720 3355 50  0000 L CNN
 F 2 "" V 6580 3400 50  0001 C CNN
@@
 $EndComp
 $Comp
-L Device:R R?
+L Device:R R49
 U 1 1 5F73A9BF
 P 6650 3800
-F 0 "R?" H 6720 3846 50  0000 L CNN
+F 0 "R49" H 6720 3846 50  0000 L CNN
 F 1 "60.4" H 6720 3755 50  0000 L CNN
 F 2 "" V 6580 3800 50  0001 C CNN
@@
 Connection ~ 6250 3600
 $Comp
-L Device:C C?
+L Device:C C45
 U 1 1 5F73B862
 P 7100 3800
-F 0 "C?" H 7215 3846 50  0000 L CNN
+F 0 "C45" H 7215 3846 50  0000 L CNN
 F 1 "0.1u" H 7215 3755 50  0000 L CNN
 F 2 "" H 7138 3650 50  0001 C CNN
@@
 	7600 2850 7600 3500
 $Comp
-L Jumper:SolderJumper_2_Open JP?
+L Jumper:SolderJumper_2_Open JP1
 U 1 1 5F73DCC4
 P 6650 3050
-F 0 "JP?" V 6604 3118 50  0000 L CNN
+F 0 "JP1" V 6604 3118 50  0000 L CNN
 F 1 "SolderJumper_2_Open" V 6695 3118 50  0000 L CNN
 F 2 "" H 6650 3050 50  0001 C CNN
@@
 	6250 3950 6250 4000
 $Comp
-L power:+5V #PWR?
+L power:+5V #PWR0230
 U 1 1 5F73F773
 P 6250 3200
-F 0 "#PWR?" H 6250 3050 50  0001 C CNN
+F 0 "#PWR0230" H 6250 3050 50  0001 C CNN
 F 1 "+5V" H 6265 3373 50  0000 C CNN
 F 2 "" H 6250 3200 50  0001 C CNN
@@
 $EndComp
 $Comp
-L power:GND #PWR?
+L power:GND #PWR0231
 U 1 1 5F73FB3D
 P 6250 4000
-F 0 "#PWR?" H 6250 3750 50  0001 C CNN
+F 0 "#PWR0231" H 6250 3750 50  0001 C CNN
 F 1 "GND" H 6255 3827 50  0000 C CNN
 F 2 "" H 6250 4000 50  0001 C CNN
@@
 	5850 4450 6650 4450
 $Comp
-L Jumper:SolderJumper_2_Open JP?
+L Jumper:SolderJumper_2_Open JP2
 U 1 1 5F740229
 P 6650 4250
-F 0 "JP?" V 6604 4318 50  0000 L CNN
+F 0 "JP2" V 6604 4318 50  0000 L CNN
 F 1 "SolderJumper_2_Open" V 6695 4318 50  0000 L CNN
 F 2 "" H 6650 4250 50  0001 C CNN
@@
 	6650 4450 7600 4450
 $Comp
-L power:GND #PWR?
+L power:GND #PWR0232
 U 1 1 5F741C20
 P 7100 4000
-F 0 "#PWR?" H 7100 3750 50  0001 C CNN
+F 0 "#PWR0232" H 7100 3750 50  0001 C CNN
 F 1 "GND" H 7105 3827 50  0000 C CNN
 F 2 "" H 7100 4000 50  0001 C CNN

Commit message: added footprints, continue layout
Parts:
- C43, C44, C45: footprint (none) -> Capacitor_SMD:C_0603_1608Metric
- JP1, JP2: footprint (none) -> Jumper:SolderJumper-2_P1.3mm_Open_RoundedPad1.0x1.5mm
- R46, R47, R48, R49: footprint (none) -> Resistor_SMD:R_0603_1608Metric
Changed lines of the file:
@@
 F 0 "C43" H 4315 2996 50  0000 L CNN
 F 1 "0.1u" H 4315 2905 50  0000 L CNN
-F 2 "" H 4238 2800 50  0001 C CNN
+F 2 "Capacitor_SMD:C_0603_1608Metric" H 4238 2800 50  0001 C CNN
 F 3 "~" H 4200 2950 50  0001 C CNN
 	1    4200 2950
@@
 F 0 "C44" H 5265 2996 50  0000 L CNN
 F 1 "0.1u" H 5265 2905 50  0000 L CNN
-F 2 "" H 5188 2800 50  0001 C CNN
+F 2 "Capacitor_SMD:C_0603_1608Metric" H 5188 2800 50  0001 C CNN
 F 3 "~" H 5150 2950 50  0001 C CNN
 	1    5150 2950
@@
 F 0 "R46" H 6320 3446 50  0000 L CNN
 F 1 "10k" H 6320 3355 50  0000 L CNN
-F 2 "" V 6180 3400 50  0001 C CNN
+F 2 "Resistor_SMD:R_0603_1608Metric" V 6180 3400 50  0001 C CNN
 F 3 "~" H 6250 3400 50  0001 C CNN
 	1    6250 3400
@@
 F 0 "R47" H 6320 3846 50  0000 L CNN
 F 1 "10k" H 6320 3755 50  0000 L CNN
-F 2 "" V 6180 3800 50  0001 C CNN
+F 2 "Resistor_SMD:R_0603_1608Metric" V 6180 3800 50  0001 C CNN
 F 3 "~" H 6250 3800 50  0001 C CNN
 	1    6250 3800
@@
 F 0 "R48" H 6720 3446 50  0000 L CNN
 F 1 "60.4" H 6720 3355 50  0000 L CNN
-F 2 "" V 6580 3400 50  0001 C CNN
+F 2 "Resistor_SMD:R_0603_1608Metric" V 6580 3400 50  0001 C CNN
 F 3 "~" H 6650 3400 50  0001 C CNN
 	1    6650 3400
@@
 F 0 "R49" H 6720 3846 50  0000 L CNN
 F 1 "60.4" H 6720 3755 50  0000 L CNN
-F 2 "" V 6580 3800 50  0001 C CNN
+F 2 "Resistor_SMD:R_0603_1608Metric" V 6580 3800 50  0001 C CNN
 F 3 "~" H 6650 3800 50  0001 C CNN
 	1    6650 3800
@@
 F 0 "C45" H 7215 3846 50  0000 L CNN
 F 1 "0.1u" H 7215 3755 50  0000 L CNN
-F 2 "" H 7138 3650 50  0001 C CNN
+F 2 "Capacitor_SMD:C_0603_1608Metric" H 7138 3650 50  0001 C CNN
 F 3 "~" H 7100 3800 50  0001 C CNN
 	1    7100 3800
@@
 F 0 "JP1" V 6604 3118 50  0000 L CNN
 F 1 "SolderJumper_2_Open" V 6695 3118 50  0000 L CNN
-F 2 "" H 6650 3050 50  0001 C CNN
+F 2 "Jumper:SolderJumper-2_P1.3mm_Open_RoundedPad1.0x1.5mm" H 6650 3050 50  0001 C CNN
 F 3 "~" H 6650 3050 50  0001 C CNN
 	1    6650 3050
@@
 F 0 "JP2" V 6604 4318 50  0000 L CNN
 F 1 "SolderJumper_2_Open" V 6695 4318 50  0000 L CNN
-F 2 "" H 6650 4250 50  0001 C CNN
+F 2 "Jumper:SolderJumper-2_P1.3mm_Open_RoundedPad1.0x1.5mm" H 6650 4250 50  0001 C CNN
 F 3 "~" H 6650 4250 50  0001 C CNN
 	1    6650 4250

Commit message: continue board layout, placed all components
Connections:
- net +3V3: no longer C43.2
- net +5V: no longer C44.2
- net GND: now also C43.2, C44.2
Changed lines of the file:
@@
 Wire Wire Line
 	4550 3000 4650 3000
-Wire Wire Line
-	4650 3000 4650 3150
 $Comp
 L power:+5V #PWR0229
@@
 Wire Wire Line
 	4900 3000 4750 3000
-Wire Wire Line
-	4750 3000 4750 3150
 $Comp
 L Device:C C43
@@
 Wire Wire Line
 	4200 3100 4200 3150
-Connection ~ 4650 3150
-Wire Wire Line
-	4650 3150 4650 3200
 Wire Wire Line
 	4200 2750 4550 2750
-Wire Wire Line
-	4200 3150 4650 3150
 $Comp
 L Device:C C44
@@
 Wire Wire Line
 	4900 2750 4900 3000
-Wire Wire Line
-	5150 3150 4750 3150
-Connection ~ 4750 3150
-Wire Wire Line
-	4750 3150 4750 3200
 Wire Wire Line
 	4250 3400 4100 3400
@@
 Wire Wire Line
 	7600 3700 7950 3700
+Wire Wire Line
+	4650 3000 4650 3200
+Wire Wire Line
+	4750 3000 4750 3200
+$Comp
+L power:GND #PWR0222
+U 1 1 5F7D2541
+P 4200 3150
+F 0 "#PWR0222" H 4200 2900 50  0001 C CNN
+F 1 "GND" H 4205 2977 50  0000 C CNN
+F 2 "" H 4200 3150 50  0001 C CNN
+F 3 "" H 4200 3150 50  0001 C CNN
+	1    4200 3150
+	1    0    0    -1
+$EndComp
+$Comp
+L power:GND #PWR0223
+U 1 1 5F7D2882
+P 5150 3150
+F 0 "#PWR0223" H 5150 2900 50  0001 C CNN
+F 1 "GND" H 5155 2977 50  0000 C CNN
+F 2 "" H 5150 3150 50  0001 C CNN
+F 3 "" H 5150 3150 50  0001 C CNN
+	1    5150 3150
+	1    0    0    -1
+$EndComp
 $EndSCHEMATC

Commit message: add resistors on mosfet driver inputs, change board corners, fix labels
Parts:
- C43, C44, C45: value 0.1u -> 100n
- R48, R49: value 60.4 -> 56R
Changed lines of the file:
@@
 P 4200 2950
 F 0 "C43" H 4315 2996 50  0000 L CNN
-F 1 "0.1u" H 4315 2905 50  0000 L CNN
+F 1 "100n" H 4315 2905 50  0000 L CNN
 F 2 "Capacitor_SMD:C_0603_1608Metric" H 4238 2800 50  0001 C CNN
 F 3 "~" H 4200 2950 50  0001 C CNN
@@
 P 5150 2950
 F 0 "C44" H 5265 2996 50  0000 L CNN
-F 1 "0.1u" H 5265 2905 50  0000 L CNN
+F 1 "100n" H 5265 2905 50  0000 L CNN
 F 2 "Capacitor_SMD:C_0603_1608Metric" H 5188 2800 50  0001 C CNN
 F 3 "~" H 5150 2950 50  0001 C CNN
@@
 P 6650 3400
 F 0 "R48" H 6720 3446 50  0000 L CNN
-F 1 "60.4" H 6720 3355 50  0000 L CNN
+F 1 "56R" H 6720 3355 50  0000 L CNN
 F 2 "Resistor_SMD:R_0603_1608Metric" V 6580 3400 50  0001 C CNN
 F 3 "~" H 6650 3400 50  0001 C CNN
@@
 P 6650 3800
 F 0 "R49" H 6720 3846 50  0000 L CNN
-F 1 "60.4" H 6720 3755 50  0000 L CNN
+F 1 "56R" H 6720 3755 50  0000 L CNN
 F 2 "Resistor_SMD:R_0603_1608Metric" V 6580 3800 50  0001 C CNN
 F 3 "~" H 6650 3800 50  0001 C CNN
@@
 P 7100 3800
 F 0 "C45" H 7215 3846 50  0000 L CNN
-F 1 "0.1u" H 7215 3755 50  0000 L CNN
+F 1 "100n" H 7215 3755 50  0000 L CNN
 F 2 "Capacitor_SMD:C_0603_1608Metric" H 7138 3650 50  0001 C CNN
 F 3 "~" H 7100 3800 50  0001 C CNN

Commit message: Changed fet driver
Parts:
- removed R46, R47: 10k, Resistor_SMD:R_0603_1608Metric, symbol Device:R
- added D12: NUP2105L, Package_TO_SOT_SMD:SOT-23, symbol Power_Protection:NUP2105L
- R48, R49: value 56R -> 60R
Connections:
- net CANH: now also D12.1 (K)
- net CANL: now also D12.2 (K)
- net GND: now also D12.3 (A)
Changed lines of the file:
@@
 L power:+5V #PWR0229
 U 1 1 5F74B31E
-P 4900 2450
-F 0 "#PWR0229" H 4900 2300 50  0001 C CNN
-F 1 "+5V" H 4915 2623 50  0000 C CNN
-F 2 "" H 4900 2450 50  0001 C CNN
-F 3 "" H 4900 2450 50  0001 C CNN
-	1    4900 2450
-	1    0    0    -1
-$EndComp
-Wire Wire Line
-	4900 2450 4900 2750
+P 4900 2700
+F 0 "#PWR0229" H 4900 2550 50  0001 C CNN
+F 1 "+5V" H 4915 2873 50  0000 C CNN
+F 2 "" H 4900 2700 50  0001 C CNN
+F 3 "" H 4900 2700 50  0001 C CNN
+	1    4900 2700
+	1    0    0    -1
+$EndComp
+Wire Wire Line
+	4900 2700 4900 2750
 Wire Wire Line
 	4900 3000 4750 3000
@@
 	4750 4100 4750 4150
 $Comp
-L Device:R R46
-U 1 1 5F739A95
-P 6250 3400
-F 0 "R46" H 6320 3446 50  0000 L CNN
-F 1 "10k" H 6320 3355 50  0000 L CNN
-F 2 "Resistor_SMD:R_0603_1608Metric" V 6180 3400 50  0001 C CNN
-F 3 "~" H 6250 3400 50  0001 C CNN
-	1    6250 3400
-	1    0    0    -1
-$EndComp
-$Comp
-L Device:R R47
-U 1 1 5F739F21
-P 6250 3800
-F 0 "R47" H 6320 3846 50  0000 L CNN
-F 1 "10k" H 6320 3755 50  0000 L CNN
-F 2 "Resistor_SMD:R_0603_1608Metric" V 6180 3800 50  0001 C CNN
-F 3 "~" H 6250 3800 50  0001 C CNN
-	1    6250 3800
-	1    0    0    -1
-$EndComp
-$Comp
 L Device:R R48
 U 1 1 5F73A83D
 P 6650 3400
 F 0 "R48" H 6720 3446 50  0000 L CNN
-F 1 "56R" H 6720 3355 50  0000 L CNN
+F 1 "60R" H 6720 3355 50  0000 L CNN
 F 2 "Resistor_SMD:R_0603_1608Metric" V 6580 3400 50  0001 C CNN
 F 3 "~" H 6650 3400 50  0001 C CNN
@@
 P 6650 3800
 F 0 "R49" H 6720 3846 50  0000 L CNN
-F 1 "56R" H 6720 3755 50  0000 L CNN
+F 1 "60R" H 6720 3755 50  0000 L CNN
 F 2 "Resistor_SMD:R_0603_1608Metric" V 6580 3800 50  0001 C CNN
 F 3 "~" H 6650 3800 50  0001 C CNN
@@
 Wire Wire Line
 	6650 3550 6650 3600
-Wire Wire Line
-	6650 3600 6250 3600
 Connection ~ 6650 3600
 Wire Wire Line
 	6650 3600 6650 3650
-Wire Wire Line
-	6250 3550 6250 3600
-Wire Wire Line
-	6250 3600 6250 3650
-Connection ~ 6250 3600
 $Comp
 L Device:C C45
@@
 	5850 2850 6650 2850
 Wire Wire Line
-	7600 2850 7600 3500
+	8150 2850 8150 3500
 $Comp
 L Jumper:SolderJumper_2_Open JP1
@@
 Connection ~ 6650 2850
 Wire Wire Line
-	6650 2850 7600 2850
-Wire Wire Line
-	6250 3250 6250 3200
-Wire Wire Line
-	6250 3950 6250 4000
-$Comp
-L power:+5V #PWR0230
-U 1 1 5F73F773
-P 6250 3200
-F 0 "#PWR0230" H 6250 3050 50  0001 C CNN
-F 1 "+5V" H 6265 3373 50  0000 C CNN
-F 2 "" H 6250 3200 50  0001 C CNN
-F 3 "" H 6250 3200 50  0001 C CNN
-	1    6250 3200
-	1    0    0    -1
-$EndComp
-$Comp
-L power:GND #PWR0231
-U 1 1 5F73FB3D
-P 6250 4000
-F 0 "#PWR0231" H 6250 3750 50  0001 C CNN
-F 1 "GND" H 6255 3827 50  0000 C CNN
-F 2 "" H 6250 4000 50  0001 C CNN
-F 3 "" H 6250 4000 50  0001 C CNN
-	1    6250 4000
-	1    0    0    -1
-$EndComp
+	6650 2850 8150 2850
 Wire Wire Line
 	5850 4450 6650 4450
@@
 Connection ~ 6650 4450
 Wire Wire Line
-	6650 4450 7600 4450
+	6650 4450 8150 4450
 $Comp
 L power:GND #PWR0232
@@
 	6650 3950 6650 4100
 Wire Wire Line
-	7600 4450 7600 3700
-Text HLabel 7950 3700 2    50   BiDi ~ 0
+	8150 4450 8150 3700
+Text HLabel 8400 3700 2    50   BiDi ~ 0
 CANL
-Text HLabel 7950 3500 2    50   BiDi ~ 0
+Text HLabel 8400 3500 2    50   BiDi ~ 0
 CANH
 Wire Wire Line
-	7600 3500 7950 3500
-Wire Wire Line
-	7600 3700 7950 3700
+	8150 3500 8400 3500
+Wire Wire Line
+	8150 3700 8400 3700
 Wire Wire Line
 	4650 3000 4650 3200
@@
 	1    0    0    -1
 $EndComp
+$Comp
+L Power_Protection:NUP2105L D12
+U 1 1 601CE5F4
+P 7950 3600
+F 0 "D12" V 7608 3600 50  0000 C CNN
+F 1 "NUP2105L" V 7699 3600 50  0000 C CNN
+F 2 "Package_TO_SOT_SMD:SOT-23" H 8175 3550 50  0001 L CNN
+F 3 "http://www.onsemi.com/pub_link/Collateral/NUP2105L-D.PDF" H 8075 3725 50  0001 C CNN
+	1    7950 3600
+	0    1    1    0
+$EndComp
+Connection ~ 8150 3500
+Connection ~ 8150 3700
+$Comp
+L power:GND #PWR07
+U 1 1 601CF80D
+P 7700 4000
+F 0 "#PWR07" H 7700 3750 50  0001 C CNN
+F 1 "GND" H 7705 3827 50  0000 C CNN
+F 2 "" H 7700 4000 50  0001 C CNN
+F 3 "" H 7700 4000 50  0001 C CNN
+	1    7700 4000
+	1    0    0    -1
+$EndComp
+Wire Wire Line
+	7700 4000 7700 3600
+Wire Wire Line
+	7700 3600 7750 3600
 $EndSCHEMATC

Commit message: Added FET for LED
Parts:
- removed U7: MCP2542FDxMF, Package_DFN_QFN:DFN-8-1EP_3x3mm_P0.65mm_EP1.55x2.4mm, symbol Interface_CAN_LIN:MCP2542FDxMF
- added U7: TJA1051T-3, Package_SO:SOIC-8_3.9x4.9mm_P1.27mm, symbol Interface_CAN_LIN:TJA1051T-3
Connections:
- net +3V3: now also U7.5 (VIO)
- net +5V: now also U7.3 (VCC)
- net CANH: now also U7.7 (CANH)
- net CANL: now also U7.6 (CANL)
- net CAN_RX: now also U7.4 (RXD)
- net CAN_TX: now also U7.1 (TXD)
- net GND: now also U7.2 (GND), U7.8 (S)
Other:
- moved on the sheet: C43
Changed lines of the file:
@@
 Comment4 ""
 $EndDescr
-$Comp
-L Interface_CAN_LIN:MCP2542FDxMF U7
-U 1 1 5F738629
-P 4750 3600
-F 0 "U7" H 5100 3200 50  0000 C CNN
-F 1 "MCP2542FDxMF" H 5100 3100 50  0000 C CNN
-F 2 "Package_DFN_QFN:DFN-8-1EP_3x3mm_P0.65mm_EP1.55x2.4mm" H 4750 3100 50  0001 C CIN
-F 3 "http://ww1.microchip.com/downloads/en/DeviceDoc/MCP2542FD-4FD-MCP2542WFD-4WFD-Data-Sheet20005514B.pdf" H 4750 3600 50  0001 C CNN
-	1    4750 3600
-	1    0    0    -1
-$EndComp
 Wire Wire Line
 	5250 3500 5850 3500
@@
 L power:+3.3V #PWR0228
 U 1 1 5F74847C
-P 4550 2700
-F 0 "#PWR0228" H 4550 2550 50  0001 C CNN
-F 1 "+3.3V" H 4565 2873 50  0000 C CNN
-F 2 "" H 4550 2700 50  0001 C CNN
-F 3 "" H 4550 2700 50  0001 C CNN
-	1    4550 2700
-	1    0    0    -1
-$EndComp
-Wire Wire Line
-	4550 2700 4550 2750
-Wire Wire Line
-	4550 3000 4650 3000
+P 3800 3700
+F 0 "#PWR0228" H 3800 3550 50  0001 C CNN
+F 1 "+3.3V" H 3650 3750 50  0000 C CNN
+F 2 "" H 3800 3700 50  0001 C CNN
+F 3 "" H 3800 3700 50  0001 C CNN
+	1    3800 3700
+	1    0    0    -1
+$EndComp
 $Comp
 L power:+5V #PWR0229
@@
 L Device:C C43
 U 1 1 5F74BE20
-P 4200 2950
-F 0 "C43" H 4315 2996 50  0000 L CNN
-F 1 "100n" H 4315 2905 50  0000 L CNN
-F 2 "Capacitor_SMD:C_0603_1608Metric" H 4238 2800 50  0001 C CNN
-F 3 "~" H 4200 2950 50  0001 C CNN
-	1    4200 2950
-	1    0    0    -1
-$EndComp
-Wire Wire Line
-	4200 2800 4200 2750
-Connection ~ 4550 2750
-Wire Wire Line
-	4550 2750 4550 3000
-Wire Wire Line
-	4200 3100 4200 3150
-Wire Wire Line
-	4200 2750 4550 2750
+P 3800 3900
+F 0 "C43" H 3915 3946 50  0000 L CNN
+F 1 "100n" H 3915 3855 50  0000 L CNN
+F 2 "Capacitor_SMD:C_0603_1608Metric" H 3838 3750 50  0001 C CNN
+F 3 "~" H 3800 3900 50  0001 C CNN
+	1    3800 3900
+	1    0    0    -1
+$EndComp
+Wire Wire Line
+	3800 3750 3800 3700
+Wire Wire Line
+	3800 4050 3800 4100
+Wire Wire Line
+	3800 3700 4250 3700
 $Comp
 L Device:C C44
@@
 	8150 3700 8400 3700
 Wire Wire Line
-	4650 3000 4650 3200
-Wire Wire Line
 	4750 3000 4750 3200
 $Comp
 L power:GND #PWR0222
 U 1 1 5F7D2541
-P 4200 3150
-F 0 "#PWR0222" H 4200 2900 50  0001 C CNN
-F 1 "GND" H 4205 2977 50  0000 C CNN
-F 2 "" H 4200 3150 50  0001 C CNN
-F 3 "" H 4200 3150 50  0001 C CNN
-	1    4200 3150
+P 3800 4100
+F 0 "#PWR0222" H 3800 3850 50  0001 C CNN
+F 1 "GND" H 3805 3927 50  0000 C CNN
+F 2 "" H 3800 4100 50  0001 C CNN
+F 3 "" H 3800 4100 50  0001 C CNN
+	1    3800 4100
 	1    0    0    -1
 $EndComp
@@
 P 5150 3150
 F 0 "#PWR0223" H 5150 2900 50  0001 C CNN
-F 1 "GND" H 5155 2977 50  0000 C CNN
+F 1 "GND" H 5000 3100 50  0000 C CNN
 F 2 "" H 5150 3150 50  0001 C CNN
 F 3 "" H 5150 3150 50  0001 C CNN
@@
 Wire Wire Line
 	7700 3600 7750 3600
+$Comp
+L Interface_CAN_LIN:TJA1051T-3 U7
+U 1 1 603E3A3E
+P 4750 3600
+F 0 "U7" H 4500 4150 50  0000 C CNN
+F 1 "TJA1051T-3" H 4500 4050 50  0000 C CNN
+F 2 "Package_SO:SOIC-8_3.9x4.9mm_P1.27mm" H 4750 3100 50  0001 C CIN
+F 3 "http://www.nxp.com/documents/data_sheet/TJA1051.pdf" H 4750 3600 50  0001 C CNN
+	1    4750 3600
+	1    0    0    -1
+$EndComp
+Connection ~ 3800 3700
 $EndSCHEMATC

Commit message: Routed FET and jumper
Parts:
- removed D12: NUP2105L, Package_TO_SOT_SMD:SOT-23, symbol Power_Protection:NUP2105L
Changed lines of the file:
@@
 $EndComp
-$Comp
-L Power_Protection:NUP2105L D12
-U 1 1 601CE5F4
-P 7950 3600
-F 0 "D12" V 7608 3600 50  0000 C CNN
-F 1 "NUP2105L" V 7699 3600 50  0000 C CNN
-F 2 "Package_TO_SOT_SMD:SOT-23" H 8175 3550 50  0001 L CNN
-F 3 "http://www.onsemi.com/pub_link/Collateral/NUP2105L-D.PDF" H 8075 3725 50  0001 C CNN
-	1    7950 3600
-	0    1    1    0
-$EndComp
-Connection ~ 8150 3500
-Connection ~ 8150 3700
-$Comp
-L power:GND #PWR07
-U 1 1 601CF80D
-P 7700 4000
-F 0 "#PWR07" H 7700 3750 50  0001 C CNN
-F 1 "GND" H 7705 3827 50  0000 C CNN
-F 2 "" H 7700 4000 50  0001 C CNN
-F 3 "" H 7700 4000 50  0001 C CNN
-	1    7700 4000
-	1    0    0    -1
-$EndComp
-Wire Wire Line
-	7700 4000 7700 3600
-Wire Wire Line
-	7700 3600 7750 3600
 $Comp
 L Interface_CAN_LIN:TJA1051T-3 U7

Commit message: Added LCSC Part # to most components
Parts:
- C43, C44, C45: value 100n -> 100nF; LCSC Part # (none) -> C14663
- R48, R49: value 60R -> 56; LCSC Part # (none) -> C25196
- U7: LCSC Part # (none) -> C38695
Changed lines of the file:
@@
 P 3800 3900
 F 0 "C43" H 3915 3946 50  0000 L CNN
-F 1 "100n" H 3915 3855 50  0000 L CNN
+F 1 "100nF" H 3915 3855 50  0000 L CNN
 F 2 "Capacitor_SMD:C_0603_1608Metric" H 3838 3750 50  0001 C CNN
 F 3 "~" H 3800 3900 50  0001 C CNN
+F 4 "C14663" H 3800 3900 50  0001 C CNN "LCSC Part #"
 	1    3800 3900
 	1    0    0    -1
@@
 P 5150 2950
 F 0 "C44" H 5265 2996 50  0000 L CNN
-F 1 "100n" H 5265 2905 50  0000 L CNN
+F 1 "100nF" H 5265 2905 50  0000 L CNN
 F 2 "Capacitor_SMD:C_0603_1608Metric" H 5188 2800 50  0001 C CNN
 F 3 "~" H 5150 2950 50  0001 C CNN
+F 4 "C14663" H 5150 2950 50  0001 C CNN "LCSC Part #"
 	1    5150 2950
 	1    0    0    -1
@@
 P 6650 3400
 F 0 "R48" H 6720 3446 50  0000 L CNN
-F 1 "60R" H 6720 3355 50  0000 L CNN
+F 1 "56" H 6720 3355 50  0000 L CNN
 F 2 "Resistor_SMD:R_0603_1608Metric" V 6580 3400 50  0001 C CNN
 F 3 "~" H 6650 3400 50  0001 C CNN
+F 4 "C25196" H 6650 3400 50  0001 C CNN "LCSC Part #"
 	1    6650 3400
 	1    0    0    -1
@@
 P 6650 3800
 F 0 "R49" H 6720 3846 50  0000 L CNN
-F 1 "60R" H 6720 3755 50  0000 L CNN
+F 1 "56" H 6720 3755 50  0000 L CNN
 F 2 "Resistor_SMD:R_0603_1608Metric" V 6580 3800 50  0001 C CNN
 F 3 "~" H 6650 3800 50  0001 C CNN
+F 4 "C25196" H 6650 3800 50  0001 C CNN "LCSC Part #"
 	1    6650 3800
 	1    0    0    -1
@@
 P 7100 3800
 F 0 "C45" H 7215 3846 50  0000 L CNN
-F 1 "100n" H 7215 3755 50  0000 L CNN
+F 1 "100nF" H 7215 3755 50  0000 L CNN
 F 2 "Capacitor_SMD:C_0603_1608Metric" H 7138 3650 50  0001 C CNN
 F 3 "~" H 7100 3800 50  0001 C CNN
+F 4 "C14663" H 7100 3800 50  0001 C CNN "LCSC Part #"
 	1    7100 3800
 	1    0    0    -1
@@
 F 2 "Package_SO:SOIC-8_3.9x4.9mm_P1.27mm" H 4750 3100 50  0001 C CIN
 F 3 "http://www.nxp.com/documents/data_sheet/TJA1051.pdf" H 4750 3600 50  0001 C CNN
+F 4 "C38695" H 4750 3600 50  0001 C CNN "LCSC Part #"
 	1    4750 3600
 	1    0    0    -1
