File: CAN.sch (KiCad schematic (older format))
At the start: 8 parts, among them U7 TJA1051T-3

Commit message: More adaptation to jlcpcb, parts checking
Parts:
- JP1, JP2: place (none) -> dnp
Changed lines of the file:
@@
 F 1 "SolderJumper_2_Open" V 6695 3118 50  0000 L CNN
 F 2 "Jumper:SolderJumper-2_P1.3mm_Open_RoundedPad1.0x1.5mm" H 6650 3050 50  0001 C CNN
-F 3 "~" H 6650 3050 50  0001 C CNN
+F 3 "" H 6650 3050 50  0001 C CNN
+F 4 "dnp" H 6650 3050 50  0001 C CNN "place"
 	1    6650 3050
 	0    1    1    0
@@
 F 1 "SolderJumper_2_Open" V 6695 4318 50  0000 L CNN
 F 2 "Jumper:SolderJumper-2_P1.3mm_Open_RoundedPad1.0x1.5mm" H 6650 4250 50  0001 C CNN
-F 3 "~" H 6650 4250 50  0001 C CNN
+F 3 "" H 6650 4250 50  0001 C CNN
+F 4 "dnp" H 6650 4250 50  0001 C CNN "place"
 	1    6650 4250
 	0    1    1    0
