File: CURRENT_SENSE.sch (KiCad schematic (older format))
At the start: 21 parts, among them Q2L1 MMBT5551, Q2R1 MMBT5551, U14 3PEAK TP09-SR

Commit message: fix some errors
Changed lines of the file:
@@
 	1    0    0    -1
 $EndComp
+Connection ~ 6950 5150
 $EndSCHEMATC

Commit message: Add TVS diode, fuse to 15 V supply
Changed lines of the file:
@@
 	1    0    0    -1
 $EndComp
-Connection ~ 6950 5150
 $EndSCHEMATC

Commit message: add silk screen, change diodes at DCDC converters, remove overcurrent detection, add 100nf
Parts:
- removed C16L1, C16R1: 100n, Capacitor_SMD:C_0603_1608Metric, symbol Device:C
- removed Q2L1, Q2R1: MMBT5551, Package_TO_SOT_SMD:SOT-23, symbol Device:Q_NPN_BCE
- removed R50L1, R50R1: 20k, Resistor_SMD:R_0603_1608Metric, symbol Device:R
- removed R51L1, R51R1: 510, Resistor_SMD:R_0603_1608Metric, symbol Device:R
- removed R52L1, R52R1: 1k, Resistor_SMD:R_0603_1608Metric, symbol Device:R
Changed lines of the file:
@@
 Comment4 ""
 $EndDescr
-$Comp
-L power:+3.3V #PWR?
-U 1 1 5F71910B
-P 2800 2900
-AR Path="/5F71910B" Ref="#PWR?"  Part="1"
-AR Path="/5F7128FA/5F71910B" Ref="#PWR0104"  Part="1"
-F 0 "#PWR0104" H 2800 2750 50  0001 C CNN
-F 1 "+3.3V" H 2815 3073 50  0000 C CNN
-F 2 "" H 2800 2900 50  0001 C CNN
-F 3 "" H 2800 2900 50  0001 C CNN
-	1    2800 2900
-	1    0    0    -1
-$EndComp
-$Comp
-L Device:R R50R?
-U 1 1 5F719111
-P 2800 3050
-AR Path="/5F719111" Ref="R50R?"  Part="1"
-AR Path="/5F7128FA/5F719111" Ref="R50R1"  Part="1"
-F 0 "R50R1" H 2870 3096 50  0000 L CNN
-F 1 "20k" H 2870 3005 50  0000 L CNN
-F 2 "Resistor_SMD:R_0603_1608Metric" V 2730 3050 50  0001 C CNN
-F 3 "~" H 2800 3050 50  0001 C CNN
-	1    2800 3050
-	1    0    0    -1
-$EndComp
-$Comp
-L Device:R R51R?
-U 1 1 5F719117
-P 3250 3200
-AR Path="/5F719117" Ref="R51R?"  Part="1"
-AR Path="/5F7128FA/5F719117" Ref="R51R1"  Part="1"
-F 0 "R51R1" V 3043 3200 50  0000 C CNN
-F 1 "510" V 3134 3200 50  0000 C CNN
-F 2 "Resistor_SMD:R_0603_1608Metric" V 3180 3200 50  0001 C CNN
-F 3 "~" H 3250 3200 50  0001 C CNN
-	1    3250 3200
-	0    1    1    0
-$EndComp
-Wire Wire Line
-	3100 3200 2800 3200
-$Comp
-L Device:C C16R?
-U 1 1 5F71911E
-P 3400 3350
-AR Path="/5F71911E" Ref="C16R?"  Part="1"
-AR Path="/5F7128FA/5F71911E" Ref="C16R1"  Part="1"
-F 0 "C16R1" H 3515 3396 50  0000 L CNN
-F 1 "100n" H 3515 3305 50  0000 L CNN
-F 2 "Capacitor_SMD:C_0603_1608Metric" H 3438 3200 50  0001 C CNN
-F 3 "~" H 3400 3350 50  0001 C CNN
-	1    3400 3350
-	1    0    0    -1
-$EndComp
-$Comp
-L power:GND #PWR?
-U 1 1 5F719124
-P 2800 3750
-AR Path="/5F719124" Ref="#PWR?"  Part="1"
-AR Path="/5F7128FA/5F719124" Ref="#PWR0105"  Part="1"
-F 0 "#PWR0105" H 2800 3500 50  0001 C CNN
-F 1 "GND" H 2805 3577 50  0000 C CNN
-F 2 "" H 2800 3750 50  0001 C CNN
-F 3 "" H 2800 3750 50  0001 C CNN
-	1    2800 3750
-	1    0    0    -1
-$EndComp
-Text HLabel 3650 3200 2    50   Input ~ 0
-R_MTR_OVERCUR
-Wire Wire Line
-	3650 3200 3400 3200
-Connection ~ 3400 3200
-Wire Wire Line
-	2800 3200 2800 3350
-Connection ~ 2800 3200
-$Comp
-L power:GND #PWR?
-U 1 1 5F71912F
-P 3400 3550
-AR Path="/5F71912F" Ref="#PWR?"  Part="1"
-AR Path="/5F7128FA/5F71912F" Ref="#PWR0106"  Part="1"
-F 0 "#PWR0106" H 3400 3300 50  0001 C CNN
-F 1 "GND" H 3405 3377 50  0000 C CNN
-F 2 "" H 3400 3550 50  0001 C CNN
-F 3 "" H 3400 3550 50  0001 C CNN
-	1    3400 3550
-	1    0    0    -1
-$EndComp
-Wire Wire Line
-	3400 3550 3400 3500
-$Comp
-L Device:Q_NPN_BCE Q2R?
-U 1 1 5F719136
-P 2700 3550
-AR Path="/5F719136" Ref="Q2R?"  Part="1"
-AR Path="/5F7128FA/5F719136" Ref="Q2R1"  Part="1"
-F 0 "Q2R1" H 2891 3596 50  0000 L CNN
-F 1 "MMBT5551" H 2891 3505 50  0000 L CNN
-F 2 "Package_TO_SOT_SMD:SOT-23" H 2900 3650 50  0001 C CNN
-F 3 "~" H 2700 3550 50  0001 C CNN
-	1    2700 3550
-	1    0    0    -1
-$EndComp
-$Comp
-L Device:R R52R?
-U 1 1 5F71913C
-P 2350 3550
-AR Path="/5F71913C" Ref="R52R?"  Part="1"
-AR Path="/5F7128FA/5F71913C" Ref="R52R1"  Part="1"
-F 0 "R52R1" V 2143 3550 50  0000 C CNN
-F 1 "1k" V 2234 3550 50  0000 C CNN
-F 2 "Resistor_SMD:R_0603_1608Metric" V 2280 3550 50  0001 C CNN
-F 3 "~" H 2350 3550 50  0001 C CNN
-	1    2350 3550
-	0    1    1    0
-$EndComp
 Text HLabel 2100 3550 0    50   Input ~ 0
 R_MTR_SHUNT
@@
 Wire Wire Line
 	2100 3550 2200 3550
-Connection ~ 2200 3550
 $Comp
 L Device:R R37R1
@@
 Wire Wire Line
 	3850 4600 3750 4600
-$Comp
-L power:+3.3V #PWR?
-U 1 1 5F732D9C
-P 6750 2800
-AR Path="/5F732D9C" Ref="#PWR?"  Part="1"
-AR Path="/5F7128FA/5F732D9C" Ref="#PWR0112"  Part="1"
-F 0 "#PWR0112" H 6750 2650 50  0001 C CNN
-F 1 "+3.3V" H 6765 2973 50  0000 C CNN
-F 2 "" H 6750 2800 50  0001 C CNN
-F 3 "" H 6750 2800 50  0001 C CNN
-	1    6750 2800
-	1    0    0    -1
-$EndComp
-$Comp
-L Device:R R50R?
-U 1 1 5F732DA2
-P 6750 2950
-AR Path="/5F732DA2" Ref="R50R?"  Part="1"
-AR Path="/5F7128FA/5F732DA2" Ref="R50L1"  Part="1"
-F 0 "R50L1" H 6820 2996 50  0000 L CNN
-F 1 "20k" H 6820 2905 50  0000 L CNN
-F 2 "Resistor_SMD:R_0603_1608Metric" V 6680 2950 50  0001 C CNN
-F 3 "~" H 6750 2950 50  0001 C CNN
-	1    6750 2950
-	1    0    0    -1
-$EndComp
-$Comp
-L Device:R R51R?
-U 1 1 5F732DA8
-P 7200 3100
-AR Path="/5F732DA8" Ref="R51R?"  Part="1"
-AR Path="/5F7128FA/5F732DA8" Ref="R51L1"  Part="1"
-F 0 "R51L1" V 6993 3100 50  0000 C CNN
-F 1 "510" V 7084 3100 50  0000 C CNN
-F 2 "Resistor_SMD:R_0603_1608Metric" V 7130 3100 50  0001 C CNN
-F 3 "~" H 7200 3100 50  0001 C CNN
-	1    7200 3100
-	0    1    1    0
-$EndComp
-Wire Wire Line
-	7050 3100 6750 3100
-$Comp
-L Device:C C16R?
-U 1 1 5F732DAF
-P 7350 3250
-AR Path="/5F732DAF" Ref="C16R?"  Part="1"
-AR Path="/5F7128FA/5F732DAF" Ref="C16L1"  Part="1"
-F 0 "C16L1" H 7465 3296 50  0000 L CNN
-F 1 "100n" H 7465 3205 50  0000 L CNN
-F 2 "Capacitor_SMD:C_0603_1608Metric" H 7388 3100 50  0001 C CNN
-F 3 "~" H 7350 3250 50  0001 C CNN
-	1    7350 3250
-	1    0    0    -1
-$EndComp
-$Comp
-L power:GND #PWR?
-U 1 1 5F732DB5
-P 6750 3650
-AR Path="/5F732DB5" Ref="#PWR?"  Part="1"
-AR Path="/5F7128FA/5F732DB5" Ref="#PWR0113"  Part="1"
-F 0 "#PWR0113" H 6750 3400 50  0001 C CNN
-F 1 "GND" H 6755 3477 50  0000 C CNN
-F 2 "" H 6750 3650 50  0001 C CNN
-F 3 "" H 6750 3650 50  0001 C CNN
-	1    6750 3650
-	1    0    0    -1
-$EndComp
-Text HLabel 7600 3100 2    50   Input ~ 0
-L_MTR_OVERCUR
-Wire Wire Line
-	7600 3100 7350 3100
-Connection ~ 7350 3100
-Wire Wire Line
-	6750 3100 6750 3250
-Connection ~ 6750 3100
-$Comp
-L power:GND #PWR?
-U 1 1 5F732DC0
-P 7350 3450
-AR Path="/5F732DC0" Ref="#PWR?"  Part="1"
-AR Path="/5F7128FA/5F732DC0" Ref="#PWR0114"  Part="1"
-F 0 "#PWR0114" H 7350 3200 50  0001 C CNN
-F 1 "GND" H 7355 3277 50  0000 C CNN
-F 2 "" H 7350 3450 50  0001 C CNN
-F 3 "" H 7350 3450 50  0001 C CNN
-	1    7350 3450
-	1    0    0    -1
-$EndComp
-Wire Wire Line
-	7350 3450 7350 3400
-$Comp
-L Device:Q_NPN_BCE Q2R?
-U 1 1 5F732DC7
-P 6650 3450
-AR Path="/5F732DC7" Ref="Q2R?"  Part="1"
-AR Path="/5F7128FA/5F732DC7" Ref="Q2L1"  Part="1"
-F 0 "Q2L1" H 6841 3496 50  0000 L CNN
-F 1 "MMBT5551" H 6841 3405 50  0000 L CNN
-F 2 "Package_TO_SOT_SMD:SOT-23" H 6850 3550 50  0001 C CNN
-F 3 "~" H 6650 3450 50  0001 C CNN
-	1    6650 3450
-	1    0    0    -1
-$EndComp
-$Comp
-L Device:R R52R?
-U 1 1 5F732DCD
-P 6300 3450
-AR Path="/5F732DCD" Ref="R52R?"  Part="1"
-AR Path="/5F7128FA/5F732DCD" Ref="R52L1"  Part="1"
-F 0 "R52L1" V 6093 3450 50  0000 C CNN
-F 1 "1k" V 6184 3450 50  0000 C CNN
-F 2 "Resistor_SMD:R_0603_1608Metric" V 6230 3450 50  0001 C CNN
-F 3 "~" H 6300 3450 50  0001 C CNN
-	1    6300 3450
-	0    1    1    0
-$EndComp
 Text HLabel 6050 3450 0    50   Input ~ 0
 L_MTR_SHUNT
@@
 Wire Wire Line
 	6050 3450 6150 3450
-Connection ~ 6150 3450
 $Comp
 L Device:R R37L1

Commit message: Added LCSC Part # to most components
Parts:
- C82: renamed from C18R1; value 100n -> 100nF; LCSC Part # (none) -> C14663
- C83: renamed from C18L1; value 100n -> 100nF; LCSC Part # (none) -> C14663
- R37L1, R37R1: LCSC Part # (none) -> C22961
- R38L1, R38R1, R39L1, R39R1: LCSC Part # (none) -> C25804
- R40L1, R40R1: LCSC Part # (none) -> C21190
- U14: LCSC Part # (none) -> C81662
Changed lines of the file:
@@
 F 2 "Resistor_SMD:R_0603_1608Metric" V 2530 4250 50  0001 C CNN
 F 3 "~" H 2600 4250 50  0001 C CNN
+F 4 "C22961" H 2600 4250 50  0001 C CNN "LCSC Part #"
 	1    2600 4250
 	1    0    0    -1
@@
 $EndComp
 $Comp
-L Device:C C18R1
+L Device:C C82
 U 1 1 5F72440B
 P 2600 4650
-F 0 "C18R1" H 2715 4696 50  0000 L CNN
-F 1 "100n" H 2715 4605 50  0000 L CNN
+F 0 "C82" H 2715 4696 50  0000 L CNN
+F 1 "100nF" H 2715 4605 50  0000 L CNN
 F 2 "Capacitor_SMD:C_0603_1608Metric" H 2638 4500 50  0001 C CNN
 F 3 "~" H 2600 4650 50  0001 C CNN
+F 4 "C14663" H 2600 4650 50  0001 C CNN "LCSC Part #"
 	1    2600 4650
 	1    0    0    -1
@@
 F 2 "Package_SO:SOIC-8_3.9x4.9mm_P1.27mm" H 3450 4600 50  0001 C CNN
 F 3 "~" H 3450 4600 50  0001 C CNN
+F 4 "C81662" H 3450 4600 50  0001 C CNN "LCSC Part #"
 	2    3450 4600
 	1    0    0    -1
@@
 F 2 "Resistor_SMD:R_0603_1608Metric" V 2930 5100 50  0001 C CNN
 F 3 "~" H 3000 5100 50  0001 C CNN
+F 4 "C21190" H 3000 5100 50  0001 C CNN "LCSC Part #"
 	1    3000 5100
 	1    0    0    -1
@@
 F 2 "Resistor_SMD:R_0603_1608Metric" V 3330 5400 50  0001 C CNN
 F 3 "~" H 3400 5400 50  0001 C CNN
+F 4 "C25804" H 3400 5400 50  0001 C CNN "LCSC Part #"
 	1    3400 5400
 	0    1    1    0
@@
 F 2 "Resistor_SMD:R_0603_1608Metric" V 6230 4400 50  0001 C CNN
 F 3 "~" H 6300 4400 50  0001 C CNN
+F 4 "C25804" H 6300 4400 50  0001 C CNN "LCSC Part #"
 	1    6300 4400
 	0    1    1    0
@@
 F 2 "Resistor_SMD:R_0603_1608Metric" V 6480 4150 50  0001 C CNN
 F 3 "~" H 6550 4150 50  0001 C CNN
+F 4 "C22961" H 6550 4150 50  0001 C CNN "LCSC Part #"
 	1    6550 4150
 	1    0    0    -1
@@
 $EndComp
 $Comp
-L Device:C C18L1
+L Device:C C83
 U 1 1 5F732DEB
 P 6550 4550
-F 0 "C18L1" H 6665 4596 50  0000 L CNN
-F 1 "100n" H 6665 4505 50  0000 L CNN
+F 0 "C83" H 6665 4596 50  0000 L CNN
+F 1 "100nF" H 6665 4505 50  0000 L CNN
 F 2 "Capacitor_SMD:C_0603_1608Metric" H 6588 4400 50  0001 C CNN
 F 3 "~" H 6550 4550 50  0001 C CNN
+F 4 "C14663" H 6550 4550 50  0001 C CNN "LCSC Part #"
 	1    6550 4550
 	1    0    0    -1
@@
 F 2 "Resistor_SMD:R_0603_1608Metric" V 6880 5000 50  0001 C CNN
 F 3 "~" H 6950 5000 50  0001 C CNN
+F 4 "C21190" H 6950 5000 50  0001 C CNN "LCSC Part #"
 	1    6950 5000
 	1    0    0    -1
@@
 F 2 "Resistor_SMD:R_0603_1608Metric" V 7280 5300 50  0001 C CNN
 F 3 "~" H 7350 5300 50  0001 C CNN
+F 4 "C25804" H 7350 5300 50  0001 C CNN "LCSC Part #"
 	1    7350 5300
 	0    1    1    0
@@
 F 2 "Resistor_SMD:R_0603_1608Metric" V 2280 4500 50  0001 C CNN
 F 3 "~" H 2350 4500 50  0001 C CNN
+F 4 "C25804" H 2350 4500 50  0001 C CNN "LCSC Part #"
 	1    2350 4500
 	0    1    1    0
@@
 F 2 "Package_SO:SOIC-8_3.9x4.9mm_P1.27mm" H 7400 4500 50  0001 C CNN
 F 3 "~" H 7400 4500 50  0001 C CNN
+F 4 "C81662" H 7400 4500 50  0001 C CNN "LCSC Part #"
 	1    7400 4500
 	1    0    0    -1
@@
 F 2 "Package_SO:SOIC-8_3.9x4.9mm_P1.27mm" H 5250 5050 50  0001 C CNN
 F 3 "~" H 5250 5050 50  0001 C CNN
+F 4 "C81662" H 5250 5050 50  0001 C CNN "LCSC Part #"
 	3    5250 5050
 	1    0    0    -1
