File: phase_sense.sch (KiCad schematic (older format))
At the start: 14 parts, among them U4 3PEAK TP09-SR

Commit message: Added LCSC Part # to most components
Parts:
- C10: value 100n -> 100nF; LCSC Part # (none) -> C14663
- D4, D5: value 1n4148w -> 1N4148W; LCSC Part # (none) -> C81598
- R1, R23, R24, R29: LCSC Part # (none) -> C4184
- R22, R27: LCSC Part # (none) -> C22961
- R25, R30: value 2k2 -> 2.2k; LCSC Part # (none) -> C4190
- R26, R31: LCSC Part # (none) -> C21190
- U4: LCSC Part # (none) -> C81662
Changed lines of the file:
@@
 AR Path="/5F7C96F7/5F7C98DC" Ref="#PWR0159"  Part="1"
 AR Path="/5F7E81D5/5F7C98DC" Ref="#PWR0165"  Part="1"
-F 0 "#PWR0165" H 8950 1600 50  0001 C CNN
+F 0 "#PWR0159" H 8950 1600 50  0001 C CNN
 F 1 "+3.3V" H 8965 1923 50  0000 C CNN
 F 2 "" H 8950 1750 50  0001 C CNN
@@
 AR Path="/5F7C96F7/5F7C9ADD" Ref="C10"  Part="1"
 AR Path="/5F7E81D5/5F7C9ADD" Ref="C7"  Part="1"
-F 0 "C7" H 9065 1946 50  0000 L CNN
-F 1 "100n" H 9065 1855 50  0000 L CNN
+F 0 "C10" H 9065 1946 50  0000 L CNN
+F 1 "100nF" H 9065 1855 50  0000 L CNN
 F 2 "Capacitor_SMD:C_0603_1608Metric" H 8988 1750 50  0001 C CNN
 F 3 "~" H 8950 1900 50  0001 C CNN
+F 4 "C14663" H 8950 1900 50  0001 C CNN "LCSC Part #"
 	1    8950 1900
 	1    0    0    -1
@@
 AR Path="/5F7C96F7/5F7C9C6F" Ref="#PWR0160"  Part="1"
 AR Path="/5F7E81D5/5F7C9C6F" Ref="#PWR0166"  Part="1"
-F 0 "#PWR0166" H 8950 1800 50  0001 C CNN
+F 0 "#PWR0160" H 8950 1800 50  0001 C CNN
 F 1 "GND" H 8955 1877 50  0000 C CNN
 F 2 "" H 8950 2050 50  0001 C CNN
@@
 AR Path="/5F7C96F7/5F7C9F32" Ref="R24"  Part="1"
 AR Path="/5F7E81D5/5F7C9F32" Ref="R2"  Part="1"
-F 0 "R2" V 4807 1650 50  0000 C CNN
+F 0 "R24" V 4807 1650 50  0000 C CNN
 F 1 "20k" V 4716 1650 50  0000 C CNN
 F 2 "Resistor_SMD:R_0603_1608Metric" V 4530 1650 50  0001 C CNN
 F 3 "~" H 4600 1650 50  0001 C CNN
+F 4 "C4184" H 4600 1650 50  0001 C CNN "LCSC Part #"
 	1    4600 1650
 	0    -1   -1   0
@@
 AR Path="/5F7C96F7/5F7CA82E" Ref="R23"  Part="1"
 AR Path="/5F7E81D5/5F7CA82E" Ref="R6"  Part="1"
-F 0 "R6" V 5107 1650 50  0000 C CNN
+F 0 "R23" V 5107 1650 50  0000 C CNN
 F 1 "20k" V 5016 1650 50  0000 C CNN
 F 2 "Resistor_SMD:R_0603_1608Metric" V 4830 1650 50  0001 C CNN
 F 3 "~" H 4900 1650 50  0001 C CNN
+F 4 "C4184" H 4900 1650 50  0001 C CNN "LCSC Part #"
 	1    4900 1650
 	0    -1   -1   0
@@
 AR Path="/5F7C96F7/5F7CA9C0" Ref="R26"  Part="1"
 AR Path="/5F7E81D5/5F7CA9C0" Ref="R3"  Part="1"
-F 0 "R3" V 4807 2000 50  0000 C CNN
+F 0 "R26" V 4807 2000 50  0000 C CNN
 F 1 "1k" V 4716 2000 50  0000 C CNN
 F 2 "Resistor_SMD:R_0603_1608Metric" V 4530 2000 50  0001 C CNN
 F 3 "~" H 4600 2000 50  0001 C CNN
+F 4 "C21190" H 4600 2000 50  0001 C CNN "LCSC Part #"
 	1    4600 2000
 	0    -1   -1   0
@@
 AR Path="/5F7C96F7/5F7CAE77" Ref="D4"  Part="1"
 AR Path="/5F7E81D5/5F7CAE77" Ref="D3"  Part="1"
-F 0 "D3" V 5096 1721 50  0000 R CNN
-F 1 "1n4148w" V 5005 1721 50  0000 R CNN
+F 0 "D4" V 5096 1721 50  0000 R CNN
+F 1 "1N4148W" V 5005 1721 50  0000 R CNN
 F 2 "Diode_SMD:D_SOD-123" H 5050 1800 50  0001 C CNN
 F 3 "~" H 5050 1800 50  0001 C CNN
+F 4 "C81598" H 5050 1800 50  0001 C CNN "LCSC Part #"
 	1    5050 1800
 	0    -1   -1   0
@@
 AR Path="/5F7C96F7/5F7CB464" Ref="#PWR0161"  Part="1"
 AR Path="/5F7E81D5/5F7CB464" Ref="#PWR0167"  Part="1"
-F 0 "#PWR0167" H 6050 1150 50  0001 C CNN
+F 0 "#PWR0161" H 6050 1150 50  0001 C CNN
 F 1 "+3.3V" H 6065 1473 50  0000 C CNN
 F 2 "" H 6050 1300 50  0001 C CNN
@@
 AR Path="/5F7C96F7/5F7CB568" Ref="R22"  Part="1"
 AR Path="/5F7E81D5/5F7CB568" Ref="R8"  Part="1"
-F 0 "R8" V 5957 1300 50  0000 C CNN
+F 0 "R22" V 5957 1300 50  0000 C CNN
 F 1 "220k" V 5866 1300 50  0000 C CNN
 F 2 "Resistor_SMD:R_0603_1608Metric" V 5680 1300 50  0001 C CNN
 F 3 "~" H 5750 1300 50  0001 C CNN
+F 4 "C22961" H 5750 1300 50  0001 C CNN "LCSC Part #"
 	1    5750 1300
 	0    -1   -1   0
@@
 AR Path="/5F7C96F7/5F7CBE46" Ref="U4"  Part="1"
 AR Path="/5F7E81D5/5F7CBE46" Ref="U6"  Part="1"
-F 0 "U6" H 6150 2025 50  0000 C CNN
+F 0 "U4" H 6150 2025 50  0000 C CNN
 F 1 "3PEAK TP09-SR" H 6150 2026 50  0001 C CNN
 F 2 "Package_SO:SOIC-8_3.9x4.9mm_P1.27mm" H 6150 1750 50  0001 C CNN
 F 3 "~" H 6150 1750 50  0001 C CNN
+F 4 "C81662" H 6150 1750 50  0001 C CNN "LCSC Part #"
 	1    6150 1750
 	1    0    0    -1
@@
 AR Path="/5F7C96F7/5F7CE17C" Ref="R25"  Part="1"
 AR Path="/5F7E81D5/5F7CE17C" Ref="R11"  Part="1"
-F 0 "R11" V 6093 2000 50  0000 C CNN
-F 1 "2k2" V 6184 2000 50  0000 C CNN
+F 0 "R25" V 6093 2000 50  0000 C CNN
+F 1 "2.2k" V 6184 2000 50  0000 C CNN
 F 2 "Resistor_SMD:R_0603_1608Metric" V 6230 2000 50  0001 C CNN
 F 3 "~" H 6300 2000 50  0001 C CNN
+F 4 "C4190" H 6300 2000 50  0001 C CNN "LCSC Part #"
 	1    6300 2000
 	0    1    1    0
@@
 AR Path="/5F7C96F7/5F7DF5DA" Ref="R29"  Part="1"
 AR Path="/5F7E81D5/5F7DF5DA" Ref="R4"  Part="1"
-F 0 "R4" V 4807 3350 50  0000 C CNN
+F 0 "R29" V 4807 3350 50  0000 C CNN
 F 1 "20k" V 4716 3350 50  0000 C CNN
 F 2 "Resistor_SMD:R_0603_1608Metric" V 4530 3350 50  0001 C CNN
 F 3 "~" H 4600 3350 50  0001 C CNN
+F 4 "C4184" H 4600 3350 50  0001 C CNN "LCSC Part #"
 	1    4600 3350
 	0    -1   -1   0
@@
 AR Path="/5F7C96F7/5F7DF5E0" Ref="R1"  Part="1"
 AR Path="/5F7E81D5/5F7DF5E0" Ref="R7"  Part="1"
-F 0 "R7" V 5107 3350 50  0000 C CNN
+F 0 "R1" V 5107 3350 50  0000 C CNN
 F 1 "20k" V 5016 3350 50  0000 C CNN
 F 2 "Resistor_SMD:R_0603_1608Metric" V 4830 3350 50  0001 C CNN
 F 3 "~" H 4900 3350 50  0001 C CNN
+F 4 "C4184" H 4900 3350 50  0001 C CNN "LCSC Part #"
 	1    4900 3350
 	0    -1   -1   0
@@
 AR Path="/5F7C96F7/5F7DF5E6" Ref="R31"  Part="1"
 AR Path="/5F7E81D5/5F7DF5E6" Ref="R5"  Part="1"
-F 0 "R5" V 4807 3700 50  0000 C CNN
+F 0 "R31" V 4807 3700 50  0000 C CNN
 F 1 "1k" V 4716 3700 50  0000 C CNN
 F 2 "Resistor_SMD:R_0603_1608Metric" V 4530 3700 50  0001 C CNN
 F 3 "~" H 4600 3700 50  0001 C CNN
+F 4 "C21190" H 4600 3700 50  0001 C CNN "LCSC Part #"
 	1    4600 3700
 	0    -1   -1   0
@@
 AR Path="/5F7C96F7/5F7DF5EC" Ref="D5"  Part="1"
 AR Path="/5F7E81D5/5F7DF5EC" Ref="D6"  Part="1"
-F 0 "D6" V 5096 3421 50  0000 R CNN
-F 1 "1n4148w" V 5005 3421 50  0000 R CNN
+F 0 "D5" V 5096 3421 50  0000 R CNN
+F 1 "1N4148W" V 5005 3421 50  0000 R CNN
 F 2 "Diode_SMD:D_SOD-123" H 5050 3500 50  0001 C CNN
 F 3 "~" H 5050 3500 50  0001 C CNN
+F 4 "C81598" H 5050 3500 50  0001 C CNN "LCSC Part #"
 	1    5050 3500
 	0    -1   -1   0
@@
 AR Path="/5F7C96F7/5F7DF5F4" Ref="#PWR0163"  Part="1"
 AR Path="/5F7E81D5/5F7DF5F4" Ref="#PWR0169"  Part="1"
-F 0 "#PWR0169" H 6050 2850 50  0001 C CNN
+F 0 "#PWR0163" H 6050 2850 50  0001 C CNN
 F 1 "+3.3V" H 6065 3173 50  0000 C CNN
 F 2 "" H 6050 3000 50  0001 C CNN
@@
 AR Path="/5F7C96F7/5F7DF5FA" Ref="R27"  Part="1"
 AR Path="/5F7E81D5/5F7DF5FA" Ref="R9"  Part="1"
-F 0 "R9" V 5957 3000 50  0000 C CNN
+F 0 "R27" V 5957 3000 50  0000 C CNN
 F 1 "220k" V 5866 3000 50  0000 C CNN
 F 2 "Resistor_SMD:R_0603_1608Metric" V 5680 3000 50  0001 C CNN
 F 3 "~" H 5750 3000 50  0001 C CNN
+F 4 "C22961" H 5750 3000 50  0001 C CNN "LCSC Part #"
 	1    5750 3000
 	0    -1   -1   0
@@
 AR Path="/5F7C96F7/5F7DF60A" Ref="U4"  Part="3"
 AR Path="/5F7E81D5/5F7DF60A" Ref="U6"  Part="3"
-F 0 "U6" H 7558 3496 50  0000 L CNN
+F 0 "U4" H 7558 3496 50  0000 L CNN
 F 1 "3PEAK TP09-SR" H 7558 3405 50  0000 L CNN
 F 2 "Package_SO:SOIC-8_3.9x4.9mm_P1.27mm" H 7600 3450 50  0001 C CNN
 F 3 "~" H 7600 3450 50  0001 C CNN
+F 4 "C81662" H 7600 3450 50  0001 C CNN "LCSC Part #"
 	3    7600 3450
 	1    0    0    -1
@@
 AR Path="/5F7C96F7/5F7DF613" Ref="#PWR0164"  Part="1"
 AR Path="/5F7E81D5/5F7DF613" Ref="#PWR0170"  Part="1"
-F 0 "#PWR0170" H 7500 3500 50  0001 C CNN
+F 0 "#PWR0164" H 7500 3500 50  0001 C CNN
 F 1 "GND" H 7505 3577 50  0000 C CNN
 F 2 "" H 7500 3750 50  0001 C CNN
@@
 AR Path="/5F7C96F7/5F7DF61A" Ref="R30"  Part="1"
 AR Path="/5F7E81D5/5F7DF61A" Ref="R12"  Part="1"
-F 0 "R12" V 6093 3700 50  0000 C CNN
-F 1 "2k2" V 6184 3700 50  0000 C CNN
+F 0 "R30" V 6093 3700 50  0000 C CNN
+F 1 "2.2k" V 6184 3700 50  0000 C CNN
 F 2 "Resistor_SMD:R_0603_1608Metric" V 6230 3700 50  0001 C CNN
 F 3 "~" H 6300 3700 50  0001 C CNN
+F 4 "C4190" H 6300 3700 50  0001 C CNN "LCSC Part #"
 	1    6300 3700
 	0    1    1    0
@@
 AR Path="/5F7C96F7/5F7E240A" Ref="U4"  Part="2"
 AR Path="/5F7E81D5/5F7E240A" Ref="U6"  Part="2"
-F 0 "U6" H 6150 3725 50  0000 C CNN
+F 0 "U4" H 6150 3725 50  0000 C CNN
 F 1 "3PEAK TP09-SR" H 6150 3726 50  0001 C CNN
 F 2 "Package_SO:SOIC-8_3.9x4.9mm_P1.27mm" H 6150 3450 50  0001 C CNN
 F 3 "~" H 6150 3450 50  0001 C CNN
+F 4 "C81662" H 6150 3450 50  0001 C CNN "LCSC Part #"
 	2    6150 3450
 	1    0    0    -1

Commit message: Added emergency-break connector
Changed lines of the file:
@@
 AR Path="/5F7C96F7/5F7C98DC" Ref="#PWR0159"  Part="1"
 AR Path="/5F7E81D5/5F7C98DC" Ref="#PWR0165"  Part="1"
-F 0 "#PWR0159" H 8950 1600 50  0001 C CNN
+F 0 "#PWR0165" H 8950 1600 50  0001 C CNN
 F 1 "+3.3V" H 8965 1923 50  0000 C CNN
 F 2 "" H 8950 1750 50  0001 C CNN
@@
 AR Path="/5F7C96F7/5F7C9ADD" Ref="C10"  Part="1"
 AR Path="/5F7E81D5/5F7C9ADD" Ref="C7"  Part="1"
-F 0 "C10" H 9065 1946 50  0000 L CNN
+F 0 "C7" H 9065 1946 50  0000 L CNN
 F 1 "100nF" H 9065 1855 50  0000 L CNN
 F 2 "Capacitor_SMD:C_0603_1608Metric" H 8988 1750 50  0001 C CNN
@@
 AR Path="/5F7C96F7/5F7C9C6F" Ref="#PWR0160"  Part="1"
 AR Path="/5F7E81D5/5F7C9C6F" Ref="#PWR0166"  Part="1"
-F 0 "#PWR0160" H 8950 1800 50  0001 C CNN
+F 0 "#PWR0166" H 8950 1800 50  0001 C CNN
 F 1 "GND" H 8955 1877 50  0000 C CNN
 F 2 "" H 8950 2050 50  0001 C CNN
@@
 AR Path="/5F7C96F7/5F7C9F32" Ref="R24"  Part="1"
 AR Path="/5F7E81D5/5F7C9F32" Ref="R2"  Part="1"
-F 0 "R24" V 4807 1650 50  0000 C CNN
+F 0 "R2" V 4807 1650 50  0000 C CNN
 F 1 "20k" V 4716 1650 50  0000 C CNN
 F 2 "Resistor_SMD:R_0603_1608Metric" V 4530 1650 50  0001 C CNN
@@
 AR Path="/5F7C96F7/5F7CA82E" Ref="R23"  Part="1"
 AR Path="/5F7E81D5/5F7CA82E" Ref="R6"  Part="1"
-F 0 "R23" V 5107 1650 50  0000 C CNN
+F 0 "R6" V 5107 1650 50  0000 C CNN
 F 1 "20k" V 5016 1650 50  0000 C CNN
 F 2 "Resistor_SMD:R_0603_1608Metric" V 4830 1650 50  0001 C CNN
@@
 AR Path="/5F7C96F7/5F7CA9C0" Ref="R26"  Part="1"
 AR Path="/5F7E81D5/5F7CA9C0" Ref="R3"  Part="1"
-F 0 "R26" V 4807 2000 50  0000 C CNN
+F 0 "R3" V 4807 2000 50  0000 C CNN
 F 1 "1k" V 4716 2000 50  0000 C CNN
 F 2 "Resistor_SMD:R_0603_1608Metric" V 4530 2000 50  0001 C CNN
@@
 AR Path="/5F7C96F7/5F7CAE77" Ref="D4"  Part="1"
 AR Path="/5F7E81D5/5F7CAE77" Ref="D3"  Part="1"
-F 0 "D4" V 5096 1721 50  0000 R CNN
+F 0 "D3" V 5096 1721 50  0000 R CNN
 F 1 "1N4148W" V 5005 1721 50  0000 R CNN
 F 2 "Diode_SMD:D_SOD-123" H 5050 1800 50  0001 C CNN
@@
 AR Path="/5F7C96F7/5F7CB464" Ref="#PWR0161"  Part="1"
 AR Path="/5F7E81D5/5F7CB464" Ref="#PWR0167"  Part="1"
-F 0 "#PWR0161" H 6050 1150 50  0001 C CNN
+F 0 "#PWR0167" H 6050 1150 50  0001 C CNN
 F 1 "+3.3V" H 6065 1473 50  0000 C CNN
 F 2 "" H 6050 1300 50  0001 C CNN
@@
 AR Path="/5F7C96F7/5F7CB568" Ref="R22"  Part="1"
 AR Path="/5F7E81D5/5F7CB568" Ref="R8"  Part="1"
-F 0 "R22" V 5957 1300 50  0000 C CNN
+F 0 "R8" V 5957 1300 50  0000 C CNN
 F 1 "220k" V 5866 1300 50  0000 C CNN
 F 2 "Resistor_SMD:R_0603_1608Metric" V 5680 1300 50  0001 C CNN
@@
 AR Path="/5F7C96F7/5F7CBE46" Ref="U4"  Part="1"
 AR Path="/5F7E81D5/5F7CBE46" Ref="U6"  Part="1"
-F 0 "U4" H 6150 2025 50  0000 C CNN
+F 0 "U6" H 6150 2025 50  0000 C CNN
 F 1 "3PEAK TP09-SR" H 6150 2026 50  0001 C CNN
 F 2 "Package_SO:SOIC-8_3.9x4.9mm_P1.27mm" H 6150 1750 50  0001 C CNN
@@
 AR Path="/5F7C96F7/5F7CE17C" Ref="R25"  Part="1"
 AR Path="/5F7E81D5/5F7CE17C" Ref="R11"  Part="1"
-F 0 "R25" V 6093 2000 50  0000 C CNN
+F 0 "R11" V 6093 2000 50  0000 C CNN
 F 1 "2.2k" V 6184 2000 50  0000 C CNN
 F 2 "Resistor_SMD:R_0603_1608Metric" V 6230 2000 50  0001 C CNN
@@
 AR Path="/5F7C96F7/5F7DF5DA" Ref="R29"  Part="1"
 AR Path="/5F7E81D5/5F7DF5DA" Ref="R4"  Part="1"
-F 0 "R29" V 4807 3350 50  0000 C CNN
+F 0 "R4" V 4807 3350 50  0000 C CNN
 F 1 "20k" V 4716 3350 50  0000 C CNN
 F 2 "Resistor_SMD:R_0603_1608Metric" V 4530 3350 50  0001 C CNN
@@
 AR Path="/5F7C96F7/5F7DF5E0" Ref="R1"  Part="1"
 AR Path="/5F7E81D5/5F7DF5E0" Ref="R7"  Part="1"
-F 0 "R1" V 5107 3350 50  0000 C CNN
+F 0 "R7" V 5107 3350 50  0000 C CNN
 F 1 "20k" V 5016 3350 50  0000 C CNN
 F 2 "Resistor_SMD:R_0603_1608Metric" V 4830 3350 50  0001 C CNN
@@
 AR Path="/5F7C96F7/5F7DF5E6" Ref="R31"  Part="1"
 AR Path="/5F7E81D5/5F7DF5E6" Ref="R5"  Part="1"
-F 0 "R31" V 4807 3700 50  0000 C CNN
+F 0 "R5" V 4807 3700 50  0000 C CNN
 F 1 "1k" V 4716 3700 50  0000 C CNN
 F 2 "Resistor_SMD:R_0603_1608Metric" V 4530 3700 50  0001 C CNN
@@
 AR Path="/5F7C96F7/5F7DF5EC" Ref="D5"  Part="1"
 AR Path="/5F7E81D5/5F7DF5EC" Ref="D6"  Part="1"
-F 0 "D5" V 5096 3421 50  0000 R CNN
+F 0 "D6" V 5096 3421 50  0000 R CNN
 F 1 "1N4148W" V 5005 3421 50  0000 R CNN
 F 2 "Diode_SMD:D_SOD-123" H 5050 3500 50  0001 C CNN
@@
 AR Path="/5F7C96F7/5F7DF5F4" Ref="#PWR0163"  Part="1"
 AR Path="/5F7E81D5/5F7DF5F4" Ref="#PWR0169"  Part="1"
-F 0 "#PWR0163" H 6050 2850 50  0001 C CNN
+F 0 "#PWR0169" H 6050 2850 50  0001 C CNN
 F 1 "+3.3V" H 6065 3173 50  0000 C CNN
 F 2 "" H 6050 3000 50  0001 C CNN
@@
 AR Path="/5F7C96F7/5F7DF5FA" Ref="R27"  Part="1"
 AR Path="/5F7E81D5/5F7DF5FA" Ref="R9"  Part="1"
-F 0 "R27" V 5957 3000 50  0000 C CNN
+F 0 "R9" V 5957 3000 50  0000 C CNN
 F 1 "220k" V 5866 3000 50  0000 C CNN
 F 2 "Resistor_SMD:R_0603_1608Metric" V 5680 3000 50  0001 C CNN
@@
 AR Path="/5F7C96F7/5F7DF60A" Ref="U4"  Part="3"
 AR Path="/5F7E81D5/5F7DF60A" Ref="U6"  Part="3"
-F 0 "U4" H 7558 3496 50  0000 L CNN
+F 0 "U6" H 7558 3496 50  0000 L CNN
 F 1 "3PEAK TP09-SR" H 7558 3405 50  0000 L CNN
 F 2 "Package_SO:SOIC-8_3.9x4.9mm_P1.27mm" H 7600 3450 50  0001 C CNN
@@
 AR Path="/5F7C96F7/5F7DF613" Ref="#PWR0164"  Part="1"
 AR Path="/5F7E81D5/5F7DF613" Ref="#PWR0170"  Part="1"
-F 0 "#PWR0164" H 7500 3500 50  0001 C CNN
+F 0 "#PWR0170" H 7500 3500 50  0001 C CNN
 F 1 "GND" H 7505 3577 50  0000 C CNN
 F 2 "" H 7500 3750 50  0001 C CNN
@@
 AR Path="/5F7C96F7/5F7DF61A" Ref="R30"  Part="1"
 AR Path="/5F7E81D5/5F7DF61A" Ref="R12"  Part="1"
-F 0 "R30" V 6093 3700 50  0000 C CNN
+F 0 "R12" V 6093 3700 50  0000 C CNN
 F 1 "2.2k" V 6184 3700 50  0000 C CNN
 F 2 "Resistor_SMD:R_0603_1608Metric" V 6230 3700 50  0001 C CNN
@@
 AR Path="/5F7C96F7/5F7E240A" Ref="U4"  Part="2"
 AR Path="/5F7E81D5/5F7E240A" Ref="U6"  Part="2"
-F 0 "U4" H 6150 3725 50  0000 C CNN
+F 0 "U6" H 6150 3725 50  0000 C CNN
 F 1 "3PEAK TP09-SR" H 6150 3726 50  0001 C CNN
 F 2 "Package_SO:SOIC-8_3.9x4.9mm_P1.27mm" H 6150 3450 50  0001 C CNN
