File: Bobbycontroller.kicad_sch (KiCad schematic)
At the start: 37 parts, among them J1 Conn_01x01_Male, J11 Conn_01x01, J12 Conn_01x01, J13 Conn_01x01, J14 Conn_01x01, J15 -BATT, J16 +BATT, J2 Conn_01x01_Male, J3 Conn_01x01_Male, J5 Conn_01x01_Male, J6 Conn_01x01_Male, J7 Conn_01x01_Male

Commit message: Silkscreen and naming fixes
Parts:
- renumbered C46 to C1, C53 to C10, C29 to C11, C54 to C12, C55 to C13, C30 to C14, C56 to C15, C57 to C16, C58 to C17, C59 to C18, C47 to C2, C27 to C3, C48 to C4, C49 to C5, C28 to C6, C50 to C7, C51 to C8, C52 to C9, J12 to J10, J13 to J11, J14 to J12, J5 to J4, J6 to J5, J7 to J6, J15 to J7, J16 to J8, J11 to J9, NT2 to NT1, NT1 to NT2, R0NL1 to R1, R0NL2 to R2, R0N1L1 to R3, R0N1L2 to R4

Commit message: added esp on bottom side
Parts:
- added J20: Conn_01x06, Connector_JST:JST_XH_B6B-XH-A_1x06_P2.50mm_Vertical, symbol Connector_Generic:Conn_01x06
- added R113, R114: 10k, Resistor_SMD:R_0603_1608Metric, symbol Device:R
- added U18: ESP32-WROOM-32, RF_Module:ESP32-WROOM-32, symbol RF_Module:ESP32-WROOM-32
- added U19: TJA1051T-3, Package_SO:SOIC-8_3.9x4.9mm_P1.27mm, symbol Interface_CAN_LIN:TJA1051T-3
- added U20, U21: LM75B, Package_SO:VSSOP-8_3.0x3.0mm_P0.65mm, symbol Sensor_Temperature:LM75B
Connections:
- net GND: now also J20.1 (Pin_1), U18.1 (GND), U18.15 (GND), U18.38 (GND), U18.39 (GND), U19.2 (GND), U19.8 (S), U20.4 (GND), U20.5 (A2), U20.6 (A1), U20.7 (A0), U21.4 (GND), U21.5 (A2), U21.6 (A1)
- new net +3V3: R113.1, R114.1, U18.2 (VDD), U19.5 (VIO), U20.8 (+Vs), U21.7 (A0), U21.8 (+Vs)
- new net +5V: J20.6 (Pin_6), U19.3 (VCC)
- new net CANH: U19.7 (CANH)
- new net CANL: U19.6 (CANL)
- new net ESP_CAN_RX: U18.36 (IO22), U19.4 (RXD)
- new net ESP_CAN_TX: U18.33 (IO21), U19.1 (TXD)
- new net ESP_EN: J20.4 (Pin_4), R113.2, U18.3 (EN)
- new net ESP_IO0: J20.5 (Pin_5), R114.2, U18.25 (IO0)
- new net ESP_RX: J20.2 (Pin_2), U18.34 (RXD0/IO3)
- new net ESP_TX: J20.3 (Pin_3), U18.35 (TXD0/IO1)
- new net SCL: U18.31 (IO19), U20.2 (SCL), U21.2 (SCL)
- new net SDA: U18.30 (IO18), U20.1 (SDA), U21.1 (SDA)
- new net U1_RX: U18.26 (IO4)
- new net U1_TX: U18.24 (IO2)

Commit message: Update a few library symbols
Parts:
- C11, C14, C3, C6: symbol Device:CP -> Device:C_Polarized
- NT1, NT2: value Net-Tie_2 -> NetTie_2; symbol Device:Net-Tie_2 -> Device:NetTie_2
Changed lines of the file:
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@@
     (pin "1")
   )
-  (symbol (lib_id "Device:Net-Tie_2") (at 262.89 53.34 0) (unit 1)
-    (in_bom yes) (on_board yes)
-    (property "Reference" "NT2" (id 0) (at 262.89 48.7426 0))
-    (property "Value" "Net-Tie_2" (id 1) (at 262.89 51.054 0))
+  (symbol (lib_id "Device:NetTie_2") (at 262.89 53.34 0) (unit 1)
+    (in_bom yes) (on_board yes)
+    (property "Reference" "NT2" (id 0) (at 262.89 52.07 0))
+    (property "Value" "NetTie_2" (id 1) (at 262.89 54.61 0))
     (property "Footprint" "NetTie:NetTie-2_SMD_Pad2.0mm" (id 2) (at 262.89 53.34 0)
       (effects (font (size 1.27 1.27)) hide)
@@
     (pin "2")
   )
-  (symbol (lib_id "Device:Net-Tie_2") (at 262.89 45.72 0) (unit 1)
-    (in_bom yes) (on_board yes)
-    (property "Reference" "NT1" (id 0) (at 262.89 41.1226 0))
-    (property "Value" "Net-Tie_2" (id 1) (at 262.89 43.434 0))
+  (symbol (lib_id "Device:NetTie_2") (at 262.89 45.72 0) (unit 1)
+    (in_bom yes) (on_board yes)
+    (property "Reference" "NT1" (id 0) (at 262.89 44.45 0))
+    (property "Value" "NetTie_2" (id 1) (at 262.89 46.99 0))
     (property "Footprint" "NetTie:NetTie-2_SMD_Pad2.0mm" (id 2) (at 262.89 45.72 0)
       (effects (font (size 1.27 1.27)) hide)
@@
     (pin "1")
   )
-  (symbol (lib_id "Device:CP") (at 248.92 129.54 0) (unit 1)
+  (symbol (lib_id "Device:C_Polarized") (at 248.92 129.54 0) (unit 1)
     (in_bom yes) (on_board yes)
     (property "Reference" "C3" (id 0) (at 251.9172 128.3716 0)
@@
     (pin "2")
   )
-  (symbol (lib_id "Device:CP") (at 256.54 129.54 0) (unit 1)
+  (symbol (lib_id "Device:C_Polarized") (at 256.54 129.54 0) (unit 1)
     (in_bom yes) (on_board yes)
     (property "Reference" "C6" (id 0) (at 259.5372 128.3716 0)
@@
     (pin "2")
   )
-  (symbol (lib_id "Device:CP") (at 262.89 129.54 0) (unit 1)
+  (symbol (lib_id "Device:C_Polarized") (at 262.89 129.54 0) (unit 1)
     (in_bom yes) (on_board yes)
     (property "Reference" "C11" (id 0) (at 265.8872 128.3716 0)
@@
     (pin "2")
   )
-  (symbol (lib_id "Device:CP") (at 269.24 129.54 0) (unit 1)
+  (symbol (lib_id "Device:C_Polarized") (at 269.24 129.54 0) (unit 1)
     (in_bom yes) (on_board yes)
     (property "Reference" "C14" (id 0) (at 272.2372 128.3716 0)
@@
     )
     (path "/00000000-0000-0000-0000-00005f7403be"
-      (reference "NT1") (unit 1) (value "Net-Tie_2") (footprint "NetTie:NetTie-2_SMD_Pad2.0mm")
+      (reference "NT1") (unit 1) (value "NetTie_2") (footprint "NetTie:NetTie-2_SMD_Pad2.0mm")
     )
     (path "/00000000-0000-0000-0000-00005f73becd"
-      (reference "NT2") (unit 1) (value "Net-Tie_2") (footprint "NetTie:NetTie-2_SMD_Pad2.0mm")
+      (reference "NT2") (unit 1) (value "NetTie_2") (footprint "NetTie:NetTie-2_SMD_Pad2.0mm")
     )
     (path "/00000000-0000-0000-0000-00005f7395da/10039648-85bc-4600-9881-23c4fdfcfb85"
