File: Bobbycontroller.kicad_sch (KiCad schematic)
At the start: 44 parts, among them J1 Conn_01x01_Male, J10 Conn_01x01, J11 Conn_01x01, J12 Conn_01x01, J2 Conn_01x01_Male, J20 Conn_01x06, J3 Conn_01x01_Male, J4 Conn_01x01_Male, J5 Conn_01x01_Male, J6 Conn_01x01_Male, J7 -BATT, J8 +BATT, J9 Conn_01x01, U18 ESP32-WROOM-32, U19 TJA1051T-3, U20 LM75B, U21 LM75B

Commit message: Some ERC fixes and other cleanups
Connections:
- no-connect marks 2 -> 29
Other:
- sheet CURRENT_SENSE ports: added none; removed L_MTR_OVERCUR, R_MTR_OVERCUR

Commit message: Add some decoupling caps; some more cleanups
Parts:
- removed J20: Conn_01x06, Connector_JST:JST_XH_B6B-XH-A_1x06_P2.50mm_Vertical, symbol Connector_Generic:Conn_01x06
- removed R113, R114: 10k, Resistor_SMD:R_0603_1608Metric, symbol Device:R
- removed U18: ESP32-WROOM-32, RF_Module:ESP32-WROOM-32, symbol RF_Module:ESP32-WROOM-32
- removed U19: TJA1051T-3, Package_SO:SOIC-8_3.9x4.9mm_P1.27mm, symbol Interface_CAN_LIN:TJA1051T-3
- removed U20, U21: LM75B, Package_SO:VSSOP-8_3.0x3.0mm_P0.65mm, symbol Sensor_Temperature:LM75B
Connections:
- no-connect marks 29 -> 4
Other:
- added sheet ESP32 (ESP32.kicad_sch)
- moved on the sheet: J7, J8

Commit message: Updated diodes, added LCSC numbers for all parts
Parts:
- C1, C10, C12, C13, C15, C16, C17, C18, C2, C4, C5, C7, C8, C9: LCSC (none) -> C577211
- C11, C14, C3, C6: LCSC (none) -> C443080
- J1, J10, J11, J12, J2, J3, J4, J5, J6, J7, J8, J9, LOGO1, NT1, NT2: now not fitted; now left out of the parts list
- R1, R2, R3, R4: LCSC (none) -> C270946; LCSC Part # C270946 -> (none)

Commit message: update lcsc numbers
Parts:
- C1, C10, C12, C13, C15, C16, C17, C18, C2, C4, C5, C7, C8, C9: now not fitted; now left out of the parts list
- C11, C14, C3, C6: place hand -> (none)

Commit message: Exchanged more components, DNP and bridge 4.7R resistor, DNP 51V TVS diode
Parts:
- R1, R2, R3, R4: LCSC C270946 -> C46634448
Changed lines of the file:
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@@
 			)
 		)
-		(property "LCSC" "C270946"
+		(property "LCSC" "C46634448"
 			(at 215.9 67.31 0)
 			(effects
@@
 			)
 		)
-		(property "LCSC" "C270946"
+		(property "LCSC" "C46634448"
 			(at 205.74 67.31 0)
 			(effects
@@
 			)
 		)
-		(property "LCSC" "C270946"
+		(property "LCSC" "C46634448"
 			(at 215.9 157.48 0)
 			(effects
@@
 			)
 		)
-		(property "LCSC" "C270946"
+		(property "LCSC" "C46634448"
 			(at 205.74 157.48 0)
 			(effects
