File: connectors.kicad_sch (KiCad schematic)
At the start: 56 parts, among them J10 UART_R1, J18 JST XH 4P, J4 Conn_01x04_Male, J8 JST XH 4P, J9 UART_L1, U15 SRV05-4, U5 SRV05-4

Commit message: Silkscreen and naming fixes
Parts:
- renumbered C60 to C22, C2 to C23, C37 to C24, C41 to C25, C72 to C26, C73 to C27, C84 to C28, C85 to C29, C86 to C30, C42 to C31, D0AL2 to D1, D34 to D10, D12 to D11, D17 to D12, D18 to D13, D19 to D14, D0AL1 to D2, D0AL3 to D3, D0AL4 to D4, D29 to D5, D30 to D6, D31 to D7, D32 to D8, D33 to D9, J9 to J13, J10 to J14, J8 to J15, J18 to J16, J4 to J17, R16L1 to R10, R16L2 to R11, R36 to R12, R17L3 to R13, R17L4 to R14, R37 to R15, R38 to R16, R17L1 to R17, R17L2 to R18, R18L3 to R19, R18L4 to R20, R18L1 to R21, R18L2 to R22, R21L1 to R23, R21L2 to R24, R82 to R25, R20L1 to R26, R20L2 to R27, R19L1 to R28, R19L2 to R29, R16L3 to R7, R16L4 to R8, R35 to R9, U5 to U2, U15 to U3

Commit message: added esp on bottom side
Changed lines of the file:
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@@
   (symbol (lib_id "Device:R") (at 83.82 139.7 270) (unit 1)
     (in_bom yes) (on_board yes)
-    (property "Reference" "R15" (id 0) (at 83.82 132.08 90))
-    (property "Value" "100" (id 1) (at 83.82 134.62 90))
+    (property "Reference" "R15" (id 0) (at 83.82 142.24 90))
+    (property "Value" "100" (id 1) (at 83.82 144.78 90))
     (property "Footprint" "Resistor_SMD:R_0603_1608Metric" (id 2) (at 83.82 137.922 90)
       (effects (font (size 1.27 1.27)) hide)
@@
   (symbol (lib_id "Device:C") (at 91.44 143.51 0) (unit 1)
     (in_bom yes) (on_board yes)
-    (property "Reference" "C28" (id 0) (at 82.55 142.24 0)
-      (effects (font (size 1.27 1.27)) (justify left))
-    )
-    (property "Value" "100nF" (id 1) (at 82.55 144.78 0)
-      (effects (font (size 1.27 1.27)) (justify left))
-    )
+    (property "Reference" "C28" (id 0) (at 88.9 140.97 0)
+      (effects (font (size 1.27 1.27)) (justify left))
+    )
+    (property "Value" "100nF" (id 1) (at 88.9 146.05 0)
+      (effects (font (size 1.27 1.27)) (justify left))
+    )

Commit message: Update CAN VBUS diode in schematic
fixes 4326932b17624209b9845990315cd6ab7ab2b5f4
Parts:
- D13: value B5819W -> SS36-E3/57T; footprint Diode_SMD:D_SOD-123 -> Diode_SMD:D_SMC; LCSC Part # C8598 -> C35722
Changed lines of the file:
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@@
   (junction (at 53.34 93.98) (diameter 0) (color 0 0 0 0)
   )
+  (junction (at 148.59 167.64) (diameter 0) (color 0 0 0 0)
+  )
   (junction (at 83.82 116.84) (diameter 0) (color 0 0 0 0)
   )
@@
   (junction (at 97.79 167.64) (diameter 0) (color 0 0 0 0)
   )
-  (junction (at 148.59 168.91) (diameter 0) (color 0 0 0 0)
-  )
   (junction (at 77.47 97.79) (diameter 0) (color 0 0 0 0)
   )
@@
   (junction (at 77.47 52.07) (diameter 0) (color 0 0 0 0)
   )
-  (junction (at 158.75 168.91) (diameter 0) (color 0 0 0 0)
-  )
   (junction (at 97.79 162.56) (diameter 0) (color 0 0 0 0)
   )
@@
   )
   (junction (at 135.89 163.83) (diameter 0) (color 0 0 0 0)
+  )
+  (junction (at 158.75 167.64) (diameter 0) (color 0 0 0 0)
   )
   (junction (at 83.82 71.12) (diameter 0) (color 0 0 0 0)
@@
     (stroke (width 0) (type default) (color 0 0 0 0))
   )
-  (wire (pts (xy 148.59 167.64) (xy 148.59 168.91))
-    (stroke (width 0) (type default) (color 0 0 0 0))
-  )
   (wire (pts (xy 95.25 67.31) (xy 95.25 73.66))
     (stroke (width 0) (type default) (color 0 0 0 0))
@@
     (stroke (width 0) (type default) (color 0 0 0 0))
   )
-  (wire (pts (xy 148.59 168.91) (xy 158.75 168.91))
+  (wire (pts (xy 148.59 167.64) (xy 158.75 167.64))
     (stroke (width 0) (type default) (color 0 0 0 0))
   )
@@
     (stroke (width 0) (type default) (color 0 0 0 0))
   )
-  (wire (pts (xy 158.75 168.91) (xy 158.75 165.1))
-    (stroke (width 0) (type default) (color 0 0 0 0))
-  )
   (wire (pts (xy 87.63 129.54) (xy 90.17 129.54))
     (stroke (width 0) (type default) (color 0 0 0 0))
@@
     (stroke (width 0) (type default) (color 0 0 0 0))
   )
+  (wire (pts (xy 158.75 167.64) (xy 158.75 173.99))
+    (stroke (width 0) (type default) (color 0 0 0 0))
+  )
   (wire (pts (xy 88.9 170.18) (xy 97.79 170.18))
     (stroke (width 0) (type default) (color 0 0 0 0))
@@
     (stroke (width 0) (type default) (color 0 0 0 0))
   )
+  (wire (pts (xy 148.59 167.64) (xy 148.59 173.99))
+    (stroke (width 0) (type default) (color 0 0 0 0))
+  )
   (wire (pts (xy 68.58 111.76) (xy 68.58 109.22))
     (stroke (width 0) (type default) (color 0 0 0 0))
@@
     (stroke (width 0) (type default) (color 0 0 0 0))
   )
-  (wire (pts (xy 158.75 168.91) (xy 158.75 173.99))
-    (stroke (width 0) (type default) (color 0 0 0 0))
-  )
   (wire (pts (xy 86.36 113.03) (xy 86.36 116.84))
     (stroke (width 0) (type default) (color 0 0 0 0))
@@
     (stroke (width 0) (type default) (color 0 0 0 0))
   )
+  (wire (pts (xy 158.75 167.64) (xy 158.75 165.1))
+    (stroke (width 0) (type default) (color 0 0 0 0))
+  )
   (wire (pts (xy 125.73 34.29) (xy 124.46 34.29))
     (stroke (width 0) (type default) (color 0 0 0 0))
@@
   )
   (wire (pts (xy 57.15 109.22) (xy 57.15 114.3))
-    (stroke (width 0) (type default) (color 0 0 0 0))
-  )
-  (wire (pts (xy 148.59 168.91) (xy 148.59 173.99))
     (stroke (width 0) (type default) (color 0 0 0 0))
   )
@@
       (effects (font (size 1.27 1.27)) (justify right))
     )
-    (property "Value" "B5819W" (id 1) (at 160.782 162.433 90)
+    (property "Value" "SS36-E3/57T" (id 1) (at 160.782 162.433 90)
       (effects (font (size 1.27 1.27)) (justify right))
     )
-    (property "Footprint" "Diode_SMD:D_SOD-123" (id 2) (at 158.75 161.29 0)
+    (property "Footprint" "Diode_SMD:D_SMC" (id 2) (at 158.75 161.29 0)
       (effects (font (size 1.27 1.27)) hide)
     )
@@
       (effects (font (size 1.27 1.27)) hide)
     )
-    (property "LCSC Part #" "C8598" (id 4) (at 158.75 161.29 0)
-      (effects (font (size 1.27 1.27)) hide)
-    )
+    (property "LCSC Part #" "C35722" (id 4) (at 158.75 161.29 0)
+      (effects (font (size 1.27 1.27)) hide)
+    )

Commit message: Refactor stuff adjacent to hall sensor pins
Parts:
- removed C22, C23, C24, C25, C26, C27, C29, C30: 100nF, Capacitor_SMD:C_0603_1608Metric, symbol Device:C
- removed D1, D2: 1N4148W, Diode_SMD:D_SOD-123, symbol Device:D
- removed D10, D5, D6, D7, D8, D9: LED, LED_SMD:LED_0603_1608Metric, symbol Device:LED
- removed R10, R11, R13, R14, R17, R18, R19, R20, R21, R22, R7, R8: 2.2k, Resistor_SMD:R_0603_1608Metric, symbol Device:R
- removed R23, R24, R26, R27, R28, R29: 3.3k, Resistor_SMD:R_0603_1608Metric, symbol Device:R
Connections:
- net GND: no longer HALL_L1.1 (Pin_1), HALL_R1.1 (Pin_1)
- net Hall_R_1: now also U3.6 (IO4); no longer U3.4 (IO3)
- net Hall_R_2: now also U3.4 (IO3); no longer U3.6 (IO4)
- net Hall_VCC renamed Hall_L_VCC
- net Hall_VCC_2 renamed Hall_R_VCC
- new net Hall Left/HALL_GND: HALL_L1.1 (Pin_1)
- new net Hall Right/HALL_GND: HALL_R1.1 (Pin_1)
Other:
- added sheet Hall Left (hall_conn.kicad_sch)
- added sheet Hall Right (hall_conn.kicad_sch)
- note added: "TVS diodes"
- moved on the sheet: HALL_R1

Commit message: Update a few library symbols
Parts:
- D12: symbol Device:D_TVS_x2_AAC -> Device:D_TVS_Dual_AAC
Changed lines of the file:
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@@
     (pin "2")
   )
-  (symbol (lib_id "Device:D_TVS_x2_AAC") (at 125.73 149.86 0) (unit 1)
+  (symbol (lib_id "Device:D_TVS_Dual_AAC") (at 125.73 149.86 0) (unit 1)
     (in_bom yes) (on_board yes)
     (property "Reference" "D12" (id 0) (at 125.73 144.3482 0))

Commit message: Some ERC fixes and other cleanups
Parts:
- D11: symbol input-board:CDSOD323-boardcomputer -> Device:D_TVS
Changed lines of the file:
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@@
     (pin "1")
   )
-  (symbol (lib_id "input-board:CDSOD323-boardcomputer") (at 97.79 142.24 270) (unit 1)
+  (symbol (lib_id "Device:D_TVS") (at 97.79 143.51 270) (unit 1)
     (in_bom yes) (on_board yes)
     (property "Reference" "D11" (id 0) (at 100.33 146.05 90)
       (effects (font (size 1.27 1.27)) (justify left))
     )
-    (property "Value" "CDSOD323" (id 1) (at 101.6 143.51 90)
+    (property "Value" "CDSOD323" (id 1) (at 100.33 143.51 90)
       (effects (font (size 1.27 1.27)) (justify left))
     )
-    (property "Footprint" "Diode_SMD:D_SOD-323" (id 2) (at 101.6 142.24 0)
+    (property "Footprint" "Diode_SMD:D_SOD-323" (id 2) (at 101.6 143.51 0)
       (effects (font (size 1.27 1.27)) hide)
     )
-    (property "Datasheet" "" (id 3) (at 101.6 142.24 0)
+    (property "Datasheet" "" (id 3) (at 101.6 143.51 0)
       (effects (font (size 1.27 1.27)) hide)
     )
-    (property "LCSC Part #" "C127526" (id 4) (at 97.79 142.24 90)
+    (property "LCSC Part #" "C127526" (id 4) (at 97.79 143.51 90)
       (effects (font (size 1.27 1.27)) hide)
     )

Commit message: Add some decoupling caps; some more cleanups
Connections:
- net Hall_R_1: now also U3.4 (IO3); no longer U3.6 (IO4)
- net Hall_R_2: now also U3.6 (IO4); no longer U3.4 (IO3)
Changed lines of the file:
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@@
     (effects (font (size 1.27 1.27)) (justify right bottom))
   )
-  (label "Hall_R_2" (at 49.53 107.95 0)
+  (label "Hall_R_2" (at 49.53 113.03 0)
     (effects (font (size 1.27 1.27)) (justify left bottom))
   )
@@
     (effects (font (size 1.27 1.27)) (justify left bottom))
   )
-  (label "Hall_R_1" (at 49.53 113.03 0)
+  (label "Hall_R_1" (at 49.53 107.95 0)
     (effects (font (size 1.27 1.27)) (justify left bottom))
   )
