File: connectors.kicad_sch (KiCad schematic)
At the start: 22 parts, among them J13 UART_L1, J14 UART_R1, J15 JST XH 4P, J16 JST XH 4P, J17 Conn_01x04_Male, U2 SRV05-4, U3 SRV05-4

Commit message: Updated diodes, added LCSC numbers for all parts
Parts:
- C28: LCSC (none) -> C14663; LCSC Part # C14663 -> (none)
- C31: LCSC (none) -> C28323; LCSC Part # C28323 -> (none)
- D11: LCSC (none) -> C127526; LCSC Part # C127526 -> (none)
- D12: LCSC (none) -> C38838; LCSC Part # C38838 -> (none)
- D13: LCSC (none) -> C35722; LCSC Part # C35722 -> (none)
- D14: LCSC (none) -> C78409; LCSC Part # C78409 -> (none)
- D3, D4: LCSC (none) -> C81598; LCSC Part # C81598 -> (none)
- HALL_L1, HALL_R1: LCSC (none) -> C57142
- J13: value UART_L1 -> UART_L1; LCSC (none) -> C192885
- J14: value UART_R1 -> UART_R1; LCSC (none) -> C192885
- J15, J16: value JST XH 4P -> CAN BUS JST XH 4P; LCSC (none) -> C68117
- J17: LCSC (none) -> C2691448
- R12, R15, R16, R9: LCSC (none) -> C22775; LCSC Part # C22775 -> (none)
- R25: LCSC (none) -> C21190; LCSC Part # C21190 -> (none)
- U2, U3: LCSC (none) -> C384887; LCSC Part # C384887 -> (none)

Commit message: update lcsc numbers
Parts:
- D11: value CDSOD323 -> 3.3V TVS; LCSC C127526 -> C314254
- HALL_L1, HALL_R1, J13, J14, J17: place dnp -> (none)
Changed lines of the file:
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@@
 			)
 		)
-		(property "place" "dnp"
+		(property "place" ""
 			(at 59.69 39.37 0)
 			(effects
@@
 			)
 		)
+		(property "alternative" ""
+			(at 59.69 39.37 0)
+			(effects
+				(font
+					(size 1.27 1.27)
+				)
+				(hide yes)
+			)
+		)
 		(pin "1"
 		)
@@
 			)
 		)
-		(property "place" "dnp"
+		(property "place" ""
 			(at 60.96 71.12 0)
 			(effects
@@
 			)
 		)
+		(property "alternative" ""
+			(at 60.96 71.12 0)
+			(effects
+				(font
+					(size 1.27 1.27)
+				)
+				(hide yes)
+			)
+		)
 		(pin "1"
 		)
@@
 			)
 		)
-		(property "place" "dnp"
+		(property "place" ""
 			(at 60.96 109.22 0)
 			(effects
@@
 		)
 		(property "LCSC" "C57142"
+			(at 60.96 109.22 0)
+			(effects
+				(font
+					(size 1.27 1.27)
+				)
+				(hide yes)
+			)
+		)
+		(property "alternative" ""
 			(at 60.96 109.22 0)
 			(effects
@@
 			)
 		)
-		(property "place" "dnp"
+		(property "place" ""
 			(at 60.96 139.7 0)
 			(effects
@@
 			)
 		)
+		(property "alternative" ""
+			(at 60.96 139.7 0)
+			(effects
+				(font
+					(size 1.27 1.27)
+				)
+				(hide yes)
+			)
+		)
 		(pin "1"
 		)
@@
 			)
 		)
+		(property "alternative" ""
+			(at 78.74 36.83 90)
+			(effects
+				(font
+					(size 1.27 1.27)
+				)
+				(hide yes)
+			)
+		)
 		(pin "1"
 		)
@@
 			)
 		)
+		(property "alternative" ""
+			(at 85.09 39.37 90)
+			(effects
+				(font
+					(size 1.27 1.27)
+				)
+				(hide yes)
+			)
+		)
 		(pin "1"
 		)
@@
 			)
 		)
+		(property "alternative" ""
+			(at 76.2 137.16 90)
+			(effects
+				(font
+					(size 1.27 1.27)
+				)
+				(hide yes)
+			)
+		)
 		(pin "1"
 		)
@@
 			)
 		)
+		(property "alternative" ""
+			(at 83.82 139.7 90)
+			(effects
+				(font
+					(size 1.27 1.27)
+				)
+				(hide yes)
+			)
+		)
 		(pin "1"
 		)
@@
 			)
 		)
+		(property "alternative" ""
+			(at 125.73 149.86 0)
+			(effects
+				(font
+					(size 1.27 1.27)
+				)
+				(hide yes)
+			)
+		)
 		(pin "1"
 		)
@@
 			)
 		)
+		(property "alternative" ""
+			(at 158.75 161.29 90)
+			(effects
+				(font
+					(size 1.27 1.27)
+				)
+				(hide yes)
+			)
+		)
 		(pin "1"
 		)
@@
 			)
 		)
+		(property "alternative" ""
+			(at 158.75 177.8 90)
+			(effects
+				(font
+					(size 1.27 1.27)
+				)
+				(hide yes)
+			)
+		)
 		(pin "1"
 		)
@@
 			)
 		)
+		(property "alternative" ""
+			(at 148.59 177.8 0)
+			(effects
+				(font
+					(size 1.27 1.27)
+				)
+				(hide yes)
+			)
+		)
 		(pin "1"
 		)
@@
 			)
 		)
+		(property "alternative" ""
+			(at 69.85 134.62 90)
+			(effects
+				(font
+					(size 1.27 1.27)
+				)
+				(hide yes)
+			)
+		)
 		(pin "1"
 		)
@@
 			)
 		)
+		(property "alternative" ""
+			(at 68.58 34.29 90)
+			(effects
+				(font
+					(size 1.27 1.27)
+				)
+				(hide yes)
+			)
+		)
 		(pin "1"
 		)
@@
 			)
 		)
-		(property "place" "dnp"
+		(property "place" ""
 			(at 119.38 31.75 0)
 			(effects
@@
 			)
 		)
+		(property "alternative" ""
+			(at 119.38 31.75 0)
+			(effects
+				(font
+					(size 1.27 1.27)
+				)
+				(hide yes)
+			)
+		)
 		(pin "1"
 		)
@@
 			)
 		)
+		(property "alternative" ""
+			(at 106.68 135.89 90)
+			(effects
+				(font
+					(size 1.27 1.27)
+				)
+				(hide yes)
+			)
+		)
 		(pin "1"
 		)
@@
 			)
 		)
-		(property "Value" "CDSOD323"
+		(property "Value" "3.3V TVS"
 			(at 100.33 143.51 90)
 			(effects
@@
 			)
 		)
-		(property "LCSC" "C127526"
+		(property "LCSC" "C314254"
+			(at 97.79 143.51 90)
+			(effects
+				(font
+					(size 1.27 1.27)
+				)
+				(hide yes)
+			)
+		)
+		(property "alternative" ""
 			(at 97.79 143.51 90)
 			(effects
@@
 			)
 		)
+		(property "alternative" ""
+			(at 91.44 143.51 0)
+			(effects
+				(font
+					(size 1.27 1.27)
+				)
+				(hide yes)
+			)
+		)
 		(pin "1"
 		)
@@
 			)
 		)
+		(property "alternative" ""
+			(at 83.82 167.64 0)
+			(effects
+				(font
+					(size 1.27 1.27)
+				)
+				(hide yes)
+			)
+		)
 		(pin "1"
 		)
@@
 			)
 		)
+		(property "alternative" ""
+			(at 36.83 72.39 0)
+			(effects
+				(font
+					(size 1.27 1.27)
+				)
+				(hide yes)
+			)
+		)
 		(pin "1"
 		)
@@
 			)
 		)
+		(property "alternative" ""
+			(at 92.71 167.64 0)
+			(effects
+				(font
+					(size 1.27 1.27)
+				)
+				(hide yes)
+			)
+		)
 		(pin "1"
 		)
@@
 			(at 36.83 110.49 0)
 			(effects
+				(font
+					(size 1.27 1.27)
+				)
+				(hide yes)
+			)
+		)
+		(property "alternative" ""
+			(at 36.83 110.49 0)
+			(effects
