File: CAN.kicad_sch (KiCad schematic)
At the start: 8 parts, among them U7 TJA1051T-3

Commit message: Silkscreen and naming fixes
Parts:
- renumbered C43 to C19, C44 to C20, C45 to C21, R48 to R5, R49 to R6, U7 to U1
Changed lines of the file:
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@@
   (symbol (lib_id "Device:R") (at 168.91 86.36 0) (unit 1)
     (in_bom yes) (on_board yes)
-    (property "Reference" "R48" (id 0) (at 170.688 85.1916 0)
+    (property "Reference" "R5" (id 0) (at 170.688 85.1916 0)
       (effects (font (size 1.27 1.27)) (justify left))
     )
@@
   (symbol (lib_id "Device:R") (at 168.91 96.52 0) (unit 1)
     (in_bom yes) (on_board yes)
-    (property "Reference" "R49" (id 0) (at 170.688 95.3516 0)
+    (property "Reference" "R6" (id 0) (at 170.688 95.3516 0)
       (effects (font (size 1.27 1.27)) (justify left))
     )
@@
   (symbol (lib_id "Device:C") (at 180.34 96.52 0) (unit 1)
     (in_bom yes) (on_board yes)
-    (property "Reference" "C45" (id 0) (at 183.261 95.3516 0)
+    (property "Reference" "C21" (id 0) (at 183.261 95.3516 0)
       (effects (font (size 1.27 1.27)) (justify left))
     )
@@
   (symbol (lib_id "power:GND") (at 180.34 101.6 0) (unit 1)
     (in_bom yes) (on_board yes)
-    (property "Reference" "#PWR0232" (id 0) (at 180.34 107.95 0)
+    (property "Reference" "#PWR021" (id 0) (at 180.34 107.95 0)
       (effects (font (size 1.27 1.27)) hide)
     )
@@
   (symbol (lib_id "power:GND") (at 120.65 105.41 0) (unit 1)
     (in_bom yes) (on_board yes)
-    (property "Reference" "#PWR0227" (id 0) (at 120.65 111.76 0)
+    (property "Reference" "#PWR018" (id 0) (at 120.65 111.76 0)
       (effects (font (size 1.27 1.27)) hide)
     )
@@
   (symbol (lib_id "power:+3.3V") (at 96.52 93.98 0) (unit 1)
     (in_bom yes) (on_board yes)
-    (property "Reference" "#PWR0228" (id 0) (at 96.52 97.79 0)
+    (property "Reference" "#PWR016" (id 0) (at 96.52 97.79 0)
       (effects (font (size 1.27 1.27)) hide)
     )
@@
   (symbol (lib_id "power:+5V") (at 124.46 68.58 0) (unit 1)
     (in_bom yes) (on_board yes)
-    (property "Reference" "#PWR0229" (id 0) (at 124.46 72.39 0)
+    (property "Reference" "#PWR019" (id 0) (at 124.46 72.39 0)
       (effects (font (size 1.27 1.27)) hide)
     )
@@
   (symbol (lib_id "Device:C") (at 96.52 99.06 0) (unit 1)
     (in_bom yes) (on_board yes)
-    (property "Reference" "C43" (id 0) (at 99.441 97.8916 0)
+    (property "Reference" "C19" (id 0) (at 99.441 97.8916 0)
       (effects (font (size 1.27 1.27)) (justify left))
     )
@@
   (symbol (lib_id "Device:C") (at 130.81 74.93 0) (unit 1)
     (in_bom yes) (on_board yes)
-    (property "Reference" "C44" (id 0) (at 133.731 73.7616 0)
+    (property "Reference" "C20" (id 0) (at 133.731 73.7616 0)
       (effects (font (size 1.27 1.27)) (justify left))
     )
@@
   (symbol (lib_id "power:GND") (at 96.52 104.14 0) (unit 1)
     (in_bom yes) (on_board yes)
-    (property "Reference" "#PWR0222" (id 0) (at 96.52 110.49 0)
+    (property "Reference" "#PWR017" (id 0) (at 96.52 110.49 0)
       (effects (font (size 1.27 1.27)) hide)
     )
@@
   (symbol (lib_id "power:GND") (at 130.81 80.01 0) (unit 1)
     (in_bom yes) (on_board yes)
-    (property "Reference" "#PWR0223" (id 0) (at 130.81 86.36 0)
+    (property "Reference" "#PWR020" (id 0) (at 130.81 86.36 0)
       (effects (font (size 1.27 1.27)) hide)
     )
@@
   (symbol (lib_id "Interface_CAN_LIN:TJA1051T-3") (at 120.65 91.44 0) (unit 1)
     (in_bom yes) (on_board yes)
-    (property "Reference" "U7" (id 0) (at 114.3 77.47 0))
+    (property "Reference" "U1" (id 0) (at 114.3 77.47 0))
     (property "Value" "TJA1051T-3" (id 1) (at 114.3 80.01 0))
     (property "Footprint" "Package_SO:SOIC-8_3.9x4.9mm_P1.27mm" (id 2) (at 120.65 104.14 0)

Commit message: Add some decoupling caps; some more cleanups
Parts:
- removed C19, C20, C21: 100nF, Capacitor_SMD:C_0603_1608Metric, symbol Device:C
- removed JP1, JP2: SolderJumper_2_Open, Jumper:SolderJumper-2_P1.3mm_Open_RoundedPad1.0x1.5mm, symbol Jumper:SolderJumper_2_Open
- removed R5, R6: 56, Resistor_SMD:R_0603_1608Metric, symbol Device:R
- removed U1: TJA1051T-3, Package_SO:SOIC-8_3.9x4.9mm_P1.27mm, symbol Interface_CAN_LIN:TJA1051T-3
Other:
- added sheet CAN TRX (CAN_TRX.kicad_sch)
- added sheet CAN Termination (can_termination.kicad_sch)
