File: CURRENT_SENSE.kicad_sch (KiCad schematic)
At the start: 11 parts, among them U14 3PEAK TP09-SR

Commit message: Silkscreen and naming fixes
Parts:
- renumbered C82 to C32, C83 to C33, R38R1 to R30, R37R1 to R31, R40R1 to R32, R39R1 to R33, R38L1 to R34, R37L1 to R35, R40L1 to R36, R39L1 to R37, U14 to U4
Changed lines of the file:
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@@
   (symbol (lib_id "Device:R") (at 59.69 114.3 270) (unit 1)
     (in_bom yes) (on_board yes)
-    (property "Reference" "R38R1" (id 0) (at 59.69 109.0422 90))
+    (property "Reference" "R30" (id 0) (at 59.69 109.0422 90))
     (property "Value" "10k" (id 1) (at 59.69 111.3536 90))
     (property "Footprint" "Resistor_SMD:R_0603_1608Metric" (id 2) (at 59.69 112.522 90)
@@
   (symbol (lib_id "Device:R") (at 66.04 107.95 0) (unit 1)
     (in_bom yes) (on_board yes)
-    (property "Reference" "R37R1" (id 0) (at 67.818 106.7816 0)
+    (property "Reference" "R31" (id 0) (at 67.818 106.7816 0)
       (effects (font (size 1.27 1.27)) (justify left))
     )
@@
   (symbol (lib_id "power:+3.3V") (at 66.04 104.14 0) (unit 1)
     (in_bom yes) (on_board yes)
-    (property "Reference" "#PWR0107" (id 0) (at 66.04 107.95 0)
+    (property "Reference" "#PWR046" (id 0) (at 66.04 107.95 0)
       (effects (font (size 1.27 1.27)) hide)
     )
@@
   (symbol (lib_id "Device:C") (at 66.04 118.11 0) (unit 1)
     (in_bom yes) (on_board yes)
-    (property "Reference" "C82" (id 0) (at 68.961 116.9416 0)
+    (property "Reference" "C32" (id 0) (at 68.961 116.9416 0)
       (effects (font (size 1.27 1.27)) (justify left))
     )
@@
   (symbol (lib_id "power:GND") (at 66.04 121.92 0) (unit 1)
     (in_bom yes) (on_board yes)
-    (property "Reference" "#PWR0108" (id 0) (at 66.04 128.27 0)
+    (property "Reference" "#PWR047" (id 0) (at 66.04 128.27 0)
       (effects (font (size 1.27 1.27)) hide)
     )
@@
   (symbol (lib_id "Device:Opamp_Dual_Generic") (at 87.63 116.84 0) (unit 2)
     (in_bom yes) (on_board yes)
-    (property "Reference" "U14" (id 0) (at 87.63 109.855 0))
+    (property "Reference" "U4" (id 0) (at 87.63 109.855 0))
     (property "Value" "3PEAK TP09-SR" (id 1) (at 87.63 109.8296 0)
       (effects (font (size 1.27 1.27)) hide)
@@
   (symbol (lib_id "Device:R") (at 76.2 129.54 0) (unit 1)
     (in_bom yes) (on_board yes)
-    (property "Reference" "R40R1" (id 0) (at 77.978 128.3716 0)
+    (property "Reference" "R32" (id 0) (at 77.978 128.3716 0)
       (effects (font (size 1.27 1.27)) (justify left))
     )
@@
   (symbol (lib_id "power:GND") (at 76.2 133.35 0) (unit 1)
     (in_bom yes) (on_board yes)
-    (property "Reference" "#PWR0110" (id 0) (at 76.2 139.7 0)
+    (property "Reference" "#PWR048" (id 0) (at 76.2 139.7 0)
       (effects (font (size 1.27 1.27)) hide)
     )
@@
   (symbol (lib_id "Device:R") (at 86.36 137.16 270) (unit 1)
     (in_bom yes) (on_board yes)
-    (property "Reference" "R39R1" (id 0) (at 86.36 131.9022 90))
+    (property "Reference" "R33" (id 0) (at 86.36 131.9022 90))
     (property "Value" "10k" (id 1) (at 86.36 134.2136 90))
     (property "Footprint" "Resistor_SMD:R_0603_1608Metric" (id 2) (at 86.36 135.382 90)
@@
   (symbol (lib_id "Device:R") (at 160.02 111.76 270) (unit 1)
     (in_bom yes) (on_board yes)
-    (property "Reference" "R38L1" (id 0) (at 160.02 106.5022 90))
+    (property "Reference" "R34" (id 0) (at 160.02 106.5022 90))
     (property "Value" "10k" (id 1) (at 160.02 108.8136 90))
     (property "Footprint" "Resistor_SMD:R_0603_1608Metric" (id 2) (at 160.02 109.982 90)
@@
   (symbol (lib_id "Device:R") (at 166.37 105.41 0) (unit 1)
     (in_bom yes) (on_board yes)
-    (property "Reference" "R37L1" (id 0) (at 168.148 104.2416 0)
+    (property "Reference" "R35" (id 0) (at 168.148 104.2416 0)
       (effects (font (size 1.27 1.27)) (justify left))
     )
@@
   (symbol (lib_id "power:+3.3V") (at 166.37 101.6 0) (unit 1)
     (in_bom yes) (on_board yes)
-    (property "Reference" "#PWR0115" (id 0) (at 166.37 105.41 0)
+    (property "Reference" "#PWR051" (id 0) (at 166.37 105.41 0)
       (effects (font (size 1.27 1.27)) hide)
     )
@@
   (symbol (lib_id "Device:C") (at 166.37 115.57 0) (unit 1)
     (in_bom yes) (on_board yes)
-    (property "Reference" "C83" (id 0) (at 169.291 114.4016 0)
+    (property "Reference" "C33" (id 0) (at 169.291 114.4016 0)
       (effects (font (size 1.27 1.27)) (justify left))
     )
@@
   (symbol (lib_id "power:GND") (at 166.37 119.38 0) (unit 1)
     (in_bom yes) (on_board yes)
-    (property "Reference" "#PWR0116" (id 0) (at 166.37 125.73 0)
+    (property "Reference" "#PWR052" (id 0) (at 166.37 125.73 0)
       (effects (font (size 1.27 1.27)) hide)
     )
@@
   (symbol (lib_id "power:+3.3V") (at 130.81 120.65 0) (unit 1)
     (in_bom yes) (on_board yes)
-    (property "Reference" "#PWR0117" (id 0) (at 130.81 124.46 0)
+    (property "Reference" "#PWR049" (id 0) (at 130.81 124.46 0)
       (effects (font (size 1.27 1.27)) hide)
     )
@@
   (symbol (lib_id "Device:R") (at 176.53 127 0) (unit 1)
     (in_bom yes) (on_board yes)
-    (property "Reference" "R40L1" (id 0) (at 178.308 125.8316 0)
+    (property "Reference" "R36" (id 0) (at 178.308 125.8316 0)
       (effects (font (size 1.27 1.27)) (justify left))
     )
@@
   (symbol (lib_id "power:GND") (at 176.53 130.81 0) (unit 1)
     (in_bom yes) (on_board yes)
-    (property "Reference" "#PWR0118" (id 0) (at 176.53 137.16 0)
+    (property "Reference" "#PWR053" (id 0) (at 176.53 137.16 0)
       (effects (font (size 1.27 1.27)) hide)
     )
@@
   (symbol (lib_id "power:GND") (at 130.81 135.89 0) (unit 1)
     (in_bom yes) (on_board yes)
-    (property "Reference" "#PWR0119" (id 0) (at 130.81 142.24 0)
+    (property "Reference" "#PWR050" (id 0) (at 130.81 142.24 0)
       (effects (font (size 1.27 1.27)) hide)
     )
@@
   (symbol (lib_id "Device:R") (at 186.69 134.62 270) (unit 1)
     (in_bom yes) (on_board yes)
-    (property "Reference" "R39L1" (id 0) (at 186.69 129.3622 90))
+    (property "Reference" "R37" (id 0) (at 186.69 129.3622 90))
     (property "Value" "10k" (id 1) (at 186.69 131.6736 90))
     (property "Footprint" "Resistor_SMD:R_0603_1608Metric" (id 2) (at 186.69 132.842 90)
@@
   (symbol (lib_id "Device:Opamp_Dual_Generic") (at 187.96 114.3 0) (unit 1)
     (in_bom yes) (on_board yes)
-    (property "Reference" "U14" (id 0) (at 187.96 107.315 0))
+    (property "Reference" "U4" (id 0) (at 187.96 107.315 0))
     (property "Value" "3PEAK TP09-SR" (id 1) (at 187.96 107.2896 0)
       (effects (font (size 1.27 1.27)) hide)
@@
   (symbol (lib_id "Device:Opamp_Dual_Generic") (at 133.35 128.27 0) (unit 3)
     (in_bom yes) (on_board yes)
-    (property "Reference" "U14" (id 0) (at 132.2832 127.1016 0)
-      (effects (font (size 1.27 1.27)) (justify left))
-    )
+    (property "Reference" "U4" (id 0) (at 132.2832 127.1016 0)
+      (effects (font (size 1.27 1.27)) (justify left))
+    )

Commit message: Updated Current sense circuit
Parts:
- removed C33: 100nF, Capacitor_SMD:C_0603_1608Metric, symbol Device:C
- removed R35: 220k, Resistor_SMD:R_0603_1608Metric, symbol Device:R
- added C32, C34, C35, C36, C37: 100nF, Capacitor_SMD:C_0603_1608Metric, symbol Device:C
- added D15, D16, D17, D18: 1N4148W, Diode_SMD:D_SOD-123, symbol Device:D
- added R30, R31, R38, R39, R40: 10k, Resistor_SMD:R_0603_1608Metric, symbol Device:R
- added U4: 3PEAK TP09-SR, Package_SO:SOIC-8_3.9x4.9mm_P1.27mm, symbol Device:Opamp_Dual_Generic
- R32: value 1k -> 10k; LCSC Part # C21190 -> C25804
- R34: value 10k -> 220k; LCSC Part # C25804 -> C22961
- R36: value 1k -> 100k; LCSC Part # C21190 -> (none)
- R37: value 10k -> 100k; LCSC Part # C25804 -> (none)
- renumbered C32 to C33, R31 to R35, R30 to R41, U4 to U5
Connections:
- net +3V3: now also R34.1, C36.2, C37.2, D15.1 (K), D16.1 (K), U4.8 (V+)
- net GND: now also R33.2, C32.2, C36.1, C37.1, D17.2 (A), D18.2 (A), R31.2, U4.4 (V-); no longer R32.2, R36.2
- net L_MTR_CURR: now also C34.2, U4.6 (-), U4.7; no longer R37.1, U5.1
- net L_MTR_SHUNT: now also R30.2; no longer R34.2
- net R_MTR_CURR: now also U5.6 (-), C35.2; no longer R33.1
- net R_MTR_SHUNT: now also R32.2; no longer R41.2
- net at C33.1, R41.1, U5.5 (+): no longer R35.2
- net at U5.3 (+): now also R32.1, R35.2, D16.2 (A); no longer R34.1
- new net: C35.1, R39.1, R41.2
- new net: D18.1 (K), R33.1, R37.1, U5.2 (-)
- new net: R37.2, R39.2, U5.1
- new net: D15.2 (A), R30.1, R34.2, U4.3 (+)
- new net: C32.1, R40.1, U4.5 (+)
- new net: C34.1, R38.1, R40.2
- new net: D17.1 (K), R31.1, R36.1, U4.2 (-)
- new net: R36.2, R38.2, U4.1
Other:
- note added: "route sense line directly to shunt insides both for shunt and gnd"
- moved on the sheet: C33, R33, R35, R41, U5A, U5B, U5C

Commit message: routed new diodes and opamp
Connections:
- net GND: no longer R31.2, R33.2
- new net -BATT: R31.2, R33.2
Changed lines of the file:
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@@
     (pin "7")
-  )
-  (symbol (lib_id "power:GND") (at 93.98 127 0) (unit 1)
-    (in_bom yes) (on_board yes)
-    (property "Reference" "#PWR047" (id 0) (at 93.98 133.35 0)
-      (effects (font (size 1.27 1.27)) hide)
-    )
-    (property "Value" "GND" (id 1) (at 94.107 131.3942 0))
-    (property "Footprint" "" (id 2) (at 93.98 127 0)
-      (effects (font (size 1.27 1.27)) hide)
-    )
-    (property "Datasheet" "" (id 3) (at 93.98 127 0)
-      (effects (font (size 1.27 1.27)) hide)
-    )
-    (pin "1")
   )
   (symbol (lib_id "Device:R") (at 105.41 127 270) (unit 1)
@@
     (pin "2")
   )
+  (symbol (lib_id "power:-BATT") (at 93.98 127 180) (unit 1)
+    (in_bom yes) (on_board yes)
+    (property "Reference" "#PWR?" (id 0) (at 93.98 123.19 0)
+      (effects (font (size 1.27 1.27)) hide)
+    )
+    (property "Value" "-BATT" (id 1) (at 93.599 131.3942 0))
+    (property "Footprint" "" (id 2) (at 93.98 127 0)
+      (effects (font (size 1.27 1.27)) hide)
+    )
+    (property "Datasheet" "" (id 3) (at 93.98 127 0)
+      (effects (font (size 1.27 1.27)) hide)
+    )
+    (pin "1")
+  )
   (symbol (lib_id "power:GND") (at 114.3 134.62 0) (unit 1)
     (in_bom yes) (on_board yes)
@@
     (pin "3")
   )
+  (symbol (lib_id "power:-BATT") (at 93.98 76.2 180) (unit 1)
+    (in_bom yes) (on_board yes)
+    (property "Reference" "#PWR?" (id 0) (at 93.98 72.39 0)
+      (effects (font (size 1.27 1.27)) hide)
+    )
+    (property "Value" "-BATT" (id 1) (at 93.599 80.5942 0))
+    (property "Footprint" "" (id 2) (at 93.98 76.2 0)
+      (effects (font (size 1.27 1.27)) hide)
+    )
+    (property "Datasheet" "" (id 3) (at 93.98 76.2 0)
+      (effects (font (size 1.27 1.27)) hide)
+    )
+    (pin "1")
+  )
   (symbol (lib_id "Device:Opamp_Dual_Generic") (at 185.42 76.2 0) (unit 2)
     (in_bom yes) (on_board yes)
@@
     (pin "2")
   )
-  (symbol (lib_id "power:GND") (at 93.98 76.2 0) (unit 1)
-    (in_bom yes) (on_board yes)
-    (property "Reference" "#PWR046" (id 0) (at 93.98 82.55 0)
-      (effects (font (size 1.27 1.27)) hide)
-    )
-    (property "Value" "GND" (id 1) (at 94.107 80.5942 0))
-    (property "Footprint" "" (id 2) (at 93.98 76.2 0)
-      (effects (font (size 1.27 1.27)) hide)
-    )
-    (property "Datasheet" "" (id 3) (at 93.98 76.2 0)
-      (effects (font (size 1.27 1.27)) hide)
-    )
-    (pin "1")
-  )
   (symbol (lib_id "Device:R") (at 127 137.16 90) (unit 1)

Commit message: Update a few library symbols
Parts:
- U4, U5: symbol Device:Opamp_Dual_Generic -> Device:Opamp_Dual
Changed lines of the file:
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@@
     (pin "1")
   )
-  (symbol (lib_id "Device:Opamp_Dual_Generic") (at 185.42 127 0) (unit 2)
+  (symbol (lib_id "Device:Opamp_Dual") (at 185.42 127 0) (unit 2)
     (in_bom yes) (on_board yes)
     (property "Reference" "U5" (id 0) (at 185.42 120.015 0))
@@
     (pin "1")
   )
-  (symbol (lib_id "Device:Opamp_Dual_Generic") (at 130.81 124.46 0) (unit 1)
+  (symbol (lib_id "Device:Opamp_Dual") (at 130.81 124.46 0) (unit 1)
     (in_bom yes) (on_board yes)
     (property "Reference" "U5" (id 0) (at 130.81 117.475 0))
@@
     (pin "8")
   )
-  (symbol (lib_id "Device:Opamp_Dual_Generic") (at 228.6 125.73 0) (unit 3)
+  (symbol (lib_id "Device:Opamp_Dual") (at 228.6 125.73 0) (unit 3)
     (in_bom yes) (on_board yes)
     (property "Reference" "U5" (id 0) (at 227.5332 124.5616 0)
@@
     (pin "1")
   )
-  (symbol (lib_id "Device:Opamp_Dual_Generic") (at 228.6 74.93 0) (unit 3)
+  (symbol (lib_id "Device:Opamp_Dual") (at 228.6 74.93 0) (unit 3)
     (in_bom yes) (on_board yes)
     (property "Reference" "U4" (id 0) (at 227.5332 73.7616 0)
@@
     (pin "1")
   )
-  (symbol (lib_id "Device:Opamp_Dual_Generic") (at 130.81 73.66 0) (unit 1)
+  (symbol (lib_id "Device:Opamp_Dual") (at 130.81 73.66 0) (unit 1)
     (in_bom yes) (on_board yes)
     (property "Reference" "U4" (id 0) (at 130.81 66.675 0))
@@
     (pin "1")
   )
-  (symbol (lib_id "Device:Opamp_Dual_Generic") (at 185.42 76.2 0) (unit 2)
+  (symbol (lib_id "Device:Opamp_Dual") (at 185.42 76.2 0) (unit 2)
     (in_bom yes) (on_board yes)
     (property "Reference" "U4" (id 0) (at 185.42 69.215 0))

Commit message: Updated diodes, added LCSC numbers for all parts
Parts:
- C32, C33, C34, C35, C36, C37: LCSC (none) -> C14663; LCSC Part # C14663 -> (none)
- D15, D16, D17, D18: LCSC (none) -> C81598; LCSC Part # C81598 -> (none)
- R30, R31, R32, R33, R38, R39, R40, R41: LCSC (none) -> C25804; LCSC Part # C25804 -> (none)
- R34, R35: LCSC (none) -> C22961; LCSC Part # C22961 -> (none)
- R36, R37: LCSC (none) -> C25803
- U4, U5: LCSC (none) -> C81662; LCSC Part # C81662 -> (none)
