File: CURRENT_SENSE.kicad_sch (KiCad schematic)
At the start: 24 parts, among them U4 3PEAK TP09-SR, U5 3PEAK TP09-SR

Commit message: update lcsc numbers
Parts:
- U4, U5: value 3PEAK TP09-SR -> TLV9362IDR; LCSC C81662 -> C4367884
