File: hh_bridge.kicad_sch (KiCad schematic)
At the start: 15 parts, among them U10 UCC27712

Commit message: add 0R resistor on BOOT0 against GND
Parts:
- renumbered C12 to C18, C13 to C24, C33 to C36, C66 to C69, D8 to D11, R16 to R33, R17 to R34, R60 to R69, R61 to R70, R68 to R76, R71 to R77, RV3 to RV6, U10 to U13, V4 to V10, V5 to V11
Changed lines of the file:
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@@
   (symbol (lib_id "Device:CP") (at 114.3 83.82 0)
     (in_bom yes) (on_board yes)
-    (property "Reference" "C13" (id 0) (at 117.2972 82.6516 0)
+    (property "Reference" "C24" (id 0) (at 117.2972 82.6516 0)
       (effects (font (size 1.27 1.27)) (justify left))
     )
@@
   (symbol (lib_id "Device:D") (at 109.22 63.5 180)
     (in_bom yes) (on_board yes)
-    (property "Reference" "D8" (id 0) (at 109.22 57.9882 0))
+    (property "Reference" "D11" (id 0) (at 109.22 57.9882 0))
     (property "Value" "1N4148W" (id 1) (at 109.22 60.2996 0))
     (property "Footprint" "Diode_SMD:D_SOD-123" (id 2) (at 109.22 63.5 0)
@@
   (symbol (lib_id "Transistor_FET:BSP89") (at 140.97 78.74 0)
     (in_bom yes) (on_board yes)
-    (property "Reference" "V4" (id 0) (at 146.1516 77.5716 0)
+    (property "Reference" "V10" (id 0) (at 146.1516 77.5716 0)
       (effects (font (size 1.27 1.27)) (justify left))
     )
@@
   (symbol (lib_id "Device:R") (at 132.08 91.44 270)
     (in_bom yes) (on_board yes)
-    (property "Reference" "R17" (id 0) (at 132.08 91.44 90))
+    (property "Reference" "R34" (id 0) (at 132.08 91.44 90))
     (property "Value" "4.7" (id 1) (at 130.81 88.9 90))
     (property "Footprint" "Resistor_SMD:R_1206_3216Metric" (id 2) (at 132.08 89.662 90)
@@
   (symbol (lib_id "Transistor_FET:BSP89") (at 140.97 91.44 0)
     (in_bom yes) (on_board yes)
-    (property "Reference" "V5" (id 0) (at 146.1516 90.2716 0)
+    (property "Reference" "V11" (id 0) (at 146.1516 90.2716 0)
       (effects (font (size 1.27 1.27)) (justify left))
     )
@@
   (symbol (lib_id "Device:R") (at 125.73 95.25 180)
     (in_bom yes) (on_board yes)
-    (property "Reference" "R61" (id 0) (at 123.9774 94.0816 0)
+    (property "Reference" "R70" (id 0) (at 123.9774 94.0816 0)
       (effects (font (size 1.27 1.27)) (justify left))
     )
@@
   (symbol (lib_id "Device:R") (at 123.19 83.82 180)
     (in_bom yes) (on_board yes)
-    (property "Reference" "R60" (id 0) (at 124.968 82.6516 0)
+    (property "Reference" "R69" (id 0) (at 124.968 82.6516 0)
       (effects (font (size 1.27 1.27)) (justify right))
     )
@@
   (symbol (lib_id "Driver_FET:IRS2304") (at 100.33 83.82 0)
     (in_bom yes) (on_board yes)
-    (property "Reference" "U10" (id 0) (at 100.33 66.5226 0))
+    (property "Reference" "U13" (id 0) (at 100.33 66.5226 0))
     (property "Value" "UCC27712" (id 1) (at 100.33 68.834 0))
     (property "Footprint" "Package_SO:SOIC-8_3.9x4.9mm_P1.27mm" (id 2) (at 100.33 83.82 0)
@@
   (symbol (lib_id "power:+VSW") (at 100.33 60.96 0)
     (in_bom yes) (on_board yes)
-    (property "Reference" "#PWR0179" (id 0) (at 100.33 64.77 0)
+    (property "Reference" "#PWR0191" (id 0) (at 100.33 64.77 0)
       (effects (font (size 1.27 1.27)) hide)
     )
@@
   (symbol (lib_id "Device:CP") (at 88.9 100.33 0)
     (in_bom yes) (on_board yes)
-    (property "Reference" "C12" (id 0) (at 85.9028 99.1616 0)
+    (property "Reference" "C18" (id 0) (at 85.9028 99.1616 0)
       (effects (font (size 1.27 1.27)) (justify right))
     )
@@
   (symbol (lib_id "power:+VSW") (at 88.9 95.25 0)
     (in_bom yes) (on_board yes)
-    (property "Reference" "#PWR0180" (id 0) (at 88.9 99.06 0)
+    (property "Reference" "#PWR0192" (id 0) (at 88.9 99.06 0)
       (effects (font (size 1.27 1.27)) hide)
     )
@@
   (symbol (lib_id "power:GND") (at 97.79 105.41 0)
     (in_bom yes) (on_board yes)
-    (property "Reference" "#PWR0181" (id 0) (at 97.79 111.76 0)
+    (property "Reference" "#PWR0193" (id 0) (at 97.79 111.76 0)
       (effects (font (size 1.27 1.27)) hide)
     )
@@
   (symbol (lib_id "Device:R") (at 132.08 78.74 270)
     (in_bom yes) (on_board yes)
-    (property "Reference" "R16" (id 0) (at 132.08 78.74 90))
+    (property "Reference" "R33" (id 0) (at 132.08 78.74 90))
     (property "Value" "4.7" (id 1) (at 132.08 75.7936 90))
     (property "Footprint" "Resistor_SMD:R_1206_3216Metric" (id 2) (at 132.08 76.962 90)
@@
   (symbol (lib_id "Device:C") (at 171.45 76.2 0)
     (in_bom yes) (on_board yes)
-    (property "Reference" "C66" (id 0) (at 168.529 75.0316 0)
+    (property "Reference" "C69" (id 0) (at 168.529 75.0316 0)
       (effects (font (size 1.27 1.27)) (justify right))
     )
@@
   (symbol (lib_id "power:+BATT") (at 143.51 71.12 0)
     (in_bom yes) (on_board yes)
-    (property "Reference" "#PWR0182" (id 0) (at 143.51 74.93 0)
+    (property "Reference" "#PWR0194" (id 0) (at 143.51 74.93 0)
       (effects (font (size 1.27 1.27)) hide)
     )
@@
   (symbol (lib_id "Device:R") (at 88.9 83.82 270)
     (in_bom yes) (on_board yes)
-    (property "Reference" "R68" (id 0) (at 88.9 76.2762 90))
+    (property "Reference" "R76" (id 0) (at 88.9 76.2762 90))
     (property "Value" "1k" (id 1) (at 88.9 78.5876 90))
     (property "Footprint" "Resistor_SMD:R_0603_1608Metric" (id 2) (at 68.58 77.47 90)
@@
   (symbol (lib_id "Device:R") (at 88.9 86.36 270)
     (in_bom yes) (on_board yes)
-    (property "Reference" "R71" (id 0) (at 88.9 81.1022 90))
+    (property "Reference" "R77" (id 0) (at 88.9 81.1022 90))
     (property "Value" "1k" (id 1) (at 88.9 83.4136 90))
     (property "Footprint" "Resistor_SMD:R_0603_1608Metric" (id 2) (at 88.9 84.582 90)
@@
   (symbol (lib_id "Device:CP") (at 180.34 76.2 0)
     (in_bom yes) (on_board yes)
-    (property "Reference" "C33" (id 0) (at 183.3372 75.0316 0)
+    (property "Reference" "C36" (id 0) (at 183.3372 75.0316 0)
       (effects (font (size 1.27 1.27)) (justify left))
     )
@@
   (symbol (lib_id "power:+BATT") (at 180.34 71.12 0)
     (in_bom yes) (on_board yes)
-    (property "Reference" "#PWR0199" (id 0) (at 180.34 74.93 0)
+    (property "Reference" "#PWR0202" (id 0) (at 180.34 74.93 0)
       (effects (font (size 1.27 1.27)) hide)
     )
@@
   (symbol (lib_id "Device:Varistor") (at 208.28 76.2 0)
     (in_bom yes) (on_board yes)
-    (property "Reference" "RV3" (id 0) (at 210.8962 75.0316 0)
-      (effects (font (size 1.27 1.27)) (justify left))
-    )
+    (property "Reference" "RV6" (id 0) (at 210.8962 75.0316 0)
+      (effects (font (size 1.27 1.27)) (justify left))
+    )

Commit message: removed faulty vias and connections
Parts:
- renumbered C18 to C14, C24 to C15, C36 to C34, C69 to C67, D11 to D9, R33 to R18, R34 to R21, R69 to R63, R70 to R64, R76 to R72, R77 to R73, RV6 to RV4, U13 to U11, V10 to V6, V11 to V7
Changed lines of the file:
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@@
   (symbol (lib_id "Device:CP") (at 114.3 83.82 0)
     (in_bom yes) (on_board yes)
-    (property "Reference" "C24" (id 0) (at 117.2972 82.6516 0)
+    (property "Reference" "C15" (id 0) (at 117.2972 82.6516 0)
       (effects (font (size 1.27 1.27)) (justify left))
     )
@@
   (symbol (lib_id "Device:D") (at 109.22 63.5 180)
     (in_bom yes) (on_board yes)
-    (property "Reference" "D11" (id 0) (at 109.22 57.9882 0))
+    (property "Reference" "D9" (id 0) (at 109.22 57.9882 0))
     (property "Value" "1N4148W" (id 1) (at 109.22 60.2996 0))
     (property "Footprint" "Diode_SMD:D_SOD-123" (id 2) (at 109.22 63.5 0)
@@
   (symbol (lib_id "Transistor_FET:BSP89") (at 140.97 78.74 0)
     (in_bom yes) (on_board yes)
-    (property "Reference" "V10" (id 0) (at 146.1516 77.5716 0)
+    (property "Reference" "V6" (id 0) (at 146.1516 77.5716 0)
       (effects (font (size 1.27 1.27)) (justify left))
     )
@@
   (symbol (lib_id "Device:R") (at 132.08 91.44 270)
     (in_bom yes) (on_board yes)
-    (property "Reference" "R34" (id 0) (at 132.08 91.44 90))
+    (property "Reference" "R21" (id 0) (at 132.08 91.44 90))
     (property "Value" "4.7" (id 1) (at 130.81 88.9 90))
     (property "Footprint" "Resistor_SMD:R_1206_3216Metric" (id 2) (at 132.08 89.662 90)
@@
   (symbol (lib_id "Transistor_FET:BSP89") (at 140.97 91.44 0)
     (in_bom yes) (on_board yes)
-    (property "Reference" "V11" (id 0) (at 146.1516 90.2716 0)
+    (property "Reference" "V7" (id 0) (at 146.1516 90.2716 0)
       (effects (font (size 1.27 1.27)) (justify left))
     )
@@
   (symbol (lib_id "Device:R") (at 125.73 95.25 180)
     (in_bom yes) (on_board yes)
-    (property "Reference" "R70" (id 0) (at 123.9774 94.0816 0)
+    (property "Reference" "R64" (id 0) (at 123.9774 94.0816 0)
       (effects (font (size 1.27 1.27)) (justify left))
     )
@@
   (symbol (lib_id "Device:R") (at 123.19 83.82 180)
     (in_bom yes) (on_board yes)
-    (property "Reference" "R69" (id 0) (at 124.968 82.6516 0)
+    (property "Reference" "R63" (id 0) (at 124.968 82.6516 0)
       (effects (font (size 1.27 1.27)) (justify right))
     )
@@
   (symbol (lib_id "Driver_FET:IRS2304") (at 100.33 83.82 0)
     (in_bom yes) (on_board yes)
-    (property "Reference" "U13" (id 0) (at 100.33 66.5226 0))
+    (property "Reference" "U11" (id 0) (at 100.33 66.5226 0))
     (property "Value" "UCC27712" (id 1) (at 100.33 68.834 0))
     (property "Footprint" "Package_SO:SOIC-8_3.9x4.9mm_P1.27mm" (id 2) (at 100.33 83.82 0)
@@
   (symbol (lib_id "power:+VSW") (at 100.33 60.96 0)
     (in_bom yes) (on_board yes)
-    (property "Reference" "#PWR0191" (id 0) (at 100.33 64.77 0)
+    (property "Reference" "#PWR0183" (id 0) (at 100.33 64.77 0)
       (effects (font (size 1.27 1.27)) hide)
     )
@@
   (symbol (lib_id "Device:CP") (at 88.9 100.33 0)
     (in_bom yes) (on_board yes)
-    (property "Reference" "C18" (id 0) (at 85.9028 99.1616 0)
+    (property "Reference" "C14" (id 0) (at 85.9028 99.1616 0)
       (effects (font (size 1.27 1.27)) (justify right))
     )
@@
   (symbol (lib_id "power:+VSW") (at 88.9 95.25 0)
     (in_bom yes) (on_board yes)
-    (property "Reference" "#PWR0192" (id 0) (at 88.9 99.06 0)
+    (property "Reference" "#PWR0184" (id 0) (at 88.9 99.06 0)
       (effects (font (size 1.27 1.27)) hide)
     )
@@
   (symbol (lib_id "power:GND") (at 97.79 105.41 0)
     (in_bom yes) (on_board yes)
-    (property "Reference" "#PWR0193" (id 0) (at 97.79 111.76 0)
+    (property "Reference" "#PWR0185" (id 0) (at 97.79 111.76 0)
       (effects (font (size 1.27 1.27)) hide)
     )
@@
   (symbol (lib_id "Device:R") (at 132.08 78.74 270)
     (in_bom yes) (on_board yes)
-    (property "Reference" "R33" (id 0) (at 132.08 78.74 90))
+    (property "Reference" "R18" (id 0) (at 132.08 78.74 90))
     (property "Value" "4.7" (id 1) (at 132.08 75.7936 90))
     (property "Footprint" "Resistor_SMD:R_1206_3216Metric" (id 2) (at 132.08 76.962 90)
@@
   (symbol (lib_id "Device:C") (at 171.45 76.2 0)
     (in_bom yes) (on_board yes)
-    (property "Reference" "C69" (id 0) (at 168.529 75.0316 0)
+    (property "Reference" "C67" (id 0) (at 168.529 75.0316 0)
       (effects (font (size 1.27 1.27)) (justify right))
     )
@@
   (symbol (lib_id "power:+BATT") (at 143.51 71.12 0)
     (in_bom yes) (on_board yes)
-    (property "Reference" "#PWR0194" (id 0) (at 143.51 74.93 0)
+    (property "Reference" "#PWR0186" (id 0) (at 143.51 74.93 0)
       (effects (font (size 1.27 1.27)) hide)
     )
@@
   (symbol (lib_id "Device:R") (at 88.9 83.82 270)
     (in_bom yes) (on_board yes)
-    (property "Reference" "R76" (id 0) (at 88.9 76.2762 90))
+    (property "Reference" "R72" (id 0) (at 88.9 76.2762 90))
     (property "Value" "1k" (id 1) (at 88.9 78.5876 90))
     (property "Footprint" "Resistor_SMD:R_0603_1608Metric" (id 2) (at 68.58 77.47 90)
@@
   (symbol (lib_id "Device:R") (at 88.9 86.36 270)
     (in_bom yes) (on_board yes)
-    (property "Reference" "R77" (id 0) (at 88.9 81.1022 90))
+    (property "Reference" "R73" (id 0) (at 88.9 81.1022 90))
     (property "Value" "1k" (id 1) (at 88.9 83.4136 90))
     (property "Footprint" "Resistor_SMD:R_0603_1608Metric" (id 2) (at 88.9 84.582 90)
@@
   (symbol (lib_id "Device:CP") (at 180.34 76.2 0)
     (in_bom yes) (on_board yes)
-    (property "Reference" "C36" (id 0) (at 183.3372 75.0316 0)
+    (property "Reference" "C34" (id 0) (at 183.3372 75.0316 0)
       (effects (font (size 1.27 1.27)) (justify left))
     )
@@
   (symbol (lib_id "power:+BATT") (at 180.34 71.12 0)
     (in_bom yes) (on_board yes)
-    (property "Reference" "#PWR0202" (id 0) (at 180.34 74.93 0)
+    (property "Reference" "#PWR0200" (id 0) (at 180.34 74.93 0)
       (effects (font (size 1.27 1.27)) hide)
     )
@@
   (symbol (lib_id "Device:Varistor") (at 208.28 76.2 0)
     (in_bom yes) (on_board yes)
-    (property "Reference" "RV6" (id 0) (at 210.8962 75.0316 0)
-      (effects (font (size 1.27 1.27)) (justify left))
-    )
+    (property "Reference" "RV4" (id 0) (at 210.8962 75.0316 0)
+      (effects (font (size 1.27 1.27)) (justify left))
+    )

Commit message: Silkscreen and naming fixes
Parts:
- renumbered C14 to C42, C15 to C43, C67 to C44, C34 to C45, D9 to D17, R72 to R50, R73 to R51, R63 to R52, R64 to R53, R18 to R54, R21 to R55, RV4 to RV3, U11 to U7, V6 to V5, V7 to V6
Changed lines of the file:
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@@
   (symbol (lib_id "Device:CP") (at 114.3 83.82 0)
     (in_bom yes) (on_board yes)
-    (property "Reference" "C15" (id 0) (at 117.2972 82.6516 0)
+    (property "Reference" "C43" (id 0) (at 117.2972 82.6516 0)
       (effects (font (size 1.27 1.27)) (justify left))
     )
@@
   (symbol (lib_id "Device:D") (at 109.22 63.5 180)
     (in_bom yes) (on_board yes)
-    (property "Reference" "D9" (id 0) (at 109.22 57.9882 0))
+    (property "Reference" "D17" (id 0) (at 109.22 57.9882 0))
     (property "Value" "1N4148W" (id 1) (at 109.22 60.2996 0))
     (property "Footprint" "Diode_SMD:D_SOD-123" (id 2) (at 109.22 63.5 0)
@@
   (symbol (lib_id "Transistor_FET:BSP89") (at 140.97 78.74 0)
     (in_bom yes) (on_board yes)
-    (property "Reference" "V6" (id 0) (at 146.1516 77.5716 0)
+    (property "Reference" "V5" (id 0) (at 146.1516 77.5716 0)
       (effects (font (size 1.27 1.27)) (justify left))
     )
@@
   (symbol (lib_id "Device:R") (at 132.08 91.44 270)
     (in_bom yes) (on_board yes)
-    (property "Reference" "R21" (id 0) (at 132.08 91.44 90))
+    (property "Reference" "R55" (id 0) (at 132.08 91.44 90))
     (property "Value" "4.7" (id 1) (at 130.81 88.9 90))
     (property "Footprint" "Resistor_SMD:R_1206_3216Metric" (id 2) (at 132.08 89.662 90)
@@
   (symbol (lib_id "Transistor_FET:BSP89") (at 140.97 91.44 0)
     (in_bom yes) (on_board yes)
-    (property "Reference" "V7" (id 0) (at 146.1516 90.2716 0)
+    (property "Reference" "V6" (id 0) (at 146.1516 90.2716 0)
       (effects (font (size 1.27 1.27)) (justify left))
     )
@@
   (symbol (lib_id "Device:R") (at 125.73 95.25 180)
     (in_bom yes) (on_board yes)
-    (property "Reference" "R64" (id 0) (at 123.9774 94.0816 0)
+    (property "Reference" "R53" (id 0) (at 123.9774 94.0816 0)
       (effects (font (size 1.27 1.27)) (justify left))
     )
@@
   (symbol (lib_id "Device:R") (at 123.19 83.82 180)
     (in_bom yes) (on_board yes)
-    (property "Reference" "R63" (id 0) (at 124.968 82.6516 0)
+    (property "Reference" "R52" (id 0) (at 124.968 82.6516 0)
       (effects (font (size 1.27 1.27)) (justify right))
     )
@@
   (symbol (lib_id "Driver_FET:IRS2304") (at 100.33 83.82 0)
     (in_bom yes) (on_board yes)
-    (property "Reference" "U11" (id 0) (at 100.33 66.5226 0))
+    (property "Reference" "U7" (id 0) (at 100.33 66.5226 0))
     (property "Value" "UCC27712" (id 1) (at 100.33 68.834 0))
     (property "Footprint" "Package_SO:SOIC-8_3.9x4.9mm_P1.27mm" (id 2) (at 100.33 83.82 0)
@@
   (symbol (lib_id "power:+VSW") (at 100.33 60.96 0)
     (in_bom yes) (on_board yes)
-    (property "Reference" "#PWR0183" (id 0) (at 100.33 64.77 0)
+    (property "Reference" "#PWR066" (id 0) (at 100.33 64.77 0)
       (effects (font (size 1.27 1.27)) hide)
     )
@@
   (symbol (lib_id "Device:CP") (at 88.9 100.33 0)
     (in_bom yes) (on_board yes)
-    (property "Reference" "C14" (id 0) (at 85.9028 99.1616 0)
+    (property "Reference" "C42" (id 0) (at 85.9028 99.1616 0)
       (effects (font (size 1.27 1.27)) (justify right))
     )
@@
   (symbol (lib_id "power:+VSW") (at 88.9 95.25 0)
     (in_bom yes) (on_board yes)
-    (property "Reference" "#PWR0184" (id 0) (at 88.9 99.06 0)
+    (property "Reference" "#PWR064" (id 0) (at 88.9 99.06 0)
       (effects (font (size 1.27 1.27)) hide)
     )
@@
   (symbol (lib_id "power:GND") (at 97.79 105.41 0)
     (in_bom yes) (on_board yes)
-    (property "Reference" "#PWR0185" (id 0) (at 97.79 111.76 0)
+    (property "Reference" "#PWR065" (id 0) (at 97.79 111.76 0)
       (effects (font (size 1.27 1.27)) hide)
     )
@@
   (symbol (lib_id "Device:R") (at 132.08 78.74 270)
     (in_bom yes) (on_board yes)
-    (property "Reference" "R18" (id 0) (at 132.08 78.74 90))
+    (property "Reference" "R54" (id 0) (at 132.08 78.74 90))
     (property "Value" "4.7" (id 1) (at 132.08 75.7936 90))
     (property "Footprint" "Resistor_SMD:R_1206_3216Metric" (id 2) (at 132.08 76.962 90)
@@
   (symbol (lib_id "Device:C") (at 171.45 76.2 0)
     (in_bom yes) (on_board yes)
-    (property "Reference" "C67" (id 0) (at 168.529 75.0316 0)
+    (property "Reference" "C44" (id 0) (at 168.529 75.0316 0)
       (effects (font (size 1.27 1.27)) (justify right))
     )
@@
   (symbol (lib_id "power:+BATT") (at 143.51 71.12 0)
     (in_bom yes) (on_board yes)
-    (property "Reference" "#PWR0186" (id 0) (at 143.51 74.93 0)
+    (property "Reference" "#PWR067" (id 0) (at 143.51 74.93 0)
       (effects (font (size 1.27 1.27)) hide)
     )
@@
   (symbol (lib_id "Device:R") (at 88.9 83.82 270)
     (in_bom yes) (on_board yes)
-    (property "Reference" "R72" (id 0) (at 88.9 76.2762 90))
+    (property "Reference" "R50" (id 0) (at 88.9 76.2762 90))
     (property "Value" "1k" (id 1) (at 88.9 78.5876 90))
     (property "Footprint" "Resistor_SMD:R_0603_1608Metric" (id 2) (at 68.58 77.47 90)
@@
   (symbol (lib_id "Device:R") (at 88.9 86.36 270)
     (in_bom yes) (on_board yes)
-    (property "Reference" "R73" (id 0) (at 88.9 81.1022 90))
+    (property "Reference" "R51" (id 0) (at 88.9 81.1022 90))
     (property "Value" "1k" (id 1) (at 88.9 83.4136 90))
     (property "Footprint" "Resistor_SMD:R_0603_1608Metric" (id 2) (at 88.9 84.582 90)
@@
   (symbol (lib_id "Device:CP") (at 180.34 76.2 0)
     (in_bom yes) (on_board yes)
-    (property "Reference" "C34" (id 0) (at 183.3372 75.0316 0)
+    (property "Reference" "C45" (id 0) (at 183.3372 75.0316 0)
       (effects (font (size 1.27 1.27)) (justify left))
     )
@@
   (symbol (lib_id "power:+BATT") (at 180.34 71.12 0)
     (in_bom yes) (on_board yes)
-    (property "Reference" "#PWR0200" (id 0) (at 180.34 74.93 0)
+    (property "Reference" "#PWR068" (id 0) (at 180.34 74.93 0)
       (effects (font (size 1.27 1.27)) hide)
     )
@@
   (symbol (lib_id "Device:Varistor") (at 208.28 76.2 0)
     (in_bom yes) (on_board yes)
-    (property "Reference" "RV4" (id 0) (at 210.8962 75.0316 0)
-      (effects (font (size 1.27 1.27)) (justify left))
-    )
+    (property "Reference" "RV3" (id 0) (at 210.8962 75.0316 0)
+      (effects (font (size 1.27 1.27)) (justify left))
+    )
