File: hh_bridge.kicad_sch (KiCad schematic)
At the start: 15 parts, among them U7 UCC27712

Commit message: Updated Current sense circuit
Parts:
- renumbered C42 to C70, C43 to C71, C44 to C72, C45 to C73, D17 to D34, R50 to R93, R51 to R94, R52 to R95, R53 to R96, R54 to R97, R55 to R98, RV3 to RV6, U7 to U14, V5 to V12, V6 to V13
Changed lines of the file:
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@@
   (symbol (lib_id "Device:CP") (at 114.3 83.82 0)
     (in_bom yes) (on_board yes)
-    (property "Reference" "C43" (id 0) (at 117.2972 82.6516 0)
+    (property "Reference" "C71" (id 0) (at 117.2972 82.6516 0)
       (effects (font (size 1.27 1.27)) (justify left))
     )
@@
   (symbol (lib_id "Device:D") (at 109.22 63.5 180)
     (in_bom yes) (on_board yes)
-    (property "Reference" "D17" (id 0) (at 109.22 57.9882 0))
+    (property "Reference" "D34" (id 0) (at 109.22 57.9882 0))
     (property "Value" "1N4148W" (id 1) (at 109.22 60.2996 0))
     (property "Footprint" "Diode_SMD:D_SOD-123" (id 2) (at 109.22 63.5 0)
@@
   (symbol (lib_id "Transistor_FET:BSP89") (at 140.97 78.74 0)
     (in_bom yes) (on_board yes)
-    (property "Reference" "V5" (id 0) (at 146.1516 77.5716 0)
+    (property "Reference" "V12" (id 0) (at 146.1516 77.5716 0)
       (effects (font (size 1.27 1.27)) (justify left))
     )
@@
   (symbol (lib_id "Device:R") (at 132.08 91.44 270)
     (in_bom yes) (on_board yes)
-    (property "Reference" "R55" (id 0) (at 132.08 91.44 90))
+    (property "Reference" "R98" (id 0) (at 132.08 91.44 90))
     (property "Value" "4.7" (id 1) (at 130.81 88.9 90))
     (property "Footprint" "Resistor_SMD:R_1206_3216Metric" (id 2) (at 132.08 89.662 90)
@@
   (symbol (lib_id "Transistor_FET:BSP89") (at 140.97 91.44 0)
     (in_bom yes) (on_board yes)
-    (property "Reference" "V6" (id 0) (at 146.1516 90.2716 0)
+    (property "Reference" "V13" (id 0) (at 146.1516 90.2716 0)
       (effects (font (size 1.27 1.27)) (justify left))
     )
@@
   (symbol (lib_id "Device:R") (at 125.73 95.25 180)
     (in_bom yes) (on_board yes)
-    (property "Reference" "R53" (id 0) (at 123.9774 94.0816 0)
+    (property "Reference" "R96" (id 0) (at 123.9774 94.0816 0)
       (effects (font (size 1.27 1.27)) (justify left))
     )
@@
   (symbol (lib_id "Device:R") (at 123.19 83.82 180)
     (in_bom yes) (on_board yes)
-    (property "Reference" "R52" (id 0) (at 124.968 82.6516 0)
+    (property "Reference" "R95" (id 0) (at 124.968 82.6516 0)
       (effects (font (size 1.27 1.27)) (justify right))
     )
@@
   (symbol (lib_id "Driver_FET:IRS2304") (at 100.33 83.82 0)
     (in_bom yes) (on_board yes)
-    (property "Reference" "U7" (id 0) (at 100.33 66.5226 0))
+    (property "Reference" "U14" (id 0) (at 100.33 66.5226 0))
     (property "Value" "UCC27712" (id 1) (at 100.33 68.834 0))
     (property "Footprint" "Package_SO:SOIC-8_3.9x4.9mm_P1.27mm" (id 2) (at 100.33 83.82 0)
@@
   (symbol (lib_id "power:+VSW") (at 100.33 60.96 0)
     (in_bom yes) (on_board yes)
-    (property "Reference" "#PWR066" (id 0) (at 100.33 64.77 0)
+    (property "Reference" "#PWR0134" (id 0) (at 100.33 64.77 0)
       (effects (font (size 1.27 1.27)) hide)
     )
@@
   (symbol (lib_id "Device:CP") (at 88.9 100.33 0)
     (in_bom yes) (on_board yes)
-    (property "Reference" "C42" (id 0) (at 85.9028 99.1616 0)
+    (property "Reference" "C70" (id 0) (at 85.9028 99.1616 0)
       (effects (font (size 1.27 1.27)) (justify right))
     )
@@
   (symbol (lib_id "power:+VSW") (at 88.9 95.25 0)
     (in_bom yes) (on_board yes)
-    (property "Reference" "#PWR064" (id 0) (at 88.9 99.06 0)
+    (property "Reference" "#PWR0132" (id 0) (at 88.9 99.06 0)
       (effects (font (size 1.27 1.27)) hide)
     )
@@
   (symbol (lib_id "power:GND") (at 97.79 105.41 0)
     (in_bom yes) (on_board yes)
-    (property "Reference" "#PWR065" (id 0) (at 97.79 111.76 0)
+    (property "Reference" "#PWR0133" (id 0) (at 97.79 111.76 0)
       (effects (font (size 1.27 1.27)) hide)
     )
@@
   (symbol (lib_id "Device:R") (at 132.08 78.74 270)
     (in_bom yes) (on_board yes)
-    (property "Reference" "R54" (id 0) (at 132.08 78.74 90))
+    (property "Reference" "R97" (id 0) (at 132.08 78.74 90))
     (property "Value" "4.7" (id 1) (at 132.08 75.7936 90))
     (property "Footprint" "Resistor_SMD:R_1206_3216Metric" (id 2) (at 132.08 76.962 90)
@@
   (symbol (lib_id "Device:C") (at 171.45 76.2 0)
     (in_bom yes) (on_board yes)
-    (property "Reference" "C44" (id 0) (at 168.529 75.0316 0)
+    (property "Reference" "C72" (id 0) (at 168.529 75.0316 0)
       (effects (font (size 1.27 1.27)) (justify right))
     )
@@
   (symbol (lib_id "power:+BATT") (at 143.51 71.12 0)
     (in_bom yes) (on_board yes)
-    (property "Reference" "#PWR067" (id 0) (at 143.51 74.93 0)
+    (property "Reference" "#PWR0135" (id 0) (at 143.51 74.93 0)
       (effects (font (size 1.27 1.27)) hide)
     )
@@
   (symbol (lib_id "Device:R") (at 88.9 83.82 270)
     (in_bom yes) (on_board yes)
-    (property "Reference" "R50" (id 0) (at 88.9 76.2762 90))
+    (property "Reference" "R93" (id 0) (at 88.9 76.2762 90))
     (property "Value" "1k" (id 1) (at 88.9 78.5876 90))
     (property "Footprint" "Resistor_SMD:R_0603_1608Metric" (id 2) (at 68.58 77.47 90)
@@
   (symbol (lib_id "Device:R") (at 88.9 86.36 270)
     (in_bom yes) (on_board yes)
-    (property "Reference" "R51" (id 0) (at 88.9 81.1022 90))
+    (property "Reference" "R94" (id 0) (at 88.9 81.1022 90))
     (property "Value" "1k" (id 1) (at 88.9 83.4136 90))
     (property "Footprint" "Resistor_SMD:R_0603_1608Metric" (id 2) (at 88.9 84.582 90)
@@
   (symbol (lib_id "Device:CP") (at 180.34 76.2 0)
     (in_bom yes) (on_board yes)
-    (property "Reference" "C45" (id 0) (at 183.3372 75.0316 0)
+    (property "Reference" "C73" (id 0) (at 183.3372 75.0316 0)
       (effects (font (size 1.27 1.27)) (justify left))
     )
@@
   (symbol (lib_id "power:+BATT") (at 180.34 71.12 0)
     (in_bom yes) (on_board yes)
-    (property "Reference" "#PWR068" (id 0) (at 180.34 74.93 0)
+    (property "Reference" "#PWR0136" (id 0) (at 180.34 74.93 0)
       (effects (font (size 1.27 1.27)) hide)
     )
@@
   (symbol (lib_id "Device:Varistor") (at 208.28 76.2 0)
     (in_bom yes) (on_board yes)
-    (property "Reference" "RV3" (id 0) (at 210.8962 75.0316 0)
-      (effects (font (size 1.27 1.27)) (justify left))
-    )
+    (property "Reference" "RV6" (id 0) (at 210.8962 75.0316 0)
+      (effects (font (size 1.27 1.27)) (justify left))
+    )

Commit message: Refactor stuff adjacent to hall sensor pins
Parts:
- renumbered C70 to C38, C71 to C39, C72 to C40, C73 to C41, D34 to D19, R93 to R42, R94 to R43, R95 to R44, R96 to R45, R97 to R46, R98 to R47, RV6 to RV1, U14 to U6, V12 to V1, V13 to V2
Changed lines of the file:
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@@
     (effects (font (size 1.27 1.27)) (justify left))
   )
-  (symbol (lib_id "Device:CP") (at 114.3 83.82 0)
-    (in_bom yes) (on_board yes)
-    (property "Reference" "C71" (id 0) (at 117.2972 82.6516 0)
+  (symbol (lib_id "Device:CP") (at 114.3 83.82 0) (unit 1)
+    (in_bom yes) (on_board yes)
+    (property "Reference" "C39" (id 0) (at 117.2972 82.6516 0)
       (effects (font (size 1.27 1.27)) (justify left))
     )
@@
     (pin "2")
   )
-  (symbol (lib_id "Device:D") (at 109.22 63.5 180)
-    (in_bom yes) (on_board yes)
-    (property "Reference" "D34" (id 0) (at 109.22 57.9882 0))
+  (symbol (lib_id "Device:D") (at 109.22 63.5 180) (unit 1)
+    (in_bom yes) (on_board yes)
+    (property "Reference" "D19" (id 0) (at 109.22 57.9882 0))
     (property "Value" "1N4148W" (id 1) (at 109.22 60.2996 0))
     (property "Footprint" "Diode_SMD:D_SOD-123" (id 2) (at 109.22 63.5 0)
@@
     (pin "2")
   )
-  (symbol (lib_id "Transistor_FET:BSP89") (at 140.97 78.74 0)
-    (in_bom yes) (on_board yes)
-    (property "Reference" "V12" (id 0) (at 146.1516 77.5716 0)
+  (symbol (lib_id "Transistor_FET:BSP89") (at 140.97 78.74 0) (unit 1)
+    (in_bom yes) (on_board yes)
+    (property "Reference" "V1" (id 0) (at 146.1516 77.5716 0)
       (effects (font (size 1.27 1.27)) (justify left))
     )
@@
     (pin "3")
   )
-  (symbol (lib_id "Device:R") (at 132.08 91.44 270)
-    (in_bom yes) (on_board yes)
-    (property "Reference" "R98" (id 0) (at 132.08 91.44 90))
+  (symbol (lib_id "Device:R") (at 132.08 91.44 270) (unit 1)
+    (in_bom yes) (on_board yes)
+    (property "Reference" "R47" (id 0) (at 132.08 91.44 90))
     (property "Value" "4.7" (id 1) (at 130.81 88.9 90))
     (property "Footprint" "Resistor_SMD:R_1206_3216Metric" (id 2) (at 132.08 89.662 90)
@@
     (pin "2")
   )
-  (symbol (lib_id "Transistor_FET:BSP89") (at 140.97 91.44 0)
-    (in_bom yes) (on_board yes)
-    (property "Reference" "V13" (id 0) (at 146.1516 90.2716 0)
+  (symbol (lib_id "Transistor_FET:BSP89") (at 140.97 91.44 0) (unit 1)
+    (in_bom yes) (on_board yes)
+    (property "Reference" "V2" (id 0) (at 146.1516 90.2716 0)
       (effects (font (size 1.27 1.27)) (justify left))
     )
@@
     (pin "3")
   )
-  (symbol (lib_id "Device:R") (at 125.73 95.25 180)
-    (in_bom yes) (on_board yes)
-    (property "Reference" "R96" (id 0) (at 123.9774 94.0816 0)
+  (symbol (lib_id "Device:R") (at 125.73 95.25 180) (unit 1)
+    (in_bom yes) (on_board yes)
+    (property "Reference" "R45" (id 0) (at 123.9774 94.0816 0)
       (effects (font (size 1.27 1.27)) (justify left))
     )
@@
     (pin "2")
   )
-  (symbol (lib_id "Device:R") (at 123.19 83.82 180)
-    (in_bom yes) (on_board yes)
-    (property "Reference" "R95" (id 0) (at 124.968 82.6516 0)
+  (symbol (lib_id "Device:R") (at 123.19 83.82 180) (unit 1)
+    (in_bom yes) (on_board yes)
+    (property "Reference" "R44" (id 0) (at 124.968 82.6516 0)
       (effects (font (size 1.27 1.27)) (justify right))
     )
@@
     (pin "2")
   )
-  (symbol (lib_id "Driver_FET:IRS2304") (at 100.33 83.82 0)
-    (in_bom yes) (on_board yes)
-    (property "Reference" "U14" (id 0) (at 100.33 66.5226 0))
+  (symbol (lib_id "Driver_FET:IRS2304") (at 100.33 83.82 0) (unit 1)
+    (in_bom yes) (on_board yes)
+    (property "Reference" "U6" (id 0) (at 100.33 66.5226 0))
     (property "Value" "UCC27712" (id 1) (at 100.33 68.834 0))
     (property "Footprint" "Package_SO:SOIC-8_3.9x4.9mm_P1.27mm" (id 2) (at 100.33 83.82 0)
@@
     (pin "8")
   )
-  (symbol (lib_id "power:+VSW") (at 100.33 60.96 0)
-    (in_bom yes) (on_board yes)
-    (property "Reference" "#PWR0134" (id 0) (at 100.33 64.77 0)
+  (symbol (lib_id "power:+VSW") (at 100.33 60.96 0) (unit 1)
+    (in_bom yes) (on_board yes)
+    (property "Reference" "#PWR062" (id 0) (at 100.33 64.77 0)
       (effects (font (size 1.27 1.27)) hide)
     )
@@
     (pin "1")
   )
-  (symbol (lib_id "Device:CP") (at 88.9 100.33 0)
-    (in_bom yes) (on_board yes)
-    (property "Reference" "C70" (id 0) (at 85.9028 99.1616 0)
+  (symbol (lib_id "Device:CP") (at 88.9 100.33 0) (unit 1)
+    (in_bom yes) (on_board yes)
+    (property "Reference" "C38" (id 0) (at 85.9028 99.1616 0)
       (effects (font (size 1.27 1.27)) (justify right))
     )
@@
     (pin "2")
   )
-  (symbol (lib_id "power:+VSW") (at 88.9 95.25 0)
-    (in_bom yes) (on_board yes)
-    (property "Reference" "#PWR0132" (id 0) (at 88.9 99.06 0)
+  (symbol (lib_id "power:+VSW") (at 88.9 95.25 0) (unit 1)
+    (in_bom yes) (on_board yes)
+    (property "Reference" "#PWR060" (id 0) (at 88.9 99.06 0)
       (effects (font (size 1.27 1.27)) hide)
     )
@@
     (pin "1")
   )
-  (symbol (lib_id "power:GND") (at 97.79 105.41 0)
-    (in_bom yes) (on_board yes)
-    (property "Reference" "#PWR0133" (id 0) (at 97.79 111.76 0)
+  (symbol (lib_id "power:GND") (at 97.79 105.41 0) (unit 1)
+    (in_bom yes) (on_board yes)
+    (property "Reference" "#PWR061" (id 0) (at 97.79 111.76 0)
       (effects (font (size 1.27 1.27)) hide)
     )
@@
     (pin "1")
   )
-  (symbol (lib_id "Device:R") (at 132.08 78.74 270)
-    (in_bom yes) (on_board yes)
-    (property "Reference" "R97" (id 0) (at 132.08 78.74 90))
+  (symbol (lib_id "Device:R") (at 132.08 78.74 270) (unit 1)
+    (in_bom yes) (on_board yes)
+    (property "Reference" "R46" (id 0) (at 132.08 78.74 90))
     (property "Value" "4.7" (id 1) (at 132.08 75.7936 90))
     (property "Footprint" "Resistor_SMD:R_1206_3216Metric" (id 2) (at 132.08 76.962 90)
@@
     (pin "2")
   )
-  (symbol (lib_id "Device:C") (at 171.45 76.2 0)
-    (in_bom yes) (on_board yes)
-    (property "Reference" "C72" (id 0) (at 168.529 75.0316 0)
+  (symbol (lib_id "Device:C") (at 171.45 76.2 0) (unit 1)
+    (in_bom yes) (on_board yes)
+    (property "Reference" "C40" (id 0) (at 168.529 75.0316 0)
       (effects (font (size 1.27 1.27)) (justify right))
     )
@@
     (pin "2")
   )
-  (symbol (lib_id "power:+BATT") (at 143.51 71.12 0)
-    (in_bom yes) (on_board yes)
-    (property "Reference" "#PWR0135" (id 0) (at 143.51 74.93 0)
+  (symbol (lib_id "power:+BATT") (at 143.51 71.12 0) (unit 1)
+    (in_bom yes) (on_board yes)
+    (property "Reference" "#PWR063" (id 0) (at 143.51 74.93 0)
       (effects (font (size 1.27 1.27)) hide)
     )
@@
     (pin "1")
   )
-  (symbol (lib_id "Device:R") (at 88.9 83.82 270)
-    (in_bom yes) (on_board yes)
-    (property "Reference" "R93" (id 0) (at 88.9 76.2762 90))
+  (symbol (lib_id "Device:R") (at 88.9 83.82 270) (unit 1)
+    (in_bom yes) (on_board yes)
+    (property "Reference" "R42" (id 0) (at 88.9 76.2762 90))
     (property "Value" "1k" (id 1) (at 88.9 78.5876 90))
     (property "Footprint" "Resistor_SMD:R_0603_1608Metric" (id 2) (at 68.58 77.47 90)
@@
     (pin "2")
   )
-  (symbol (lib_id "Device:R") (at 88.9 86.36 270)
-    (in_bom yes) (on_board yes)
-    (property "Reference" "R94" (id 0) (at 88.9 81.1022 90))
+  (symbol (lib_id "Device:R") (at 88.9 86.36 270) (unit 1)
+    (in_bom yes) (on_board yes)
+    (property "Reference" "R43" (id 0) (at 88.9 81.1022 90))
     (property "Value" "1k" (id 1) (at 88.9 83.4136 90))
     (property "Footprint" "Resistor_SMD:R_0603_1608Metric" (id 2) (at 88.9 84.582 90)
@@
     (pin "2")
   )
-  (symbol (lib_id "Device:CP") (at 180.34 76.2 0)
-    (in_bom yes) (on_board yes)
-    (property "Reference" "C73" (id 0) (at 183.3372 75.0316 0)
+  (symbol (lib_id "Device:CP") (at 180.34 76.2 0) (unit 1)
+    (in_bom yes) (on_board yes)
+    (property "Reference" "C41" (id 0) (at 183.3372 75.0316 0)
       (effects (font (size 1.27 1.27)) (justify left))
     )
@@
     (pin "2")
   )
-  (symbol (lib_id "power:+BATT") (at 180.34 71.12 0)
-    (in_bom yes) (on_board yes)
-    (property "Reference" "#PWR0136" (id 0) (at 180.34 74.93 0)
+  (symbol (lib_id "power:+BATT") (at 180.34 71.12 0) (unit 1)
+    (in_bom yes) (on_board yes)
+    (property "Reference" "#PWR064" (id 0) (at 180.34 74.93 0)
       (effects (font (size 1.27 1.27)) hide)
     )
@@
     (pin "1")
   )
-  (symbol (lib_id "Device:Varistor") (at 208.28 76.2 0)
-    (in_bom yes) (on_board yes)
-    (property "Reference" "RV6" (id 0) (at 210.8962 75.0316 0)
-      (effects (font (size 1.27 1.27)) (justify left))
-    )
+  (symbol (lib_id "Device:Varistor") (at 208.28 76.2 0) (unit 1)
+    (in_bom yes) (on_board yes)
+    (property "Reference" "RV1" (id 0) (at 210.8962 75.0316 0)
+      (effects (font (size 1.27 1.27)) (justify left))
+    )

Commit message: Update a few library symbols
Parts:
- C38, C39, C41: symbol Device:CP -> Device:C_Polarized
Changed lines of the file:
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@@
     (effects (font (size 1.27 1.27)) (justify left))
   )
-  (symbol (lib_id "Device:CP") (at 114.3 83.82 0) (unit 1)
+  (symbol (lib_id "Device:C_Polarized") (at 114.3 83.82 0) (unit 1)
     (in_bom yes) (on_board yes)
     (property "Reference" "C39" (id 0) (at 117.2972 82.6516 0)
@@
     (pin "1")
   )
-  (symbol (lib_id "Device:CP") (at 88.9 100.33 0) (unit 1)
+  (symbol (lib_id "Device:C_Polarized") (at 88.9 100.33 0) (unit 1)
     (in_bom yes) (on_board yes)
     (property "Reference" "C38" (id 0) (at 85.9028 99.1616 0)
@@
     (pin "2")
   )
-  (symbol (lib_id "Device:CP") (at 180.34 76.2 0) (unit 1)
+  (symbol (lib_id "Device:C_Polarized") (at 180.34 76.2 0) (unit 1)
     (in_bom yes) (on_board yes)
     (property "Reference" "C41" (id 0) (at 183.3372 75.0316 0)
