File: hh_bridge.kicad_sch (KiCad schematic)
At the start: 15 parts, among them U6 UCC27712

Commit message: ordered this on jlcpcb
Parts:
- renumbered C38 to C70, C39 to C71, C40 to C72, C41 to C73, D19 to D34, R42 to R93, R43 to R94, R44 to R95, R45 to R96, R46 to R97, R47 to R98, RV1 to RV6, U6 to U14, V1 to V12, V2 to V13
Changed lines of the file:
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@@
     (effects (font (size 1.27 1.27)) (justify left))
   )
-  (symbol (lib_id "Device:C_Polarized") (at 114.3 83.82 0) (unit 1)
-    (in_bom yes) (on_board yes)
-    (property "Reference" "C39" (id 0) (at 117.2972 82.6516 0)
+  (symbol (lib_id "Device:C_Polarized") (at 114.3 83.82 0)
+    (in_bom yes) (on_board yes)
+    (property "Reference" "C71" (id 0) (at 117.2972 82.6516 0)
       (effects (font (size 1.27 1.27)) (justify left))
     )
@@
     (pin "2")
   )
-  (symbol (lib_id "Device:D") (at 109.22 63.5 180) (unit 1)
-    (in_bom yes) (on_board yes)
-    (property "Reference" "D19" (id 0) (at 109.22 57.9882 0))
+  (symbol (lib_id "Device:D") (at 109.22 63.5 180)
+    (in_bom yes) (on_board yes)
+    (property "Reference" "D34" (id 0) (at 109.22 57.9882 0))
     (property "Value" "1N4148W" (id 1) (at 109.22 60.2996 0))
     (property "Footprint" "Diode_SMD:D_SOD-123" (id 2) (at 109.22 63.5 0)
@@
     (pin "2")
   )
-  (symbol (lib_id "Transistor_FET:BSP89") (at 140.97 78.74 0) (unit 1)
-    (in_bom yes) (on_board yes)
-    (property "Reference" "V1" (id 0) (at 146.1516 77.5716 0)
+  (symbol (lib_id "Transistor_FET:BSP89") (at 140.97 78.74 0)
+    (in_bom yes) (on_board yes)
+    (property "Reference" "V12" (id 0) (at 146.1516 77.5716 0)
       (effects (font (size 1.27 1.27)) (justify left))
     )
@@
     (pin "3")
   )
-  (symbol (lib_id "Device:R") (at 132.08 91.44 270) (unit 1)
-    (in_bom yes) (on_board yes)
-    (property "Reference" "R47" (id 0) (at 132.08 91.44 90))
+  (symbol (lib_id "Device:R") (at 132.08 91.44 270)
+    (in_bom yes) (on_board yes)
+    (property "Reference" "R98" (id 0) (at 132.08 91.44 90))
     (property "Value" "4.7" (id 1) (at 130.81 88.9 90))
     (property "Footprint" "Resistor_SMD:R_1206_3216Metric" (id 2) (at 132.08 89.662 90)
@@
     (pin "2")
   )
-  (symbol (lib_id "Transistor_FET:BSP89") (at 140.97 91.44 0) (unit 1)
-    (in_bom yes) (on_board yes)
-    (property "Reference" "V2" (id 0) (at 146.1516 90.2716 0)
+  (symbol (lib_id "Transistor_FET:BSP89") (at 140.97 91.44 0)
+    (in_bom yes) (on_board yes)
+    (property "Reference" "V13" (id 0) (at 146.1516 90.2716 0)
       (effects (font (size 1.27 1.27)) (justify left))
     )
@@
     (pin "3")
   )
-  (symbol (lib_id "Device:R") (at 125.73 95.25 180) (unit 1)
-    (in_bom yes) (on_board yes)
-    (property "Reference" "R45" (id 0) (at 123.9774 94.0816 0)
+  (symbol (lib_id "Device:R") (at 125.73 95.25 180)
+    (in_bom yes) (on_board yes)
+    (property "Reference" "R96" (id 0) (at 123.9774 94.0816 0)
       (effects (font (size 1.27 1.27)) (justify left))
     )
@@
     (pin "2")
   )
-  (symbol (lib_id "Device:R") (at 123.19 83.82 180) (unit 1)
-    (in_bom yes) (on_board yes)
-    (property "Reference" "R44" (id 0) (at 124.968 82.6516 0)
+  (symbol (lib_id "Device:R") (at 123.19 83.82 180)
+    (in_bom yes) (on_board yes)
+    (property "Reference" "R95" (id 0) (at 124.968 82.6516 0)
       (effects (font (size 1.27 1.27)) (justify right))
     )
@@
     (pin "2")
   )
-  (symbol (lib_id "Driver_FET:IRS2304") (at 100.33 83.82 0) (unit 1)
-    (in_bom yes) (on_board yes)
-    (property "Reference" "U6" (id 0) (at 100.33 66.5226 0))
+  (symbol (lib_id "Driver_FET:IRS2304") (at 100.33 83.82 0)
+    (in_bom yes) (on_board yes)
+    (property "Reference" "U14" (id 0) (at 100.33 66.5226 0))
     (property "Value" "UCC27712" (id 1) (at 100.33 68.834 0))
     (property "Footprint" "Package_SO:SOIC-8_3.9x4.9mm_P1.27mm" (id 2) (at 100.33 83.82 0)
@@
     (pin "8")
   )
-  (symbol (lib_id "power:+VSW") (at 100.33 60.96 0) (unit 1)
-    (in_bom yes) (on_board yes)
-    (property "Reference" "#PWR062" (id 0) (at 100.33 64.77 0)
+  (symbol (lib_id "power:+VSW") (at 100.33 60.96 0)
+    (in_bom yes) (on_board yes)
+    (property "Reference" "#PWR0134" (id 0) (at 100.33 64.77 0)
       (effects (font (size 1.27 1.27)) hide)
     )
@@
     (pin "1")
   )
-  (symbol (lib_id "Device:C_Polarized") (at 88.9 100.33 0) (unit 1)
-    (in_bom yes) (on_board yes)
-    (property "Reference" "C38" (id 0) (at 85.9028 99.1616 0)
+  (symbol (lib_id "Device:C_Polarized") (at 88.9 100.33 0)
+    (in_bom yes) (on_board yes)
+    (property "Reference" "C70" (id 0) (at 85.9028 99.1616 0)
       (effects (font (size 1.27 1.27)) (justify right))
     )
@@
     (pin "2")
   )
-  (symbol (lib_id "power:+VSW") (at 88.9 95.25 0) (unit 1)
-    (in_bom yes) (on_board yes)
-    (property "Reference" "#PWR060" (id 0) (at 88.9 99.06 0)
+  (symbol (lib_id "power:+VSW") (at 88.9 95.25 0)
+    (in_bom yes) (on_board yes)
+    (property "Reference" "#PWR0132" (id 0) (at 88.9 99.06 0)
       (effects (font (size 1.27 1.27)) hide)
     )
@@
     (pin "1")
   )
-  (symbol (lib_id "power:GND") (at 97.79 105.41 0) (unit 1)
-    (in_bom yes) (on_board yes)
-    (property "Reference" "#PWR061" (id 0) (at 97.79 111.76 0)
+  (symbol (lib_id "power:GND") (at 97.79 105.41 0)
+    (in_bom yes) (on_board yes)
+    (property "Reference" "#PWR0133" (id 0) (at 97.79 111.76 0)
       (effects (font (size 1.27 1.27)) hide)
     )
@@
     (pin "1")
   )
-  (symbol (lib_id "Device:R") (at 132.08 78.74 270) (unit 1)
-    (in_bom yes) (on_board yes)
-    (property "Reference" "R46" (id 0) (at 132.08 78.74 90))
+  (symbol (lib_id "Device:R") (at 132.08 78.74 270)
+    (in_bom yes) (on_board yes)
+    (property "Reference" "R97" (id 0) (at 132.08 78.74 90))
     (property "Value" "4.7" (id 1) (at 132.08 75.7936 90))
     (property "Footprint" "Resistor_SMD:R_1206_3216Metric" (id 2) (at 132.08 76.962 90)
@@
     (pin "2")
   )
-  (symbol (lib_id "Device:C") (at 171.45 76.2 0) (unit 1)
-    (in_bom yes) (on_board yes)
-    (property "Reference" "C40" (id 0) (at 168.529 75.0316 0)
+  (symbol (lib_id "Device:C") (at 171.45 76.2 0)
+    (in_bom yes) (on_board yes)
+    (property "Reference" "C72" (id 0) (at 168.529 75.0316 0)
       (effects (font (size 1.27 1.27)) (justify right))
     )
@@
     (pin "2")
   )
-  (symbol (lib_id "power:+BATT") (at 143.51 71.12 0) (unit 1)
-    (in_bom yes) (on_board yes)
-    (property "Reference" "#PWR063" (id 0) (at 143.51 74.93 0)
+  (symbol (lib_id "power:+BATT") (at 143.51 71.12 0)
+    (in_bom yes) (on_board yes)
+    (property "Reference" "#PWR0135" (id 0) (at 143.51 74.93 0)
       (effects (font (size 1.27 1.27)) hide)
     )
@@
     (pin "1")
   )
-  (symbol (lib_id "Device:R") (at 88.9 83.82 270) (unit 1)
-    (in_bom yes) (on_board yes)
-    (property "Reference" "R42" (id 0) (at 88.9 76.2762 90))
+  (symbol (lib_id "Device:R") (at 88.9 83.82 270)
+    (in_bom yes) (on_board yes)
+    (property "Reference" "R93" (id 0) (at 88.9 76.2762 90))
     (property "Value" "1k" (id 1) (at 88.9 78.5876 90))
     (property "Footprint" "Resistor_SMD:R_0603_1608Metric" (id 2) (at 68.58 77.47 90)
@@
     (pin "2")
   )
-  (symbol (lib_id "Device:R") (at 88.9 86.36 270) (unit 1)
-    (in_bom yes) (on_board yes)
-    (property "Reference" "R43" (id 0) (at 88.9 81.1022 90))
+  (symbol (lib_id "Device:R") (at 88.9 86.36 270)
+    (in_bom yes) (on_board yes)
+    (property "Reference" "R94" (id 0) (at 88.9 81.1022 90))
     (property "Value" "1k" (id 1) (at 88.9 83.4136 90))
     (property "Footprint" "Resistor_SMD:R_0603_1608Metric" (id 2) (at 88.9 84.582 90)
@@
     (pin "2")
   )
-  (symbol (lib_id "Device:C_Polarized") (at 180.34 76.2 0) (unit 1)
-    (in_bom yes) (on_board yes)
-    (property "Reference" "C41" (id 0) (at 183.3372 75.0316 0)
+  (symbol (lib_id "Device:C_Polarized") (at 180.34 76.2 0)
+    (in_bom yes) (on_board yes)
+    (property "Reference" "C73" (id 0) (at 183.3372 75.0316 0)
       (effects (font (size 1.27 1.27)) (justify left))
     )
@@
     (pin "2")
   )
-  (symbol (lib_id "power:+BATT") (at 180.34 71.12 0) (unit 1)
-    (in_bom yes) (on_board yes)
-    (property "Reference" "#PWR064" (id 0) (at 180.34 74.93 0)
+  (symbol (lib_id "power:+BATT") (at 180.34 71.12 0)
+    (in_bom yes) (on_board yes)
+    (property "Reference" "#PWR0136" (id 0) (at 180.34 74.93 0)
       (effects (font (size 1.27 1.27)) hide)
     )
@@
     (pin "1")
   )
-  (symbol (lib_id "Device:Varistor") (at 208.28 76.2 0) (unit 1)
-    (in_bom yes) (on_board yes)
-    (property "Reference" "RV1" (id 0) (at 210.8962 75.0316 0)
-      (effects (font (size 1.27 1.27)) (justify left))
-    )
+  (symbol (lib_id "Device:Varistor") (at 208.28 76.2 0)
+    (in_bom yes) (on_board yes)
+    (property "Reference" "RV6" (id 0) (at 210.8962 75.0316 0)
+      (effects (font (size 1.27 1.27)) (justify left))
+    )

Commit message: Updated diodes, added LCSC numbers for all parts
Parts:
- C38: renamed from C70; LCSC (none) -> C399576; LCSC Part # C399576 -> (none)
- C39: renamed from C71; LCSC (none) -> C106686; LCSC Part # C106686 -> (none)
- C40: renamed from C72; LCSC (none) -> C577211
- C41: renamed from C73; LCSC (none) -> C106686; LCSC Part # C106686 -> (none)
- D19: renamed from D34; LCSC (none) -> C81598; LCSC Part # C81598 -> (none)
- R42: renamed from R93; LCSC (none) -> C21190; LCSC Part # C21190 -> (none)
- R43: renamed from R94; LCSC (none) -> C21190; LCSC Part # C21190 -> (none)
- R44: renamed from R95; LCSC (none) -> C17902; LCSC Part # C17902 -> (none)
- R45: renamed from R96; LCSC (none) -> C17902; LCSC Part # C17902 -> (none)
- R46: renamed from R97; LCSC (none) -> C17937; LCSC Part # C17937 -> (none)
- R47: renamed from R98; LCSC (none) -> C17937; LCSC Part # C17937 -> (none)
- RV1: renamed from RV6; value Varistor -> V20P35P; LCSC (none) -> C1528974
- U6: renamed from U14; value UCC27712 -> IRS2304; LCSC (none) -> C82060; LCSC Part # C485818 -> (none); alternative IRS2304 old -> (none)
- V1: renamed from V12; LCSC (none) -> C410926
- V2: renamed from V13; LCSC (none) -> C410926
