File: hh_bridge.kicad_sch (KiCad schematic)
At the start: 15 parts, among them U6 IRS2304

Commit message: update lcsc numbers
Parts:
- C40, RV1, V1, V2: place hand -> (none)
Changed lines of the file:
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@@
+			)
+		)
+		(property "alternative" ""
+			(at 114.3 83.82 0)
+			(effects
+				(font
+					(size 1.27 1.27)
+				)
+				(hide yes)
 			)
 		)
@@
 			)
 		)
+		(property "alternative" ""
+			(at 109.22 63.5 0)
+			(effects
+				(font
+					(size 1.27 1.27)
+				)
+				(hide yes)
+			)
+		)
 		(pin "1"
 		)
@@
 			)
 		)
-		(property "place" "hand"
+		(property "place" ""
 			(at 140.97 78.74 0)
 			(effects
@@
 		)
 		(property "LCSC" "C410926"
+			(at 140.97 78.74 0)
+			(effects
+				(font
+					(size 1.27 1.27)
+				)
+				(hide yes)
+			)
+		)
+		(property "alternative" ""
 			(at 140.97 78.74 0)
 			(effects
@@
 			)
 		)
+		(property "alternative" ""
+			(at 132.08 91.44 90)
+			(effects
+				(font
+					(size 1.27 1.27)
+				)
+				(hide yes)
+			)
+		)
 		(pin "1"
 		)
@@
 			)
 		)
-		(property "place" "hand"
+		(property "place" ""
 			(at 140.97 91.44 0)
 			(effects
@@
 		)
 		(property "LCSC" "C410926"
+			(at 140.97 91.44 0)
+			(effects
+				(font
+					(size 1.27 1.27)
+				)
+				(hide yes)
+			)
+		)
+		(property "alternative" ""
 			(at 140.97 91.44 0)
 			(effects
@@
 			)
 		)
+		(property "alternative" ""
+			(at 125.73 95.25 0)
+			(effects
+				(font
+					(size 1.27 1.27)
+				)
+				(hide yes)
+			)
+		)
 		(pin "1"
 		)
@@
 			)
 		)
+		(property "alternative" ""
+			(at 123.19 83.82 0)
+			(effects
+				(font
+					(size 1.27 1.27)
+				)
+				(hide yes)
+			)
+		)
 		(pin "1"
 		)
@@
 			)
 		)
+		(property "alternative" ""
+			(at 100.33 83.82 0)
+			(effects
+				(font
+					(size 1.27 1.27)
+				)
+				(hide yes)
+			)
+		)
 		(pin "1"
 		)
@@
 			)
 		)
+		(property "alternative" ""
+			(at 88.9 100.33 0)
+			(effects
+				(font
+					(size 1.27 1.27)
+				)
+				(hide yes)
+			)
+		)
 		(pin "1"
 		)
@@
 			)
 		)
+		(property "alternative" ""
+			(at 132.08 78.74 90)
+			(effects
+				(font
+					(size 1.27 1.27)
+				)
+				(hide yes)
+			)
+		)
 		(pin "1"
 		)
@@
 			)
 		)
-		(property "place" "hand"
+		(property "LCSC" "C577211"
 			(at 171.45 76.2 0)
 			(effects
@@
 			)
 		)
-		(property "LCSC" "C577211"
+		(property "alternative" ""
 			(at 171.45 76.2 0)
 			(effects
@@
 			)
 		)
+		(property "alternative" ""
+			(at 88.9 83.82 90)
+			(effects
+				(font
+					(size 1.27 1.27)
+				)
+				(hide yes)
+			)
+		)
 		(pin "1"
 		)
@@
 			)
 		)
+		(property "alternative" ""
+			(at 88.9 86.36 90)
+			(effects
+				(font
+					(size 1.27 1.27)
+				)
+				(hide yes)
+			)
+		)
 		(pin "1"
 		)
@@
 			)
 		)
+		(property "alternative" ""
+			(at 180.34 76.2 0)
+			(effects
+				(font
+					(size 1.27 1.27)
+				)
+				(hide yes)
+			)
+		)
 		(pin "1"
 		)
@@
 			)
 		)
-		(property "place" "hand"
+		(property "place" ""
 			(at 208.28 76.2 0)
 			(effects
@@
 			(at 208.28 76.2 0)
 			(effects
+				(font
+					(size 1.27 1.27)
+				)
+				(hide yes)
+			)
+		)
+		(property "alternative" ""
+			(at 208.28 76.2 0)
+			(effects

Commit message: Exchanged more components, DNP and bridge 4.7R resistor, DNP 51V TVS diode
Parts:
- C38: value 220u25V LKMD0901E221MF -> 220u25V; LCSC C399576 -> C106697
Changed lines of the file:
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@@
 			)
 		)
-		(property "Value" "220u25V LKMD0901E221MF"
+		(property "Value" "220u25V"
 			(at 85.9028 101.473 0)
 			(effects
@@
 			)
 		)
-		(property "LCSC" "C399576"
+		(property "LCSC" "C106697"
 			(at 88.9 100.33 0)
 			(effects
