File: phase_sense.kicad_sch (KiCad schematic)
At the start: 18 parts, among them U4 3PEAK TP09-SR

Commit message: removed faulty vias and connections
Other:
- moved on the sheet: D25, D26
Changed lines of the file:
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@@
 (kicad_sch (version 20211123) (generator eeschema)
   (paper "A4")
-  (junction (at 134.62 41.91) (diameter 0) (color 0 0 0 0)
-  )
   (junction (at 153.67 76.2) (diameter 0) (color 0 0 0 0)
   )
@@
   (junction (at 163.83 87.63) (diameter 0) (color 0 0 0 0)
   )
-  (junction (at 134.62 50.8) (diameter 0) (color 0 0 0 0)
+  (junction (at 140.97 41.91) (diameter 0) (color 0 0 0 0)
+  )
+  (junction (at 140.97 50.8) (diameter 0) (color 0 0 0 0)
   )
   (junction (at 153.67 33.02) (diameter 0) (color 0 0 0 0)
@@
   (junction (at 128.27 93.98) (diameter 0) (color 0 0 0 0)
   )
-  (junction (at 133.35 93.98) (diameter 0) (color 0 0 0 0)
+  (junction (at 140.97 85.09) (diameter 0) (color 0 0 0 0)
+  )
+  (junction (at 140.97 93.98) (diameter 0) (color 0 0 0 0)
   )
   (junction (at 190.5 76.2) (diameter 0) (color 0 0 0 0)
   )
-  (junction (at 133.35 85.09) (diameter 0) (color 0 0 0 0)
-  )
   (junction (at 128.27 50.8) (diameter 0) (color 0 0 0 0)
   )
-  (wire (pts (xy 133.35 93.98) (xy 128.27 93.98))
+  (wire (pts (xy 140.97 93.98) (xy 128.27 93.98))
     (stroke (width 0) (type default) (color 0 0 0 0))
   )
@@
     (stroke (width 0) (type default) (color 0 0 0 0))
   )
-  (wire (pts (xy 134.62 49.53) (xy 134.62 50.8))
-    (stroke (width 0) (type default) (color 0 0 0 0))
-  )
-  (wire (pts (xy 134.62 41.91) (xy 128.27 41.91))
-    (stroke (width 0) (type default) (color 0 0 0 0))
-  )
-  (wire (pts (xy 148.59 41.91) (xy 134.62 41.91))
+  (wire (pts (xy 140.97 49.53) (xy 140.97 50.8))
+    (stroke (width 0) (type default) (color 0 0 0 0))
+  )
+  (wire (pts (xy 148.59 41.91) (xy 140.97 41.91))
     (stroke (width 0) (type default) (color 0 0 0 0))
   )
@@
     (stroke (width 0) (type default) (color 0 0 0 0))
   )
-  (wire (pts (xy 148.59 85.09) (xy 133.35 85.09))
+  (wire (pts (xy 148.59 85.09) (xy 140.97 85.09))
     (stroke (width 0) (type default) (color 0 0 0 0))
   )
@@
     (stroke (width 0) (type default) (color 0 0 0 0))
   )
+  (wire (pts (xy 128.27 41.91) (xy 140.97 41.91))
+    (stroke (width 0) (type default) (color 0 0 0 0))
+  )
   (wire (pts (xy 167.64 87.63) (xy 163.83 87.63))
     (stroke (width 0) (type default) (color 0 0 0 0))
@@
     (stroke (width 0) (type default) (color 0 0 0 0))
   )
-  (wire (pts (xy 133.35 85.09) (xy 128.27 85.09))
+  (wire (pts (xy 128.27 85.09) (xy 140.97 85.09))
     (stroke (width 0) (type default) (color 0 0 0 0))
   )
@@
     (stroke (width 0) (type default) (color 0 0 0 0))
   )
-  (wire (pts (xy 134.62 50.8) (xy 128.27 50.8))
+  (wire (pts (xy 140.97 50.8) (xy 128.27 50.8))
     (stroke (width 0) (type default) (color 0 0 0 0))
   )
@@
     (stroke (width 0) (type default) (color 0 0 0 0))
   )
-  (wire (pts (xy 148.59 93.98) (xy 133.35 93.98))
-    (stroke (width 0) (type default) (color 0 0 0 0))
-  )
-  (wire (pts (xy 148.59 50.8) (xy 134.62 50.8))
+  (wire (pts (xy 148.59 93.98) (xy 140.97 93.98))
+    (stroke (width 0) (type default) (color 0 0 0 0))
+  )
+  (wire (pts (xy 148.59 50.8) (xy 140.97 50.8))
     (stroke (width 0) (type default) (color 0 0 0 0))
   )
@@
     (stroke (width 0) (type default) (color 0 0 0 0))
   )
-  (wire (pts (xy 133.35 92.71) (xy 133.35 93.98))
+  (wire (pts (xy 140.97 92.71) (xy 140.97 93.98))
     (stroke (width 0) (type default) (color 0 0 0 0))
   )
@@
     (pin "7")
   )
-  (symbol (lib_id "Diode:BAS20") (at 134.62 45.72 90)
+  (symbol (lib_id "Diode:BAS20") (at 140.97 45.72 90)
     (in_bom yes) (on_board yes) (fields_autoplaced)
-    (property "Reference" "D26" (id 0) (at 136.652 44.8115 90)
-      (effects (font (size 1.27 1.27)) (justify right))
-    )
-    (property "Value" "BAS20" (id 1) (at 136.652 47.5866 90)
-      (effects (font (size 1.27 1.27)) (justify right))
-    )
-    (property "Footprint" "Package_TO_SOT_SMD:SOT-23" (id 2) (at 139.065 45.72 0)
-      (effects (font (size 1.27 1.27)) hide)
-    )
-    (property "Datasheet" "https://www.diodes.com/assets/Datasheets/Ds12004.pdf" (id 3) (at 134.62 45.72 0)
+    (property "Reference" "D26" (id 0) (at 143.002 44.8115 90)
+      (effects (font (size 1.27 1.27)) (justify right))
+    )
+    (property "Value" "BAS20" (id 1) (at 143.002 47.5866 90)
+      (effects (font (size 1.27 1.27)) (justify right))
+    )
+    (property "Footprint" "Package_TO_SOT_SMD:SOT-23" (id 2) (at 145.415 45.72 0)
+      (effects (font (size 1.27 1.27)) hide)
+    )
+    (property "Datasheet" "https://www.diodes.com/assets/Datasheets/Ds12004.pdf" (id 3) (at 140.97 45.72 0)
       (effects (font (size 1.27 1.27)) hide)
     )
@@
     (pin "3")
   )
-  (symbol (lib_id "Diode:BAS20") (at 133.35 88.9 90)
+  (symbol (lib_id "Diode:BAS20") (at 140.97 88.9 90)
     (in_bom yes) (on_board yes) (fields_autoplaced)
-    (property "Reference" "D25" (id 0) (at 135.382 87.9915 90)
-      (effects (font (size 1.27 1.27)) (justify right))
-    )
-    (property "Value" "BAS20" (id 1) (at 135.382 90.7666 90)
-      (effects (font (size 1.27 1.27)) (justify right))
-    )
-    (property "Footprint" "Package_TO_SOT_SMD:SOT-23" (id 2) (at 137.795 88.9 0)
-      (effects (font (size 1.27 1.27)) hide)
-    )
-    (property "Datasheet" "https://www.diodes.com/assets/Datasheets/Ds12004.pdf" (id 3) (at 133.35 88.9 0)
-      (effects (font (size 1.27 1.27)) hide)
-    )
+    (property "Reference" "D25" (id 0) (at 143.002 87.9915 90)
+      (effects (font (size 1.27 1.27)) (justify right))
+    )
+    (property "Value" "BAS20" (id 1) (at 143.002 90.7666 90)
+      (effects (font (size 1.27 1.27)) (justify right))
+    )
+    (property "Footprint" "Package_TO_SOT_SMD:SOT-23" (id 2) (at 145.415 88.9 0)
+      (effects (font (size 1.27 1.27)) hide)
+    )
+    (property "Datasheet" "https://www.diodes.com/assets/Datasheets/Ds12004.pdf" (id 3) (at 140.97 88.9 0)
+      (effects (font (size 1.27 1.27)) hide)
+    )

Commit message: Silkscreen and naming fixes
Parts:
- renumbered C10 to C70, D4 to D31, D5 to D32, D26 to D33, D25 to D34, R1 to R100, R22 to R101, R27 to R102, R25 to R103, R30 to R104, R24 to R95, R26 to R96, R29 to R97, R31 to R98, R23 to R99, U4 to U14
Changed lines of the file:
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@@
   (symbol (lib_id "power:+3.3V") (at 227.33 44.45 0)
     (in_bom yes) (on_board yes)
-    (property "Reference" "#PWR0159" (id 0) (at 227.33 48.26 0)
+    (property "Reference" "#PWR0132" (id 0) (at 227.33 48.26 0)
       (effects (font (size 1.27 1.27)) hide)
     )
@@
   (symbol (lib_id "Device:C") (at 227.33 48.26 0)
     (in_bom yes) (on_board yes)
-    (property "Reference" "C10" (id 0) (at 230.251 47.0916 0)
+    (property "Reference" "C70" (id 0) (at 230.251 47.0916 0)
       (effects (font (size 1.27 1.27)) (justify left))
     )
@@
   (symbol (lib_id "power:GND") (at 227.33 52.07 0)
     (in_bom yes) (on_board yes)
-    (property "Reference" "#PWR0160" (id 0) (at 227.33 58.42 0)
+    (property "Reference" "#PWR0133" (id 0) (at 227.33 58.42 0)
       (effects (font (size 1.27 1.27)) hide)
     )
@@
   (symbol (lib_id "Device:R") (at 116.84 41.91 90)
     (in_bom yes) (on_board yes)
-    (property "Reference" "R24" (id 0) (at 116.84 36.6522 90))
+    (property "Reference" "R95" (id 0) (at 116.84 36.6522 90))
     (property "Value" "20k" (id 1) (at 116.84 38.9636 90))
     (property "Footprint" "Resistor_SMD:R_0603_1608Metric" (id 2) (at 116.84 43.688 90)
@@
   (symbol (lib_id "Device:R") (at 124.46 41.91 90)
     (in_bom yes) (on_board yes)
-    (property "Reference" "R23" (id 0) (at 124.46 36.6522 90))
+    (property "Reference" "R99" (id 0) (at 124.46 36.6522 90))
     (property "Value" "20k" (id 1) (at 124.46 38.9636 90))
     (property "Footprint" "Resistor_SMD:R_0603_1608Metric" (id 2) (at 124.46 43.688 90)
@@
   (symbol (lib_id "Device:R") (at 116.84 50.8 90)
     (in_bom yes) (on_board yes)
-    (property "Reference" "R26" (id 0) (at 116.84 45.5422 90))
+    (property "Reference" "R96" (id 0) (at 116.84 45.5422 90))
     (property "Value" "1k" (id 1) (at 116.84 47.8536 90))
     (property "Footprint" "Resistor_SMD:R_0603_1608Metric" (id 2) (at 116.84 52.578 90)
@@
   (symbol (lib_id "Device:D") (at 128.27 45.72 90)
     (in_bom yes) (on_board yes)
-    (property "Reference" "D4" (id 0) (at 130.2766 44.5516 90)
+    (property "Reference" "D31" (id 0) (at 130.2766 44.5516 90)
       (effects (font (size 1.27 1.27)) (justify right))
     )
@@
   (symbol (lib_id "power:+3.3V") (at 153.67 33.02 0)
     (in_bom yes) (on_board yes)
-    (property "Reference" "#PWR0161" (id 0) (at 153.67 36.83 0)
+    (property "Reference" "#PWR0129" (id 0) (at 153.67 36.83 0)
       (effects (font (size 1.27 1.27)) hide)
     )
@@
   (symbol (lib_id "Device:R") (at 146.05 33.02 90)
     (in_bom yes) (on_board yes)
-    (property "Reference" "R22" (id 0) (at 146.05 27.7622 90))
+    (property "Reference" "R101" (id 0) (at 146.05 27.7622 90))
     (property "Value" "220k" (id 1) (at 146.05 30.0736 90))
     (property "Footprint" "Resistor_SMD:R_0603_1608Metric" (id 2) (at 146.05 34.798 90)
@@
   (symbol (lib_id "Device:Opamp_Dual_Generic") (at 156.21 44.45 0)
     (in_bom yes) (on_board yes)
-    (property "Reference" "U4" (id 0) (at 156.21 37.465 0))
+    (property "Reference" "U14" (id 0) (at 156.21 37.465 0))
     (property "Value" "3PEAK TP09-SR" (id 1) (at 156.21 37.4396 0)
       (effects (font (size 1.27 1.27)) hide)
@@
   (symbol (lib_id "Device:R") (at 160.02 50.8 270)
     (in_bom yes) (on_board yes)
-    (property "Reference" "R25" (id 0) (at 160.02 45.5422 90))
+    (property "Reference" "R103" (id 0) (at 160.02 45.5422 90))
     (property "Value" "2.2k" (id 1) (at 160.02 47.8536 90))
     (property "Footprint" "Resistor_SMD:R_0603_1608Metric" (id 2) (at 160.02 49.022 90)
@@
   (symbol (lib_id "Device:R") (at 116.84 85.09 90)
     (in_bom yes) (on_board yes)
-    (property "Reference" "R29" (id 0) (at 116.84 79.8322 90))
+    (property "Reference" "R97" (id 0) (at 116.84 79.8322 90))
     (property "Value" "20k" (id 1) (at 116.84 82.1436 90))
     (property "Footprint" "Resistor_SMD:R_0603_1608Metric" (id 2) (at 116.84 86.868 90)
@@
   (symbol (lib_id "Device:R") (at 124.46 85.09 90)
     (in_bom yes) (on_board yes)
-    (property "Reference" "R1" (id 0) (at 124.46 79.8322 90))
+    (property "Reference" "R100" (id 0) (at 124.46 79.8322 90))
     (property "Value" "20k" (id 1) (at 124.46 82.1436 90))
     (property "Footprint" "Resistor_SMD:R_0603_1608Metric" (id 2) (at 124.46 86.868 90)
@@
   (symbol (lib_id "Device:R") (at 116.84 93.98 90)
     (in_bom yes) (on_board yes)
-    (property "Reference" "R31" (id 0) (at 116.84 88.7222 90))
+    (property "Reference" "R98" (id 0) (at 116.84 88.7222 90))
     (property "Value" "1k" (id 1) (at 116.84 91.0336 90))
     (property "Footprint" "Resistor_SMD:R_0603_1608Metric" (id 2) (at 116.84 95.758 90)
@@
   (symbol (lib_id "Device:D") (at 128.27 88.9 90)
     (in_bom yes) (on_board yes)
-    (property "Reference" "D5" (id 0) (at 130.2766 87.7316 90)
+    (property "Reference" "D32" (id 0) (at 130.2766 87.7316 90)
       (effects (font (size 1.27 1.27)) (justify right))
     )
@@
   (symbol (lib_id "power:+3.3V") (at 153.67 76.2 0)
     (in_bom yes) (on_board yes)
-    (property "Reference" "#PWR0163" (id 0) (at 153.67 80.01 0)
+    (property "Reference" "#PWR0130" (id 0) (at 153.67 80.01 0)
       (effects (font (size 1.27 1.27)) hide)
     )
@@
   (symbol (lib_id "Device:R") (at 146.05 76.2 90)
     (in_bom yes) (on_board yes)
-    (property "Reference" "R27" (id 0) (at 146.05 70.9422 90))
+    (property "Reference" "R102" (id 0) (at 146.05 70.9422 90))
     (property "Value" "220k" (id 1) (at 146.05 73.2536 90))
     (property "Footprint" "Resistor_SMD:R_0603_1608Metric" (id 2) (at 146.05 77.978 90)
@@
   (symbol (lib_id "Device:Opamp_Dual_Generic") (at 193.04 87.63 0)
     (in_bom yes) (on_board yes)
-    (property "Reference" "U4" (id 0) (at 191.9732 86.4616 0)
+    (property "Reference" "U14" (id 0) (at 191.9732 86.4616 0)
       (effects (font (size 1.27 1.27)) (justify left))
     )
@@
   (symbol (lib_id "power:GND") (at 190.5 95.25 0)
     (in_bom yes) (on_board yes)
-    (property "Reference" "#PWR0164" (id 0) (at 190.5 101.6 0)
+    (property "Reference" "#PWR0131" (id 0) (at 190.5 101.6 0)
       (effects (font (size 1.27 1.27)) hide)
     )
@@
   (symbol (lib_id "Device:R") (at 160.02 93.98 270)
     (in_bom yes) (on_board yes)
-    (property "Reference" "R30" (id 0) (at 160.02 88.7222 90))
+    (property "Reference" "R104" (id 0) (at 160.02 88.7222 90))
     (property "Value" "2.2k" (id 1) (at 160.02 91.0336 90))
     (property "Footprint" "Resistor_SMD:R_0603_1608Metric" (id 2) (at 160.02 92.202 90)
@@
   (symbol (lib_id "Device:Opamp_Dual_Generic") (at 156.21 87.63 0)
     (in_bom yes) (on_board yes)
-    (property "Reference" "U4" (id 0) (at 156.21 80.645 0))
+    (property "Reference" "U14" (id 0) (at 156.21 80.645 0))
     (property "Value" "3PEAK TP09-SR" (id 1) (at 156.21 80.6196 0)
       (effects (font (size 1.27 1.27)) hide)
@@
   (symbol (lib_id "Diode:BAS20") (at 140.97 45.72 90)
     (in_bom yes) (on_board yes) (fields_autoplaced)
-    (property "Reference" "D26" (id 0) (at 143.002 44.8115 90)
+    (property "Reference" "D33" (id 0) (at 143.002 44.8115 90)
       (effects (font (size 1.27 1.27)) (justify right))
     )
@@
   (symbol (lib_id "Diode:BAS20") (at 140.97 88.9 90)
     (in_bom yes) (on_board yes) (fields_autoplaced)
-    (property "Reference" "D25" (id 0) (at 143.002 87.9915 90)
-      (effects (font (size 1.27 1.27)) (justify right))
-    )
+    (property "Reference" "D34" (id 0) (at 143.002 87.9915 90)
+      (effects (font (size 1.27 1.27)) (justify right))
+    )

Commit message: Updated Current sense circuit
Parts:
- removed D31, D32: 1N4148W, Diode_SMD:D_SOD-123, symbol Device:D
- removed D33, D34: BAS20, Package_TO_SOT_SMD:SOT-23, symbol Diode:BAS20
- added D22, D23, D24, D25: SM4007, Diode_SMD:D_SOD-123, symbol Diode:SM4007
- renumbered C70 to C50, R95 to R60, R96 to R61, R97 to R62, R98 to R63, R99 to R64, R100 to R65, R101 to R66, R102 to R67, R103 to R68, R104 to R69, U14 to U9
Connections:
- net GND: now also D23.2 (A), D25.2 (A)
- net at R64.2, R66.1, U9.3 (+): now also D22.2 (A)
- net at R61.2, R68.2, U9.2 (-): now also D22.1 (K), D23.1 (K)
- net at R65.2, R67.1, U9.3 (+): now also D24.2 (A)
- net at R63.2, R69.2, U9.2 (-): now also D24.1 (K), D25.1 (K)

Commit message: added esp on bottom side
Parts:
- added D49, D50: SM4007, Diode_SMD:D_SOD-123, symbol Diode:SM4007
- renumbered C50 to C74, D22 to D35, D23 to D36, D24 to D37, D25 to D38, R61 to R100, R62 to R101, R63 to R102, R64 to R103, R65 to R104, R66 to R105, R67 to R106, R68 to R107, R69 to R108, R60 to R99, U9 to U15
Connections:
- net GND: now also D49.2 (A), D50.2 (A)
- net at D35.2 (A), R103.2, R105.1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: now also D49.1 (K)
- net at D37.2 (A), R104.2, R106.1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: now also D50.1 (K)

Commit message: Refactor stuff adjacent to hall sensor pins
Parts:
- renumbered C74 to C50, D35 to D22, D36 to D23, D37 to D24, D38 to D25, D49 to D47, D50 to D48, R99 to R60, R100 to R61, R101 to R62, R102 to R63, R103 to R64, R104 to R65, R105 to R66, R106 to R67, R107 to R68, R108 to R69, U15 to U9
Connections:
- net +3V3: now also U9.8 (V+)
- net GND: now also U9.4 (V-)
- net PH_AMP_B_OUT: now also U9.7; no longer U9.1
- net at D24.2 (A), D48.1 (K), R65.2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: now also U9.5 (+); no longer U9.3 (+)
- net at D24.1 (K), D25.1 (K), R63.2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: now also U9.6 (-); no longer U9.2 (-)

Commit message: Update a few library symbols
Parts:
- U9: symbol Device:Opamp_Dual_Generic -> Device:Opamp_Dual
Changed lines of the file:
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@@
     (pin "2")
   )
-  (symbol (lib_id "Device:Opamp_Dual_Generic") (at 156.21 44.45 0) (unit 1)
+  (symbol (lib_id "Device:Opamp_Dual") (at 156.21 44.45 0) (unit 1)
     (in_bom yes) (on_board yes)
     (property "Reference" "U9" (id 0) (at 156.21 37.465 0))
@@
     (pin "2")
   )
-  (symbol (lib_id "Device:Opamp_Dual_Generic") (at 193.04 87.63 0) (unit 3)
+  (symbol (lib_id "Device:Opamp_Dual") (at 193.04 87.63 0) (unit 3)
     (in_bom yes) (on_board yes)
     (property "Reference" "U9" (id 0) (at 191.9732 86.4616 0)
@@
     (pin "2")
   )
-  (symbol (lib_id "Device:Opamp_Dual_Generic") (at 156.21 87.63 0) (unit 2)
+  (symbol (lib_id "Device:Opamp_Dual") (at 156.21 87.63 0) (unit 2)
     (in_bom yes) (on_board yes)
     (property "Reference" "U9" (id 0) (at 156.21 80.645 0))

Commit message: ordered this on jlcpcb
Parts:
- renumbered C50 to C74, D22 to D35, D23 to D36, D24 to D37, D25 to D38, D47 to D49, D48 to D50, R61 to R100, R62 to R101, R63 to R102, R64 to R103, R65 to R104, R66 to R105, R67 to R106, R68 to R107, R69 to R108, R60 to R99, U9 to U15
Connections:
- net +3V3: no longer U15.8 (V+)
- net GND: no longer U15.4 (V-)
- net PH_AMP_B_OUT: now also U15.1; no longer U15.7
- net at D37.2 (A), D50.1 (K), R104.2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: now also U15.3 (+); no longer U15.5 (+)
- net at D37.1 (K), D38.1 (K), R102.2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: now also U15.2 (-); no longer U15.6 (-)

Commit message: Updated diodes, added LCSC numbers for all parts
Parts:
- C50: renamed from C74; LCSC (none) -> C14663; LCSC Part # C14663 -> (none)
- D22: renamed from D35; value SM4007 -> 1N4148W; symbol Diode:SM4007 -> Diode:1N4148W; LCSC (none) -> C81598; LCSC Part # C64898 -> (none)
- D23: renamed from D36; value SM4007 -> 1N4148W; symbol Diode:SM4007 -> Diode:1N4148W; LCSC (none) -> C81598; LCSC Part # C64898 -> (none)
- D24: renamed from D37; value SM4007 -> 1N4148W; symbol Diode:SM4007 -> Diode:1N4148W; LCSC (none) -> C81598; LCSC Part # C64898 -> (none)
- D25: renamed from D38; value SM4007 -> 1N4148W; symbol Diode:SM4007 -> Diode:1N4148W; LCSC (none) -> C81598; LCSC Part # C64898 -> (none)
- D47: renamed from D49; value SM4007 -> 1N4148W; symbol Diode:SM4007 -> Diode:1N4148W; LCSC (none) -> C81598; LCSC Part # C64898 -> (none)
- D48: renamed from D50; value SM4007 -> 1N4148W; symbol Diode:SM4007 -> Diode:1N4148W; LCSC (none) -> C81598; LCSC Part # C64898 -> (none)
- R60: renamed from R99; LCSC (none) -> C4184; LCSC Part # C4184 -> (none)
- R61: renamed from R100; LCSC (none) -> C21190; LCSC Part # C21190 -> (none)
- R62: renamed from R101; LCSC (none) -> C4184; LCSC Part # C4184 -> (none)
- R63: renamed from R102; LCSC (none) -> C21190; LCSC Part # C21190 -> (none)
- R64: renamed from R103; LCSC (none) -> C4184; LCSC Part # C4184 -> (none)
- R65: renamed from R104; LCSC (none) -> C4184; LCSC Part # C4184 -> (none)
- R66: renamed from R105; LCSC (none) -> C22961; LCSC Part # C22961 -> (none)
- R67: renamed from R106; LCSC (none) -> C22961; LCSC Part # C22961 -> (none)
- R68: renamed from R107; LCSC (none) -> C4190; LCSC Part # C4190 -> (none)
- R69: renamed from R108; LCSC (none) -> C4190; LCSC Part # C4190 -> (none)
- U9: renamed from U15; LCSC (none) -> C81662; LCSC Part # C81662 -> (none)
Connections:
- net +3V3: now also U9.8 (V+)
- net GND: now also U9.4 (V-)
- net PH_AMP_B_OUT: now also U9.7; no longer U9.1
- net at D24.2 (A), D48.1 (K), R65.2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: now also U9.5 (+); no longer U9.3 (+)
- net at D24.1 (K), D25.1 (K), R63.2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: now also U9.6 (-); no longer U9.2 (-)
