File: phase_sense.kicad_sch (KiCad schematic)
At the start: 18 parts, among them U9 3PEAK TP09-SR

Commit message: Exchanged more components, DNP and bridge 4.7R resistor, DNP 51V TVS diode
Parts:
- U9: value 3PEAK TP09-SR -> TLV9362IDR; LCSC C81662 -> C4367884
Changed lines of the file:
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@@
 			)
 		)
-		(property "Value" "3PEAK TP09-SR"
+		(property "Value" "TLV9362IDR"
 			(at 156.21 37.4396 0)
 			(effects
@@
 			)
 		)
-		(property "LCSC" "C81662"
+		(property "LCSC" "C4367884"
 			(at 156.21 44.45 0)
 			(effects
@@
 			)
 		)
-		(property "Value" "3PEAK TP09-SR"
+		(property "Value" "TLV9362IDR"
 			(at 191.9732 88.773 0)
 			(effects
@@
 			)
 		)
-		(property "LCSC" "C81662"
+		(property "LCSC" "C4367884"
 			(at 193.04 87.63 0)
 			(effects
@@
 			)
 		)
-		(property "Value" "3PEAK TP09-SR"
+		(property "Value" "TLV9362IDR"
 			(at 156.21 80.6196 0)
 			(effects
@@
 			)
 		)
-		(property "LCSC" "C81662"
+		(property "LCSC" "C4367884"
 			(at 156.21 87.63 0)
 			(effects
