File: CAN_TRX.kicad_sch (KiCad schematic)
At the start: 3 parts, among them U1 TJA1051T-3

Commit message: Updated diodes, added LCSC numbers for all parts
Parts:
- C19, C20: LCSC (none) -> C14663; LCSC Part # C14663 -> (none)
- U1: LCSC (none) -> C38695; LCSC Part # C38695 -> (none)
