File: ESP32.kicad_sch (KiCad schematic)
At the start: 11 parts, among them J20 Conn_01x06, U18 ESP32-WROOM-32, U20 LM75B, U21 LM75B

Commit message: Updated diodes, added LCSC numbers for all parts
Parts:
- C86, C87: LCSC (none) -> C1779; LCSC Part # C1779 -> (none)
- C88, C89, C90: LCSC (none) -> C14663; LCSC Part # C14663 -> (none)
- J20: now not fitted; now left out of the parts list
- R113, R114: LCSC (none) -> C25804
- U18: LCSC (none) -> C701343; now not fitted
- U20, U21: value LM75B -> LM75BDP; LCSC (none) -> C33099
