File: can_termination.kicad_sch (KiCad schematic)
At the start: 5 parts

Commit message: Updated diodes, added LCSC numbers for all parts
Parts:
- C21: LCSC (none) -> C14663; LCSC Part # C14663 -> (none)
- JP1, JP2: now not fitted; now left out of the parts list
- R5, R6: LCSC (none) -> C25196; LCSC Part # C25196 -> (none)
