File: hall_conn.kicad_sch (KiCad schematic)
At the start: 17 parts

Commit message: Some ERC fixes and other cleanups
Changed lines of the file:
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@@
     (effects (font (size 1.27 1.27)) (justify right bottom))
-  )
-  (label "Hall_1" (at 124.46 81.28 0)
-    (effects (font (size 1.27 1.27)) (justify left bottom))
-  )
-  (label "Hall_VCC" (at 130.81 128.27 0)
-    (effects (font (size 1.27 1.27)) (justify left bottom))
-  )
-  (label "Hall_2" (at 124.46 86.36 0)
-    (effects (font (size 1.27 1.27)) (justify left bottom))
-  )
-  (label "Hall_3" (at 124.46 91.44 0)
-    (effects (font (size 1.27 1.27)) (justify left bottom))
   )
   (hierarchical_label "HALL_VCC" (shape output) (at 121.92 128.27 180)

Commit message: ordered this on jlcpcb
Parts:
- renumbered C23 to C22, C24 to C25, C26 to C27, C29 to C30, D2 to D1, D9 to D10, D5 to D6, D7 to D8, R10 to R11, R13 to R14, R17 to R18, R19 to R20, R21 to R22, R23 to R24, R26 to R27, R28 to R29, R7 to R8
Changed lines of the file:
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@@
     (effects (font (size 1.27 1.27)) (justify right))
   )
-  (symbol (lib_id "power:GND") (at 124.46 74.93 90) (unit 1)
-    (in_bom yes) (on_board yes)
-    (property "Reference" "#PWR0192" (id 0) (at 130.81 74.93 0)
+  (symbol (lib_id "power:GND") (at 124.46 74.93 90)
+    (in_bom yes) (on_board yes)
+    (property "Reference" "#PWR0198" (id 0) (at 130.81 74.93 0)
       (effects (font (size 1.27 1.27)) hide)
     )
@@
     (pin "1")
   )
-  (symbol (lib_id "power:GND") (at 151.13 102.87 0) (unit 1)
-    (in_bom yes) (on_board yes)
-    (property "Reference" "#PWR0194" (id 0) (at 151.13 109.22 0)
+  (symbol (lib_id "power:GND") (at 151.13 102.87 0)
+    (in_bom yes) (on_board yes)
+    (property "Reference" "#PWR0200" (id 0) (at 151.13 109.22 0)
       (effects (font (size 1.27 1.27)) hide)
     )
@@
     (pin "1")
   )
-  (symbol (lib_id "Device:C") (at 139.7 96.52 0) (unit 1)
-    (in_bom yes) (on_board yes)
-    (property "Reference" "C24" (id 0) (at 142.24 95.25 0)
+  (symbol (lib_id "Device:C") (at 139.7 96.52 0)
+    (in_bom yes) (on_board yes)
+    (property "Reference" "C25" (id 0) (at 142.24 95.25 0)
       (effects (font (size 1.27 1.27)) (justify left))
     )
@@
     (pin "2")
   )
-  (symbol (lib_id "Device:C") (at 162.56 96.52 0) (unit 1)
-    (in_bom yes) (on_board yes)
-    (property "Reference" "C29" (id 0) (at 165.1 95.25 0)
+  (symbol (lib_id "Device:C") (at 162.56 96.52 0)
+    (in_bom yes) (on_board yes)
+    (property "Reference" "C30" (id 0) (at 165.1 95.25 0)
       (effects (font (size 1.27 1.27)) (justify left))
     )
@@
     (pin "2")
   )
-  (symbol (lib_id "Device:C") (at 130.81 133.35 0) (unit 1)
-    (in_bom yes) (on_board yes)
-    (property "Reference" "C23" (id 0) (at 133.35 132.08 0)
+  (symbol (lib_id "Device:C") (at 130.81 133.35 0)
+    (in_bom yes) (on_board yes)
+    (property "Reference" "C22" (id 0) (at 133.35 132.08 0)
       (effects (font (size 1.27 1.27)) (justify left))
     )
@@
     (pin "2")
   )
-  (symbol (lib_id "Device:LED") (at 184.15 64.77 90) (unit 1)
-    (in_bom yes) (on_board yes)
-    (property "Reference" "D9" (id 0) (at 190.627 64.9478 0)
+  (symbol (lib_id "Device:LED") (at 184.15 64.77 90)
+    (in_bom yes) (on_board yes)
+    (property "Reference" "D10" (id 0) (at 190.627 64.9478 0)
       (effects (font (size 1.27 1.27)) hide)
     )
@@
     (pin "2")
   )
-  (symbol (lib_id "Device:LED") (at 171.45 64.77 90) (unit 1)
-    (in_bom yes) (on_board yes)
-    (property "Reference" "D7" (id 0) (at 177.927 64.9478 0)
+  (symbol (lib_id "Device:LED") (at 171.45 64.77 90)
+    (in_bom yes) (on_board yes)
+    (property "Reference" "D8" (id 0) (at 177.927 64.9478 0)
       (effects (font (size 1.27 1.27)) hide)
     )
@@
     (pin "2")
   )
-  (symbol (lib_id "power:GND") (at 130.81 138.43 0) (unit 1)
-    (in_bom yes) (on_board yes)
-    (property "Reference" "#PWR0195" (id 0) (at 130.81 144.78 0)
+  (symbol (lib_id "power:GND") (at 130.81 138.43 0)
+    (in_bom yes) (on_board yes)
+    (property "Reference" "#PWR0201" (id 0) (at 130.81 144.78 0)
       (effects (font (size 1.27 1.27)) hide)
     )
@@
     (pin "1")
   )
-  (symbol (lib_id "Device:R") (at 199.39 86.36 90) (unit 1)
-    (in_bom yes) (on_board yes)
-    (property "Reference" "R26" (id 0) (at 199.39 83.82 90))
+  (symbol (lib_id "Device:R") (at 199.39 86.36 90)
+    (in_bom yes) (on_board yes)
+    (property "Reference" "R27" (id 0) (at 199.39 83.82 90))
     (property "Value" "3.3k" (id 1) (at 199.39 86.36 90))
     (property "Footprint" "Resistor_SMD:R_0603_1608Metric" (id 2) (at 199.39 88.138 90)
@@
     (pin "2")
   )
-  (symbol (lib_id "power:+3.3V") (at 167.64 58.42 0) (unit 1)
-    (in_bom yes) (on_board yes)
-    (property "Reference" "#PWR0197" (id 0) (at 167.64 62.23 0)
+  (symbol (lib_id "power:+3.3V") (at 167.64 58.42 0)
+    (in_bom yes) (on_board yes)
+    (property "Reference" "#PWR0203" (id 0) (at 167.64 62.23 0)
       (effects (font (size 1.27 1.27)) hide)
     )
@@
     (pin "1")
   )
-  (symbol (lib_id "Device:R") (at 180.34 72.39 0) (unit 1)
-    (in_bom yes) (on_board yes)
-    (property "Reference" "R19" (id 0) (at 177.8 72.39 90))
+  (symbol (lib_id "Device:R") (at 180.34 72.39 0)
+    (in_bom yes) (on_board yes)
+    (property "Reference" "R20" (id 0) (at 177.8 72.39 90))
     (property "Value" "2.2k" (id 1) (at 180.34 72.39 90))
     (property "Footprint" "Resistor_SMD:R_0603_1608Metric" (id 2) (at 178.562 72.39 90)
@@
     (pin "2")
   )
-  (symbol (lib_id "Device:R") (at 205.74 91.44 90) (unit 1)
-    (in_bom yes) (on_board yes)
-    (property "Reference" "R28" (id 0) (at 205.74 88.9 90))
+  (symbol (lib_id "Device:R") (at 205.74 91.44 90)
+    (in_bom yes) (on_board yes)
+    (property "Reference" "R29" (id 0) (at 205.74 88.9 90))
     (property "Value" "3.3k" (id 1) (at 205.74 91.44 90))
     (property "Footprint" "Resistor_SMD:R_0603_1608Metric" (id 2) (at 205.74 93.218 90)
@@
     (pin "2")
   )
-  (symbol (lib_id "Device:R") (at 167.64 72.39 0) (unit 1)
-    (in_bom yes) (on_board yes)
-    (property "Reference" "R13" (id 0) (at 165.1 72.39 90))
+  (symbol (lib_id "Device:R") (at 167.64 72.39 0)
+    (in_bom yes) (on_board yes)
+    (property "Reference" "R14" (id 0) (at 165.1 72.39 90))
     (property "Value" "2.2k" (id 1) (at 167.64 72.39 90))
     (property "Footprint" "Resistor_SMD:R_0603_1608Metric" (id 2) (at 165.862 72.39 90)
@@
     (pin "2")
   )
-  (symbol (lib_id "Device:R") (at 193.04 81.28 90) (unit 1)
-    (in_bom yes) (on_board yes)
-    (property "Reference" "R23" (id 0) (at 193.04 78.74 90))
+  (symbol (lib_id "Device:R") (at 193.04 81.28 90)
+    (in_bom yes) (on_board yes)
+    (property "Reference" "R24" (id 0) (at 193.04 78.74 90))
     (property "Value" "3.3k" (id 1) (at 193.04 81.28 90))
     (property "Footprint" "Resistor_SMD:R_0603_1608Metric" (id 2) (at 193.04 83.058 90)
@@
     (pin "2")
   )
-  (symbol (lib_id "Device:R") (at 171.45 72.39 0) (unit 1)
-    (in_bom yes) (on_board yes)
-    (property "Reference" "R17" (id 0) (at 173.99 72.39 90))
+  (symbol (lib_id "Device:R") (at 171.45 72.39 0)
+    (in_bom yes) (on_board yes)
+    (property "Reference" "R18" (id 0) (at 173.99 72.39 90))
     (property "Value" "2.2k" (id 1) (at 171.45 72.39 90))
     (property "Footprint" "Resistor_SMD:R_0603_1608Metric" (id 2) (at 169.672 72.39 90)
@@
     (pin "2")
   )
-  (symbol (lib_id "Device:C") (at 151.13 96.52 0) (unit 1)
-    (in_bom yes) (on_board yes)
-    (property "Reference" "C26" (id 0) (at 153.67 95.25 0)
+  (symbol (lib_id "Device:C") (at 151.13 96.52 0)
+    (in_bom yes) (on_board yes)
+    (property "Reference" "C27" (id 0) (at 153.67 95.25 0)
       (effects (font (size 1.27 1.27)) (justify left))
     )
@@
     (pin "2")
   )
-  (symbol (lib_id "Device:LED") (at 158.75 64.77 90) (unit 1)
-    (in_bom yes) (on_board yes)
-    (property "Reference" "D5" (id 0) (at 165.227 64.9478 0)
+  (symbol (lib_id "Device:LED") (at 158.75 64.77 90)
+    (in_bom yes) (on_board yes)
+    (property "Reference" "D6" (id 0) (at 165.227 64.9478 0)
       (effects (font (size 1.27 1.27)) hide)
     )
@@
     (pin "2")
   )
-  (symbol (lib_id "Device:D") (at 130.81 121.92 90) (unit 1)
-    (in_bom yes) (on_board yes)
-    (property "Reference" "D2" (id 0) (at 132.8166 120.7516 90)
+  (symbol (lib_id "Device:D") (at 130.81 121.92 90)
+    (in_bom yes) (on_board yes)
+    (property "Reference" "D1" (id 0) (at 132.8166 120.7516 90)
       (effects (font (size 1.27 1.27)) (justify right))
     )
@@
     (pin "2")
   )
-  (symbol (lib_id "Device:R") (at 184.15 72.39 0) (unit 1)
-    (in_bom yes) (on_board yes)
-    (property "Reference" "R21" (id 0) (at 186.69 72.39 90))
+  (symbol (lib_id "Device:R") (at 184.15 72.39 0)
+    (in_bom yes) (on_board yes)
+    (property "Reference" "R22" (id 0) (at 186.69 72.39 90))
     (property "Value" "2.2k" (id 1) (at 184.15 72.39 90))
     (property "Footprint" "Resistor_SMD:R_0603_1608Metric" (id 2) (at 182.372 72.39 90)
@@
     (pin "2")
   )
-  (symbol (lib_id "Device:R") (at 154.94 72.39 0) (unit 1)
-    (in_bom yes) (on_board yes)
-    (property "Reference" "R7" (id 0) (at 152.4 72.39 90))
+  (symbol (lib_id "Device:R") (at 154.94 72.39 0)
+    (in_bom yes) (on_board yes)
+    (property "Reference" "R8" (id 0) (at 152.4 72.39 90))
     (property "Value" "2.2k" (id 1) (at 154.94 72.39 90))
     (property "Footprint" "Resistor_SMD:R_0603_1608Metric" (id 2) (at 153.162 72.39 90)
@@
     (pin "2")
   )
-  (symbol (lib_id "Device:R") (at 158.75 72.39 0) (unit 1)
-    (in_bom yes) (on_board yes)
-    (property "Reference" "R10" (id 0) (at 161.29 72.39 90))
+  (symbol (lib_id "Device:R") (at 158.75 72.39 0)
+    (in_bom yes) (on_board yes)
+    (property "Reference" "R11" (id 0) (at 161.29 72.39 90))
     (property "Value" "2.2k" (id 1) (at 158.75 72.39 90))
     (property "Footprint" "Resistor_SMD:R_0603_1608Metric" (id 2) (at 156.972 72.39 90)
@@
     (pin "2")
   )
-  (symbol (lib_id "power:+5V") (at 130.81 116.84 0) (unit 1)
-    (in_bom yes) (on_board yes)
-    (property "Reference" "#PWR0193" (id 0) (at 130.81 120.65 0)
-      (effects (font (size 1.27 1.27)) hide)
-    )
+  (symbol (lib_id "power:+5V") (at 130.81 116.84 0)
+    (in_bom yes) (on_board yes)
+    (property "Reference" "#PWR0199" (id 0) (at 130.81 120.65 0)
+      (effects (font (size 1.27 1.27)) hide)
+    )

Commit message: Updated diodes, added LCSC numbers for all parts
Parts:
- C23: renamed from C22; LCSC (none) -> C14663; LCSC Part # C14663 -> (none)
- C24: renamed from C25; LCSC (none) -> C14663; LCSC Part # C14663 -> (none)
- C26: renamed from C27; LCSC (none) -> C14663; LCSC Part # C14663 -> (none)
- C29: renamed from C30; LCSC (none) -> C14663; LCSC Part # C14663 -> (none)
- D2: renamed from D1; LCSC (none) -> C81598; LCSC Part # C81598 -> (none)
- D5: renamed from D6; LCSC (none) -> C2290; LCSC Part # C2290 -> (none)
- D7: renamed from D8; LCSC (none) -> C2290; LCSC Part # C2290 -> (none)
- D9: renamed from D10; LCSC (none) -> C2290; LCSC Part # C2290 -> (none)
- R10: renamed from R11; LCSC (none) -> C4190; LCSC Part # C4190 -> (none)
- R13: renamed from R14; LCSC (none) -> C4190; LCSC Part # C4190 -> (none)
- R17: renamed from R18; LCSC (none) -> C4190; LCSC Part # C4190 -> (none)
- R19: renamed from R20; LCSC (none) -> C4190; LCSC Part # C4190 -> (none)
- R21: renamed from R22; LCSC (none) -> C4190; LCSC Part # C4190 -> (none)
- R23: renamed from R24; LCSC (none) -> C22978; LCSC Part # C22978 -> (none)
- R26: renamed from R27; LCSC (none) -> C22978; LCSC Part # C22978 -> (none)
- R28: renamed from R29; LCSC (none) -> C22978; LCSC Part # C22978 -> (none)
- R7: renamed from R8; LCSC (none) -> C4190; LCSC Part # C4190 -> (none)
