File: mcu.kicad_sch (KiCad schematic)
At the start: 34 parts, among them J17 Conn_01x01_Male, Q6 MMBT5551, U17 UCC27517, U3 STM32F103RCT, X1 8MHz 2520

Commit message: add 0R resistor on BOOT0 against GND
Parts:
- added R13: 0R, Resistor_SMD:R_0603_1608Metric, symbol Device:R
Connections:
- net GND: now also R13.2
- net at U3.60 (BOOT0): now also R13.1
- no-connect marks 9 -> 8
Changed lines of the file:
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@@
   (no_connect (at 161.29 96.52))
   (no_connect (at 125.73 96.52))
-  (no_connect (at 125.73 63.5))
   (no_connect (at 125.73 93.98))
   (no_connect (at 125.73 134.62))
@@
     (pin "1")
   )
-  (symbol (lib_id "Transistor_FET:BSP89") (at 245.11 121.92 0)
+  (symbol (lib_id "Transistor_FET:BSP89") (at 245.11 121.92 0) (unit 1)
     (in_bom yes) (on_board yes)
     (property "Reference" "V12" (id 0) (at 250.2916 120.7516 0)
@@
     (pin "3")
   )
-  (symbol (lib_id "Device:R") (at 234.95 121.92 270)
+  (symbol (lib_id "Device:R") (at 234.95 121.92 270) (unit 1)
     (in_bom yes) (on_board yes)
     (property "Reference" "R79" (id 0) (at 234.95 121.92 90))
@@
     (pin "2")
   )
-  (symbol (lib_id "Connector:Conn_01x01_Male") (at 252.73 114.3 180)
+  (symbol (lib_id "Connector:Conn_01x01_Male") (at 252.73 114.3 180) (unit 1)
     (in_bom yes) (on_board yes)
     (property "Reference" "J17" (id 0) (at 253.4412 113.7412 0)
@@
       (effects (font (size 1.27 1.27)) hide)
     )
+    (pin "1")
+    (pin "2")
+  )
+  (symbol (lib_id "power:GND") (at 118.11 63.5 0) (unit 1)
+    (in_bom yes) (on_board yes)
+    (property "Reference" "#PWR0131" (id 0) (at 118.11 69.85 0)
+      (effects (font (size 1.27 1.27)) hide)
+    )
+    (property "Value" "GND" (id 1) (at 118.237 67.8942 0))
+    (property "Footprint" "" (id 2) (at 118.11 63.5 0)
+      (effects (font (size 1.27 1.27)) hide)
+    )
+    (property "Datasheet" "" (id 3) (at 118.11 63.5 0)
+      (effects (font (size 1.27 1.27)) hide)
+    )
+    (pin "1")
+  )
+  (symbol (lib_id "Device:R") (at 121.92 63.5 270) (unit 1)
+    (in_bom yes) (on_board yes)
+    (property "Reference" "R13" (id 0) (at 121.92 58.2422 90))
+    (property "Value" "0R" (id 1) (at 121.92 60.5536 90))
+    (property "Footprint" "Resistor_SMD:R_0603_1608Metric" (id 2) (at 121.92 61.722 90)
+      (effects (font (size 1.27 1.27)) hide)
+    )
+    (property "Datasheet" "~" (id 3) (at 121.92 63.5 0)
+      (effects (font (size 1.27 1.27)) hide)
+    )
+    (property "LCSC Part #" "C22962" (id 4) (at 121.92 63.5 0)
+      (effects (font (size 1.27 1.27)) hide)
+    )

Commit message: Silkscreen and naming fixes
Parts:
- renumbered C70 to C47, C4 to C48, C23 to C49, C21 to C50, C19 to C51, C20 to C52, C22 to C53, C39 to C54, C40 to C55, C75 to C56, C76 to C57, D1AR1 to D22, D2 to D23, D13 to D24, D14 to D25, D15 to D26, D16 to D27, J17 to J18, Q6 to Q1, R19 to R66, R13 to R67, R20 to R68, R56 to R69, R46 to R70, R47 to R71, R79 to R72, R41 to R73, R42 to R74, R43 to R75, R44 to R76, U17 to U10, U3 to U9, V12 to V7

Commit message: Updated Current sense circuit
Parts:
- renumbered C47 to C51, C48 to C52, C49 to C53, C50 to C54, C51 to C55, C52 to C56, C53 to C57, C54 to C58, C55 to C59, C56 to C60, C57 to C61, D22 to D26, D23 to D27, D24 to D28, D25 to D29, D26 to D30, D27 to D31, R66 to R70, R67 to R71, R68 to R72, R69 to R73, R70 to R74, R71 to R75, R72 to R76, R73 to R77, R74 to R78, R75 to R79, R76 to R80, U9 to U10, U10 to U11

Commit message: added esp on bottom side
Connections:
- net +BATT renamed KEY_IN
Changed lines of the file:
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@@
     (effects (font (size 1.27 1.27)) (justify left bottom))
+  )
+  (global_label "KEY_IN" (shape input) (at 250.19 50.8 180) (fields_autoplaced)
+    (effects (font (size 1.27 1.27)) (justify right))
+    (property "Intersheet References" "${INTERSHEET_REFS}" (id 0) (at 241.4553 50.7206 0)
+      (effects (font (size 1.27 1.27)) (justify right) hide)
+    )
   )
   (hierarchical_label "CAN_TX" (shape output) (at 161.29 124.46 0)
@@
     (pin "2")
   )
-  (symbol (lib_id "power:+BATT") (at 250.19 50.8 0) (unit 1)
-    (in_bom yes) (on_board yes)
-    (property "Reference" "#PWR0114" (id 0) (at 250.19 54.61 0)
-      (effects (font (size 1.27 1.27)) hide)
-    )
-    (property "Value" "+BATT" (id 1) (at 250.571 46.4058 0))
-    (property "Footprint" "" (id 2) (at 250.19 50.8 0)
-      (effects (font (size 1.27 1.27)) hide)
-    )
-    (property "Datasheet" "" (id 3) (at 250.19 50.8 0)
-      (effects (font (size 1.27 1.27)) hide)
-    )
-    (pin "1")
-  )
   (symbol (lib_id "power:+VSW") (at 250.19 62.23 0) (unit 1)

Commit message: Some ERC fixes and other cleanups
Connections:
- no-connect marks 8 -> 9
Changed lines of the file:
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@@
   (junction (at 157.48 29.21) (diameter 0) (color 0 0 0 0)
   )
+  (no_connect (at 161.29 88.9))
   (no_connect (at 161.29 96.52))
   (no_connect (at 125.73 96.52))

Commit message: Updated diodes, added LCSC numbers for all parts
Parts:
- C51, C52, C53, C54, C55, C56, C60: LCSC (none) -> C14663; LCSC Part # C14663 -> (none)
- C57: LCSC (none) -> C1779; LCSC Part # C1779 -> (none)
- C58: LCSC (none) -> C57112; LCSC Part # C57112 -> (none)
- C59, C61: LCSC (none) -> C28323; LCSC Part # C28323 -> (none)
- D26: LCSC (none) -> C81598; LCSC Part # C81598 -> (none)
- D27, D28, D29, D30, D31: LCSC (none) -> C2290; LCSC Part # C2290 -> (none)
- J18: now not fitted; now left out of the parts list
- LS1: value FS1212 #Rastermaß 6.5 -> FS1212; LCSC (none) -> C482353; place hand -> (none)
- Q1: LCSC (none) -> C2145; LCSC Part # C2145 -> (none)
- R70: LCSC (none) -> C25804; LCSC Part # C25804 -> (none)
- R71, R73: LCSC (none) -> C22962; LCSC Part # C22962 -> (none)
- R72: LCSC (none) -> C4190; LCSC Part # C4190 -> (none)
- R74, R75, R80: LCSC (none) -> C21190; LCSC Part # C21190 -> (none)
- R76: LCSC (none) -> C17937; LCSC Part # C17937 -> (none)
- R77: LCSC (none) -> C25803; LCSC Part # C25803 -> (none)
- R78: LCSC (none) -> C4184; LCSC Part # C4184 -> (none)
- R79: LCSC (none) -> C22978; LCSC Part # C22978 -> (none)
- U10: LCSC (none) -> C8323
- U11: LCSC (none) -> C99395; LCSC Part # C99395 -> (none)
- V7: LCSC (none) -> C108637; LCSC Part # C108637 -> (none)
- X1: LCSC (none) -> C390520; LCSC Part # C390520 -> (none)

Commit message: update lcsc numbers
Parts:
- U10: place hand -> (none)
