File: supplies.kicad_sch (KiCad schematic)
At the start: 27 parts, among them U1 L7805, U2 AMS1117-3.3

Commit message: Silkscreen and naming fixes
Parts:
- renumbered C61 to C72, C3 to C73, C25 to C74, C5 to C75, C74 to C76, C62 to C77, C63 to C78, C38 to C79, C6 to C80, C26 to C81, D21 to D35, D20 to D36, D22 to D37, D35 to D38, D36 to D39, D37 to D40, D38 to D41, D39 to D42, R81 to R105, R53 to R106, R54 to R107, R55 to R108, U1 to U15, U2 to U16

Commit message: Updated Current sense circuit
Parts:
- renumbered C71 to C75, C72 to C76, C73 to C77, C74 to C78, C75 to C79, C76 to C80, C77 to C81, C78 to C82, C79 to C83, C80 to C84, C81 to C85, D35 to D39, D36 to D40, D37 to D41, D38 to D42, D39 to D43, D40 to D44, D41 to D45, D42 to D46, R105 to R109, R106 to R110, R107 to R111, R108 to R112, U15 to U16, U16 to U17

Commit message: added esp on bottom side
Parts:
- added J19: KEY_SWITCH, Connector_JST:JST_XH_B2B-XH-A_1x02_P2.50mm_Vertical, symbol Connector_Generic:Conn_01x02
- added JP3: Jumper_2_Open, Jumper:SolderJumper-2_P1.3mm_Open_RoundedPad1.0x1.5mm, symbol Jumper:Jumper_2_Open
Connections:
- net +BATT: now also J19.1 (Pin_1), JP3.2 (B); no longer F1.2
- new net KEY_IN: F1.2, J19.2 (Pin_2), JP3.1 (A)
Changed lines of the file:
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@@
   (junction (at 257.81 91.44) (diameter 0) (color 0 0 0 0)
   )
+  (junction (at 58.42 76.2) (diameter 0) (color 0 0 0 0)
+  )
   (junction (at 93.98 57.15) (diameter 0) (color 0 0 0 0)
   )
@@
   (junction (at 247.65 91.44) (diameter 0) (color 0 0 0 0)
   )
+  (junction (at 58.42 66.04) (diameter 0) (color 0 0 0 0)
+  )
   (junction (at 242.57 83.82) (diameter 0) (color 0 0 0 0)
   )
@@
     (stroke (width 0) (type default) (color 0 0 0 0))
   )
+  (wire (pts (xy 52.07 66.04) (xy 58.42 66.04))
+    (stroke (width 0) (type default) (color 0 0 0 0))
+  )
   (wire (pts (xy 231.14 99.06) (xy 231.14 106.68))
     (stroke (width 0) (type default) (color 0 0 0 0))
@@
     (stroke (width 0) (type default) (color 0 0 0 0))
   )
+  (wire (pts (xy 58.42 66.04) (xy 58.42 69.85))
+    (stroke (width 0) (type default) (color 0 0 0 0))
+  )
   (wire (pts (xy 240.03 36.83) (xy 242.57 36.83))
     (stroke (width 0) (type default) (color 0 0 0 0))
@@
     (stroke (width 0) (type default) (color 0 0 0 0))
   )
+  (wire (pts (xy 52.07 76.2) (xy 58.42 76.2))
+    (stroke (width 0) (type default) (color 0 0 0 0))
+  )
   (wire (pts (xy 78.74 83.82) (xy 101.6 83.82))
     (stroke (width 0) (type default) (color 0 0 0 0))
@@
     (stroke (width 0) (type default) (color 0 0 0 0))
   )
-  (wire (pts (xy 58.42 83.82) (xy 58.42 76.2))
+  (wire (pts (xy 58.42 72.39) (xy 58.42 76.2))
     (stroke (width 0) (type default) (color 0 0 0 0))
   )
@@
   )
   (wire (pts (xy 93.98 66.04) (xy 93.98 67.31))
+    (stroke (width 0) (type default) (color 0 0 0 0))
+  )
+  (wire (pts (xy 58.42 76.2) (xy 58.42 83.82))
     (stroke (width 0) (type default) (color 0 0 0 0))
   )
@@
   (text "beefy" (at 222.25 104.14 90)
     (effects (font (size 1.27 1.27)) (justify left bottom))
+  )
+  (global_label "KEY_IN" (shape input) (at 58.42 80.01 180) (fields_autoplaced)
+    (effects (font (size 1.27 1.27)) (justify right))
+    (property "Intersheet References" "${INTERSHEET_REFS}" (id 0) (at 49.6853 79.9306 0)
+      (effects (font (size 1.27 1.27)) (justify right) hide)
+    )
   )
   (hierarchical_label "V_BATT_MEAS" (shape input) (at 88.9 57.15 180)
@@
     (in_bom yes) (on_board yes)
     (property "Reference" "F1" (id 0) (at 67.31 81.28 90))
-    (property "Value" "2A permanent fuse" (id 1) (at 62.23 86.36 90))
+    (property "Value" "2A permanent fuse" (id 1) (at 69.85 83.82 0))
     (property "Footprint" "Fuse:Fuse_1206_3216Metric" (id 2) (at 67.31 82.042 90)
       (effects (font (size 1.27 1.27)) hide)
@@
     (pin "1")
   )
-  (symbol (lib_id "power:+BATT") (at 58.42 76.2 0) (unit 1)
-    (in_bom yes) (on_board yes)
-    (property "Reference" "#PWR0144" (id 0) (at 58.42 80.01 0)
-      (effects (font (size 1.27 1.27)) hide)
-    )
-    (property "Value" "+BATT" (id 1) (at 58.801 71.8058 0))
-    (property "Footprint" "" (id 2) (at 58.42 76.2 0)
-      (effects (font (size 1.27 1.27)) hide)
-    )
-    (property "Datasheet" "" (id 3) (at 58.42 76.2 0)
+  (symbol (lib_id "power:+BATT") (at 58.42 66.04 0) (unit 1)
+    (in_bom yes) (on_board yes)
+    (property "Reference" "#PWR0144" (id 0) (at 58.42 69.85 0)
+      (effects (font (size 1.27 1.27)) hide)
+    )
+    (property "Value" "+BATT" (id 1) (at 58.801 61.6458 0))
+    (property "Footprint" "" (id 2) (at 58.42 66.04 0)
+      (effects (font (size 1.27 1.27)) hide)
+    )
+    (property "Datasheet" "" (id 3) (at 58.42 66.04 0)
       (effects (font (size 1.27 1.27)) hide)
     )
@@
     (pin "1")
   )
+  (symbol (lib_id "Connector_Generic:Conn_01x02") (at 63.5 69.85 0) (unit 1)
+    (in_bom yes) (on_board yes) (fields_autoplaced)
+    (property "Reference" "J19" (id 0) (at 65.532 70.2115 0)
+      (effects (font (size 1.27 1.27)) (justify left))
+    )
+    (property "Value" "KEY_SWITCH" (id 1) (at 65.532 72.9866 0)
+      (effects (font (size 1.27 1.27)) (justify left))
+    )
+    (property "Footprint" "Connector_JST:JST_XH_B2B-XH-A_1x02_P2.50mm_Vertical" (id 2) (at 63.5 69.85 0)
+      (effects (font (size 1.27 1.27)) hide)
+    )
+    (property "Datasheet" "~" (id 3) (at 63.5 69.85 0)
+      (effects (font (size 1.27 1.27)) hide)
+    )
+    (pin "1")
+    (pin "2")
+  )
   (symbol (lib_id "power:GND") (at 121.92 88.9 0) (unit 1)
     (in_bom yes) (on_board yes)
@@
     (pin "1")
   )
+  (symbol (lib_id "Jumper:Jumper_2_Open") (at 52.07 71.12 90) (unit 1)
+    (in_bom yes) (on_board yes)
+    (property "Reference" "JP3" (id 0) (at 43.18 71.12 90)
+      (effects (font (size 1.27 1.27)) (justify right))
+    )
+    (property "Value" "Jumper_2_Open" (id 1) (at 48.26 63.5 0)
+      (effects (font (size 1.27 1.27)) (justify right))
+    )
+    (property "Footprint" "Jumper:SolderJumper-2_P1.3mm_Open_RoundedPad1.0x1.5mm" (id 2) (at 52.07 71.12 0)
+      (effects (font (size 1.27 1.27)) hide)
+    )
+    (property "Datasheet" "~" (id 3) (at 52.07 71.12 0)
+      (effects (font (size 1.27 1.27)) hide)
+    )
+    (pin "1")
+    (pin "2")
+  )
 )

Commit message: Update a few library symbols
Parts:
- C78, C83, C85: symbol Device:CP -> Device:C_Polarized
Changed lines of the file:
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@@
     (pin "1")
   )
-  (symbol (lib_id "Device:CP") (at 194.31 46.99 0) (unit 1)
+  (symbol (lib_id "Device:C_Polarized") (at 194.31 46.99 0) (unit 1)
     (in_bom yes) (on_board yes)
     (property "Reference" "C78" (id 0) (at 197.3072 45.8216 0)
@@
     (pin "2")
   )
-  (symbol (lib_id "Device:CP") (at 252.73 44.45 0) (unit 1)
+  (symbol (lib_id "Device:C_Polarized") (at 252.73 44.45 0) (unit 1)
     (in_bom yes) (on_board yes)
     (property "Reference" "C85" (id 0) (at 255.7272 43.2816 0)
@@
     (pin "1")
   )
-  (symbol (lib_id "Device:CP") (at 231.14 95.25 0) (unit 1)
+  (symbol (lib_id "Device:C_Polarized") (at 231.14 95.25 0) (unit 1)
     (in_bom yes) (on_board yes)
     (property "Reference" "C83" (id 0) (at 234.1372 94.0816 0)

Commit message: Some ERC fixes and other cleanups
Parts:
- PS1: value 120V DC DC converterr -> 120V DC DC converter; symbol Converter_DCDC:MEE1S0303SC -> Bobbycontroller:120V_DCDC
Other:
- moved on the sheet: C77, C79, C80, C81, C83, D39, D40, D41, D42, D43, D44, D45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

Commit message: Updated diodes, added LCSC numbers for all parts
Parts:
- C75, C80: LCSC (none) -> C76685; LCSC Part # C76685 -> (none)
- C76: LCSC (none) -> C113803; LCSC Part # C113803 -> (none)
- C77, C79, C81, C82, C84: LCSC (none) -> C14663; LCSC Part # C14663 -> (none)
- C78, C83, C85: LCSC (none) -> C105289; LCSC Part # C105289 -> (none)
- D39: LCSC (none) -> C10374; LCSC Part # C10374 -> (none)
- D40: LCSC (none) -> C8598; LCSC Part # C8598 -> (none)
- D41, D42, D43, D44, D45, D46: LCSC (none) -> C78409; LCSC Part # C78409 -> (none)
- F1: LCSC (none) -> C182310; LCSC Part # C182310 -> (none)
- J19: LCSC (none) -> C24192
- JP3: now not fitted; now left out of the parts list
- PS1: now not fitted
- R109: LCSC (none) -> C17937; LCSC Part # C17937 -> (none)
- R110, R111: LCSC (none) -> C22809; LCSC Part # C22809 -> (none)
- R112: LCSC (none) -> C21190; LCSC Part # C21190 -> (none)
- U16: LCSC (none) -> C15077; LCSC Part # C15077 -> (none)
- U17: LCSC (none) -> C426566; LCSC Part # C426566 -> (none)

Commit message: update lcsc numbers
Parts:
- C75, C80: place hand -> (none)
- D39, R109: now not fitted; now left out of the parts list
- F1: LCSC C182310 -> C99538
Connections:
- net at C75.1, C76.1, D39.1 (K)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: now also F1.1, R109.2
